Commit message: Remove inertia from hm structure

File: urdf/structures/summit_hm/summit_hm_structure.xacro (robot description, xacro)
@@ -10,9 +10,4 @@
 	  </joint>
 	  <link name="${prefix}_link">
-	    <inertial>
-	      <mass value="0.001"/>
-	      <origin rpy="0 0 0" xyz="0 0 0"/>
-	      <inertia ixx="0.0001" ixy="0" ixz="0" iyy="0.000001" iyz="0" izz="0.0001"/>
-	    </inertial>
 	    <visual>
 	      <origin rpy="0 0 0" xyz="0 0 0"/>
