Commit message: Increase the mass of the summit-hm model

File: urdf/bases/summit_hm_base.urdf.xacro (robot description, xacro)
@@ -37,5 +37,5 @@
 		<link name="${prefix}base_link">
 		<inertial>
-			<mass value="25.0" />
+			<mass value="50.0" />
 			<origin xyz="0 0 0" />
 			<inertia  ixx="1.391" ixy="0.004"  ixz="0.0"  iyy="6.853"  iyz="0.0"  izz="6.125" />
