Commit message: Update rb_theron.urdf.xacro
- added vectornav (random position)
- ros2 changes made with rafael

File: robots/rb_theron.urdf.xacro (robot description, xacro)
@@ -32,5 +32,5 @@
 	<xacro:property name="elevator_y" value="0.0" />
 	<xacro:property name="elevator_z" value="0.2238" />
-	<xacro:arg name="prefix" default="robot_"/>
+	<xacro:arg name="prefix" default=""/>
 	<xacro:arg name="ros_planar_move_plugin" default="false"/>
     <xacro:arg name="ros_planar_move_plugin_force_based" default="false"/>
@@ -66,22 +66,23 @@
 		<origin xyz="0.3305 0.0 0.1748" rpy="0 0 0"/>
 	</xacro:sensor_orbbec_astra-->
-	<xacro:sensor_intel_d435 prefix="$(arg prefix)front_rgbd_camera" parent="$(arg prefix)base_link" prefix_topic="front_rgbd_camera">
+    <xacro:sensor_intel_realsense_d435 frame_prefix="$(arg prefix)front_rgbd_camera_" parent="$(arg prefix)base_link" topic_prefix="front_rgbd_camera">
 		<origin xyz="0.3045 0.0 0.1898" rpy="0 0 0"/>
-	</xacro:sensor_intel_d435>
-	<xacro:sensor_intel_d435 prefix="$(arg prefix)rear_rgbd_camera" parent="$(arg prefix)base_link" prefix_topic="rear_rgbd_camera">
-		<origin xyz="-0.3045 0.0 0.1158" rpy="0 0 3.1416"/>
-	</xacro:sensor_intel_d435>
-	<xacro:sensor_imu_hector prefix="$(arg prefix)imu" parent="$(arg prefix)base_link">
+    </xacro:sensor_intel_realsense_d435>
+	<xacro:sensor_intel_realsense_d435 frame_prefix="$(arg prefix)rear_rgbd_camera_" parent="$(arg prefix)base_link" topic_prefix="rear_rgbd_camera">
+		<origin xyz="-0.3045 0.0 0.1898" rpy="0 0 3.1416"/>
+	</xacro:sensor_intel_realsense_d435>
+	<!-- TODO determine correct imu position-->
+	<xacro:sensor_vectornav frame_prefix="$(arg prefix)imu_" parent="$(arg prefix)base_link">
 		<origin xyz="-0.1975 0.0 0.1598" rpy="0 0 0"/>
-	</xacro:sensor_imu_hector>
-	<xacro:sensor_hokuyo_ust20lx prefix="$(arg prefix)front_laser" parent="$(arg prefix)base_link" prefix_topic="front_laser" min_angle="-2.0507619" max_angle="2.0507619">
+	</xacro:sensor_vectornav>
+	<!-- <xacro:sensor_hokuyo_ust20lx prefix="$(arg prefix)front_laser" parent="$(arg prefix)base_link" prefix_topic="front_laser" min_angle="-2.0507619" max_angle="2.0507619">
 		<origin xyz="0.2675 -0.215 0.1613" rpy="0 -3.1416 2.3562"/>
 	</xacro:sensor_hokuyo_ust20lx>
 	<xacro:sensor_hokuyo_ust20lx prefix="$(arg prefix)rear_laser" parent="$(arg prefix)base_link" prefix_topic="rear_laser" min_angle="-2.0507619" max_angle="2.0507619">
 		<origin xyz="-0.2675 0.215 0.1613" rpy="0 -3.1416 -0.7854"/>
-	</xacro:sensor_hokuyo_ust20lx>
-	<!--xacro:sensor_sick_nanoscan3 prefix="$(arg prefix)front_laser" parent="$(arg prefix)base_link" prefix_topic="front_laser" min_angle="-2.0507619" max_angle="2.0507619">
+	</xacro:sensor_hokuyo_ust20lx> -->
+	<xacro:sensor_sick_nanoscan3 frame_prefix="$(arg prefix)front_laser_" parent="$(arg prefix)base_link" topic_prefix="front_laser">
 		<origin xyz="0.250 0.0 0.1643" rpy="0 3.1416 3.1416"/>
-	</xacro:sensor_sick_nanoscan3-->
+	</xacro:sensor_sick_nanoscan3>
 	<!--xacro:sensor_sick_tim571 prefix="$(arg prefix)front_laser" parent="$(arg prefix)base_link" prefix_topic="front_laser" min_angle="-2.0507619" max_angle="2.0507619">
 		<origin xyz="0.2675 -0.215 0.1613" rpy="0 -3.1416 2.3562"/>
