Commit message: Robocomp urdf

File: robots/rbrobout.urdf.xacro (robot description, xacro)
@@ -11,4 +11,10 @@
 	<!-- Import all available sensors -->
 	<xacro:include filename="$(find robotnik_sensors)/urdf/all_sensors.urdf.xacro" />
+	<!-- Import robocomp structures -->
+	<xacro:include filename="$(find robot_description)/urdf/robocomp/cajon.urdf.xacro" />
+	<xacro:include filename="$(find robot_description)/urdf/robocomp/telescopico.urdf.xacro" />
+	<xacro:include filename="$(find robot_description)/urdf/robocomp/tool_changer.urdf.xacro" />
+	<!-- UR-20 arm -->
+	<xacro:include filename="$(find ur_description)/urdf/inc/ur20_macro.xacro" />
 	<xacro:property name="PI" value="3.1415926535897931"/>
 	<!-- Wheel parameters -->
@@ -57,16 +63,27 @@
     	</xacro:sensor_intel_d435>
     		<xacro:sensor_intel_d435 prefix="$(arg prefix)rear_rgbd_camera" parent="$(arg prefix)base_link" prefix_topic="rear_rgbd_camera">
-      		<origin xyz="-0.835 0  0.1555" rpy="0 ${PI} 0"/>
+      		<origin xyz="-0.835 0  0.1555" rpy="0 0 ${PI}"/>
     	</xacro:sensor_intel_d435>
-		<!-- magnetic sensors  -->
-		<!--xacro:sick_mls prefix="$(arg prefix)left_mls" parent="$(arg prefix)base_link">
-			<origin xyz="0.1085 -0.3045 -0.09137" rpy="0 0 ${1/2*PI}"/>
-		</xacro:sick_mls>
-		<xacro:sick_mls prefix="$(arg prefix)right_mls" parent="$(arg prefix)base_link">
-			<origin xyz="-0.1085 0.3045 -0.09137" rpy="0 0 ${-1/2*PI}"/>
-		</xacro:sick_mls>
-		<xacro:sick_mls prefix="$(arg prefix)front_mls" parent="$(arg prefix)base_link">
-			<origin xyz="0.7725 -0.1085 -0.09137" rpy="0 0 0"/>
-		</xacro:sick_mls!-->
+		<xacro:sensor_rs_helios_16p prefix="$(arg prefix)3d_laser" parent="$(arg prefix)base_link" prefix_topic="top_3d_laser">
+      		<origin xyz="0.4015 -0.44544 1.45476" rpy="0 0 ${PI}"/>
+    	</xacro:sensor_rs_helios_16p>
+		<!-- Robocomp structures -->
+		<xacro:structure_robocomp_cajon prefix="$(arg prefix)cajon" parent="$(arg prefix)base_link">
+      		<origin xyz="0 0 0" rpy="0 0 0"/>
+    	</xacro:structure_robocomp_cajon>
+		<xacro:structure_robocomp_telescopico prefix="$(arg prefix)telescopico" parent="$(arg prefix)cajon_link">
+      		<origin xyz="-0.7605 0 1.05" rpy="0 0 0"/>
+    	</xacro:structure_robocomp_telescopico>
+		<xacro:structure_robocomp_tool_changer prefix="$(arg prefix)tool_changer" parent="$(arg prefix)arm_tool0">
+      		<origin xyz="0 0 0" rpy="0 ${-PI/2} 0"/>
+    	</xacro:structure_robocomp_tool_changer>
+		<!-- UR-20 ARM -->
+		<xacro:ur20_robot prefix="$(arg prefix)arm_">
+		</xacro:ur20_robot>
+		<joint name="$(arg prefix)arm_base_joint" type="fixed">
+			<origin xyz="0 0 0" rpy="0 0 0"/>
+			<parent link="$(arg prefix)telescopico_link" />
+			<child link="$(arg prefix)arm_base_link" />
+		</joint>
    </xacro:macro>
    <!-- Gazebo ros control plugins -->

Commit message: Working lift

File: robots/rbrobout.urdf.xacro (robot description, xacro)
@@ -13,5 +13,5 @@
 	<!-- Import robocomp structures -->
 	<xacro:include filename="$(find robot_description)/urdf/robocomp/cajon.urdf.xacro" />
-	<xacro:include filename="$(find robot_description)/urdf/robocomp/telescopico.urdf.xacro" />
+	<xacro:include filename="$(find robot_description)/urdf/robocomp/Linak_LC3_lift.urdf.xacro" />
 	<xacro:include filename="$(find robot_description)/urdf/robocomp/tool_changer.urdf.xacro" />
 	<!-- UR-20 arm -->
@@ -62,5 +62,5 @@
       		<origin xyz="0.835 0  0.1555" rpy="0 0 0"/>
     	</xacro:sensor_intel_d435>
-    		<xacro:sensor_intel_d435 prefix="$(arg prefix)rear_rgbd_camera" parent="$(arg prefix)base_link" prefix_topic="rear_rgbd_camera">
+    	<xacro:sensor_intel_d435 prefix="$(arg prefix)rear_rgbd_camera" parent="$(arg prefix)base_link" prefix_topic="rear_rgbd_camera">
       		<origin xyz="-0.835 0  0.1555" rpy="0 0 ${PI}"/>
     	</xacro:sensor_intel_d435>
@@ -72,10 +72,7 @@
       		<origin xyz="0 0 0" rpy="0 0 0"/>
     	</xacro:structure_robocomp_cajon>
-		<xacro:structure_robocomp_telescopico prefix="$(arg prefix)telescopico" parent="$(arg prefix)cajon_link">
+		<xacro:linak_lc3_lift prefix="$(arg prefix)elevator" parent="$(arg prefix)cajon_link">
       		<origin xyz="-0.7605 0 1.05" rpy="0 0 0"/>
-    	</xacro:structure_robocomp_telescopico>
-		<xacro:structure_robocomp_tool_changer prefix="$(arg prefix)tool_changer" parent="$(arg prefix)arm_tool0">
-      		<origin xyz="0 0 0" rpy="0 ${-PI/2} 0"/>
-    	</xacro:structure_robocomp_tool_changer>
+    	</xacro:linak_lc3_lift>
 		<!-- UR-20 ARM -->
 		<xacro:ur20_robot prefix="$(arg prefix)arm_">
@@ -83,7 +80,10 @@
 		<joint name="$(arg prefix)arm_base_joint" type="fixed">
 			<origin xyz="0 0 0" rpy="0 0 0"/>
-			<parent link="$(arg prefix)telescopico_link" />
+			<parent link="$(arg prefix)elevator_linak_lc3_top_link" />
 			<child link="$(arg prefix)arm_base_link" />
 		</joint>
+		<xacro:structure_robocomp_tool_changer prefix="$(arg prefix)tool_changer" parent="$(arg prefix)arm_tool0">
+      		<origin xyz="0 0 0" rpy="0 ${-PI/2} 0"/>
+    	</xacro:structure_robocomp_tool_changer>
    </xacro:macro>
    <!-- Gazebo ros control plugins -->

Commit message: updated links and joints, changed meshes

File: robots/rbrobout.urdf.xacro (robot description, xacro)
@@ -73,4 +73,5 @@
     	</xacro:structure_robocomp_cajon>
 		<xacro:linak_lc3_lift prefix="$(arg prefix)elevator" parent="$(arg prefix)cajon_link">
+      		<!-- <origin xyz="0 0 1.05" rpy="0 0 0"/> -->
       		<origin xyz="-0.7605 0 1.05" rpy="0 0 0"/>
     	</xacro:linak_lc3_lift>
@@ -84,5 +85,6 @@
 		</joint>
 		<xacro:structure_robocomp_tool_changer prefix="$(arg prefix)tool_changer" parent="$(arg prefix)arm_tool0">
-      		<origin xyz="0 0 0" rpy="0 ${-PI/2} 0"/>
+      		<origin xyz="0 0 0" rpy="0 0 0"/>
+      		<!-- <origin xyz="0 0 0" rpy="0 ${-PI/2} 0"/> -->
     	</xacro:structure_robocomp_tool_changer>
    </xacro:macro>

File: urdf/robocomp/Linak_LC3_lift.urdf.xacro (robot description, xacro)
@@ -14,5 +14,5 @@
         </material>
 	      <geometry>
-	        <mesh filename="package://robot_description/meshes/robocomp/Linak_LC3_lift.stl"/>
+	        <!-- <mesh filename="package://robot_description/meshes/robocomp/Linak_LC3_lift.stl"/> -->
 	      </geometry>
 	    </visual>
@@ -20,5 +20,5 @@
 	      <origin rpy="0 0 0" xyz="0 0 0"/>
 	      <geometry>
-	        <mesh filename="package://robot_description/meshes/robocomp/Linak_LC3_lift.stl"/>
+	        <!-- <mesh filename="package://robot_description/meshes/robocomp/Linak_LC3_lift.stl"/> -->
 	      </geometry>
 	    </collision>
@@ -55,7 +55,5 @@
       <joint name="${prefix}_linak_lc3_top_joint" type="prismatic">
 	    <axis xyz="0 0 1"/>
-	    <xacro:insert_block name="origin"/>
-	    <!-- <parent link="${prefix}_linak_lc3_base_link"/> -->
-		<parent link="${parent}"/>
+	    <parent link="${prefix}_linak_lc3_base_link"/>
 	    <child link="${prefix}_linak_lc3_top_link"/>
         <limit lower="0" upper="0.9" effort="100.0" velocity="0.5" />
@@ -71,11 +69,11 @@
       </joint>
     </transmission>
-	  <gazebo reference="${prefix}_linak_lc3_base_link">
+	  <!-- <gazebo reference="${prefix}_linak_lc3_base_link">
 	    <material>Gazebo/Gray</material>
-	    <!-- <gravity>true</gravity> -->
-	  </gazebo>
+	    <gravity>true</gravity>
+	  </gazebo> -->
 	  <gazebo reference="${prefix}_linak_lc3_top_link">
 	    <material>Gazebo/Gray</material>
-	    <!-- <gravity>true</gravity> -->
+	    <gravity>true</gravity>
 	  </gazebo>
   </xacro:macro>

File: urdf/robocomp/cajon.urdf.xacro (robot description, xacro)
@@ -29,4 +29,26 @@
 	    <gravity>true</gravity>
 	  </gazebo>
+	  <!-- Could be an option to always provide link for any elevator in there -->
+ 	  <!-- <link name="${prefix}_elevator_mount_link">
+	    <visual>
+	      <origin rpy="0 0 0" xyz="0 0 0"/>
+	      <material name="alu_color">
+           <color rgba="0.5 0.5 0.5 1"/>
+        </material>
+	      <geometry>
+	      </geometry>
+	    </visual>
+	    <collision>
+	      <origin rpy="0 0 0" xyz="0 0 0"/>
+	      <geometry>
+	      </geometry>
+	    </collision>
+	  </link>
+	  <joint name="${prefix}_elevator_mount_joint" type="fixed">
+	    <axis xyz="0 1 0"/>
+      	<origin xyz="-0.7605 0 0" rpy="0 0 0"/>
+	    <parent link="${prefix}_link"/>
+	    <child link="${prefix}_elevator_mount_link"/>
+	  </joint> -->
   </xacro:macro>
 </robot>

File: urdf/robocomp/tool_changer.urdf.xacro (robot description, xacro)
@@ -2,16 +2,16 @@
 <robot name="structure" xmlns:xacro="http://wiki.ros.org/xacro">
   <xacro:macro name="structure_robocomp_tool_changer" params="prefix parent *origin">
-	  <joint name="${prefix}_joint" type="fixed">
+	  <joint name="${prefix}__base_joint" type="fixed">
 	    <axis xyz="0 1 0"/>
 	    <xacro:insert_block name="origin"/>
 	    <parent link="${parent}"/>
-	    <child link="${prefix}_link"/>
+	    <child link="${prefix}_base_link"/>
 	  </joint>
-	  <link name="${prefix}_link">
-	    <!-- <inertial>
-	      <mass value="0.001"/>
-	      <origin rpy="0 0 0" xyz="0 0 0"/>
-	      <inertia ixx="0.0001" ixy="0" ixz="0" iyy="0.000001" iyz="0" izz="0.0001"/>
-	    </inertial> -->
+	  <link name="${prefix}_base_link">
+		<inertial>
+			<mass value="2" />
+			<origin xyz="0 0 0" rpy="0 0 0"/>
+			<inertia ixx="1e-1" ixy="0" ixz="0" iyy="1e-1" iyz="0" izz="1e-1" />
+		</inertial>
 	    <visual>
 	      <origin rpy="0 0 0" xyz="0 0 0"/>
@@ -30,5 +30,30 @@
 	    </collision>
 	  </link>
-	  <gazebo reference="${prefix}_link">
+	  <joint name="${prefix}_tool_joint" type="fixed">
+	    <axis xyz="0 1 0"/>
+	      <origin rpy="0 0 0" xyz="0 0 0.05"/>
+	    <parent link="${prefix}_base_link"/>
+	    <child link="${prefix}_tool_link"/>
+	  </joint>
+	  <link name="${prefix}_tool_link">
+	    <visual>
+	      <origin rpy="0 0 0" xyz="0 0 0"/>
+	      <material name="alu_color">
+           <color rgba="0.5 0.5 0.5 1"/>
+        </material>
+	      <geometry>
+	      </geometry>
+	    </visual>
+	    <collision>
+	      <origin rpy="0 0 0" xyz="0 0 0"/>
+	      <geometry>
+	      </geometry>
+	    </collision>
+	  </link>
+	  <gazebo reference="${prefix}_base_link">
+	    <material>Gazebo/White</material>
+	    <gravity>true</gravity>
+	  </gazebo>
+	  <gazebo reference="${prefix}_tool_link">
 	    <material>Gazebo/White</material>
 	    <gravity>true</gravity>

Commit message: Fix wheels collision, add new version of cajon structure and fix rs helios origin

File: robots/rbrobout.urdf.xacro (robot description, xacro)
@@ -66,5 +66,5 @@
     	</xacro:sensor_intel_d435>
 		<xacro:sensor_rs_helios_16p prefix="$(arg prefix)3d_laser" parent="$(arg prefix)base_link" prefix_topic="top_3d_laser">
-      		<origin xyz="0.4015 -0.44544 1.45476" rpy="0 0 ${PI}"/>
+      		<origin xyz="0.4015 -0.451 1.45475" rpy="0 0 ${PI}"/>
     	</xacro:sensor_rs_helios_16p>
 		<!-- Robocomp structures -->

File: urdf/robocomp/cajon.urdf.xacro (robot description, xacro)
@@ -9,5 +9,5 @@
         </material>
 	      <geometry>
-	        <mesh filename="package://robot_description/meshes/robocomp/cajon.stl"/>
+	        <mesh filename="package://robot_description/meshes/robocomp/cajonv2.stl"/>
 	      </geometry>
 	    </visual>
@@ -15,5 +15,5 @@
 	      <origin rpy="0 0 0" xyz="0 0 0"/>
 	      <geometry>
-	        <mesh filename="package://robot_description/meshes/robocomp/cajon.stl"/>
+	        <mesh filename="package://robot_description/meshes/robocomp/cajonv2.stl"/>
 	      </geometry>
 	    </collision>
