Commit message: Add use_sim for caster and rocker in rbsherkan and correct naming in rb_theron and rb1 for wheel prefix

File: robots/rb1_base.urdf.xacro (robot description, xacro)
@@ -57,8 +57,8 @@
 	<xacro:gazebo_colors prefix="$(arg prefix)"/>
 	<!-- WHEELS -->
-	<xacro:rubber_wheel prefix="$(arg prefix)right" parent="$(arg prefix)base_link" hq="${hq}">
+	<xacro:rubber_wheel prefix="$(arg prefix)right_" parent="$(arg prefix)base_link" hq="${hq}">
 		<origin xyz="${wheel_offset_x} -${wheel_offset_y} ${wheel_offset_z}" rpy="0 0 0"/>
 	</xacro:rubber_wheel>
-	<xacro:rubber_wheel prefix="$(arg prefix)left" parent="$(arg prefix)base_link" hq="${hq}">
+	<xacro:rubber_wheel prefix="$(arg prefix)left_" parent="$(arg prefix)base_link" hq="${hq}">
 		<origin xyz="${wheel_offset_x} ${wheel_offset_y} ${wheel_offset_z}" rpy="0 0 0"/>
 	</xacro:rubber_wheel>

File: robots/rbsherkan_std.urdf.xacro (robot description, xacro)
@@ -18,18 +18,27 @@
     <xacro:arg name="prefix" default="robot_" />
     <xacro:property name="hq" value="true" />
+    <xacro:arg name="use_sim" default="false"/>
+    <xacro:arg name="ros_planar_move_plugin" default="false"/>
     <xacro:macro name="rbsherkan" params="prefix hq">
       <xacro:rbsherkan_base prefix="${prefix}" hq="${hq}"/>
+  <!-- Gazebo ros control pluggins -->
+	<!--xacro:ros_control namespace="$(arg namespace)"/-->
+	<xacro:ros_control/>
+	<xacro:if value="$(arg ros_planar_move_plugin)">
+    <xacro:omni_steering prefix="$(arg prefix)" publish_tf="true"/>
+  </xacro:if>
+    <xacro:gazebo_colors prefix="$(arg prefix)"/>
       <!-- Rocker -->
-      <xacro:rocker_front prefix="${prefix}left" parent="${prefix}base_link" hq="true" reflect="true">
+      <xacro:rocker_front prefix="${prefix}left_" parent="${prefix}base_link" hq="true" reflect="true" use_sim="$(arg use_sim)" >
         <origin xyz="0.095 0.16975 -0.0125" rpy="0 0 0"/>
       </xacro:rocker_front>
-      <xacro:rocker_front prefix="${prefix}right" parent="${prefix}base_link" hq="true" reflect="false">
+      <xacro:rocker_front prefix="${prefix}right_" parent="${prefix}base_link" hq="true" reflect="false" use_sim="$(arg use_sim)">
         <origin xyz="0.095 -0.16975 -0.0125" rpy="0 0 0"/>
       </xacro:rocker_front>
       <!-- Casters -->
-      <xacro:caster prefix="${prefix}rear_left_caster_" parent="${prefix}base_link" hq="true">
+      <xacro:caster prefix="${prefix}rear_left_caster_" parent="${prefix}base_link" hq="true" use_sim="$(arg use_sim)">
         <origin xyz="-0.185 0.16975 0.0302" rpy="0 0 0"/>
       </xacro:caster>
-      <xacro:caster prefix="${prefix}rear_right_caster_" parent="${prefix}base_link" hq="true">
+      <xacro:caster prefix="${prefix}rear_right_caster_" parent="${prefix}base_link" hq="true" use_sim="$(arg use_sim)">
         <origin xyz="-0.185 -0.16975 0.0302" rpy="0 0 0"/>
       </xacro:caster>
@@ -47,16 +56,4 @@
       </xacro:sensor_sick_nanoscan3>
     </xacro:macro>
-  <!-- Gazebo ros control pluggins -->
-  <!-- ros control plugin -->
-  <xacro:macro name="ros_control">
-    <gazebo>
-      <plugin name="ros_control" filename="libgazebo_ros_control.so">
-		    <robotParam>robot_description</robotParam>
-        <controlPeriod>0.001</controlPeriod>
-	      <robotSimType>gazebo_ros_control/DefaultRobotHWSim</robotSimType>
-		    <legacyModeNS>true</legacyModeNS>
-      </plugin>
-    </gazebo>
-	</xacro:macro>
   <xacro:rbsherkan prefix="$(arg prefix)" hq="${hq}" />
 </robot>

File: urdf/bases/rb_theron_base.urdf.xacro (robot description, xacro)
@@ -25,26 +25,26 @@
 	<!-- Robots Elements -->
 	<!-- *************** -->
-  <xacro:macro name="rb_theron_base" params="prefix hq use_sim">
+  <xacro:macro name="rb_theron_base" params="prefix hq use_sim:=^|false">
     <!-- rb_theron base -->
   	<xacro:rb_theron_base_v4 prefix="${prefix}" publish_bf="true" hq="${hq}" />
     <xacro:gazebo_colors prefix="${prefix}"/>
   	<!-- WHEELS -->
-  	<xacro:rubber_wheel prefix="${prefix}right" parent="${prefix}base_link" hq="${hq}">
+	<xacro:rubber_wheel prefix="${prefix}right_" parent="${prefix}base_link" hq="${hq}">
   		<origin xyz="${wheel_offset_x} ${-wheel_offset_y} ${wheel_offset_z}" rpy="0 0 0"/>
   	</xacro:rubber_wheel>
-  	<xacro:rubber_wheel prefix="${prefix}left" parent="${prefix}base_link" hq="${hq}">
+	<xacro:rubber_wheel prefix="${prefix}left_" parent="${prefix}base_link" hq="${hq}">
   		<origin xyz="${wheel_offset_x} ${wheel_offset_y} ${wheel_offset_z}" rpy="0 0 0"/>
   	</xacro:rubber_wheel>
 <!-- Castor wheels-->
-	<xacro:caster prefix="${prefix}front_left" parent="${prefix}base_link" hq="${hq}" use_sim="$(arg use_sim)">
+	<xacro:caster prefix="${prefix}front_left_" parent="${prefix}base_link" hq="${hq}" use_sim="$(arg use_sim)">
 		<origin xyz="0.235 0.1825 0.0448" rpy="0 0 0"/>
 	</xacro:caster>
-	<xacro:caster prefix="${prefix}front_right" parent="${prefix}base_link" hq="${hq}" use_sim="$(arg use_sim)">
+	<xacro:caster prefix="${prefix}front_right_" parent="${prefix}base_link" hq="${hq}" use_sim="$(arg use_sim)">
 		<origin xyz="0.235 -0.1825 0.0448" rpy="0 0 0"/>
 	</xacro:caster>
-	<xacro:caster prefix="${prefix}rear_left" parent="${prefix}base_link" hq="${hq}" use_sim="$(arg use_sim)">
+	<xacro:caster prefix="${prefix}rear_left_" parent="${prefix}base_link" hq="${hq}" use_sim="$(arg use_sim)">
 		<origin xyz="-0.235 0.1825 0.0448" rpy="0 0 0"/>
 	</xacro:caster>
-	<xacro:caster prefix="${prefix}rear_right" parent="${prefix}base_link" hq="${hq}" use_sim="$(arg use_sim)">
+	<xacro:caster prefix="${prefix}rear_right_" parent="${prefix}base_link" hq="${hq}" use_sim="$(arg use_sim)">
 		<origin xyz="-0.235 -0.1825 0.0448" rpy="0 0 0"/>
 	</xacro:caster>

File: urdf/structures/rbsherkan_chassis/rbsherkan_rocker.urdf.xacro (robot description, xacro)
@@ -1,8 +1,32 @@
 <?xml version="1.0"?>
 <robot name="caster_wheel" xmlns:xacro="http://www.ros.org/wiki/xacro">
-  <xacro:macro name="rocker_front" params="prefix parent *origin hq reflect">
+  <xacro:macro name="rocker_front" params="prefix parent *origin hq reflect use_sim:=^|false">
     <xacro:include filename="$(find robot_description)/urdf/wheels/caster_wheel/rbsherkan_caster.urdf.xacro" />
     <xacro:include filename="$(find robot_description)/urdf/wheels/rubber_wheel/rubber_wheel_150.urdf.xacro" />
     <!-- Base link -->
+    <xacro:if value="${use_sim}">
+    <joint name="${prefix}rocker_joint" type="revolute">
+      <xacro:insert_block name="origin" />
+      <parent link="${parent}"/>
+      <child link="${prefix}rocker_link"/>
+      <axis xyz="0 1 0" />
+      <limit effort="7000.0" lower="-1.0" upper="1.0" velocity="10.0"/>
+      <dynamics damping="0.01" friction="0.1"/>
+    </joint>
+    <transmission name="${prefix}rocker_joint_trans">
+			<type>transmission_interface/SimpleTransmission</type>
+			<joint name="${prefix}rocker_joint">
+				<!-- for the gazebo plugin -->
+				<!--hardwareInterface>EffortJointInterface</hardwareInterface-->
+				<!-- for ros control controller -->
+				<hardwareInterface>hardware_interface/EffortJointInterface</hardwareInterface>
+			</joint>
+			<actuator name="${prefix}rocker_joint_motor">
+				<mechanicalReduction>1</mechanicalReduction>
+				<motorTorqueConstant>20</motorTorqueConstant>
+			</actuator>
+		</transmission>
+  </xacro:if>
+  <xacro:unless value="${use_sim}">
     <joint name="${prefix}rocker_joint" type="fixed">
       <xacro:insert_block name="origin" />
@@ -11,4 +35,5 @@
       <axis xyz="0 1 0" />
     </joint>
+  </xacro:unless>
     <link name="${prefix}rocker_link">
       <visual>
@@ -51,5 +76,5 @@
       </xacro:unless>
     </xacro:rubber_wheel>
-    <xacro:caster prefix="${prefix}caster_" parent="${prefix}rocker_link" hq="${hq}">
+    <xacro:caster prefix="${prefix}caster_" parent="${prefix}rocker_link" hq="${hq}" use_sim="$(arg use_sim)">
       <origin xyz="0.090 0 0.0427" rpy="0 0 0" />
     </xacro:caster>

File: urdf/wheels/caster_wheel/rb_theron_caster.urdf.xacro (robot description, xacro)
@@ -18,10 +18,10 @@
               izz="${m*r*r/2}" />
   </xacro:macro>
-  <xacro:macro name="caster" params="prefix parent *origin hq use_sim">
+  <xacro:macro name="caster" params="prefix parent *origin hq use_sim:=^|false">
   <!--CASTER SUPPORT -->
   <xacro:if value="${use_sim}">
     <joint name="${prefix}joint_support" type="continuous">
       <parent link="${parent}"/>
-      <child link="${prefix}_support"/>
+      <child link="${prefix}support"/>
       <xacro:insert_block name="origin" />
       <axis xyz="0 0 1" rpy="0 ${M_PI} 0" />
@@ -34,5 +34,5 @@
     <joint name="${prefix}joint_support" type="fixed">
         <parent link="${parent}"/>
-        <child link="${prefix}_support"/>
+        <child link="${prefix}support"/>
         <xacro:insert_block name="origin" />
         <axis xyz="0 0 1" rpy="0 ${M_PI} 0" />
@@ -42,5 +42,5 @@
       </joint>
   </xacro:unless>
-    <link name="${prefix}_support">
+    <link name="${prefix}support">
       <visual>
         <origin xyz="0 0 0" rpy="0 0 0" />
@@ -62,6 +62,6 @@
     </link>
   <!--CASTER WHEEL -->
-  <!-- xacro:caster_wheel prefix="${prefix}" parent="${prefix}_support" hq="${hq}" -->
-  <xacro:caster_wheel prefix="${prefix}" parent="${prefix}_support" hq="${hq}" use_sim="$(arg use_sim)">
+  <!-- xacro:caster_wheel prefix="${prefix}" parent="${prefix}support" hq="${hq}" -->
+  <xacro:caster_wheel prefix="${prefix}" parent="${prefix}support" hq="${hq}" use_sim="$(arg use_sim)">
 		<origin xyz="${caster_wheel_offset_x} ${caster_wheel_offset_y} ${caster_wheel_offset_z}" rpy="0 0 0"/>
    </xacro:caster_wheel>
@@ -71,6 +71,6 @@
     <joint name="${prefix}joint_wheel" type="continuous">
       <parent link="${parent}"/>
-      <child link="${prefix}_wheel"/>
-      <insert_block name="origin" />
+      <child link="${prefix}wheel"/>
+      <xacro:insert_block name="origin" />
       <axis xyz="0 1 0" rpy="0 0 0" />
       <limit effort="100" velocity="100"/>
@@ -81,6 +81,6 @@
      <joint name="${prefix}joint_wheel" type="fixed">
        <parent link="${parent}"/>
-       <child link="${prefix}_wheel"/>
-       <insert_block name="origin" />
+       <child link="${prefix}wheel"/>
+       <xacro:insert_block name="origin" />
        <axis xyz="0 1 0" rpy="0 0 0" />
        <!-- <limit effort="100" velocity="100"/> -->
@@ -88,22 +88,5 @@
     </joint>
   </xacro:unless>
-    <link name="${prefix}_wheel">
-      <visual>
-        <!-- HIGH RESOLUTION WHEELS -->
-     <!-- xacro:if value="${hq}">
-          <origin xyz="0 0 0" rpy="0 0 0" />
-          <geometry>
-		<mesh filename="package://robot_description/meshes/wheels/mcq_prototype_caster_wheel.dae" />
-          </geometry>
-        </xacro:if -->
-       <!-- LOW RESOLUTION WHEELS -->
-       <!-- xacro:unless value="${hq}" -->
-          <origin xyz="0 0 0" rpy="0 0 0" />
-          <geometry>
-            <cylinder length="${caster_height}" radius="${caster_radius}" />
-            <!-- sphere radius="${caster_radius}"/ -->
-          </geometry>
-        <!-- /xacro:unless -->
-      </visual>
+    <link name="${prefix}wheel">
      <collision>
 	  <origin xyz="0 0 0" rpy="${M_PI/2} 0 0" />
@@ -126,20 +109,20 @@
   <!-- Transmission is important to link the joints and the controller-->
   <xacro:if value="${use_sim}">
-    <transmission name="${prefix}_support_joint_trans">
+    <transmission name="${prefix}support_joint_trans">
       <type>transmission_interface/SimpleTransmission</type>
       <joint name="${prefix}joint_support">
           <hardwareInterface>hardware_interface/EffortJointInterface</hardwareInterface>
       </joint>
-      <actuator name="${prefix}_support_joint_motor">
+      <actuator name="${prefix}support_joint_motor">
         <mechanicalReduction>1</mechanicalReduction>
       	<motorTorqueConstant>1</motorTorqueConstant>
       </actuator>
     </transmission>
-    <transmission name="${prefix}_wheel_joint_trans">
+    <transmission name="${prefix}wheel_joint_trans">
       <type>transmission_interface/SimpleTransmission</type>
       <joint name="${prefix}joint_wheel">
           <hardwareInterface>hardware_interface/EffortJointInterface</hardwareInterface>
       </joint>
-      <actuator name="${prefix}_wheel_joint_motor">
+      <actuator name="${prefix}wheel_joint_motor">
         <mechanicalReduction>1</mechanicalReduction>
 		<motorTorqueConstant>1</motorTorqueConstant>
@@ -147,5 +130,5 @@
     </transmission>
   </xacro:if>
-    <gazebo reference="${prefix}_support">
+    <gazebo reference="${prefix}support">
 			<mu1 value="5.0"/>
 			<mu2 value="0.5"/>
@@ -155,5 +138,5 @@
       <turnGravityOff>false</turnGravityOff>
     </gazebo>
-     <gazebo reference="${prefix}_wheel">
+     <gazebo reference="${prefix}wheel">
 			<mu1 value="100.0"/>
 			<mu2 value="100.0"/>

File: urdf/wheels/caster_wheel/rbsherkan_caster.urdf.xacro (robot description, xacro)
@@ -1,5 +1,5 @@
 <?xml version="1.0"?>
 <robot name="caster" xmlns:xacro="http://www.ros.org/wiki/xacro">
-  <xacro:macro name="caster" params="prefix parent *origin hq">
+  <xacro:macro name="caster" params="prefix parent *origin hq use_sim:=^|false">
     <!-- Caster support parameters -->
     <xacro:property name="caster_support_mass" value="1.5" /> <!-- in kg-->
@@ -18,11 +18,22 @@
     </xacro:macro>
     <!--CASTER SUPPORT -->
-    <joint name="${prefix}support_joint" type="continuous">
-      <xacro:insert_block name="origin" />
-      <parent link="${parent}"/>
-      <child link="${prefix}base_link"/>
-      <axis xyz="0 0 1" />
-      <dynamics damping="0.01" friction="0.1"/>
-    </joint>
+    <xacro:if value="${use_sim}">
+      <joint name="${prefix}support_joint" type="continuous">
+        <xacro:insert_block name="origin" />
+        <parent link="${parent}"/>
+        <child link="${prefix}base_link"/>
+        <axis xyz="0 0 1" />
+        <dynamics damping="0.01" friction="0.1"/>
+      </joint>
+    </xacro:if>
+    <xacro:unless value="${use_sim}">
+      <joint name="${prefix}support_joint" type="fixed">
+        <xacro:insert_block name="origin" />
+        <parent link="${parent}"/>
+        <child link="${prefix}base_link"/>
+        <axis xyz="0 0 1" />
+        <dynamics damping="0.01" friction="0.1"/>
+      </joint>
+    </xacro:unless>
     <link name="${prefix}base_link">
       <visual>
@@ -41,11 +52,22 @@
       </inertial>
     </link>
-    <joint name="${prefix}joint" type="continuous">
-      <origin xyz="${caster_wheel_offset_x} ${caster_wheel_offset_y} ${caster_wheel_offset_z}" rpy="0 0 0" />
-      <parent link="${prefix}base_link"/>
-      <child link="${prefix}link"/>
-      <axis xyz="0 1 0"/>
-      <dynamics damping="0.01" friction="0.1"/>
-    </joint>
+    <xacro:if value="${use_sim}">
+      <joint name="${prefix}joint" type="continuous">
+        <origin xyz="${caster_wheel_offset_x} ${caster_wheel_offset_y} ${caster_wheel_offset_z}" rpy="0 0 0" />
+        <parent link="${prefix}base_link"/>
+        <child link="${prefix}link"/>
+        <axis xyz="0 1 0"/>
+        <dynamics damping="0.01" friction="0.1"/>
+      </joint>
+    </xacro:if>
+    <xacro:unless value="${use_sim}">
+      <joint name="${prefix}joint" type="fixed">
+        <origin xyz="${caster_wheel_offset_x} ${caster_wheel_offset_y} ${caster_wheel_offset_z}" rpy="0 0 0" />
+        <parent link="${prefix}base_link"/>
+        <child link="${prefix}link"/>
+        <axis xyz="0 1 0"/>
+        <dynamics damping="0.01" friction="0.1"/>
+      </joint>
+    </xacro:unless>
     <link name="${prefix}link">
       <!--visual>
@@ -67,4 +89,27 @@
       </inertial>
     </link>
+  <!-- Transmission is important to link the joints and the controller-->
+  <xacro:if value="${use_sim}">
+    <transmission name="${prefix}_support_joint_trans">
+      <type>transmission_interface/SimpleTransmission</type>
+      <joint name="${prefix}support_joint">
+          <hardwareInterface>hardware_interface/EffortJointInterface</hardwareInterface>
+      </joint>
+      <actuator name="${prefix}_support_joint_motor">
+        <mechanicalReduction>1</mechanicalReduction>
+        <motorTorqueConstant>1</motorTorqueConstant>
+      </actuator>
+    </transmission>
+    <transmission name="${prefix}_wheel_joint_trans">
+      <type>transmission_interface/SimpleTransmission</type>
+      <joint name="${prefix}joint">
+          <hardwareInterface>hardware_interface/EffortJointInterface</hardwareInterface>
+      </joint>
+      <actuator name="${prefix}_wheel_joint_motor">
+        <mechanicalReduction>1</mechanicalReduction>
+		<motorTorqueConstant>1</motorTorqueConstant>
+      </actuator>
+    </transmission>
+  </xacro:if>
     <gazebo reference="${prefix}support">
       <mu1>0.45</mu1>

File: urdf/wheels/rubber_wheel/gazebo/rubber_wheel.transmission.xacro (robot description, xacro)
@@ -4,7 +4,7 @@
 	<xacro:macro name="rubber_wheel_transmission" params="prefix">
 	<!-- Transmission is important to link the joints and the controller (see rb_theron_control/config/rb_theron_control.yaml)-->
-		<transmission name="${prefix}_wheel_joint_trans">
+		<transmission name="${prefix}wheel_joint_trans">
 			<type>transmission_interface/SimpleTransmission</type>
-			<joint name="${prefix}_wheel_joint">
+			<joint name="${prefix}wheel_joint">
 				<!-- for the gazebo plugin -->
 				<!--hardwareInterface>EffortJointInterface</hardwareInterface-->
@@ -12,5 +12,5 @@
 				<hardwareInterface>hardware_interface/VelocityJointInterface</hardwareInterface>
 			</joint>
-			<actuator name="${prefix}_wheel_joint_motor">
+			<actuator name="${prefix}wheel_joint_motor">
 				<mechanicalReduction>1</mechanicalReduction>
 				<motorTorqueConstant>20</motorTorqueConstant>

File: urdf/wheels/rubber_wheel/rubber_wheel_150.urdf.xacro (robot description, xacro)
@@ -17,7 +17,7 @@
 	<xacro:macro name="rubber_wheel" params="prefix parent *origin hq">
 		<!--WHEEL TIRE -->
-		<joint name="${prefix}_wheel_joint" type="continuous">
+		<joint name="${prefix}wheel_joint" type="continuous">
 			<parent link="${parent}"/>
-			<child link="${prefix}_wheel_link"/>
+			<child link="${prefix}wheel_link"/>
 			<xacro:insert_block name="origin" />
 			<axis xyz="0 1 0" rpy="0 0 0" />
@@ -25,5 +25,5 @@
 			<joint_properties damping="0.0" friction="0.0"/>
 		</joint>
-		<link name="${prefix}_wheel_link">
+		<link name="${prefix}wheel_link">
 			<visual>
 				<!-- HIGH RESOLUTION WHEELS -->
@@ -46,10 +46,10 @@
 			</inertial>
 		</link>
-		<joint name="${prefix}_wheel_tire_joint" type="fixed">
-			<parent link="${prefix}_wheel_link"/>
-			<child link="${prefix}_wheel_tire_link"/>
+		<joint name="${prefix}wheel_tire_joint" type="fixed">
+			<parent link="${prefix}wheel_link"/>
+			<child link="${prefix}wheel_tire_link"/>
 			<origin xyz="0 0 0" rpy="0 0 0" />
 		</joint>
-		<link name="${prefix}_wheel_tire_link">
+		<link name="${prefix}wheel_tire_link">
 			<visual>
         <origin xyz="0 0 0" rpy="${M_PI/2} 0 0" />
