Commit message: URDF change to the POC gassco

File: robots/rbwatcher_std.urdf.xacro (robot description, xacro)
@@ -42,5 +42,5 @@
     	<!-- RGBD -->
     	<xacro:sensor_intel_d435 prefix="${prefix}front_rgbd_camera" parent="${prefix}base_link" prefix_topic="front_rgbd_camera">
-			<origin xyz="0.29881 0.0 0.15243" rpy="0 0 0"/>
+			<origin xyz="0.3003 0.0 0.15184" rpy="0 0 0"/>
     	</xacro:sensor_intel_d435>
 		<!--xacro:sensor_intel_d435 prefix="${prefix}rear_rgbd_camera" parent="${prefix}base_link" prefix_topic="rear_rgbd_camera">
@@ -49,13 +49,13 @@
         <!-- GPS -->
         <xacro:sensor_ublox prefix="${prefix}gps" parent="${prefix}base_link" use_mast="false">
-            <origin xyz="-0.24824 0.095 0.76359" rpy="0 0 0"/>
+            <origin xyz="-0.24702 0.095 0.773" rpy="0 0 0"/>
         </xacro:sensor_ublox>
     	<!-- LIDAR -->
     	<xacro:sensor_rs_helios_16p prefix="${prefix}top_3d_laser" prefix_topic="top_3d_laser" parent="${prefix}base_link" gpu="$(arg gpu)" suffix_topic="_raw">
-    	  	<origin xyz="-0.11924 0.0 0.38609" rpy="0 0 0"/>
+    	  	<origin xyz="-0.11802 0.0 0.3855" rpy="0 0 0"/>
     	</xacro:sensor_rs_helios_16p>
 		<!-- Antenna -->
 		<xacro:sensor_antena_std prefix="${prefix}antenna" parent="${prefix}base_link" mesh_file="${antenna_mesh}">
-			<origin xyz="-0.24124 0.0 0.31109" rpy="0 0 0"/>
+			<origin xyz="-0.24004 0.0 0.31005" rpy="0 0 0"/>
 		</xacro:sensor_antena_std>
 		<!-- PTZ camera -->

File: urdf/bases/rbwatcher_base.urdf.xacro (robot description, xacro)
@@ -8,6 +8,6 @@
 		<xacro:property name="PI" value="3.1415926535897931"/>
 		<!-- Wheel parameters -->
-		<xacro:property name="wheel_offset_x" value="0.22795" />    <!-- x,y,z in translation from base_link to the center of the wheel -->
-		<xacro:property name="wheel_offset_y" value="0.155" />
+		<xacro:property name="wheel_offset_x" value="0.234585" />    <!-- x,y,z in translation from base_link to the center of the wheel -->
+		<xacro:property name="wheel_offset_y" value="0.118" />
 		<xacro:property name="wheel_offset_z" value="0.0" />
 		<xacro:property name="docking_contact_offset_x" value="0.29378" />
