Commit message: Fix rbrobout_omni_wheel collision

File: urdf/wheels/omni_wheel/rbrobout_omni_wheel.urdf.xacro (robot description, xacro)
@@ -4,6 +4,6 @@
   <!-- Wheels -->
   <xacro:property name="omni_wheel_radius" value="0.127" />
-  <xacro:property name="omni_wheel_height" value="0.087" />
-  <xacro:property name="omni_wheel_mass" value="6.5" /> <!-- in kg-->
+  <xacro:property name="omni_wheel_height" value="0.128" />
+  <xacro:property name="omni_wheel_mass" value="15" /> <!-- in kg-->
   <xacro:macro name="cylinder_inertia" params="m r h">
     <inertia  ixx="${m*(3*r*r+h*h)/12}" ixy = "0" ixz = "0"
@@ -39,5 +39,5 @@
       </visual>
       <collision>
-				<origin xyz="0 0 0" rpy="${PI/2} 0 0" />
+				<origin xyz="0 0 0" rpy="0 0 0" />
         <geometry>
 					<cylinder length="${omni_wheel_height}" radius="${omni_wheel_radius}" />
