Commit message: fix for real kairos:
- modified launcher
- put wheels in the right directions
- added kairos urdf without arm

File: urdf/wheels/omni_wheel/omni_wheel.urdf.xacro (robot description, xacro)
@@ -16,5 +16,10 @@
       <child link="${prefix}_wheel_link"/>
       <xacro:insert_block name="origin" />
-      <axis xyz="0 1 0" rpy="0 0 0" />
+      <xacro:if value="${reflect}">
+        <axis xyz="0 1 0" rpy="0 0 0" />
+       </xacro:if>
+       <xacro:unless value="${reflect}">
+            <axis xyz="0 -1 0" rpy="0 0 0" />
+       </xacro:unless>
       <limit effort="100" velocity="100"/>
       <joint_properties damping="0.0" friction="0.0"/>
