Commit message: Fix kairos base urdf

File: robots/macros/rbkairos_macro.urdf.xacro (robot description, xacro)
@@ -6,5 +6,5 @@
   	<!-- First we import all posible elements defined in the urdf.xacro files. All these elements are defined as macro:xacros -->
   	<!-- Import summit XL base elements -->
-  	<xacro:include filename="$(find robot_description)/urdf/bases/rbkairos/rbkairos_base.urdf.xacro" />
+	<xacro:include filename="$(find robot_description)/urdf/bases/rbkairos/rbkairos_plus_base.urdf.xacro" />
   	<!-- Import summit XL wheels -->
   	<xacro:include filename="$(find robot_description)/urdf/wheels/omni_wheel/omni_wheel.urdf.xacro" />
@@ -12,6 +12,6 @@
   	<!-- Wheel parameters -->
   	<!-- Wheel parameters -->
-  	<xacro:property name="wheel_offset_x" value="0.2225" />    <!-- x,y,z in translation from base_link to the center of the wheel -->
-  	<xacro:property name="wheel_offset_y" value="0.2045" />
+  	<xacro:property name="wheel_offset_x" value="0.21528" />    <!-- x,y,z in translation from base_link to the center of the wheel -->
+  	<xacro:property name="wheel_offset_y" value="0.2590" />
   	<xacro:property name="wheel_offset_z" value="0.0" />
     <xacro:macro name="rbkairos">
@@ -20,5 +20,5 @@
   		<!-- *************** -->
   		<!-- Here we create the robot elements using the xacro:macros imported at the beggining of this file -->
-  		<xacro:rbkairos_base />
+  		<xacro:rbkairos_plus_base />
   		<xacro:omni_wheel robot_id="rbkairos_front_right" parent="rbkairos_base_link" reflect="false" hq="true">
   			<origin xyz="${wheel_offset_x} -${wheel_offset_y} ${wheel_offset_z}" rpy="0 0 0"/>
