Commit message: reestructure robot_description, robot_ prefix substituted by robot name

File: gazebo/ignition/rbkairos_control.urdf.xacro (robot description, xacro)
@@ -1,10 +1,13 @@
 <?xml version="1.0"?>
 <robot xmlns:xacro="http://wiki.ros.org/xacro">
-    <xacro:macro name="ros2_control" params="controllers">
+    <xacro:macro name="rbkairos_gz_ignition_control" params="namespace">
         <gazebo>
-          <plugin name="ros_control" filename="libgazebo_ros2_control.so">
+          <plugin name="ign_ros2_control::IgnitionROS2ControlPlugin" filename="ign_ros2_control-system">
             <robot_param>robot_description</robot_param>
             <robot_param_node>robot_state_publisher</robot_param_node>
-            <parameters>${controllers}</parameters>
+            <parameters>$(find robotnik_controller)/config/rbkairos_controller_example_params.yaml</parameters>
+            <ros>
+                <namespace>/${namespace}</namespace>
+            </ros>
           </plugin>
         </gazebo>
@@ -22,5 +25,5 @@
         <ros2_control name="GazeboSystem" type="system">
           <hardware>
-              <plugin>gazebo_ros2_control/GazeboSystem</plugin>
+            <plugin>ign_ros2_control/IgnitionSystem</plugin>
           </hardware>
           <xacro:ros2_joint interface="velocity" jmin="-10" jmax="10" name="rbkairos_front_left_wheel_joint"/>

File: gazebo/ignition/rbsummit_control.urdf.xacro (robot description, xacro)
@@ -1,10 +1,13 @@
 <?xml version="1.0"?>
 <robot xmlns:xacro="http://wiki.ros.org/xacro">
-    <xacro:macro name="rbsummit_gz_control" params="controllers">
+    <xacro:macro name="rbsummit_gz_ignition_control" params="namespace">
         <gazebo>
-          <plugin name="ros_control" filename="libgazebo_ros2_control.so">
+          <plugin name="ign_ros2_control::IgnitionROS2ControlPlugin" filename="ign_ros2_control-system">
             <robot_param>robot_description</robot_param>
             <robot_param_node>robot_state_publisher</robot_param_node>
-            <parameters>${controllers}</parameters>
+            <parameters>$(find robotnik_controller)/config/rbsummit_controller_example_params.yaml</parameters>
+            <ros>
+                <namespace>/${namespace}</namespace>
+            </ros>
           </plugin>
         </gazebo>
@@ -22,5 +25,5 @@
         <ros2_control name="GazeboSystem" type="system">
           <hardware>
-              <plugin>gazebo_ros2_control/GazeboSystem</plugin>
+            <plugin>ign_ros2_control/IgnitionSystem</plugin>
           </hardware>
           <xacro:ros2_joint interface="velocity" jmin="-30" jmax="30" name="rbsummit_front_left_wheel_joint"/>

File: gazebo/ignition/rbtheron_control.urdf.xacro (robot description, xacro)
@@ -1,10 +1,13 @@
 <?xml version="1.0"?>
 <robot xmlns:xacro="http://wiki.ros.org/xacro">
-    <xacro:macro name="rbtheron_gz_control" params="controllers">
+    <xacro:macro name="rbtheron_gz_ignition_control" params="namespace">
         <gazebo>
-          <plugin name="ros_control" filename="libgazebo_ros2_control.so">
+          <plugin name="ign_ros2_control::IgnitionROS2ControlPlugin" filename="ign_ros2_control-system">
             <robot_param>robot_description</robot_param>
             <robot_param_node>robot_state_publisher</robot_param_node>
-            <parameters>${controllers}</parameters>
+            <parameters>$(find robotnik_controller)/config/rbtheron_controller_example_params.yaml</parameters>
+            <ros>
+                <namespace>/${namespace}</namespace>
+            </ros>
           </plugin>
         </gazebo>
@@ -22,5 +25,5 @@
         <ros2_control name="GazeboSystem" type="system">
           <hardware>
-              <plugin>gazebo_ros2_control/GazeboSystem</plugin>
+            <plugin>ign_ros2_control/IgnitionSystem</plugin>
           </hardware>
           <xacro:ros2_joint interface="velocity" jmin="-10" jmax="10" name="rbtheron_left_wheel_joint"/>

File: gazebo/ignition/rbvogui_control.urdf.xacro (robot description, xacro)
@@ -1,10 +1,13 @@
 <?xml version="1.0"?>
 <robot xmlns:xacro="http://wiki.ros.org/xacro">
-    <xacro:macro name="rbvogui_gz_control" params="controllers">
+    <xacro:macro name="rbvogui_gz_ignition_control" params="namespace">
         <gazebo>
-          <plugin name="ros_control" filename="libgazebo_ros2_control.so">
+          <plugin name="ign_ros2_control::IgnitionROS2ControlPlugin" filename="ign_ros2_control-system">
             <robot_param>robot_description</robot_param>
             <robot_param_node>robot_state_publisher</robot_param_node>
-            <parameters>${controllers}</parameters>
+            <parameters>$(find robotnik_controller)/config/rbvogui_controller_example_params.yaml</parameters>
+            <ros>
+                <namespace>/${namespace}</namespace>
+            </ros>
           </plugin>
         </gazebo>
@@ -22,5 +25,5 @@
         <ros2_control name="GazeboSystem" type="system">
           <hardware>
-              <plugin>gazebo_ros2_control/GazeboSystem</plugin>
+            <plugin>ign_ros2_control/IgnitionSystem</plugin>
           </hardware>
           <xacro:ros2_joint interface="position" jmin="-2" jmax="2" name="rbvogui_front_left_steering_joint"/>

File: robots/rbkairos/rbkairos_ur5e.urdf.xacro (robot description, xacro)
@@ -8,4 +8,5 @@
   <xacro:include filename="$(find robot_description)/gazebo/classic/rbkairos_control.urdf.xacro"/>
   <xacro:include filename="$(find robot_description)/gazebo/ignition/rbkairos_control.urdf.xacro"/>
+  <xacro:include filename="$(find ur_description)/urdf/ur_macro.xacro"/>
   <!-- Import all available sensors -->
   <xacro:include filename="$(find robotnik_sensors)/urdf/all_sensors.urdf.xacro" />
@@ -33,9 +34,91 @@
   <xacro:property name="gps_offset_z" value="0.302"/>
   <!-- Launch Arguments -->
-  <xacro:arg name="use_gazebo_classic" default="false" />
+  <xacro:arg name="use_gazebo_classic" default="true" />
   <xacro:arg name="use_gazebo_ignition" default="false" />
   <xacro:arg name="gpu" default="true" />
   <xacro:arg name="namespace" default="robot" />
+  <!-- UR Arm -->
+   <xacro:arg name="ur_type" default="ur10e"/>
+  <xacro:arg name="joint_limit_params" default="$(find ur_description)/config/$(arg ur_type)/joint_limits.yaml"/>
+  <xacro:arg name="kinematics_params" default="$(find ur_description)/config/$(arg ur_type)/default_kinematics.yaml"/>
+  <xacro:arg name="physical_params" default="$(find ur_description)/config/$(arg ur_type)/physical_parameters.yaml"/>
+  <xacro:arg name="visual_params" default="$(find ur_description)/config/$(arg ur_type)/visual_parameters.yaml"/>
+  <xacro:arg name="transmission_hw_interface" default=""/>
+  <xacro:arg name="safety_limits" default="false"/>
+  <xacro:arg name="safety_pos_margin" default="0.15"/>
+  <xacro:arg name="safety_k_position" default="20"/>
+  <!-- ros2_control related parameters -->
+  <xacro:arg name="headless_mode" default="false" />
+  <xacro:arg name="robot_ip" default="192.168.0.210" />
+  <xacro:arg name="script_filename" default=""/>
+  <xacro:arg name="output_recipe_filename" default=""/>
+  <xacro:arg name="input_recipe_filename" default=""/>
+  <xacro:arg name="reverse_ip" default="0.0.0.0"/>
+  <xacro:arg name="script_command_port" default="50004"/>
+  <xacro:arg name="reverse_port" default="50001"/>
+  <xacro:arg name="script_sender_port" default="50002"/>
+  <xacro:arg name="trajectory_port" default="50003"/>
+  <!--   tool communication related parameters-->
+  <xacro:arg name="use_tool_communication" default="false" />
+  <xacro:arg name="tool_voltage" default="0" />
+  <xacro:arg name="tool_parity" default="0" />
+  <xacro:arg name="tool_baud_rate" default="115200" />
+  <xacro:arg name="tool_stop_bits" default="1" />
+  <xacro:arg name="tool_rx_idle_chars" default="1.5" />
+  <xacro:arg name="tool_tx_idle_chars" default="3.5" />
+  <xacro:arg name="tool_device_name" default="/tmp/ttyUR" />
+  <xacro:arg name="tool_tcp_port" default="54321" />
+    <!-- Simulation parameters -->
+  <xacro:arg name="use_fake_hardware" default="true" />
+  <xacro:arg name="fake_sensor_commands" default="true" />
+  <xacro:arg name="sim_gazebo" default="$(arg use_gazebo_classic)" />
+  <xacro:arg name="sim_ignition" default="$(arg use_gazebo_ignition)" />
+  <xacro:arg name="simulation_controllers" default="" />
+  <!-- initial position for simulations (Fake Hardware, Gazebo, Ignition) -->
+  <xacro:arg name="initial_positions_file" default="$(find ur_description)/config/initial_positions.yaml"/>
+  <!-- convert to property to use substitution in function -->
+  <xacro:property name="initial_positions_file" default="$(arg initial_positions_file)"/>
+  <xacro:property name="is_sim_gazebo" value="$(arg sim_gazebo)"/>
+  <xacro:property name="is_sim_ignition" value="$(arg sim_ignition)"/>
   <xacro:rbkairos/>
+  <xacro:ur_robot
+     name="$(arg ur_type)"
+     tf_prefix="$(arg ur_type)_"
+     parent="rbkairos_base_link"
+     joint_limits_parameters_file="$(arg joint_limit_params)"
+     kinematics_parameters_file="$(arg kinematics_params)"
+     physical_parameters_file="$(arg physical_params)"
+     visual_parameters_file="$(arg visual_params)"
+     transmission_hw_interface="$(arg transmission_hw_interface)"
+     safety_limits="$(arg safety_limits)"
+     safety_pos_margin="$(arg safety_pos_margin)"
+     safety_k_position="$(arg safety_k_position)"
+     use_fake_hardware="$(arg use_fake_hardware)"
+     fake_sensor_commands="$(arg fake_sensor_commands)"
+     sim_gazebo="$(arg sim_gazebo)"
+     sim_ignition="$(arg sim_ignition)"
+     headless_mode="$(arg headless_mode)"
+     initial_positions="${xacro.load_yaml(initial_positions_file)}"
+     use_tool_communication="$(arg use_tool_communication)"
+     tool_voltage="$(arg tool_voltage)"
+     tool_parity="$(arg tool_parity)"
+     tool_baud_rate="$(arg tool_baud_rate)"
+     tool_stop_bits="$(arg tool_stop_bits)"
+     tool_rx_idle_chars="$(arg tool_rx_idle_chars)"
+     tool_tx_idle_chars="$(arg tool_tx_idle_chars)"
+     tool_device_name="$(arg tool_device_name)"
+     tool_tcp_port="$(arg tool_tcp_port)"
+     robot_ip="$(arg robot_ip)"
+     script_filename="$(arg script_filename)"
+     output_recipe_filename="$(arg output_recipe_filename)"
+     input_recipe_filename="$(arg input_recipe_filename)"
+     reverse_ip="$(arg reverse_ip)"
+     script_command_port="$(arg script_command_port)"
+     reverse_port="$(arg reverse_port)"
+     script_sender_port="$(arg script_sender_port)"
+     trajectory_port="$(arg trajectory_port)"
+     >
+     <origin xyz="0 0 0.5" rpy="0 0 0" />          <!-- position robot in the world -->
+   </xacro:ur_robot>
   <xacro:include filename="$(find robot_description)/gazebo/classic/rbkairos_control.urdf.xacro" />
   <xacro:include filename="$(find robot_description)/gazebo/ignition/rbkairos_control.urdf.xacro" />

File: robots/rbsummit/rbsummit.urdf.xacro (robot description, xacro)
@@ -6,10 +6,11 @@
 	<!-- First we import the robot and all the sensors. All these elements are defined as macro:xacros -->
 	<!-- Import summit XL macro -->
-	<xacro:include filename="$(find robot_description)/robots/macros/rbsummit_macro.xacro"/>
+	<xacro:include filename="$(find robot_description)/macros/rbsummit_macro.xacro"/>
 	<!-- Import all available sensors -->
 	<xacro:include filename="$(find robotnik_sensors)/urdf/all_sensors.urdf.xacro" />
 	<!-- Import antenna -->
 	<xacro:include filename="$(find robot_description)/urdf/structures/sensor_support/structure_teltonika.urdf.xacro" />
-    <xacro:include filename="$(find robot_description)/urdf/ros2_control/rbsummit_control.urdf.xacro"/>
+    <xacro:include filename="$(find robot_description)/gazebo/classic/rbsummit_control.urdf.xacro"/>
+    <xacro:include filename="$(find robot_description)/gazebo/ignition/rbsummit_control.urdf.xacro"/>
 	<!-- ***************** -->
 	<!-- Global parameters -->
@@ -19,5 +20,9 @@
 	<!-- Flag to select the high or low quality model -->
 	<xacro:property name="hq" value="true" />
-	<xacro:arg name="gpu" default="false"/>
+    <!-- Launch Arguments -->
+    <xacro:arg name="use_gazebo_classic" default="false" />
+    <xacro:arg name="use_gazebo_ignition" default="false" />
+    <xacro:arg name="gpu" default="true" />
+  	<xacro:arg name="namespace" default="robot" />
 	<xacro:arg name="gps_latitude" default="0"/>
 	<xacro:arg name="gps_longitude" default="0"/>
@@ -49,4 +54,9 @@
 			<origin xyz="-0.22528 -0.095 0.23325" rpy="0 0 0"/>
 		</xacro:structure_mastil_teltonika> -->
-  <xacro:rbsummit_gz_control controllers="$(arg controllers)"/>
+    <xacro:if value="$(arg use_gazebo_classic)">
+        <xacro:rbsummit_gz_classic_control namespace="$(arg namespace)"/>
+    </xacro:if>
+    <xacro:if value="$(arg use_gazebo_ignition)">
+        <xacro:rbsummit_gz_ignition_control namespace="$(arg namespace)"/>
+    </xacro:if>
 </robot>

File: robots/rbtheron/rbtheron.urdf.xacro (robot description, xacro)
@@ -7,5 +7,5 @@
 	<!-- First we import all posible elements defined in the urdf.xacro files. All these elements are defined as macro:xacros -->
 	<!-- Import rbtheron macro -->
-	<xacro:include filename="$(find robot_description)/robots/macros/rbtheron_macro.xacro"/>
+	<xacro:include filename="$(find robot_description)/macros/rbtheron_macro.xacro"/>
 	<!-- Import all available sensors -->
 	<xacro:include filename="$(find robotnik_sensors)/urdf/all_sensors.urdf.xacro" />
@@ -14,5 +14,6 @@
 	<!-- Import Elevator -->
 	<xacro:include filename="$(find robot_description)/urdf/structures/elevator/rb_theron_elevator.urdf.xacro"/>
-    <xacro:include filename="$(find robot_description)/urdf/ros2_control/rbtheron_control.urdf.xacro"/>
+    <xacro:include filename="$(find robot_description)/gazebo/classic/rbtheron_control.urdf.xacro"/>
+    <xacro:include filename="$(find robot_description)/gazebo/ignition/rbtheron_control.urdf.xacro"/>
 	<!-- ***************** -->
 	<!-- Global parameters -->
@@ -26,7 +27,9 @@
 	<xacro:property name="elevator_y" value="0.0" />
 	<xacro:property name="elevator_z" value="0.2238" />
-    <xacro:arg name="use_gazebo" default="true" />
+    <xacro:arg name="use_gazebo_classic" default="false" />
+    <xacro:arg name="use_gazebo_ignition" default="false" />
+    <xacro:arg name="gpu" default="true" />
+  	<xacro:arg name="namespace" default="robot" />
     <xacro:arg name="has_elevator" default="false" />
-    <xacro:arg name="controllers" default="" />
 	<!-- Here we create the robot using the xacro:macro imported at the beggining of this file -->
 	<xacro:rbtheron hq="${hq}"/>
@@ -41,6 +44,9 @@
 		<origin xyz="-0.1975 0.0 0.1598" rpy="0 0 0"/>
     </xacro:sensor_vectornav>
-    <xacro:if value="$(arg use_gazebo)">
-        <xacro:rbtheron_gz_control controllers="$(arg controllers)"/>
+    <xacro:if value="$(arg use_gazebo_classic)">
+        <xacro:rbtheron_gz_classic_control namespace="$(arg namespace)"/>
+    </xacro:if>
+    <xacro:if value="$(arg use_gazebo_ignition)">
+        <xacro:rbtheron_gz_ignition_control namespace="$(arg namespace)"/>
     </xacro:if>
 </robot>

File: robots/rbvogui/rbvogui.urdf.xacro (robot description, xacro)
@@ -7,6 +7,7 @@
     <!-- First we import all posible elements defined in the urdf.xacro files. All these elements are defined as macro:xacros -->
     <!-- Import rbvogui base elements-->
-    <xacro:include filename="$(find robot_description)/robots/macros/rbvogui_macro.urdf.xacro" />
-    <xacro:include filename="$(find robot_description)/urdf/ros2_control/rbvogui_control.urdf.xacro"/>
+    <xacro:include filename="$(find robot_description)/macros/rbvogui_macro.urdf.xacro" />
+    <xacro:include filename="$(find robot_description)/gazebo/classic/rbvogui_control.urdf.xacro"/>
+    <xacro:include filename="$(find robot_description)/gazebo/ignition/rbvogui_control.urdf.xacro"/>
     <!-- Import all available sensors -->
     <xacro:include filename="$(find robotnik_sensors)/urdf/all_sensors.urdf.xacro" />
@@ -14,10 +15,9 @@
     <!-- Flag to select the high or low quality model -->
     <xacro:property name="hq" value="true" />
-    <xacro:property name="publish_bf" value="true" />
-    <xacro:arg name="robot_id" default="robot" />
-    <xacro:arg name="use_gazebo" default="true" />
+    <!-- Launch Arguments -->
+    <xacro:arg name="use_gazebo_classic" default="false" />
+    <xacro:arg name="use_gazebo_ignition" default="false" />
+    <xacro:arg name="gpu" default="true" />
     <xacro:arg name="namespace" default="robot" />
-    <xacro:arg name="gpu" default="true" />
-    <xacro:arg name="controllers" default="$(find rbvogui_gazebo)/config/omni_controller.yaml" />
     <xacro:rbvogui gpu="$(arg gpu)" hq="${hq}"/>
     <!-- SENSORS see robotnik_sensors for the specific configuration -->
@@ -41,6 +41,9 @@
         <origin xyz="-0.53 -0.33 0.1145" rpy="${PI} 0 ${-PI*3/4}"/>
     </xacro:sensor_sick_s300>
-    <xacro:if value="$(arg use_gazebo)">
-        <xacro:rbvogui_gz_control controllers="$(arg controllers)"/>
+    <xacro:if value="$(arg use_gazebo_classic)">
+        <xacro:rbvogui_gz_classic_control namespace="$(arg namespace)"/>
+    </xacro:if>
+    <xacro:if value="$(arg use_gazebo_ignition)">
+        <xacro:rbvogui_gz_ignition_control namespace="$(arg namespace)"/>
     </xacro:if>
 </robot>
