Commit message: Fix rbrobout wheels

File: urdf/bases/rbrobout/rbrobout_base.urdf.xacro (robot description, xacro)
@@ -26,14 +26,14 @@
 		<!-- Wheels -->
 		<xacro:rbrobout_omni_wheel prefix="${prefix}front_right" parent="${prefix}base_link" reflect="false" hq="${hq}">
-			<origin xyz="${wheel_offset_x} -${wheel_offset_y} ${wheel_offset_z}" rpy="1.57 0 0"/>
+			<origin xyz="${wheel_offset_x} -${wheel_offset_y} ${wheel_offset_z}" rpy="0 0 0"/>
 		</xacro:rbrobout_omni_wheel>
 		<xacro:rbrobout_omni_wheel prefix="${prefix}front_left" parent="${prefix}base_link" reflect="true" hq="${hq}">
-			<origin xyz="${wheel_offset_x} ${wheel_offset_y} ${wheel_offset_z}" rpy="1.57 0 0"/>
+			<origin xyz="${wheel_offset_x} ${wheel_offset_y} ${wheel_offset_z}" rpy="0 0 0"/>
 		</xacro:rbrobout_omni_wheel>
 		<xacro:rbrobout_omni_wheel prefix="${prefix}back_left" parent="${prefix}base_link" reflect="true" hq="${hq}">
-			<origin xyz="-${wheel_offset_x} ${wheel_offset_y} ${wheel_offset_z}" rpy="1.57 0 0"/>
+			<origin xyz="-${wheel_offset_x} ${wheel_offset_y} ${wheel_offset_z}" rpy="0 0 0"/>
 		</xacro:rbrobout_omni_wheel>
 		<xacro:rbrobout_omni_wheel prefix="${prefix}back_right" parent="${prefix}base_link" reflect="false" hq="${hq}">
-			<origin xyz="-${wheel_offset_x} -${wheel_offset_y} ${wheel_offset_z}" rpy="1.57 0 0"/>
+			<origin xyz="-${wheel_offset_x} -${wheel_offset_y} ${wheel_offset_z}" rpy="0 0 0"/>
 		</xacro:rbrobout_omni_wheel>
    </xacro:macro>

File: urdf/wheels/omni_wheel/rbrobout_omni_wheel.urdf.xacro (robot description, xacro)
@@ -23,5 +23,5 @@
       <visual>
         <xacro:if value="${hq}">
-          <origin xyz="0 0 0" rpy="0 0 0" />
+          <origin xyz="0 0 0" rpy="${PI/2} 0 0" />
           <geometry>
             <mesh filename="package://robot_description/meshes/wheels/omni_wheel/robout_wheel.stl" />
@@ -39,5 +39,5 @@
       </visual>
       <collision>
-				<origin xyz="0 0 0" rpy="${PI/2} 0 0" />
+				<origin xyz="0 0 0" rpy="0 0 0" />
         <geometry>
 					<cylinder length="${omni_wheel_height}" radius="${omni_wheel_radius}" />
