Commit message: Fix/ros2/remove old references (#27)
* removed rb1 references

* removed sherkan references

* removed hm references

* removed ur universal robot arms references

* removed fixed wheel references

* removed unused theron wheel reference

* removed unused rubber wheel reference

* removed steel references

* removed container structures references

* removed elevator structure references

* removed old structures

* removed meshes from structures

* removed unused meshes

* working basic robots after removing references

---------

Co-authored-by: Marc Bosch <mbosch@robotnik.es>

File: urdf/bases/rbrobout/rbrobout_cameras_cover.urdf.xacro (robot description, xacro)
@@ -18,5 +18,5 @@
 			<origin xyz="0 0 0" rpy="0 0 -${PI/2}" />
 			<geometry>
-				<mesh filename="package://robotnik_description/meshes/structures/rbrobout/cameras_cover.stl"/>
+				<mesh filename="package://robotnik_description/meshes/bases/rbrobout/rbrobout_cameras_cover.stl"/>
 			</geometry>
 			<material name="grey">
@@ -27,5 +27,5 @@
 			<origin xyz="0 0 0" rpy="0 0 -${PI/2}" />
 			<geometry>
-				<mesh filename="package://robotnik_description/meshes/structures/rbrobout/cameras_cover.stl"/>
+				<mesh filename="package://robotnik_description/meshes/bases/rbrobout/rbrobout_cameras_cover.stl"/>
 			</geometry>
 		</collision>

File: urdf/bases/rbrobout/rbrobout_top_cover.urdf.xacro (robot description, xacro)
@@ -18,5 +18,5 @@
         <origin xyz="0 0 0" rpy="0 0 0" />
         <geometry>
-            <mesh filename="package://robotnik_description/meshes/structures/rbrobout/top_cover.stl"/>
+            <mesh filename="package://robotnik_description/meshes/bases/rbrobout/rbrobout_top_cover.stl"/>
         </geometry>
         <material name="darkgrey">
@@ -27,5 +27,5 @@
         <origin xyz="0 0 0" rpy="0 0 0 " />
         <geometry>
-            <mesh filename="package://robotnik_description/meshes/structures/rbrobout/top_cover.stl"/>
+            <mesh filename="package://robotnik_description/meshes/bases/rbrobout/rbrobout_top_cover.stl"/>
         </geometry>
     </collision>

File: urdf/inertia.urdf.xacro (robot description, xacro)
@@ -10,22 +10,8 @@
   </xacro:macro>
   <!-- TODO Hollow sphere of radius r and mass m-->
-  <xacro:macro name="solid_sphere_inertia" params="m r">
+  <xacro:macro name="hollow_sphere_inertia" params="m r">
     <inertia  ixx="${(2*r*r*m)/3}" ixy = "0" ixz = "0"
               iyy="${(2*r*r*m)/3}" iyz = "0"
               izz="${(2*r*r*m)/3}"
-     />
-  </xacro:macro>
-  <!-- TODO Solid ellipsoid of semi-axes a, b, c and mass m-->
-  <xacro:macro name="ellipsoid_semi_axes_inertia" params="a b c m r">
-    <inertia  ixx="${(m*(b*b+c*c))/5}" ixy = "0" ixz = "0"
-              iyy="${(m*(a*a+c*c))/5}" iyz = "0"
-              izz="${(m*(a*a+b*b))/5}"
-     />
-  </xacro:macro>
-  <!-- TODO Right circular cone with radius r, height h and mass m, about the apex -->
-  <xacro:macro name="right_circular_cone_inertia" params="m r h">
-    <inertia  ixx="${((3*m*(h*h))/5)+((3*m*(r*r))/20)}" ixy = "0" ixz = "0"
-              iyy="${((3*m*(h*h))/5)+((3*m*(r*r))/20)}" iyz = "0"
-              izz="${(3*m*(r*r))/10}"
      />
   </xacro:macro>
@@ -46,10 +32,3 @@
      />
   </xacro:macro>
-    <!-- TODO Thick-walled cylindrical tube with open ends, of inner radius r1, outer radius r2, length h and mass m -->
-    <xacro:macro name="thick_walled_cylinder_inertia" params="m r1 r2 h">
-    <inertia  ixx="${m*((3*(r1*r1+r2*r2))+(h*h))/12}" ixy = "0" ixz = "0"
-              iyy="${m*((3*(r1*r1+r2*r2))+(h*h))/12}" iyz = "0"
-              izz="${m*(r1*r1+r2*r2)/2}"
-     />
-  </xacro:macro>
 </robot>
