Commit message: add base_docking_contact link to vogui

File: urdf/bases/rbrobout/rbrobout_top_cover.urdf.xacro (robot description, xacro)
@@ -31,12 +31,4 @@
     </collision>
     </link>
-        <!-- DOCKING CONTACTS -->
-        <!-- <joint name="${prefix}base_docking_joint" type="fixed">
-            <origin xyz="0.284 0.012 0.068" rpy="0 0 0 " />
-            <parent link="${prefix}base_link"/>
-            <child link="${prefix}base_docking_contact_link" />
-        </joint> -->
-        <!-- DOCKING LINK -->
-        <!-- <link name="${prefix}base_docking_contact_link" /> -->
   </xacro:macro>
 </robot>

File: urdf/bodies/rb1/rb1_body.urdf.xacro (robot description, xacro)
@@ -93,11 +93,10 @@
   </joint>
   <link name="${prefix}top_cover_link"/>
-   <!-- DOCKING CONTACT -->
-    <link name="${prefix}base_docking_contact">
-    </link>
+    <!-- DOCKING CONTACT -->
+    <link name="${prefix}base_docking_contact"/>
     <joint name="${prefix}base_docking_joint" type="fixed">
-      <origin xyz="0.030 0.000 0.068" rpy="0 0 0 " />
-      <parent link="${prefix}base_link"/>
-      <child link="${prefix}base_docking_contact" />
+        <origin xyz="0.030 0.000 0.068" rpy="0 0 0 " />
+        <parent link="${prefix}base_link"/>
+        <child link="${prefix}base_docking_contact"/>
     </joint>
   </xacro:macro>

File: urdf/bodies/rbkairos/rbkairos_body.urdf.xacro (robot description, xacro)
@@ -130,11 +130,10 @@
     <child link="${prefix}base_logo_rear" />
   </joint>
-   <!-- DOCKING CONTACT -->
-    <link name="${prefix}base_docking_contact">
-    </link>
+    <!-- DOCKING CONTACT -->
+    <link name="${prefix}base_docking_contact"/>
     <joint name="${prefix}base_docking_joint" type="fixed">
-      <origin xyz="0.35 0 0.09" rpy="0 0 0" />
-      <parent link="${prefix}base_link"/>
-      <child link="${prefix}base_docking_contact" />
+        <origin xyz="0.35 0 0.09" rpy="0 0 0" />
+        <parent link="${prefix}base_link"/>
+        <child link="${prefix}base_docking_contact"/>
     </joint>
   </xacro:macro>

File: urdf/bodies/rbrobout/rbrobout_body.urdf.xacro (robot description, xacro)
@@ -42,12 +42,11 @@
           </collision>
       </link>
-        <!-- DOCKING CONTACTS -->
-        <joint name="${prefix}base_docking_joint" type="fixed">
-            <origin xyz="0.858 0.02 0.008" rpy="0 0 0 " />
-            <parent link="${prefix}base_footprint"/>
-            <child link="${prefix}base_docking_contact_link" />
-        </joint>
-        <!-- DOCKING LINK -->
-        <link name="${prefix}base_docking_contact_link" />
+    <!-- DOCKING CONTACT -->
+    <link name="${prefix}base_docking_contact"/>
+    <joint name="${prefix}base_docking_joint" type="fixed">
+        <origin xyz="0.858 0.02 0.008" rpy="0 0 0 " />
+        <parent link="${prefix}base_link"/>
+        <child link="${prefix}base_docking_contact" />
+    </joint>
   </xacro:macro>
 </robot>

File: urdf/bodies/rbtheron/rbtheron_body.urdf.xacro (robot description, xacro)
@@ -120,11 +120,10 @@
     <child link="${prefix}base_logo_rear" />
   </joint>
-   <!-- DOCKING CONTACT -->
-    <link name="${prefix}base_docking_contact">
-    </link>
+    <!-- DOCKING CONTACT -->
+    <link name="${prefix}base_docking_contact"/>
     <joint name="${prefix}base_docking_joint" type="fixed">
-      <origin xyz="0.35 0 0.09" rpy="0 0 0" />
-      <parent link="${prefix}base_link"/>
-      <child link="${prefix}base_docking_contact" />
+        <origin xyz="0.35 0 0.09" rpy="0 0 0" />
+        <parent link="${prefix}base_link"/>
+        <child link="${prefix}base_docking_contact" />
     </joint>
   </xacro:macro>

File: urdf/bodies/rbvogui/rbvogui_body.urdf.xacro (robot description, xacro)
@@ -156,4 +156,11 @@
     <xacro:gazebo_color_logo_link prefix="${prefix}"/>
     <xacro:gazebo_color_leds_link prefix="${prefix}"/>
+    <!-- DOCKING CONTACT -->
+    <link name="${prefix}base_docking_contact"/>
+    <joint name="${prefix}base_docking_joint" type="fixed">
+        <origin xyz="0.6405 0 0.10264" rpy="0 0 0"/>
+        <parent link="${prefix}chassis_link"/>
+        <child link="${prefix}base_docking_contact"/>
+    </joint>
   </xacro:macro>
 </robot>

File: urdf/bodies/rbvogui/rbvogui_xl_body.urdf.xacro (robot description, xacro)
@@ -159,4 +159,11 @@
     <xacro:gazebo_color_logo_link prefix="${prefix}"/>
     <xacro:gazebo_color_leds_link prefix="${prefix}"/>
+    <!-- DOCKING CONTACT -->
+    <link name="${prefix}base_docking_contact"/>
+    <joint name="${prefix}base_docking_joint" type="fixed">
+        <origin xyz="0.6405 0 0.10264" rpy="0 0 0"/>
+        <parent link="${prefix}chassis_link"/>
+        <child link="${prefix}base_docking_contact"/>
+    </joint>
   </xacro:macro>
 </robot>
