Commit message: corrected laser position in robout

File: robots/rbrobout/rbrobout.urdf.xacro (robot description, xacro)
@@ -12,13 +12,13 @@
   <xacro:arg name="prefix" default="robot_"/>
   <xacro:arg name="gazebo_classic" default="false"/>
-  <xacro:property name="front_laser_offset_x" value="0.2865"/>
-  <xacro:property name="front_laser_offset_y" value="-0.20894"/>
-  <xacro:property name="front_laser_offset_z" value="0.2973"/>
-  <xacro:property name="rear_laser_offset_x" value="-0.2865"/>
-  <xacro:property name="rear_laser_offset_y" value="0.20894"/>
-  <xacro:property name="rear_laser_offset_z" value="0.2973"/>
-  <xacro:property name="imu_offset_x" value="0.127"/>
-  <xacro:property name="imu_offset_y" value="-0.129"/>
-  <xacro:property name="imu_offset_z" value="0.212"/>
+  <xacro:property name="front_laser_offset_x" value="0.8"/>
+  <xacro:property name="front_laser_offset_y" value="0.366"/>
+  <xacro:property name="front_laser_offset_z" value="-0.06"/>
+  <xacro:property name="rear_laser_offset_x" value="-0.8"/>
+  <xacro:property name="rear_laser_offset_y" value="-0.366"/>
+  <xacro:property name="rear_laser_offset_z" value="-0.06"/>
+  <xacro:property name="imu_offset_x" value="0.3"/>
+  <xacro:property name="imu_offset_y" value="-0.3"/>
+  <xacro:property name="imu_offset_z" value="0.0725"/>
   <xacro:rbrobout prefix="$(arg prefix)"/>
   <!-- IMU -->
