Commit message: update structures for rbrobout

File: robots/rbrobout/rbrobout_plus.urdf.xacro (robot description, xacro)
@@ -18,5 +18,4 @@
   <xacro:arg name="prefix" default="robot_"/>
   <xacro:arg name="gazebo_classic" default="false"/>
-  <xacro:arg name="gazebo_ignition" default="false"/>
   <xacro:arg name="ur_type" default="ur10e"/>
   <xacro:arg name="joint_limit_params" default="$(find ur_description)/config/$(arg ur_type)/joint_limits.yaml"/>
@@ -33,25 +32,7 @@
   <xacro:property name="imu_offset_y" value="-0.3"/>
   <xacro:property name="imu_offset_z" value="0.0725"/>
-  <xacro:property name="front_rgbd_camera_offset_x" value="0.883"/>
-  <xacro:property name="front_rgbd_camera_offset_y" value="0.0"/>
-  <xacro:property name="front_rgbd_camera_offset_z" value="0.887"/>
-  <xacro:property name="front_right_rgbd_camera_offset_x" value="0.089"/>
-  <xacro:property name="front_right_rgbd_camera_offset_y" value="-0.399"/>
-  <xacro:property name="front_right_rgbd_camera_offset_z" value="0.994"/>
-  <xacro:property name="front_left_rgbd_camera_offset_x" value="0.089"/>
-  <xacro:property name="front_left_rgbd_camera_offset_y" value="0.399"/>
-  <xacro:property name="front_left_rgbd_camera_offset_z" value="0.994"/>
-  <xacro:property name="rear_rgbd_camera_offset_x" value="-0.883"/>
-  <xacro:property name="rear_rgbd_camera_offset_y" value="-0.0"/>
-  <xacro:property name="rear_rgbd_camera_offset_z" value="0.769"/>
-  <xacro:property name="rear_right_rgbd_camera_offset_x" value="-0.427"/>
-  <xacro:property name="rear_right_rgbd_camera_offset_y" value="-0.399"/>
-  <xacro:property name="rear_right_rgbd_camera_offset_z" value="0.994"/>
-  <xacro:property name="rear_left_rgbd_camera_offset_x" value="-0.427"/>
-  <xacro:property name="rear_left_rgbd_camera_offset_y" value="0.399"/>
-  <xacro:property name="rear_left_rgbd_camera_offset_z" value="0.994"/>
-  <xacro:property name="lift_position_x" value="0.72328"/>
-  <xacro:property name="lift_position_y" value="0"/>
-  <xacro:property name="lift_position_z" value="0.38"/>
+  <xacro:property name="lift_position_x" value="-0.76"/>
+  <xacro:property name="lift_position_y" value="-0.1"/>
+  <xacro:property name="lift_position_z" value="0.18"/>
   <xacro:property name="lift_orientation_r" value="0"/>
   <xacro:property name="lift_orientation_p" value="0"/>
@@ -59,5 +40,5 @@
   <xacro:rbrobout prefix="$(arg prefix)"  gazebo_classic="$(arg gazebo_classic)" gazebo_ignition="$(arg gazebo_ignition)"/>
   <xacro:top_cover prefix="$(arg prefix)" parent="$(arg prefix)base_link">
-      <origin xyz="0 0 0" rpy="0 0 0"/>
+      <origin xyz="0 0 -0.1" rpy="0 0 0"/>
   </xacro:top_cover>
   <xacro:ewellix_lift_900mm prefix="$(arg prefix)lift_" parent="$(arg prefix)base_link">
@@ -72,5 +53,6 @@
       physical_parameters_file="$(arg physical_params)"
       visual_parameters_file="$(arg visual_params)"
-      sim_gazebo="$(arg gazebo_classic)">
+      sim_gazebo="$(arg gazebo_classic)"
+      sim_ignition="$(arg gazebo_ignition)">
       <origin xyz="0 0 0" rpy="0 0 0"/>
   </xacro:ur_robot>
@@ -84,64 +66,4 @@
         <origin xyz="${imu_offset_x} ${imu_offset_y} ${imu_offset_z}" rpy="0 0 0"/>
     </xacro:sensor_vectornav>
-    <!-- Front Camera -->
-    <xacro:sensor_intel_realsense_d435
-        frame_prefix="$(arg prefix)front_rgbd_camera_"
-        parent="$(arg prefix)base_link"
-        node_namespace="$(arg namespace)"
-        node_name="front_camera"
-        gazebo_classic="$(arg gazebo_classic)"
-        gazebo_ignition="$(arg gazebo_ignition)">
-        <origin xyz="${front_rgbd_camera_offset_x} ${front_rgbd_camera_offset_y} ${front_rgbd_camera_offset_z}" rpy="0 1.0472 0"/>
-    </xacro:sensor_intel_realsense_d435>
-    <!-- Front Right Camera -->
-    <xacro:sensor_intel_realsense_d435
-        frame_prefix="$(arg prefix)front_right_rgbd_camera_"
-        parent="$(arg prefix)base_link"
-        node_namespace="$(arg namespace)"
-        node_name="front_right_camera"
-        gazebo_classic="$(arg gazebo_classic)"
-        gazebo_ignition="$(arg gazebo_ignition)">
-        <origin xyz="${front_right_rgbd_camera_offset_x} ${front_right_rgbd_camera_offset_y} ${front_right_rgbd_camera_offset_z}" rpy="0 1.0472 -${PI/2}"/>
-    </xacro:sensor_intel_realsense_d435>
-    <!-- Front Left Camera -->
-    <xacro:sensor_intel_realsense_d435
-        frame_prefix="$(arg prefix)front_left_rgbd_camera_"
-        parent="$(arg prefix)base_link"
-        node_namespace="$(arg namespace)"
-        node_name="front_left_camera"
-        gazebo_classic="$(arg gazebo_classic)"
-        gazebo_ignition="$(arg gazebo_ignition)">
-        <origin xyz="${front_left_rgbd_camera_offset_x} ${front_left_rgbd_camera_offset_y} ${front_left_rgbd_camera_offset_z}" rpy="0 1.0472 ${PI/2}"/>
-    </xacro:sensor_intel_realsense_d435>
-    <!-- Rear Camera -->
-    <xacro:sensor_intel_realsense_d435
-        frame_prefix="$(arg prefix)rear_rgbd_camera_"
-        parent="$(arg prefix)base_link"
-        node_namespace="$(arg namespace)"
-        node_name="rear_camera"
-        gazebo_classic="$(arg gazebo_classic)"
-        gazebo_ignition="$(arg gazebo_ignition)">
-        <origin xyz="${rear_rgbd_camera_offset_x} ${rear_rgbd_camera_offset_y} ${rear_rgbd_camera_offset_z}" rpy="0 1.0472 ${PI}"/>
-    </xacro:sensor_intel_realsense_d435>
-    <!-- Rear Right Camera -->
-    <xacro:sensor_intel_realsense_d435
-        frame_prefix="$(arg prefix)rear_right_rgbd_camera_"
-        parent="$(arg prefix)base_link"
-        node_namespace="$(arg namespace)"
-        node_name="rear_right_camera"
-        gazebo_classic="$(arg gazebo_classic)"
-        gazebo_ignition="$(arg gazebo_ignition)">
-        <origin xyz="${rear_right_rgbd_camera_offset_x} ${rear_right_rgbd_camera_offset_y} ${rear_right_rgbd_camera_offset_z}" rpy="0 1.0472 -${PI/2}"/>
-    </xacro:sensor_intel_realsense_d435>
-    <!-- Rear Left Camera -->
-    <xacro:sensor_intel_realsense_d435
-        frame_prefix="$(arg prefix)rear_left_rgbd_camera_"
-        parent="$(arg prefix)base_link"
-        node_namespace="$(arg namespace)"
-        node_name="rear_left_camera"
-        gazebo_classic="$(arg gazebo_classic)"
-        gazebo_ignition="$(arg gazebo_ignition)">
-        <origin xyz="${rear_left_rgbd_camera_offset_x} ${rear_left_rgbd_camera_offset_y} ${rear_left_rgbd_camera_offset_z}" rpy="0 1.0472 ${PI/2}"/>
-    </xacro:sensor_intel_realsense_d435>
     <!-- 2d laser -->
     <xacro:sensor_sick_microscan3

Commit message: update structures for rbrobout

File: robots/rbrobout/rbrobout_plus.urdf.xacro (robot description, xacro)
@@ -32,25 +32,7 @@
   <xacro:property name="imu_offset_y" value="-0.3"/>
   <xacro:property name="imu_offset_z" value="0.0725"/>
-  <xacro:property name="front_rgbd_camera_offset_x" value="0.883"/>
-  <xacro:property name="front_rgbd_camera_offset_y" value="0.0"/>
-  <xacro:property name="front_rgbd_camera_offset_z" value="0.887"/>
-  <xacro:property name="front_right_rgbd_camera_offset_x" value="0.089"/>
-  <xacro:property name="front_right_rgbd_camera_offset_y" value="-0.399"/>
-  <xacro:property name="front_right_rgbd_camera_offset_z" value="0.994"/>
-  <xacro:property name="front_left_rgbd_camera_offset_x" value="0.089"/>
-  <xacro:property name="front_left_rgbd_camera_offset_y" value="0.399"/>
-  <xacro:property name="front_left_rgbd_camera_offset_z" value="0.994"/>
-  <xacro:property name="rear_rgbd_camera_offset_x" value="-0.883"/>
-  <xacro:property name="rear_rgbd_camera_offset_y" value="-0.0"/>
-  <xacro:property name="rear_rgbd_camera_offset_z" value="0.769"/>
-  <xacro:property name="rear_right_rgbd_camera_offset_x" value="-0.427"/>
-  <xacro:property name="rear_right_rgbd_camera_offset_y" value="-0.399"/>
-  <xacro:property name="rear_right_rgbd_camera_offset_z" value="0.994"/>
-  <xacro:property name="rear_left_rgbd_camera_offset_x" value="-0.427"/>
-  <xacro:property name="rear_left_rgbd_camera_offset_y" value="0.399"/>
-  <xacro:property name="rear_left_rgbd_camera_offset_z" value="0.994"/>
-  <xacro:property name="lift_position_x" value="0.72328"/>
-  <xacro:property name="lift_position_y" value="0"/>
-  <xacro:property name="lift_position_z" value="0.38"/>
+  <xacro:property name="lift_position_x" value="-0.76"/>
+  <xacro:property name="lift_position_y" value="-0.1"/>
+  <xacro:property name="lift_position_z" value="0.18"/>
   <xacro:property name="lift_orientation_r" value="0"/>
   <xacro:property name="lift_orientation_p" value="0"/>
@@ -58,5 +40,5 @@
   <xacro:rbrobout prefix="$(arg prefix)"  gazebo_classic="$(arg gazebo_classic)" gazebo_ignition="$(arg gazebo_ignition)"/>
   <xacro:top_cover prefix="$(arg prefix)" parent="$(arg prefix)base_link">
-      <origin xyz="0 0 0" rpy="0 0 0"/>
+      <origin xyz="0 0 -0.1" rpy="0 0 0"/>
   </xacro:top_cover>
   <xacro:ewellix_lift_900mm prefix="$(arg prefix)lift_" parent="$(arg prefix)base_link">
@@ -84,64 +66,4 @@
         <origin xyz="${imu_offset_x} ${imu_offset_y} ${imu_offset_z}" rpy="0 0 0"/>
     </xacro:sensor_vectornav>
-    <!-- Front Camera -->
-    <xacro:sensor_intel_realsense_d435
-        frame_prefix="$(arg prefix)front_rgbd_camera_"
-        parent="$(arg prefix)base_link"
-        node_namespace="$(arg namespace)"
-        node_name="front_camera"
-        gazebo_classic="$(arg gazebo_classic)"
-        gazebo_ignition="$(arg gazebo_ignition)">
-        <origin xyz="${front_rgbd_camera_offset_x} ${front_rgbd_camera_offset_y} ${front_rgbd_camera_offset_z}" rpy="0 1.0472 0"/>
-    </xacro:sensor_intel_realsense_d435>
-    <!-- Front Right Camera -->
-    <xacro:sensor_intel_realsense_d435
-        frame_prefix="$(arg prefix)front_right_rgbd_camera_"
-        parent="$(arg prefix)base_link"
-        node_namespace="$(arg namespace)"
-        node_name="front_right_camera"
-        gazebo_classic="$(arg gazebo_classic)"
-        gazebo_ignition="$(arg gazebo_ignition)">
-        <origin xyz="${front_right_rgbd_camera_offset_x} ${front_right_rgbd_camera_offset_y} ${front_right_rgbd_camera_offset_z}" rpy="0 1.0472 -${PI/2}"/>
-    </xacro:sensor_intel_realsense_d435>
-    <!-- Front Left Camera -->
-    <xacro:sensor_intel_realsense_d435
-        frame_prefix="$(arg prefix)front_left_rgbd_camera_"
-        parent="$(arg prefix)base_link"
-        node_namespace="$(arg namespace)"
-        node_name="front_left_camera"
-        gazebo_classic="$(arg gazebo_classic)"
-        gazebo_ignition="$(arg gazebo_ignition)">
-        <origin xyz="${front_left_rgbd_camera_offset_x} ${front_left_rgbd_camera_offset_y} ${front_left_rgbd_camera_offset_z}" rpy="0 1.0472 ${PI/2}"/>
-    </xacro:sensor_intel_realsense_d435>
-    <!-- Rear Camera -->
-    <xacro:sensor_intel_realsense_d435
-        frame_prefix="$(arg prefix)rear_rgbd_camera_"
-        parent="$(arg prefix)base_link"
-        node_namespace="$(arg namespace)"
-        node_name="rear_camera"
-        gazebo_classic="$(arg gazebo_classic)"
-        gazebo_ignition="$(arg gazebo_ignition)">
-        <origin xyz="${rear_rgbd_camera_offset_x} ${rear_rgbd_camera_offset_y} ${rear_rgbd_camera_offset_z}" rpy="0 1.0472 ${PI}"/>
-    </xacro:sensor_intel_realsense_d435>
-    <!-- Rear Right Camera -->
-    <xacro:sensor_intel_realsense_d435
-        frame_prefix="$(arg prefix)rear_right_rgbd_camera_"
-        parent="$(arg prefix)base_link"
-        node_namespace="$(arg namespace)"
-        node_name="rear_right_camera"
-        gazebo_classic="$(arg gazebo_classic)"
-        gazebo_ignition="$(arg gazebo_ignition)">
-        <origin xyz="${rear_right_rgbd_camera_offset_x} ${rear_right_rgbd_camera_offset_y} ${rear_right_rgbd_camera_offset_z}" rpy="0 1.0472 -${PI/2}"/>
-    </xacro:sensor_intel_realsense_d435>
-    <!-- Rear Left Camera -->
-    <xacro:sensor_intel_realsense_d435
-        frame_prefix="$(arg prefix)rear_left_rgbd_camera_"
-        parent="$(arg prefix)base_link"
-        node_namespace="$(arg namespace)"
-        node_name="rear_left_camera"
-        gazebo_classic="$(arg gazebo_classic)"
-        gazebo_ignition="$(arg gazebo_ignition)">
-        <origin xyz="${rear_left_rgbd_camera_offset_x} ${rear_left_rgbd_camera_offset_y} ${rear_left_rgbd_camera_offset_z}" rpy="0 1.0472 ${PI/2}"/>
-    </xacro:sensor_intel_realsense_d435>
     <!-- 2d laser -->
     <xacro:sensor_sick_microscan3

Commit message: humble: update structures for rbrobout (#56)
* update structures for rbrobout

* removed unused meshes

File: robots/rbrobout/rbrobout_plus.urdf.xacro (robot description, xacro)
@@ -7,5 +7,4 @@
   <xacro:include filename="$(find robotnik_description)/urdf/bases/rbrobout/rbrobout_base.urdf.xacro" />
   <xacro:include filename="$(find robotnik_description)/urdf/bases/rbrobout/rbrobout_top_cover.urdf.xacro" />
-  <xacro:include filename="$(find robotnik_description)/urdf/bases/rbrobout/rbrobout_cameras_cover.urdf.xacro" />
   <xacro:include filename="$(find robotnik_description)/urdf/base_hw/rbrobout.ros2_control.urdf" />
   <xacro:include filename="$(find robotnik_description)/simulators/gazebo_classic/rbrobout/rbrobout_control.urdf.xacro" />
@@ -18,5 +17,4 @@
   <xacro:arg name="prefix" default="robot_"/>
   <xacro:arg name="gazebo_classic" default="false"/>
-  <xacro:arg name="gazebo_ignition" default="false"/>
   <xacro:arg name="ur_type" default="ur10e"/>
   <xacro:arg name="joint_limit_params" default="$(find ur_description)/config/$(arg ur_type)/joint_limits.yaml"/>
@@ -33,25 +31,7 @@
   <xacro:property name="imu_offset_y" value="-0.3"/>
   <xacro:property name="imu_offset_z" value="0.0725"/>
-  <xacro:property name="front_rgbd_camera_offset_x" value="0.883"/>
-  <xacro:property name="front_rgbd_camera_offset_y" value="0.0"/>
-  <xacro:property name="front_rgbd_camera_offset_z" value="0.887"/>
-  <xacro:property name="front_right_rgbd_camera_offset_x" value="0.089"/>
-  <xacro:property name="front_right_rgbd_camera_offset_y" value="-0.399"/>
-  <xacro:property name="front_right_rgbd_camera_offset_z" value="0.994"/>
-  <xacro:property name="front_left_rgbd_camera_offset_x" value="0.089"/>
-  <xacro:property name="front_left_rgbd_camera_offset_y" value="0.399"/>
-  <xacro:property name="front_left_rgbd_camera_offset_z" value="0.994"/>
-  <xacro:property name="rear_rgbd_camera_offset_x" value="-0.883"/>
-  <xacro:property name="rear_rgbd_camera_offset_y" value="-0.0"/>
-  <xacro:property name="rear_rgbd_camera_offset_z" value="0.769"/>
-  <xacro:property name="rear_right_rgbd_camera_offset_x" value="-0.427"/>
-  <xacro:property name="rear_right_rgbd_camera_offset_y" value="-0.399"/>
-  <xacro:property name="rear_right_rgbd_camera_offset_z" value="0.994"/>
-  <xacro:property name="rear_left_rgbd_camera_offset_x" value="-0.427"/>
-  <xacro:property name="rear_left_rgbd_camera_offset_y" value="0.399"/>
-  <xacro:property name="rear_left_rgbd_camera_offset_z" value="0.994"/>
-  <xacro:property name="lift_position_x" value="0.72328"/>
-  <xacro:property name="lift_position_y" value="0"/>
-  <xacro:property name="lift_position_z" value="0.38"/>
+  <xacro:property name="lift_position_x" value="-0.76"/>
+  <xacro:property name="lift_position_y" value="-0.1"/>
+  <xacro:property name="lift_position_z" value="0.18"/>
   <xacro:property name="lift_orientation_r" value="0"/>
   <xacro:property name="lift_orientation_p" value="0"/>
@@ -59,5 +39,5 @@
   <xacro:rbrobout prefix="$(arg prefix)"  gazebo_classic="$(arg gazebo_classic)" gazebo_ignition="$(arg gazebo_ignition)"/>
   <xacro:top_cover prefix="$(arg prefix)" parent="$(arg prefix)base_link">
-      <origin xyz="0 0 0" rpy="0 0 0"/>
+      <origin xyz="0 0 -0.1" rpy="0 0 0"/>
   </xacro:top_cover>
   <xacro:ewellix_lift_900mm prefix="$(arg prefix)lift_" parent="$(arg prefix)base_link">
@@ -72,5 +52,6 @@
       physical_parameters_file="$(arg physical_params)"
       visual_parameters_file="$(arg visual_params)"
-      sim_gazebo="$(arg gazebo_classic)">
+      sim_gazebo="$(arg gazebo_classic)"
+      sim_ignition="$(arg gazebo_ignition)">
       <origin xyz="0 0 0" rpy="0 0 0"/>
   </xacro:ur_robot>
@@ -84,64 +65,4 @@
         <origin xyz="${imu_offset_x} ${imu_offset_y} ${imu_offset_z}" rpy="0 0 0"/>
     </xacro:sensor_vectornav>
-    <!-- Front Camera -->
-    <xacro:sensor_intel_realsense_d435
-        frame_prefix="$(arg prefix)front_rgbd_camera_"
-        parent="$(arg prefix)base_link"
-        node_namespace="$(arg namespace)"
-        node_name="front_camera"
-        gazebo_classic="$(arg gazebo_classic)"
-        gazebo_ignition="$(arg gazebo_ignition)">
-        <origin xyz="${front_rgbd_camera_offset_x} ${front_rgbd_camera_offset_y} ${front_rgbd_camera_offset_z}" rpy="0 1.0472 0"/>
-    </xacro:sensor_intel_realsense_d435>
-    <!-- Front Right Camera -->
-    <xacro:sensor_intel_realsense_d435
-        frame_prefix="$(arg prefix)front_right_rgbd_camera_"
-        parent="$(arg prefix)base_link"
-        node_namespace="$(arg namespace)"
-        node_name="front_right_camera"
-        gazebo_classic="$(arg gazebo_classic)"
-        gazebo_ignition="$(arg gazebo_ignition)">
-        <origin xyz="${front_right_rgbd_camera_offset_x} ${front_right_rgbd_camera_offset_y} ${front_right_rgbd_camera_offset_z}" rpy="0 1.0472 -${PI/2}"/>
-    </xacro:sensor_intel_realsense_d435>
-    <!-- Front Left Camera -->
-    <xacro:sensor_intel_realsense_d435
-        frame_prefix="$(arg prefix)front_left_rgbd_camera_"
-        parent="$(arg prefix)base_link"
-        node_namespace="$(arg namespace)"
-        node_name="front_left_camera"
-        gazebo_classic="$(arg gazebo_classic)"
-        gazebo_ignition="$(arg gazebo_ignition)">
-        <origin xyz="${front_left_rgbd_camera_offset_x} ${front_left_rgbd_camera_offset_y} ${front_left_rgbd_camera_offset_z}" rpy="0 1.0472 ${PI/2}"/>
-    </xacro:sensor_intel_realsense_d435>
-    <!-- Rear Camera -->
-    <xacro:sensor_intel_realsense_d435
-        frame_prefix="$(arg prefix)rear_rgbd_camera_"
-        parent="$(arg prefix)base_link"
-        node_namespace="$(arg namespace)"
-        node_name="rear_camera"
-        gazebo_classic="$(arg gazebo_classic)"
-        gazebo_ignition="$(arg gazebo_ignition)">
-        <origin xyz="${rear_rgbd_camera_offset_x} ${rear_rgbd_camera_offset_y} ${rear_rgbd_camera_offset_z}" rpy="0 1.0472 ${PI}"/>
-    </xacro:sensor_intel_realsense_d435>
-    <!-- Rear Right Camera -->
-    <xacro:sensor_intel_realsense_d435
-        frame_prefix="$(arg prefix)rear_right_rgbd_camera_"
-        parent="$(arg prefix)base_link"
-        node_namespace="$(arg namespace)"
-        node_name="rear_right_camera"
-        gazebo_classic="$(arg gazebo_classic)"
-        gazebo_ignition="$(arg gazebo_ignition)">
-        <origin xyz="${rear_right_rgbd_camera_offset_x} ${rear_right_rgbd_camera_offset_y} ${rear_right_rgbd_camera_offset_z}" rpy="0 1.0472 -${PI/2}"/>
-    </xacro:sensor_intel_realsense_d435>
-    <!-- Rear Left Camera -->
-    <xacro:sensor_intel_realsense_d435
-        frame_prefix="$(arg prefix)rear_left_rgbd_camera_"
-        parent="$(arg prefix)base_link"
-        node_namespace="$(arg namespace)"
-        node_name="rear_left_camera"
-        gazebo_classic="$(arg gazebo_classic)"
-        gazebo_ignition="$(arg gazebo_ignition)">
-        <origin xyz="${rear_left_rgbd_camera_offset_x} ${rear_left_rgbd_camera_offset_y} ${rear_left_rgbd_camera_offset_z}" rpy="0 1.0472 ${PI/2}"/>
-    </xacro:sensor_intel_realsense_d435>
     <!-- 2d laser -->
     <xacro:sensor_sick_microscan3
