Commit message: jazzy: update structures for rbrobout (#57)
* update structures for rbrobout

* removed unused meshes

---------

Co-authored-by: Marc Bosch <mbosch@robotnik.es>

File: robots/rbrobout/rbrobout_plus.urdf.xacro (robot description, xacro)
@@ -7,5 +7,4 @@
   <xacro:include filename="$(find robotnik_description)/urdf/bases/rbrobout/rbrobout_base.urdf.xacro" />
   <xacro:include filename="$(find robotnik_description)/urdf/bases/rbrobout/rbrobout_top_cover.urdf.xacro" />
-  <xacro:include filename="$(find robotnik_description)/urdf/bases/rbrobout/rbrobout_cameras_cover.urdf.xacro" />
   <xacro:include filename="$(find robotnik_description)/urdf/base_hw/rbrobout.ros2_control.urdf" />
   <xacro:include filename="$(find robotnik_description)/simulators/gazebo_classic/rbrobout/rbrobout_control.urdf.xacro" />
@@ -33,25 +32,7 @@
   <xacro:property name="imu_offset_y" value="-0.3"/>
   <xacro:property name="imu_offset_z" value="0.0725"/>
-  <xacro:property name="front_rgbd_camera_offset_x" value="0.883"/>
-  <xacro:property name="front_rgbd_camera_offset_y" value="0.0"/>
-  <xacro:property name="front_rgbd_camera_offset_z" value="0.887"/>
-  <xacro:property name="front_right_rgbd_camera_offset_x" value="0.089"/>
-  <xacro:property name="front_right_rgbd_camera_offset_y" value="-0.399"/>
-  <xacro:property name="front_right_rgbd_camera_offset_z" value="0.994"/>
-  <xacro:property name="front_left_rgbd_camera_offset_x" value="0.089"/>
-  <xacro:property name="front_left_rgbd_camera_offset_y" value="0.399"/>
-  <xacro:property name="front_left_rgbd_camera_offset_z" value="0.994"/>
-  <xacro:property name="rear_rgbd_camera_offset_x" value="-0.883"/>
-  <xacro:property name="rear_rgbd_camera_offset_y" value="-0.0"/>
-  <xacro:property name="rear_rgbd_camera_offset_z" value="0.769"/>
-  <xacro:property name="rear_right_rgbd_camera_offset_x" value="-0.427"/>
-  <xacro:property name="rear_right_rgbd_camera_offset_y" value="-0.399"/>
-  <xacro:property name="rear_right_rgbd_camera_offset_z" value="0.994"/>
-  <xacro:property name="rear_left_rgbd_camera_offset_x" value="-0.427"/>
-  <xacro:property name="rear_left_rgbd_camera_offset_y" value="0.399"/>
-  <xacro:property name="rear_left_rgbd_camera_offset_z" value="0.994"/>
-  <xacro:property name="lift_position_x" value="0.72328"/>
-  <xacro:property name="lift_position_y" value="0"/>
-  <xacro:property name="lift_position_z" value="0.38"/>
+  <xacro:property name="lift_position_x" value="-0.76"/>
+  <xacro:property name="lift_position_y" value="-0.1"/>
+  <xacro:property name="lift_position_z" value="0.18"/>
   <xacro:property name="lift_orientation_r" value="0"/>
   <xacro:property name="lift_orientation_p" value="0"/>
@@ -59,5 +40,5 @@
   <xacro:rbrobout prefix="$(arg prefix)"  gazebo_classic="$(arg gazebo_classic)" gazebo_ignition="$(arg gazebo_ignition)"/>
   <xacro:top_cover prefix="$(arg prefix)" parent="$(arg prefix)base_link">
-      <origin xyz="0 0 0" rpy="0 0 0"/>
+      <origin xyz="0 0 -0.1" rpy="0 0 0"/>
   </xacro:top_cover>
   <xacro:ewellix_lift_900mm prefix="$(arg prefix)lift_" parent="$(arg prefix)base_link">
@@ -85,64 +66,4 @@
         <origin xyz="${imu_offset_x} ${imu_offset_y} ${imu_offset_z}" rpy="0 0 0"/>
     </xacro:sensor_vectornav>
-    <!-- Front Camera -->
-    <xacro:sensor_intel_realsense_d435
-        frame_prefix="$(arg prefix)front_rgbd_camera_"
-        parent="$(arg prefix)base_link"
-        node_namespace="$(arg namespace)"
-        node_name="front_camera"
-        gazebo_classic="$(arg gazebo_classic)"
-        gazebo_ignition="$(arg gazebo_ignition)">
-        <origin xyz="${front_rgbd_camera_offset_x} ${front_rgbd_camera_offset_y} ${front_rgbd_camera_offset_z}" rpy="0 1.0472 0"/>
-    </xacro:sensor_intel_realsense_d435>
-    <!-- Front Right Camera -->
-    <xacro:sensor_intel_realsense_d435
-        frame_prefix="$(arg prefix)front_right_rgbd_camera_"
-        parent="$(arg prefix)base_link"
-        node_namespace="$(arg namespace)"
-        node_name="front_right_camera"
-        gazebo_classic="$(arg gazebo_classic)"
-        gazebo_ignition="$(arg gazebo_ignition)">
-        <origin xyz="${front_right_rgbd_camera_offset_x} ${front_right_rgbd_camera_offset_y} ${front_right_rgbd_camera_offset_z}" rpy="0 1.0472 -${PI/2}"/>
-    </xacro:sensor_intel_realsense_d435>
-    <!-- Front Left Camera -->
-    <xacro:sensor_intel_realsense_d435
-        frame_prefix="$(arg prefix)front_left_rgbd_camera_"
-        parent="$(arg prefix)base_link"
-        node_namespace="$(arg namespace)"
-        node_name="front_left_camera"
-        gazebo_classic="$(arg gazebo_classic)"
-        gazebo_ignition="$(arg gazebo_ignition)">
-        <origin xyz="${front_left_rgbd_camera_offset_x} ${front_left_rgbd_camera_offset_y} ${front_left_rgbd_camera_offset_z}" rpy="0 1.0472 ${PI/2}"/>
-    </xacro:sensor_intel_realsense_d435>
-    <!-- Rear Camera -->
-    <xacro:sensor_intel_realsense_d435
-        frame_prefix="$(arg prefix)rear_rgbd_camera_"
-        parent="$(arg prefix)base_link"
-        node_namespace="$(arg namespace)"
-        node_name="rear_camera"
-        gazebo_classic="$(arg gazebo_classic)"
-        gazebo_ignition="$(arg gazebo_ignition)">
-        <origin xyz="${rear_rgbd_camera_offset_x} ${rear_rgbd_camera_offset_y} ${rear_rgbd_camera_offset_z}" rpy="0 1.0472 ${PI}"/>
-    </xacro:sensor_intel_realsense_d435>
-    <!-- Rear Right Camera -->
-    <xacro:sensor_intel_realsense_d435
-        frame_prefix="$(arg prefix)rear_right_rgbd_camera_"
-        parent="$(arg prefix)base_link"
-        node_namespace="$(arg namespace)"
-        node_name="rear_right_camera"
-        gazebo_classic="$(arg gazebo_classic)"
-        gazebo_ignition="$(arg gazebo_ignition)">
-        <origin xyz="${rear_right_rgbd_camera_offset_x} ${rear_right_rgbd_camera_offset_y} ${rear_right_rgbd_camera_offset_z}" rpy="0 1.0472 -${PI/2}"/>
-    </xacro:sensor_intel_realsense_d435>
-    <!-- Rear Left Camera -->
-    <xacro:sensor_intel_realsense_d435
-        frame_prefix="$(arg prefix)rear_left_rgbd_camera_"
-        parent="$(arg prefix)base_link"
-        node_namespace="$(arg namespace)"
-        node_name="rear_left_camera"
-        gazebo_classic="$(arg gazebo_classic)"
-        gazebo_ignition="$(arg gazebo_ignition)">
-        <origin xyz="${rear_left_rgbd_camera_offset_x} ${rear_left_rgbd_camera_offset_y} ${rear_left_rgbd_camera_offset_z}" rpy="0 1.0472 ${PI/2}"/>
-    </xacro:sensor_intel_realsense_d435>
     <!-- 2d laser -->
     <xacro:sensor_sick_microscan3

Commit message: changes added

File: robots/rbrobout/rbrobout_plus.urdf.xacro (robot description, xacro)
@@ -13,18 +13,17 @@
   <xacro:include
     filename="$(find robotnik_sensors)/urdf/all_sensors.urdf.xacro" />
+  <xacro:include
+    filename="$(find robotnik_sensors)/urdf/depth/intel_realsense_d435.urdf.xacro" />
+  <xacro:include
+    filename="$(find robotnik_sensors)/urdf/depth/intel_realsense_d435i.urdf.xacro" />
+  <xacro:include
+    filename="$(find robotnik_description)/urdf/grippers/suction_gripper/suction_gripper.urdf.xacro" />
   <!-- ARGUMENTS -->
-  <xacro:arg
-    name="namespace"
-    default="robot" />
-  <xacro:arg
-    name="prefix"
-    default="" />
-  <xacro:arg
-    name="gazebo_ignition"
-    default="false" />
-  <xacro:arg
-    name="ur_type"
-    default="ur5e" />
-  <!-- RB-ROBOUT -->
+  <xacro:arg name="namespace"      default="robot" />
+  <xacro:arg name="prefix"         default="" />
+  <xacro:arg name="gazebo_ignition" default="false" />
+  <xacro:arg name="ur_type"        default="ur5e" />
+  <xacro:arg name="world_name" default="room_test_world"/>
+  <!-- RB-ROBOUT BASE -->
   <xacro:rbrobout
     prefix="$(arg prefix)"
@@ -34,16 +33,12 @@
     prefix="$(arg prefix)"
     parent="$(arg prefix)base_link">
-    <origin
-      xyz="0 0 -0.1"
-      rpy="0 0 0" />
+    <origin xyz="0 0 -0.1" rpy="0 0 0" />
   </xacro:top_cover>
   <xacro:ewellix_lift_900mm
     prefix="$(arg prefix)lift_"
     parent="$(arg prefix)base_link">
-    <origin
-      xyz="-0.76 0.0 0.18"
-      rpy="0 0 0" />
+    <origin xyz="-0.76 0.0 0.18" rpy="0 0 0" />
   </xacro:ewellix_lift_900mm>
-  <!-- ARMS -->
+  <!-- ARM -->
   <xacro:arm_ur
     ur_type="$(arg ur_type)"
@@ -51,8 +46,22 @@
     parent="$(arg prefix)lift_ewellix_lift_top_link"
     gazebo_ignition="$(arg gazebo_ignition)">
-    <origin
-      xyz="0 0 0"
-      rpy="0 0 0" />
+    <origin xyz="0 0 0" rpy="0 0 0" />
   </xacro:arm_ur>
+  <!-- WRIST CAMERA -->
+  <xacro:sensor_intel_realsense_d435i
+    frame_prefix="$(arg prefix)wrist_rgbd_camera_"
+    parent="$(arg prefix)arm_tool0"
+    node_namespace="$(arg namespace)"
+    node_name="wrist_camera"
+    gazebo_ignition="$(arg gazebo_ignition)">
+    <origin xyz="0.0 -0.055 0.020" rpy="0 -1.5708 1.5708" />
+  </xacro:sensor_intel_realsense_d435i>
+  <!-- SUCTION GRIPPER -->
+  <xacro:suction_gripper
+    prefix="$(arg prefix)vacuum_"
+    parent="$(arg prefix)arm_tool0"
+    ns="$(arg namespace)">
+    <origin xyz="0 0 0" rpy="0 0 0" />
+  </xacro:suction_gripper>
   <!-- IMU -->
   <xacro:sensor_vectornav
@@ -61,7 +70,5 @@
     node_namespace="$(arg namespace)"
     gazebo_ignition="$(arg gazebo_ignition)">
-    <origin
-      xyz="0.3 -0.3 0.0725"
-      rpy="0 0 0" />
+    <origin xyz="0.3 -0.3 0.0725" rpy="0 0 0" />
   </xacro:sensor_vectornav>
   <!-- LASERS -->
@@ -74,7 +81,5 @@
     max_angle="2.1"
     min_angle="-2.1">
-    <origin
-      xyz="0.8 0.366 -0.06"
-      rpy="0 0 ${1/4*pi}" />
+    <origin xyz="0.8 0.366 -0.06" rpy="0 0 ${1/4*pi}" />
   </xacro:sensor_sick_microscan3>
   <xacro:sensor_sick_microscan3
@@ -86,9 +91,7 @@
     max_angle="2.1"
     min_angle="-2.1">
-    <origin
-      xyz="-0.8 -0.366 -0.06"
-      rpy="0 0 ${-3/4*pi}" />
+    <origin xyz="-0.8 -0.366 -0.06" rpy="0 0 ${-3/4*pi}" />
   </xacro:sensor_sick_microscan3>
-  <!-- CAMERAS -->
+  <!-- FRONT CAMERA -->
   <xacro:sensor_intel_realsense_d435
     frame_prefix="$(arg prefix)front_rgbd_camera_"
@@ -97,7 +100,15 @@
     node_name="front_camera"
     gazebo_ignition="$(arg gazebo_ignition)">
-    <origin
-      xyz="0.835 0 0.1555"
-      rpy="0 0 0" />
+    <origin xyz="0.835 0 0.1555" rpy="0 0 0" />
   </xacro:sensor_intel_realsense_d435>
+  <!-- VACUUM GRIPPER PLUGIN -->
+  <gazebo>
+    <plugin filename="libVacuumGripper.so"
+            name="vacuum_gripper_plugin::VacuumGripper">
+      <suction_link>$(arg prefix)vacuum_link_suction_gripper</suction_link>
+      <contact_topic>/world/$(arg world_name)/model/$(arg namespace)/link/$(arg prefix)vacuum_link_suction_gripper/sensor/$(arg prefix)vacuum_suction_contact_sensor/contact</contact_topic>
+      <cmd_topic>/$(arg namespace)/vacuum_on</cmd_topic>
+      <max_distance>0.15</max_distance>
+    </plugin>
+  </gazebo>
 </robot>

File: urdf/arms/ur_macro.urdf.xacro (robot description, xacro)
@@ -34,13 +34,20 @@
       kinematics_parameters_file="${kinematics_params}"
       physical_parameters_file="${physical_params}"
-      visual_parameters_file="${visual_params}">
+      visual_parameters_file="${visual_params}"
+      generate_ros2_control_tag="false">
       <xacro:insert_block name="origin" />
     </xacro:ur_robot>
     <xacro:if value="$(arg gazebo_ignition)">
       <xacro:include
-        filename="$(find ur_simulation_gz)/urdf/ur_gz.ros2_control.xacro" />
+        filename="$(find ur_description)/urdf/ur.ros2_control.xacro" />
       <xacro:ur_ros2_control
-        name="${frame_prefix}"
-        tf_prefix="${frame_prefix}" />
+        name="arm"
+        sim_ignition="true"
+        tf_prefix="${frame_prefix}"
+        script_filename=""
+        output_recipe_filename=""
+        input_recipe_filename=""
+        hash_kinematics=""
+        robot_ip="" />
     </xacro:if>
   </xacro:macro>
