Commit message: removed old robot_id parameter

File: urdf/bases/rbsummit/rbsummit_base.xacro (robot description, xacro)
@@ -17,14 +17,14 @@
 		<xacro:rbsummit_body prefix="${prefix}" hq="${hq}" />
 		<!-- Summit XL wheels -->
-		<xacro:rubber_wheel robot_id="${prefix}front_right" parent="${prefix}base_link" reflect="false" hq="${hq}">
+		<xacro:rubber_wheel prefix="${prefix}front_right_" parent="${prefix}base_link" reflect="false" hq="${hq}">
 			<origin xyz="${wheel_offset_x} -${wheel_offset_y} ${wheel_offset_z}" rpy="0 0 0"/>
 		</xacro:rubber_wheel>
-		<xacro:rubber_wheel robot_id="${prefix}front_left" parent="${prefix}base_link" reflect="true" hq="${hq}">
+		<xacro:rubber_wheel prefix="${prefix}front_left_" parent="${prefix}base_link" reflect="true" hq="${hq}">
 			<origin xyz="${wheel_offset_x} ${wheel_offset_y} ${wheel_offset_z}" rpy="0 0 0"/>
 		</xacro:rubber_wheel>
-		<xacro:rubber_wheel robot_id="${prefix}back_left" parent="${prefix}base_link" reflect="true" hq="${hq}">
+		<xacro:rubber_wheel prefix="${prefix}back_left_" parent="${prefix}base_link" reflect="true" hq="${hq}">
 			<origin xyz="-${wheel_offset_x} ${wheel_offset_y} ${wheel_offset_z}" rpy="0 0 0"/>
 		</xacro:rubber_wheel>
-		<xacro:rubber_wheel robot_id="${prefix}back_right" parent="${prefix}base_link" reflect="false" hq="${hq}">
+		<xacro:rubber_wheel prefix="${prefix}back_right_" parent="${prefix}base_link" reflect="false" hq="${hq}">
 			<origin xyz="-${wheel_offset_x} -${wheel_offset_y} ${wheel_offset_z}" rpy="0 0 0"/>
 		</xacro:rubber_wheel>

File: urdf/bases/rbtheron/rbtheron_base.xacro (robot description, xacro)
@@ -23,21 +23,21 @@
 		<xacro:rbtheron_body prefix="${prefix}" hq="${hq}" />
 		<!-- WHEELS -->
-		<xacro:rubber_wheel robot_id="${prefix}right" parent="${prefix}base_link" hq="${hq}">
+		<xacro:rubber_wheel prefix="${prefix}right_" parent="${prefix}base_link" hq="${hq}">
 			<origin xyz="${wheel_offset_x} ${-wheel_offset_y} ${wheel_offset_z}" rpy="0 0 0"/>
 		</xacro:rubber_wheel>
-		<xacro:rubber_wheel robot_id="${prefix}left" parent="${prefix}base_link" hq="${hq}">
+		<xacro:rubber_wheel prefix="${prefix}left_" parent="${prefix}base_link" hq="${hq}">
 			<origin xyz="${wheel_offset_x} ${wheel_offset_y} ${wheel_offset_z}" rpy="0 0 0"/>
 		</xacro:rubber_wheel>
 		<!-- Castor wheels-->
-		<xacro:caster robot_id="${prefix}front_left" parent="${prefix}base_link" hq="${hq}" use_sim="true">
+		<xacro:caster prefix="${prefix}front_left_" parent="${prefix}base_link" hq="${hq}" use_sim="true">
 			<origin xyz="${castor_offset_x} ${castor_offset_y} ${castor_offset_z}" rpy="0 0 0"/>
 		</xacro:caster>
-		<xacro:caster robot_id="${prefix}front_right" parent="${prefix}base_link" hq="${hq}" use_sim="true">
+		<xacro:caster prefix="${prefix}front_right_" parent="${prefix}base_link" hq="${hq}" use_sim="true">
 			<origin xyz="${castor_offset_x} ${-castor_offset_y} ${castor_offset_z}" rpy="0 0 0"/>
 		</xacro:caster>
-		<xacro:caster robot_id="${prefix}rear_left" parent="${prefix}base_link" hq="${hq}" use_sim="true">
+		<xacro:caster prefix="${prefix}rear_left_" parent="${prefix}base_link" hq="${hq}" use_sim="true">
 			<origin xyz="${-castor_offset_x} ${castor_offset_y} ${castor_offset_z}" rpy="0 0 0"/>
 		</xacro:caster>
-		<xacro:caster robot_id="${prefix}rear_right" parent="${prefix}base_link" hq="${hq}" use_sim="true">
+		<xacro:caster prefix="${prefix}rear_right_" parent="${prefix}base_link" hq="${hq}" use_sim="true">
 			<origin xyz="${-castor_offset_x} ${-castor_offset_y} ${castor_offset_z}" rpy="0 0 0"/>
 		</xacro:caster>

File: urdf/wheels/rubber_wheel/rubber_wheel.urdf.xacro (robot description, xacro)
@@ -7,9 +7,9 @@
               izz="${m*(3*r*r+h*h)/12}" />
   </xacro:macro>
-  <xacro:macro name="rubber_wheel" params="robot_id parent *origin reflect hq rubber_wheel_radius:=0.11 rubber_wheel_width:=0.15 rubber_wheel_mass:=6.5">
+  <xacro:macro name="rubber_wheel" params="prefix parent *origin reflect hq rubber_wheel_radius:=0.11 rubber_wheel_width:=0.15 rubber_wheel_mass:=6.5">
 <!--WHEEL TIRE -->
-    <joint name="${robot_id}_wheel_joint" type="continuous">
+    <joint name="${prefix}wheel_joint" type="continuous">
       <parent link="${parent}"/>
-      <child link="${robot_id}_wheel"/>
+      <child link="${prefix}wheel"/>
       <xacro:insert_block name="origin" />
       <axis xyz="0 1 0" rpy="0 0 0" />
@@ -17,5 +17,5 @@
       <joint_properties damping="0.5" friction="2.0"/>
     </joint>
-    <link name="${robot_id}_wheel">
+    <link name="${prefix}wheel">
       <visual>
         <!-- HIGH RESOLUTION WHEELS -->
@@ -51,5 +51,5 @@
       </inertial>
     </link>
-    <gazebo reference="${robot_id}_wheel">
+    <gazebo reference="${prefix}wheel">
 			<!-- <material>Gazebo/Black</material> -->
       <mu1>0.9</mu1>
