Commit message: remove unused arg in axis tag

File: urdf/wheels/caster_wheel/rbtheron_caster.urdf.xacro (robot description, xacro)
@@ -25,5 +25,5 @@
         <child link="${prefix}support"/>
         <xacro:insert_block name="origin" />
-        <axis xyz="0 0 1" rpy="0 ${M_PI} 0" />
+        <axis xyz="0 0 1" />
         <limit effort="100" velocity="100"/>
         <dynamics damping="0.8" friction="0.01"/>
@@ -35,5 +35,5 @@
           <child link="${prefix}support"/>
           <xacro:insert_block name="origin" />
-          <axis xyz="0 0 1" rpy="0 ${M_PI} 0" />
+          <axis xyz="0 0 1" />
           <dynamics damping="0" friction="0.01"/>
         </joint>
@@ -62,5 +62,5 @@
       <child link="${prefix}wheel"/>
       <origin xyz="-0.033 0.0 -0.071" rpy="0 0 0"/>
-      <axis xyz="0 1 0" rpy="0 0 0" />
+      <axis xyz="0 1 0" />
       <limit effort="100" velocity="100"/>
       <joint_properties damping="0.2" friction="2.0"/>
@@ -72,5 +72,5 @@
        <child link="${prefix}wheel"/>
       <origin xyz="-0.033 0.0 -0.07" rpy="0 0 0"/>
-       <axis xyz="0 1 0" rpy="0 0 0" />
+       <axis xyz="0 1 0" />
        <joint_properties damping="0.1" friction="0.1"/>
     </joint>

File: urdf/wheels/omni_wheel/rbkairos_omni_wheel.urdf.xacro (robot description, xacro)
@@ -16,5 +16,5 @@
             <child link="${prefix}wheel_link" />
             <xacro:insert_block name="origin" />
-            <axis xyz="0 1 0" rpy="0 0 0" />
+            <axis xyz="0 1 0" />
             <limit effort="100000" velocity="100" />
             <!-- <joint_properties damping="1.0" friction="1.0"/> -->

File: urdf/wheels/omni_wheel/rbrobout_omni_wheel.urdf.xacro (robot description, xacro)
@@ -16,5 +16,5 @@
             <child link="${prefix}wheel_link" />
             <xacro:insert_block name="origin" />
-            <axis xyz="0 1 0" rpy="0 0 0" />
+            <axis xyz="0 1 0" />
             <limit effort="100000" velocity="100" />
             <!-- <joint_properties damping="1.0" friction="1.0"/> -->

File: urdf/wheels/rubber_wheel/rubber_wheel.urdf.xacro (robot description, xacro)
@@ -13,5 +13,5 @@
       <child link="${prefix}wheel"/>
       <xacro:insert_block name="origin" />
-      <axis xyz="0 1 0" rpy="0 0 0" />
+      <axis xyz="0 1 0" />
       <limit effort="100" velocity="100"/>
       <joint_properties damping="0.5" friction="2.0"/>

File: urdf/wheels/rubber_wheel/rubber_wheel_150.urdf.xacro (robot description, xacro)
@@ -21,5 +21,5 @@
 			<child link="${prefix}wheel_link"/>
 			<xacro:insert_block name="origin" />
-			<axis xyz="0 1 0" rpy="0 0 0" />
+			<axis xyz="0 1 0" />
 			<limit effort="100" velocity="100"/>
 			<joint_properties damping="0.0" friction="0.0"/>

File: urdf/wheels/steering_wheel/steering_wheel.urdf.xacro (robot description, xacro)
@@ -20,5 +20,5 @@
       <child link="${prefix}base_wheel"/>
       <xacro:insert_block name="origin" />
-      <axis xyz="0 0 1" rpy="0 0 0" />
+      <axis xyz="0 0 1"/>
       <limit effort="${steer_joint_effort_limit}" velocity="${steer_joint_velocity_limit}" lower="-3.00" upper="3.00"/>
       <dynamics damping="${steer_joint_damping}" friction="${steer_joint_friction}"/>
