Commit message: remove spanish names from rbkairos

File: urdf/bodies/rbkairos/rbkairos_plus_body.urdf.xacro (robot description, xacro)
@@ -46,9 +46,9 @@
   </gazebo>
   <!-- CHAPAS INOX TAPAS -->
-  <link name="${prefix}base_chapa">
+  <link name="${prefix}top_cover">
   <visual>
     <origin xyz="0 0 0" rpy="0 0 0" />
     <geometry>
-      <mesh filename="package://robotnik_description/meshes/bases/rbkairos/rbkairos_chapas_inox_tapas.stl"/>
+      <mesh filename="package://robotnik_description/meshes/bases/rbkairos/rbkairos_top_cover.stl"/>
     </geometry>
     <material name="darkgrey">
@@ -60,7 +60,7 @@
     <origin xyz="0.0 0 0.56162" rpy="0 0 0" />
     <parent link="${prefix}base_link"/>
-    <child link="${prefix}base_chapa" />
+    <child link="${prefix}top_cover" />
   </joint>
-  <!-- LOGO ROBOTNIK IZQUIERDO -->
+  <!-- LOGO ROBOTNIK LEFT -->
   <link name="${prefix}base_logo_left">
   <visual>
@@ -79,5 +79,5 @@
     <child link="${prefix}base_logo_left" />
   </joint>
-  <!-- LOGO ROBOTNIK DERECHO -->
+  <!-- LOGO ROBOTNIK RIGHT -->
   <link name="${prefix}base_logo_right">
   <visual>
@@ -96,5 +96,5 @@
     <child link="${prefix}base_logo_right" />
   </joint>
-  <!-- LOGO ROBOTNIK FRONTAL -->
+  <!-- LOGO ROBOTNIK FRONT -->
   <link name="${prefix}base_logo_front">
   <visual>
@@ -113,5 +113,5 @@
     <child link="${prefix}base_logo_front" />
   </joint>
-  <!-- LOGO ROBOTNIK TRASERO -->
+  <!-- LOGO ROBOTNIK REAR -->
   <link name="${prefix}base_logo_rear">
   <visual>
