Commit message: change name to mecanum wheels
Signed-off-by: cgasconb <cgascon@robotnik.es>

File: urdf/bases/rbkairos/rbkairos_base.urdf.xacro (robot description, xacro)
@@ -7,5 +7,5 @@
   	<!-- Import summit XL base elements -->
 	<xacro:include filename="$(find robotnik_description)/urdf/bodies/rbkairos/rbkairos_plus_body.urdf.xacro" />
-  	<xacro:include filename="$(find robotnik_description)/urdf/wheels/omni_wheel/rbkairos_omni_wheel.urdf.xacro" />
+  	<xacro:include filename="$(find robotnik_description)/urdf/wheels/mecanum_wheel/rbkairos_mecanum_wheel.urdf.xacro" />
   	<xacro:property name="PI" value="3.1415926535897931"/>
   	<!-- Wheel parameters -->
@@ -19,16 +19,16 @@
   		<!-- Here we create the robot elements using the xacro:macros imported at the beggining of this file -->
   		<xacro:rbkairos_plus_body prefix="${prefix}"/>
-  		<xacro:omni_wheel prefix="${prefix}front_right_" parent="${prefix}base_link" reflect="false" hq="true">
+  		<xacro:mecanum_wheel prefix="${prefix}front_right_" parent="${prefix}base_link" reflect="false" hq="true">
   			<origin xyz="${wheel_offset_x} -${wheel_offset_y} ${wheel_offset_z}" rpy="0 0 ${PI/4}"/>
-  		</xacro:omni_wheel>
-  		<xacro:omni_wheel prefix="${prefix}front_left_" parent="${prefix}base_link" reflect="true" hq="true">
+  		</xacro:mecanum_wheel>
+  		<xacro:mecanum_wheel prefix="${prefix}front_left_" parent="${prefix}base_link" reflect="true" hq="true">
   			<origin xyz="${wheel_offset_x} ${wheel_offset_y} ${wheel_offset_z}" rpy="0 0 ${-PI/4}"/>
-  		</xacro:omni_wheel>
-  		<xacro:omni_wheel prefix="${prefix}back_left_" parent="${prefix}base_link" reflect="false" hq="true">
+  		</xacro:mecanum_wheel>
+  		<xacro:mecanum_wheel prefix="${prefix}back_left_" parent="${prefix}base_link" reflect="false" hq="true">
   			<origin xyz="-${wheel_offset_x} ${wheel_offset_y} ${wheel_offset_z}" rpy="0 0 ${PI/4}"/>
-  		</xacro:omni_wheel>
-  		<xacro:omni_wheel prefix="${prefix}back_right_" parent="${prefix}base_link" reflect="true" hq="true">
+  		</xacro:mecanum_wheel>
+  		<xacro:mecanum_wheel prefix="${prefix}back_right_" parent="${prefix}base_link" reflect="true" hq="true">
   			<origin xyz="-${wheel_offset_x} -${wheel_offset_y} ${wheel_offset_z}" rpy="0 0 ${-PI/4}"/>
-  		</xacro:omni_wheel>
+  		</xacro:mecanum_wheel>
      </xacro:macro>
 </robot>

File: urdf/bases/rbrobout/rbrobout_base.urdf.xacro (robot description, xacro)
@@ -8,5 +8,5 @@
 	<xacro:include filename="$(find robotnik_description)/urdf/bodies/rbrobout/rbrobout_body.urdf.xacro" />
 	<!-- Import RB-Robout wheels -->
-  	<xacro:include filename="$(find robotnik_description)/urdf/wheels/omni_wheel/rbrobout_omni_wheel.urdf.xacro" />
+  	<xacro:include filename="$(find robotnik_description)/urdf/wheels/mecanum_wheel/rbrobout_mecanum_wheel.urdf.xacro" />
 	<!-- Import all available sensors -->
 	<xacro:include filename="$(find robotnik_sensors)/urdf/all_sensors.urdf.xacro" />
@@ -25,16 +25,16 @@
 		<xacro:rbrobout_body prefix="${prefix}" />
 		<!-- Wheels -->
-		<xacro:rbrobout_omni_wheel prefix="${prefix}front_right_" parent="${prefix}base_link" reflect="false" hq="${hq}">
+		<xacro:rbrobout_mecanum_wheel prefix="${prefix}front_right_" parent="${prefix}base_link" reflect="false" hq="${hq}">
 			<origin xyz="${wheel_offset_x} -${wheel_offset_y} ${wheel_offset_z}" rpy="0 0 ${PI/4}"/>
-		</xacro:rbrobout_omni_wheel>
-		<xacro:rbrobout_omni_wheel prefix="${prefix}front_left_" parent="${prefix}base_link" reflect="true" hq="${hq}">
+		</xacro:rbrobout_mecanum_wheel>
+		<xacro:rbrobout_mecanum_wheel prefix="${prefix}front_left_" parent="${prefix}base_link" reflect="true" hq="${hq}">
 			<origin xyz="${wheel_offset_x} ${wheel_offset_y} ${wheel_offset_z}" rpy="0 0 ${-PI/4}"/>
-		</xacro:rbrobout_omni_wheel>
-		<xacro:rbrobout_omni_wheel prefix="${prefix}back_left_" parent="${prefix}base_link" reflect="false" hq="${hq}">
+		</xacro:rbrobout_mecanum_wheel>
+		<xacro:rbrobout_mecanum_wheel prefix="${prefix}back_left_" parent="${prefix}base_link" reflect="false" hq="${hq}">
 			<origin xyz="-${wheel_offset_x} ${wheel_offset_y} ${wheel_offset_z}" rpy="0 0 ${PI/4}"/>
-		</xacro:rbrobout_omni_wheel>
-		<xacro:rbrobout_omni_wheel prefix="${prefix}back_right_" parent="${prefix}base_link" reflect="true" hq="${hq}">
+		</xacro:rbrobout_mecanum_wheel>
+		<xacro:rbrobout_mecanum_wheel prefix="${prefix}back_right_" parent="${prefix}base_link" reflect="true" hq="${hq}">
 			<origin xyz="-${wheel_offset_x} -${wheel_offset_y} ${wheel_offset_z}" rpy="0 0 ${-PI/4}"/>
-		</xacro:rbrobout_omni_wheel>
+		</xacro:rbrobout_mecanum_wheel>
    </xacro:macro>
 </robot>

File: urdf/wheels/mecanum_wheel/rbkairos_mecanum_wheel.urdf.xacro (robot description, xacro)
@@ -3,7 +3,7 @@
     <xacro:property name="M_PI" value="3.1415926535897931" />
     <!-- Wheels -->
-    <xacro:property name="omni_wheel_radius" value="0.127" />
-    <xacro:property name="omni_wheel_height" value="0.087" />
-    <xacro:property name="omni_wheel_mass" value="6.5" /> <!-- in kg-->
+    <xacro:property name="mecanum_wheel_radius" value="0.127" />
+    <xacro:property name="mecanum_wheel_height" value="0.087" />
+    <xacro:property name="mecanum_wheel_mass" value="6.5" /> <!-- in kg-->
     <xacro:macro name="cylinder_inertia" params="m r h">
         <inertia ixx="${m*(3*r*r+h*h)/12}" ixy="0" ixz="0"
@@ -11,5 +11,5 @@
             izz="${m*(3*r*r+h*h)/12}" />
     </xacro:macro>
-    <xacro:macro name="omni_wheel" params="prefix parent *origin reflect hq">
+    <xacro:macro name="mecanum_wheel" params="prefix parent *origin reflect hq">
         <joint name="${prefix}wheel_joint" type="continuous">
             <parent link="${parent}" />
@@ -33,12 +33,12 @@
                 <origin xyz="0 0 0" rpy="0 0 0" />
                 <geometry>
-                    <sphere radius="${omni_wheel_radius}" />
+                    <sphere radius="${mecanum_wheel_radius}" />
                 </geometry>
             </collision>
             <inertial>
-                <mass value="${omni_wheel_mass}" />
+                <mass value="${mecanum_wheel_mass}" />
                 <origin xyz="0 0 0" />
-                <xacro:cylinder_inertia m="${omni_wheel_mass}" r="${omni_wheel_radius}"
-                    h="${omni_wheel_height}" />
+                <xacro:cylinder_inertia m="${mecanum_wheel_mass}" r="${mecanum_wheel_radius}"
+                    h="${mecanum_wheel_height}" />
             </inertial>
         </link>
@@ -75,5 +75,5 @@
                         <geometry>
                             <mesh
-                                filename="package://robotnik_description/meshes/wheels/omni_wheel/omni_wheel_1.dae" />
+                                filename="package://robotnik_description/meshes/wheels/mecanum_wheel/mecanum_wheel_1.dae" />
                         </geometry>
                     </xacro:if>
@@ -82,5 +82,5 @@
                         <geometry>
                             <mesh
-                                filename="package://robotnik_description/meshes/wheels/omni_wheel/omni_wheel_2.dae" />
+                                filename="package://robotnik_description/meshes/wheels/mecanum_wheel/mecanum_wheel_2.dae" />
                         </geometry>
                     </xacro:unless>
@@ -89,5 +89,5 @@
                     <origin xyz="0 0 0" rpy="0 0 0" />
                     <geometry>
-                        <sphere radius="${omni_wheel_radius}" />
+                        <sphere radius="${mecanum_wheel_radius}" />
                     </geometry>
                 </xacro:unless>
@@ -103,8 +103,8 @@
             </collision>
             <inertial>
-                <mass value="${omni_wheel_mass}" />
+                <mass value="${mecanum_wheel_mass}" />
                 <origin xyz="0 0 0" />
-                <xacro:cylinder_inertia m="${omni_wheel_mass}" r="${omni_wheel_radius}"
-                    h="${omni_wheel_height}" />
+                <xacro:cylinder_inertia m="${mecanum_wheel_mass}" r="${mecanum_wheel_radius}"
+                    h="${mecanum_wheel_height}" />
             </inertial>
         </link>

File: urdf/wheels/mecanum_wheel/rbrobout_mecanum_wheel.urdf.xacro (robot description, xacro)
@@ -3,7 +3,7 @@
     <xacro:property name="M_PI" value="3.1415926535897931" />
     <!-- Wheels -->
-    <xacro:property name="omni_wheel_radius" value="0.127" />
-    <xacro:property name="omni_wheel_height" value="0.087" />
-    <xacro:property name="omni_wheel_mass" value="6.5" /> <!-- in kg-->
+    <xacro:property name="mecanum_wheel_radius" value="0.127" />
+    <xacro:property name="mecanum_wheel_height" value="0.087" />
+    <xacro:property name="mecanum_wheel_mass" value="6.5" /> <!-- in kg-->
     <xacro:macro name="cylinder_inertia" params="m r h">
         <inertia ixx="${m*(3*r*r+h*h)/12}" ixy="0" ixz="0"
@@ -11,5 +11,5 @@
             izz="${m*(3*r*r+h*h)/12}" />
     </xacro:macro>
-    <xacro:macro name="rbrobout_omni_wheel" params="prefix parent *origin reflect hq">
+    <xacro:macro name="rbrobout_mecanum_wheel" params="prefix parent *origin reflect hq">
         <joint name="${prefix}wheel_joint" type="continuous">
             <parent link="${parent}" />
@@ -33,12 +33,12 @@
                 <origin xyz="0 0 0" rpy="0 0 0" />
                 <geometry>
-                    <sphere radius="${omni_wheel_radius}" />
+                    <sphere radius="${mecanum_wheel_radius}" />
                 </geometry>
             </collision>
             <inertial>
-                <mass value="${omni_wheel_mass}" />
+                <mass value="${mecanum_wheel_mass}" />
                 <origin xyz="0 0 0" />
-                <xacro:cylinder_inertia m="${omni_wheel_mass}" r="${omni_wheel_radius}"
-                    h="${omni_wheel_height}" />
+                <xacro:cylinder_inertia m="${mecanum_wheel_mass}" r="${mecanum_wheel_radius}"
+                    h="${mecanum_wheel_height}" />
             </inertial>
         </link>
@@ -75,5 +75,5 @@
                         <geometry>
                             <mesh
-                                filename="package://robotnik_description/meshes/wheels/omni_wheel/robout_wheel.stl" />
+                                filename="package://robotnik_description/meshes/wheels/mecanum_wheel/robout_wheel.stl" />
                         </geometry>
                     </xacro:if>
@@ -82,5 +82,5 @@
                         <geometry>
                             <mesh
-                                filename="package://robotnik_description/meshes/wheels/omni_wheel/robout_wheel.stl" />
+                                filename="package://robotnik_description/meshes/wheels/mecanum_wheel/robout_wheel.stl" />
                         </geometry>
                     </xacro:unless>
@@ -89,5 +89,5 @@
                     <origin xyz="0 0 0" rpy="0 0 0" />
                     <geometry>
-                        <sphere radius="${omni_wheel_radius}" />
+                        <sphere radius="${mecanum_wheel_radius}" />
                     </geometry>
                 </xacro:unless>
@@ -103,8 +103,8 @@
             </collision>
             <inertial>
-                <mass value="${omni_wheel_mass}" />
+                <mass value="${mecanum_wheel_mass}" />
                 <origin xyz="0 0 0" />
-                <xacro:cylinder_inertia m="${omni_wheel_mass}" r="${omni_wheel_radius}"
-                    h="${omni_wheel_height}" />
+                <xacro:cylinder_inertia m="${mecanum_wheel_mass}" r="${mecanum_wheel_radius}"
+                    h="${mecanum_wheel_height}" />
             </inertial>
         </link>

Commit message: changed name mecanum wheels (#20)

File: urdf/bases/rbkairos/rbkairos_base.urdf.xacro (robot description, xacro)
@@ -19,16 +19,16 @@
   		<!-- Here we create the robot elements using the xacro:macros imported at the beggining of this file -->
   		<xacro:rbkairos_plus_body prefix="${prefix}"/>
-  		<xacro:mecanum_wheel prefix="${prefix}front_right_" parent="${prefix}base_link" reflect="false" hq="true" gazebo_classic="${gazebo_classic}" gazebo_ignition="${gazebo_ignition}"
+  		<xacro:rbkairos_mecanum_wheel prefix="${prefix}front_right_" parent="${prefix}base_link" reflect="false" hq="true" gazebo_classic="${gazebo_classic}" gazebo_ignition="${gazebo_ignition}"
 			xyz="${wheel_offset_x} -${wheel_offset_y} ${wheel_offset_z}">
-  		</xacro:mecanum_wheel>
-  		<xacro:mecanum_wheel prefix="${prefix}front_left_" parent="${prefix}base_link" reflect="true" hq="true" gazebo_classic="${gazebo_classic}" gazebo_ignition="${gazebo_ignition}"
+  		</xacro:rbkairos_mecanum_wheel>
+  		<xacro:rbkairos_mecanum_wheel prefix="${prefix}front_left_" parent="${prefix}base_link" reflect="true" hq="true" gazebo_classic="${gazebo_classic}" gazebo_ignition="${gazebo_ignition}"
 			xyz="${wheel_offset_x} ${wheel_offset_y} ${wheel_offset_z}">
-  		</xacro:mecanum_wheel>
-  		<xacro:mecanum_wheel prefix="${prefix}back_left_" parent="${prefix}base_link" reflect="false" hq="true" gazebo_classic="${gazebo_classic}" gazebo_ignition="${gazebo_ignition}"
+  		</xacro:rbkairos_mecanum_wheel>
+  		<xacro:rbkairos_mecanum_wheel prefix="${prefix}back_left_" parent="${prefix}base_link" reflect="false" hq="true" gazebo_classic="${gazebo_classic}" gazebo_ignition="${gazebo_ignition}"
 			xyz="-${wheel_offset_x} ${wheel_offset_y} ${wheel_offset_z}">
-  		</xacro:mecanum_wheel>
-  		<xacro:mecanum_wheel prefix="${prefix}back_right_" parent="${prefix}base_link" reflect="true" hq="true" gazebo_classic="${gazebo_classic}" gazebo_ignition="${gazebo_ignition}"
+  		</xacro:rbkairos_mecanum_wheel>
+  		<xacro:rbkairos_mecanum_wheel prefix="${prefix}back_right_" parent="${prefix}base_link" reflect="true" hq="true" gazebo_classic="${gazebo_classic}" gazebo_ignition="${gazebo_ignition}"
 			xyz="-${wheel_offset_x} -${wheel_offset_y} ${wheel_offset_z}">
-  		</xacro:mecanum_wheel>
+  		</xacro:rbkairos_mecanum_wheel>
      </xacro:macro>
 </robot>

File: urdf/wheels/mecanum_wheel/rbkairos_mecanum_wheel.urdf.xacro (robot description, xacro)
@@ -11,5 +11,5 @@
             izz="${m*(3*r*r+h*h)/12}" />
     </xacro:macro>
-    <xacro:macro name="mecanum_wheel" params="prefix parent xyz reflect hq gazebo_classic:=false gazebo_ignition:=false">
+    <xacro:macro name="rbkairos_mecanum_wheel" params="prefix parent xyz reflect hq gazebo_classic:=false gazebo_ignition:=false">
         <joint name="${prefix}wheel_joint" type="continuous">
             <parent link="${parent}" />
@@ -37,5 +37,5 @@
                             <geometry>
                                 <mesh
-                                    filename="package://robotnik_description/meshes/wheels/mecanum_wheel/mecanum_wheel_1.dae" />
+                                    filename="package://robotnik_description/meshes/wheels/mecanum_wheel/kairos_mecanum_wheel_1.dae" />
                             </geometry>
                         </xacro:if>
@@ -44,5 +44,5 @@
                             <geometry>
                                 <mesh
-                                    filename="package://robotnik_description/meshes/wheels/mecanum_wheel/mecanum_wheel_2.dae" />
+                                    filename="package://robotnik_description/meshes/wheels/mecanum_wheel/kairos_mecanum_wheel_2.dae" />
                             </geometry>
                         </xacro:unless>
@@ -105,5 +105,5 @@
                             <geometry>
                                 <mesh
-                                    filename="package://robotnik_description/meshes/wheels/mecanum_wheel/mecanum_wheel_1.dae" />
+                                    filename="package://robotnik_description/meshes/wheels/mecanum_wheel/kairos_mecanum_wheel_1.dae" />
                             </geometry>
                         </xacro:if>
@@ -112,5 +112,5 @@
                             <geometry>
                                 <mesh
-                                    filename="package://robotnik_description/meshes/wheels/mecanum_wheel/mecanum_wheel_2.dae" />
+                                    filename="package://robotnik_description/meshes/wheels/mecanum_wheel/kairos_mecanum_wheel_2.dae" />
                             </geometry>
                         </xacro:unless>

Commit message: Fix/ros2/change name mecanum wheels (#30)
* change name to mecanum wheels

Signed-off-by: cgasconb <cgascon@robotnik.es>

* Mecanum wheels joints adapted to simulation or real robot

* changed name mecanum wheels (#20)

---------

Signed-off-by: cgasconb <cgascon@robotnik.es>

File: urdf/bases/rbkairos/rbkairos_base.urdf.xacro (robot description, xacro)
@@ -7,5 +7,5 @@
   	<!-- Import summit XL base elements -->
 	<xacro:include filename="$(find robotnik_description)/urdf/bodies/rbkairos/rbkairos_plus_body.urdf.xacro" />
-  	<xacro:include filename="$(find robotnik_description)/urdf/wheels/omni_wheel/rbkairos_omni_wheel.urdf.xacro" />
+  	<xacro:include filename="$(find robotnik_description)/urdf/wheels/mecanum_wheel/rbkairos_mecanum_wheel.urdf.xacro" />
   	<xacro:property name="PI" value="3.1415926535897931"/>
   	<!-- Wheel parameters -->
@@ -13,5 +13,5 @@
   	<xacro:property name="wheel_offset_y" value="0.2590" />
   	<xacro:property name="wheel_offset_z" value="0.0" />
-    <xacro:macro name="rbkairos" params="prefix:=robot_">
+    <xacro:macro name="rbkairos" params="prefix:=robot_ gazebo_classic:=false gazebo_ignition:=false">
   		<!-- *************** -->
   		<!-- Robots Elements -->
@@ -19,16 +19,16 @@
   		<!-- Here we create the robot elements using the xacro:macros imported at the beggining of this file -->
   		<xacro:rbkairos_plus_body prefix="${prefix}"/>
-  		<xacro:omni_wheel prefix="${prefix}front_right_" parent="${prefix}base_link" reflect="false" hq="true">
-  			<origin xyz="${wheel_offset_x} -${wheel_offset_y} ${wheel_offset_z}" rpy="0 0 ${PI/4}"/>
-  		</xacro:omni_wheel>
-  		<xacro:omni_wheel prefix="${prefix}front_left_" parent="${prefix}base_link" reflect="true" hq="true">
-  			<origin xyz="${wheel_offset_x} ${wheel_offset_y} ${wheel_offset_z}" rpy="0 0 ${-PI/4}"/>
-  		</xacro:omni_wheel>
-  		<xacro:omni_wheel prefix="${prefix}back_left_" parent="${prefix}base_link" reflect="false" hq="true">
-  			<origin xyz="-${wheel_offset_x} ${wheel_offset_y} ${wheel_offset_z}" rpy="0 0 ${PI/4}"/>
-  		</xacro:omni_wheel>
-  		<xacro:omni_wheel prefix="${prefix}back_right_" parent="${prefix}base_link" reflect="true" hq="true">
-  			<origin xyz="-${wheel_offset_x} -${wheel_offset_y} ${wheel_offset_z}" rpy="0 0 ${-PI/4}"/>
-  		</xacro:omni_wheel>
+  		<xacro:rbkairos_mecanum_wheel prefix="${prefix}front_right_" parent="${prefix}base_link" reflect="false" hq="true" gazebo_classic="${gazebo_classic}" gazebo_ignition="${gazebo_ignition}"
+			xyz="${wheel_offset_x} -${wheel_offset_y} ${wheel_offset_z}">
+  		</xacro:rbkairos_mecanum_wheel>
+  		<xacro:rbkairos_mecanum_wheel prefix="${prefix}front_left_" parent="${prefix}base_link" reflect="true" hq="true" gazebo_classic="${gazebo_classic}" gazebo_ignition="${gazebo_ignition}"
+			xyz="${wheel_offset_x} ${wheel_offset_y} ${wheel_offset_z}">
+  		</xacro:rbkairos_mecanum_wheel>
+  		<xacro:rbkairos_mecanum_wheel prefix="${prefix}back_left_" parent="${prefix}base_link" reflect="false" hq="true" gazebo_classic="${gazebo_classic}" gazebo_ignition="${gazebo_ignition}"
+			xyz="-${wheel_offset_x} ${wheel_offset_y} ${wheel_offset_z}">
+  		</xacro:rbkairos_mecanum_wheel>
+  		<xacro:rbkairos_mecanum_wheel prefix="${prefix}back_right_" parent="${prefix}base_link" reflect="true" hq="true" gazebo_classic="${gazebo_classic}" gazebo_ignition="${gazebo_ignition}"
+			xyz="-${wheel_offset_x} -${wheel_offset_y} ${wheel_offset_z}">
+  		</xacro:rbkairos_mecanum_wheel>
      </xacro:macro>
 </robot>

File: urdf/bases/rbrobout/rbrobout_base.urdf.xacro (robot description, xacro)
@@ -8,5 +8,5 @@
 	<xacro:include filename="$(find robotnik_description)/urdf/bodies/rbrobout/rbrobout_body.urdf.xacro" />
 	<!-- Import RB-Robout wheels -->
-  	<xacro:include filename="$(find robotnik_description)/urdf/wheels/omni_wheel/rbrobout_omni_wheel.urdf.xacro" />
+  	<xacro:include filename="$(find robotnik_description)/urdf/wheels/mecanum_wheel/rbrobout_mecanum_wheel.urdf.xacro" />
 	<!-- Import all available sensors -->
 	<xacro:include filename="$(find robotnik_sensors)/urdf/all_sensors.urdf.xacro" />
@@ -18,5 +18,5 @@
 	<!-- Flag to select the high or low quality model -->
 	<xacro:property name="hq" value="true" />
-    <xacro:macro name="rbrobout" params="prefix:=robot_">
+    <xacro:macro name="rbrobout" params="prefix:=robot_ gazebo_classic:=false gazebo_ignition:=false">
 		<!-- *************** -->
 		<!-- Robots Elements -->
@@ -25,16 +25,16 @@
 		<xacro:rbrobout_body prefix="${prefix}" />
 		<!-- Wheels -->
-		<xacro:rbrobout_omni_wheel prefix="${prefix}front_right_" parent="${prefix}base_link" reflect="false" hq="${hq}">
-			<origin xyz="${wheel_offset_x} -${wheel_offset_y} ${wheel_offset_z}" rpy="0 0 ${PI/4}"/>
-		</xacro:rbrobout_omni_wheel>
-		<xacro:rbrobout_omni_wheel prefix="${prefix}front_left_" parent="${prefix}base_link" reflect="true" hq="${hq}">
-			<origin xyz="${wheel_offset_x} ${wheel_offset_y} ${wheel_offset_z}" rpy="0 0 ${-PI/4}"/>
-		</xacro:rbrobout_omni_wheel>
-		<xacro:rbrobout_omni_wheel prefix="${prefix}back_left_" parent="${prefix}base_link" reflect="false" hq="${hq}">
-			<origin xyz="-${wheel_offset_x} ${wheel_offset_y} ${wheel_offset_z}" rpy="0 0 ${PI/4}"/>
-		</xacro:rbrobout_omni_wheel>
-		<xacro:rbrobout_omni_wheel prefix="${prefix}back_right_" parent="${prefix}base_link" reflect="true" hq="${hq}">
-			<origin xyz="-${wheel_offset_x} -${wheel_offset_y} ${wheel_offset_z}" rpy="0 0 ${-PI/4}"/>
-		</xacro:rbrobout_omni_wheel>
+		<xacro:rbrobout_mecanum_wheel prefix="${prefix}front_right_" parent="${prefix}base_link" reflect="false" hq="${hq}" gazebo_classic="${gazebo_classic}" gazebo_ignition="${gazebo_ignition}"
+			xyz="${wheel_offset_x} -${wheel_offset_y} ${wheel_offset_z}">
+		</xacro:rbrobout_mecanum_wheel>
+		<xacro:rbrobout_mecanum_wheel prefix="${prefix}front_left_" parent="${prefix}base_link" reflect="true" hq="${hq}" gazebo_classic="${gazebo_classic}" gazebo_ignition="${gazebo_ignition}"
+			xyz="${wheel_offset_x} ${wheel_offset_y} ${wheel_offset_z}">
+		</xacro:rbrobout_mecanum_wheel>
+		<xacro:rbrobout_mecanum_wheel prefix="${prefix}back_left_" parent="${prefix}base_link" reflect="false" hq="${hq}" gazebo_classic="${gazebo_classic}" gazebo_ignition="${gazebo_ignition}"
+			xyz="-${wheel_offset_x} ${wheel_offset_y} ${wheel_offset_z}">
+		</xacro:rbrobout_mecanum_wheel>
+		<xacro:rbrobout_mecanum_wheel prefix="${prefix}back_right_" parent="${prefix}base_link" reflect="true" hq="${hq}" gazebo_classic="${gazebo_classic}" gazebo_ignition="${gazebo_ignition}"
+			xyz="-${wheel_offset_x} -${wheel_offset_y} ${wheel_offset_z}">
+		</xacro:rbrobout_mecanum_wheel>
    </xacro:macro>
 </robot>
