Commit message: added properties in summit

File: robots/rbsummit/rbsummit.urdf.xacro (robot description, xacro)
@@ -11,6 +11,34 @@
 	<!-- Import antenna -->
 	<xacro:include filename="$(find robot_description)/urdf/structures/sensor_support/structure_teltonika.urdf.xacro" />
-    <xacro:include filename="$(find robot_description)/gazebo/classic/rbsummit_control.urdf.xacro"/>
-    <xacro:include filename="$(find robot_description)/gazebo/ignition/rbsummit_control.urdf.xacro"/>
+	<xacro:include filename="$(find robot_description)/gazebo/classic/rbsummit_control.urdf.xacro"/>
+	<xacro:include filename="$(find robot_description)/gazebo/ignition/rbsummit_control.urdf.xacro"/>
+	<!-- ***************** -->
+	<!-- Sensor parameters -->
+	<!-- ***************** -->
+	<!-- x,y,z in translation from base_link to the center of the sensor -->
+	<xacro:property name="imu_offset_x" value="0.0385"/>
+	<xacro:property name="imu_offset_y" value="0.132"/>
+	<xacro:property name="imu_offset_z" value="0.158"/>
+	<xacro:property name="top_laser_offset_x" value="-0.11808"/>
+	<xacro:property name="top_laser_offset_y" value="0.0"/>
+	<xacro:property name="top_laser_offset_z" value="0.38509"/>
+	<xacro:property name="front_rgbd_camera_offset_x" value="0.324"/>
+	<xacro:property name="front_rgbd_camera_offset_y" value="0.012"/>
+	<xacro:property name="front_rgbd_camera_offset_z" value="0.172"/>
+	<xacro:property name="front_ptz_camera_offset_x" value="0.19"/>
+	<xacro:property name="front_ptz_camera_offset_y" value="0.0"/>
+	<xacro:property name="front_ptz_camera_offset_z" value="0.26"/>
+	<xacro:property name="gps_offset_x" value="-0.22528"/>
+	<xacro:property name="gps_offset_y" value="0.095"/>
+	<xacro:property name="gps_offset_z" value="0.275"/>
+	<!-- Other elements -->
+	<!--
+	<xacro:property name="antenna_offset_x" value="-0.22528"/>
+	<xacro:property name="antenna_offset_y" value="-0.095"/>
+	<xacro:property name="antenna_offset_z" value="0.23325"/>
+	-->
+	<xacro:property name="antenna_offset_x" value="-0.25528"/>
+	<xacro:property name="antenna_offset_y" value="0.0"/>
+	<xacro:property name="antenna_offset_z" value="0.23325"/>
 	<!-- ***************** -->
 	<!-- Global parameters -->
@@ -20,43 +48,85 @@
 	<!-- Flag to select the high or low quality model -->
 	<xacro:property name="hq" value="true" />
-    <!-- Launch Arguments -->
-    <xacro:arg name="use_gazebo_classic" default="false" />
-    <xacro:arg name="use_gazebo_ignition" default="false" />
-    <xacro:arg name="gpu" default="true" />
-  	<xacro:arg name="namespace" default="robot" />
+	<!-- Launch Arguments -->
+	<xacro:arg name="use_gazebo_classic" default="false" />
+	<xacro:arg name="use_gazebo_ignition" default="false" />
+	<xacro:arg name="gpu" default="true" />
+	<xacro:arg name="namespace" default="robot" />
 	<xacro:arg name="gps_latitude" default="0"/>
 	<xacro:arg name="gps_longitude" default="0"/>
 	<!-- Here we create the robot using the xacro:macro imported at the beggining of this file -->
-   	<xacro:rbsummit hq="${hq}"/>
+	<xacro:rbsummit hq="${hq}"/>
 	<!-- Custom Sensors -->
 	<!-- IMU -->
-	<xacro:sensor_vectornav prefix="rbsummit_" parent="rbsummit_base_link" topic="imu/data">
-		<origin xyz="0.0385 0.132 0.158" rpy="0 0 0"/>
-  </xacro:sensor_vectornav>
+	<xacro:sensor_vectornav
+		frame_prefix="rbsummit_imu_"
+		parent="rbsummit_base_link"
+	>
+		<origin
+			xyz="${imu_offset_x} ${imu_offset_y} ${imu_offset_z}"
+			rpy="0 0 0"
+		/>
+	</xacro:sensor_vectornav>
 	<!-- 3d laser -->
-	<!-- <xacro:sensor_rs_helios_16p prefix="$(arg prefix)top_3d_laser" parent="$(arg prefix)base_link" gpu="$(arg gpu)">
-		<origin xyz="-0.11808 0.0 0.38509" rpy="0 0 0"/>
-	</xacro:sensor_rs_helios_16p> -->
+	<xacro:sensor_robosense_helios
+		frame_prefix="rbsummit_top_3d_laser_"
+		parent="rbsummit_base_link"
+		gpu="$(arg gpu)"
+	>
+		<origin
+			xyz="${top_laser_offset_x} ${top_laser_offset_y} ${top_laser_offset_z}"
+			rpy="0 0 0"
+		/>
+	</xacro:sensor_robosense_helios>
 	<!-- ptz camera -->
-	<!-- <xacro:sensor_axis_m5525 prefix="$(arg prefix)front_ptz_camera" parent="$(arg prefix)base_link">
-		<origin xyz="0.19 0 0.26" rpy="0 ${15*PI/180} 0"/>
-	</xacro:sensor_axis_m5525> -->
+	<!--
+	<xacro:sensor_axis
+		prefix="rbsummit_front_ptz_camera"
+		parent="rbsummit_base_link"
+	>
+		<origin
+			xyz="0.19 0 0.26"
+			rpy="0 ${15*PI/180} 0"
+		/>
+	</xacro:sensor_axis>
+	-->
 	<!-- RGBD -->
-	<!-- <xacro:sensor_orbbec_astra prefix="$(arg prefix)front_rgbd_camera" parent="$(arg prefix)base_link">
-			<origin xyz="0.324 0.012 0.172" rpy="0 0 0"/>
-		</xacro:sensor_orbbec_astra> -->
+	<xacro:sensor_intel_realsense_d435
+		frame_prefix="rbsummit_front_rgbd_camera_"
+		parent="rbsummit_base_link"
+		topic_prefix="front_rgbd_camera"
+	>
+		<origin
+			xyz="${front_rgbd_camera_offset_x} ${front_rgbd_camera_offset_y} ${front_rgbd_camera_offset_z}"
+			rpy="0 0 0"
+		/>
+	</xacro:sensor_intel_realsense_d435>
 	<!-- GPS -->
-	<!-- <xacro:sensor_gps_with_mast prefix="$(arg prefix)gps" parent="$(arg prefix)base_link" gps_latitude="$(arg gps_latitude)" gps_longitude="$(arg gps_longitude)" update_rate="5">
-			<origin xyz="-0.22528 0.095 0.275" rpy="0 0 0"/>
-		</xacro:sensor_gps_with_mast> -->
-	<!--Antenna-->
-	<!-- <xacro:structure_mastil_teltonika prefix="$(arg prefix)antenna" parent="$(arg prefix)base_link">
-			<origin xyz="-0.22528 -0.095 0.23325" rpy="0 0 0"/>
-		</xacro:structure_mastil_teltonika> -->
-    <xacro:if value="$(arg use_gazebo_classic)">
-        <xacro:rbsummit_gz_classic_control namespace="$(arg namespace)"/>
-    </xacro:if>
-    <xacro:if value="$(arg use_gazebo_ignition)">
-        <xacro:rbsummit_gz_ignition_control namespace="$(arg namespace)"/>
-    </xacro:if>
+	<xacro:sensor_gps
+		frame_prefix="rbsummit_gps_"
+		parent="rbsummit_base_link"
+		update_rate="5"
+	>
+		<origin
+			xyz="${gps_offset_x} ${gps_offset_y} ${gps_offset_z}"
+			rpy="0 0 0"
+		/>
+	</xacro:sensor_gps>
+	<!-- Other Elements -->
+	<!-- Antenna -->
+	<xacro:structure_mastil_teltonika
+		prefix="rbsummit_antenna"
+		parent="rbsummit_base_link"
+	>
+		<origin
+			xyz="${antenna_offset_x} ${antenna_offset_y} ${antenna_offset_z}"
+			rpy="0 0 0"
+		/>
+	</xacro:structure_mastil_teltonika>
+	<xacro:if value="$(arg use_gazebo_classic)">
+		<xacro:rbsummit_gz_classic_control namespace="$(arg namespace)"/>
+	</xacro:if>
+	<xacro:if value="$(arg use_gazebo_ignition)">
+		<xacro:rbsummit_gz_ignition_control namespace="$(arg namespace)"/>
+	</xacro:if>
 </robot>

Commit message: Add planar_move sim control

File: robots/rbsummit/rbsummit.urdf.xacro (robot description, xacro)
@@ -98,4 +98,5 @@
   <xacro:if value="$(arg gazebo_classic)">
     <xacro:rbsummit_gz_classic_control namespace="$(arg namespace)" prefix="$(arg prefix)"/>
+        <xacro:ros_planar_move_gazebo_classic/>
   </xacro:if>
   <xacro:unless value="$(arg gazebo_classic)">

File: robots/rbtheron/rbtheron.urdf.xacro (robot description, xacro)
@@ -45,4 +45,5 @@
 	<xacro:if value="$(arg gazebo_classic)">
 		<xacro:rbtheron_gz_classic_control namespace="$(arg namespace)" prefix="$(arg prefix)"/>
+        <xacro:ros_planar_move_gazebo_classic/>
 	</xacro:if>
   <xacro:unless value="$(arg gazebo_classic)">

File: robots/rbvogui/rbvogui.urdf.xacro (robot description, xacro)
@@ -67,4 +67,5 @@
 	<xacro:if value="$(arg gazebo_classic)">
 		<xacro:rbvogui_gz_classic_control namespace="$(arg namespace)" prefix="$(arg prefix)"/>
+        <xacro:ros_planar_move_gazebo_classic/>
 	</xacro:if>
     <xacro:unless value="$(arg gazebo_classic)">

File: simulators/gazebo_classic/rbkairos/rbkairos_control.urdf.xacro (robot description, xacro)
@@ -43,6 +43,8 @@
             <publish_rate>10</publish_rate>
             <!-- output -->
-            <publish_odom>false</publish_odom>
-            <publish_odom_tf>false</publish_odom_tf>
+            <publish_odom>true</publish_odom>
+            <publish_odom_tf>true</publish_odom_tf>
+            <odometry_frame>robot_odom</odometry_frame>
+            <robot_base_frame>robot_base_footprint</robot_base_frame>
           </plugin>
         </gazebo>

File: simulators/gazebo_classic/rbsummit/rbsummit_control.urdf.xacro (robot description, xacro)
@@ -33,3 +33,20 @@
         </ros2_control>
     </xacro:macro>
+    <xacro:macro name="ros_planar_move_gazebo_classic">
+        <gazebo>
+          <plugin name="planar_move" filename="libgazebo_ros_planar_move.so">
+            <ros>
+              <!-- Remap the default topic -->
+              <remapping>cmd_vel:=/robot/robotnik_base_controller/cmd_vel</remapping>
+            </ros>
+            <update_rate>100</update_rate>
+            <publish_rate>10</publish_rate>
+            <!-- output -->
+            <publish_odom>true</publish_odom>
+            <publish_odom_tf>true</publish_odom_tf>
+            <odometry_frame>robot_odom</odometry_frame>
+            <robot_base_frame>robot_base_footprint</robot_base_frame>
+          </plugin>
+        </gazebo>
+    </xacro:macro>
 </robot>

File: simulators/gazebo_classic/rbtheron/rbtheron_control.urdf.xacro (robot description, xacro)
@@ -31,3 +31,20 @@
         </ros2_control>
     </xacro:macro>
+    <xacro:macro name="ros_planar_move_gazebo_classic">
+        <gazebo>
+          <plugin name="planar_move" filename="libgazebo_ros_planar_move.so">
+            <ros>
+              <!-- Remap the default topic -->
+              <remapping>cmd_vel:=/robot/robotnik_base_controller/cmd_vel</remapping>
+            </ros>
+            <update_rate>100</update_rate>
+            <publish_rate>10</publish_rate>
+            <!-- output -->
+            <publish_odom>true</publish_odom>
+            <publish_odom_tf>true</publish_odom_tf>
+            <odometry_frame>robot_odom</odometry_frame>
+            <robot_base_frame>robot_base_footprint</robot_base_frame>
+          </plugin>
+        </gazebo>
+    </xacro:macro>
 </robot>

File: simulators/gazebo_classic/rbvogui/rbvogui_control.urdf.xacro (robot description, xacro)
@@ -37,3 +37,20 @@
         </ros2_control>
     </xacro:macro>
+    <xacro:macro name="ros_planar_move_gazebo_classic">
+        <gazebo>
+          <plugin name="planar_move" filename="libgazebo_ros_planar_move.so">
+            <ros>
+              <!-- Remap the default topic -->
+              <remapping>cmd_vel:=/robot/robotnik_base_controller/cmd_vel</remapping>
+            </ros>
+            <update_rate>100</update_rate>
+            <publish_rate>10</publish_rate>
+            <!-- output -->
+            <publish_odom>true</publish_odom>
+            <publish_odom_tf>true</publish_odom_tf>
+            <odometry_frame>robot_odom</odometry_frame>
+            <robot_base_frame>robot_base_footprint</robot_base_frame>
+          </plugin>
+        </gazebo>
+    </xacro:macro>
 </robot>

Commit message: fix issue with rbsummit sensors

File: robots/rbsummit/rbsummit.urdf.xacro (robot description, xacro)
@@ -52,4 +52,5 @@
 		parent="$(arg prefix)base_link"
         node_namespace="$(arg namespace)"
+        node_name="top_lidar"
         gazebo_classic="$(arg gazebo_classic)"
         gazebo_ignition="$(arg gazebo_ignition)">
@@ -60,16 +61,13 @@
 	</xacro:sensor_robosense_helios_16p>
 	<!-- CAMERA -->
-	<xacro:sensor_intel_realsense_d435
-		frame_prefix="$(arg prefix)front_rgbd_camera_"
-		parent="$(arg prefix)base_link"
-		topic_prefix="front_rgbd_camera"
+    <xacro:sensor_intel_realsense_d435
+        frame_prefix="$(arg prefix)front_rgbd_camera_"
+        parent="$(arg prefix)base_link"
         node_namespace="$(arg namespace)"
+        node_name="front_camera"
         gazebo_classic="$(arg gazebo_classic)"
         gazebo_ignition="$(arg gazebo_ignition)">
-		<origin
-			xyz="${front_rgbd_camera_offset_x} ${front_rgbd_camera_offset_y} ${front_rgbd_camera_offset_z}"
-			rpy="0 0 0"
-		/>
-	</xacro:sensor_intel_realsense_d435>
+        <origin xyz="${front_rgbd_camera_offset_x} ${front_rgbd_camera_offset_y} ${front_rgbd_camera_offset_z}" rpy="0 0 0"/>
+    </xacro:sensor_intel_realsense_d435>
 	<!-- GPS -->
 	<xacro:sensor_ublox_with_mast
