Commit message: modify color view rbtheron body

File: urdf/bodies/rbtheron/rbtheron_body.urdf.xacro (robot description, xacro)
@@ -38,6 +38,6 @@
       </geometry>
       </xacro:unless>
-      <material name="black">
-        <color rgba="0.0 0.0 0.0 1"/>
+      <material name="grey">
+        <color rgba="0.2 0.2 0.2 1"/>
       </material>
     </visual>
@@ -65,5 +65,5 @@
   </link>
   <joint name="${prefix}base_logo_left_joint" type="fixed">
-    <origin xyz="0.0 0.28931 0.19062" rpy="0 0 0" />
+    <origin xyz="0.0 0.27531 0.19062" rpy="0 0 0" />
     <parent link="${prefix}base_link"/>
     <child link="${prefix}base_logo_left" />
@@ -82,5 +82,5 @@
   </link>
   <joint name="${prefix}base_logo_right_joint" type="fixed">
-    <origin xyz="0.0 -0.28931 0.19062" rpy="0 0 ${PI}" />
+    <origin xyz="0.0 -0.27531 0.19062" rpy="0 0 ${PI}" />
     <parent link="${prefix}base_link"/>
     <child link="${prefix}base_logo_right" />
@@ -99,5 +99,5 @@
   </link>
   <joint name="${prefix}base_logo_front_joint" type="fixed">
-    <origin xyz="0.345 0.0 0.0" rpy="0 0 ${-PI/2}" />
+    <origin xyz="0.332 0.0 0.0" rpy="0 0 ${-PI/2}" />
     <parent link="${prefix}base_link"/>
     <child link="${prefix}base_logo_front" />
@@ -116,5 +116,5 @@
   </link>
   <joint name="${prefix}base_logo_rear_joint" type="fixed">
-    <origin xyz="-0.345 0.0 0.0" rpy="0 0 ${PI/2}" />
+    <origin xyz="-0.332 0.0 0.0" rpy="0 0 ${PI/2}" />
     <parent link="${prefix}base_link"/>
     <child link="${prefix}base_logo_rear" />
