Commit message: Remove color references for gazebo

File: urdf/bodies/rbtheron/rbtheron_body.urdf.xacro (robot description, xacro)
@@ -60,6 +60,6 @@
           </geometry>
         </xacro:unless>
-        <material name="grey">
-          <color rgba="0.2 0.2 0.2 1" />
+        <material name="black">
+          <color rgba="0.0 0.0 0.0 1" />
         </material>
       </visual>
@@ -74,7 +74,4 @@
       </collision>
     </link>
-    <gazebo reference="${prefix}base_link">
-      <material>Gazebo/Black</material>
-    </gazebo>
     <!-- LOGO ROBOTNIK IZQUIERDO -->
     <link name="${prefix}base_logo_left">
