Commit message: fix rocker joint difference between simulation and real

File: robots/rbficus/rbficus.urdf.xacro (robot description, xacro)
@@ -24,5 +24,5 @@
   <xacro:property name="imu_offset_y" value="-0.129"/>
   <xacro:property name="imu_offset_z" value="0.212"/>
-  <xacro:rbficus prefix="$(arg prefix)"/>
+  <xacro:rbficus prefix="$(arg prefix)" gazebo_classic="$(arg gazebo_classic)" gazebo_ignition="$(arg gazebo_ignition)"/>
 	<!-- Controllers -->
 	<xacro:if value="$(arg gazebo_ignition)">

File: urdf/bases/rbficus/rbficus_base.urdf.xacro (robot description, xacro)
@@ -12,10 +12,10 @@
     <xacro:arg name="prefix" default="robot_" />
     <!-- <xacro:arg name="gpu" default="true" /> -->
-    <xacro:macro name="rbficus" params="prefix">
+    <xacro:macro name="rbficus" params="prefix gazebo_classic gazebo_ignition">
         <!-- *************** -->
         <!-- Robots Elements -->
         <!-- *************** -->
         <!-- Here we create the robot elements using the xacro:macros imported at the beggining of this file -->
-        <xacro:rbficus_body prefix="${prefix}"/>
+        <xacro:rbficus_body prefix="${prefix}" gazebo_classic="${gazebo_classic}" gazebo_ignition="${gazebo_ignition}"/>
         <!-- WHEELS -->
         <xacro:rbficus_steering_wheel prefix="${prefix}front_right_" parent="${prefix}chassis_link" reflect="true" hq="true">

File: urdf/bodies/rbficus/rbficus_body.urdf.xacro (robot description, xacro)
@@ -2,5 +2,5 @@
 <robot xmlns:xacro="http://www.ros.org/wiki/xacro">
     <xacro:include filename="$(find robotnik_description)/urdf/inertia.urdf.xacro" />
-    <xacro:macro name="rbficus_body" params="prefix">
+    <xacro:macro name="rbficus_body" params="prefix gazebo_classic gazebo_ignition">
         <!-- Robot mechanical and motor parameters -->
         <xacro:property name="PI" value="3.1415926535897931" />
@@ -46,11 +46,20 @@
         </link>
         <!-- Rocker Chassis Joint -->
-        <joint name="${prefix}rocker_chassis" type="revolute">
-            <axis xyz="1 0 0" />
-            <origin xyz="-0.835 0 0.047" rpy="0 0 0" />
-            <parent link="${prefix}chassis_link" />
-            <child link="${prefix}rocker_link" />
-            <limit effort="30" velocity="1.0" lower="${-15*PI/180}" upper="${15*PI/180}" />
-        </joint>
+        <xacro:if value="${gazebo_classic or gazebo_ignition}">
+            <joint name="${prefix}rocker_chassis" type="revolute">
+                <axis xyz="1 0 0" />
+                <origin xyz="-0.835 0 0.047" rpy="0 0 0" />
+                <parent link="${prefix}chassis_link" />
+                <child link="${prefix}rocker_link" />
+                <limit effort="30" velocity="1.0" lower="${-15*PI/180}" upper="${15*PI/180}" />
+            </joint>
+        </xacro:if>
+        <xacro:unless value="${gazebo_classic or gazebo_ignition}">
+            <joint name="${prefix}rocker_chassis" type="fixed">
+                <origin xyz="-0.835 0 0.047" rpy="0 0 0" />
+                <parent link="${prefix}chassis_link" />
+                <child link="${prefix}rocker_link" />
+            </joint>
+        </xacro:unless>
         <!-- Rocker -->
         <link name="${prefix}rocker_link">
