Commit message: move sensors to correct position rbvogui

File: robots/rbvogui/rbvogui.urdf.xacro (robot description, xacro)
@@ -5,95 +5,105 @@
     <!-- Imported elements -->
     <!-- ***************** -->
-    <!-- First we import all posible elements defined in the urdf.xacro files. All these elements are defined as macro:xacros -->
+    <!-- First we import all posible elements defined in the urdf.xacro files. All these elements
+    are defined as macro:xacros -->
     <!-- Import rbvogui base elements-->
-    <xacro:include filename="$(find robotnik_description)/urdf/bases/rbvogui/rbvogui_base.urdf.xacro" />
+    <xacro:include
+        filename="$(find robotnik_description)/urdf/bases/rbvogui/rbvogui_base.urdf.xacro" />
     <xacro:include filename="$(find robotnik_description)/urdf/base_hw/rbvogui.ros2_control.urdf" />
-    <xacro:include filename="$(find robotnik_description)/simulators/gazebo_classic/rbvogui/rbvogui_control.urdf.xacro" />
-    <xacro:include filename="$(find robotnik_description)/simulators/gazebo_ignition/rbvogui/rbvogui_control.urdf.xacro" />
+    <xacro:include
+        filename="$(find robotnik_description)/simulators/gazebo_classic/rbvogui/rbvogui_control.urdf.xacro" />
+    <xacro:include
+        filename="$(find robotnik_description)/simulators/gazebo_ignition/rbvogui/rbvogui_control.urdf.xacro" />
     <!-- Import all available sensors -->
     <xacro:include filename="$(find robotnik_sensors)/urdf/all_sensors.urdf.xacro" />
     <!-- Flag to select the high or low quality model -->
     <xacro:property name="hq" value="true" />
-    <xacro:property name="front_laser_offset_x" value="0.53"/>
-    <xacro:property name="front_laser_offset_y" value="0.33"/>
-    <xacro:property name="front_laser_offset_z" value="0.1145"/>
-    <xacro:property name="rear_laser_offset_x" value="-0.53"/>
-    <xacro:property name="rear_laser_offset_y" value="-0.33"/>
-    <xacro:property name="rear_laser_offset_z" value="0.1145"/>
-    <xacro:property name="imu_offset_x" value="0.3"/>
-    <xacro:property name="imu_offset_y" value="-0.3"/>
-    <xacro:property name="imu_offset_z" value="0.0725"/>
-    <xacro:property name="front_rgbd_camera_offset_x" value="0.46462"/>
-    <xacro:property name="front_rgbd_camera_offset_y" value="0.0"/>
-    <xacro:property name="front_rgbd_camera_offset_z" value="0.18258"/>
-    <xacro:property name="rear_rgbd_camera_offset_x" value="-0.503"/>
-    <xacro:property name="rear_rgbd_camera_offset_y" value="0.0"/>
-    <xacro:property name="rear_rgbd_camera_offset_z" value="0.29"/>
+    <xacro:property name="front_laser_offset_x" value="0.53" />
+    <xacro:property name="front_laser_offset_y" value="0.33" />
+    <xacro:property name="front_laser_offset_z" value="0.1145" />
+    <xacro:property name="rear_laser_offset_x" value="-0.53" />
+    <xacro:property name="rear_laser_offset_y" value="-0.33" />
+    <xacro:property name="rear_laser_offset_z" value="0.1145" />
+    <xacro:property name="imu_offset_x" value="0.127" />
+    <xacro:property name="imu_offset_y" value="-0.129" />
+    <xacro:property name="imu_offset_z" value="0.212" />
+    <xacro:property name="front_rgbd_camera_offset_x" value="0.46462" />
+    <xacro:property name="front_rgbd_camera_offset_y" value="0.0" />
+    <xacro:property name="front_rgbd_camera_offset_z" value="0.18258" />
+    <xacro:property name="rear_rgbd_camera_offset_x" value="-0.515" />
+    <xacro:property name="rear_rgbd_camera_offset_y" value="0.0" />
+    <xacro:property name="rear_rgbd_camera_offset_z" value="0.29" />
     <!-- Launch Arguments -->
-	<xacro:arg name="namespace" default="robot"/>
-	<xacro:arg name="prefix" default="robot_"/>
-	<xacro:arg name="gazebo_classic" default="false"/>
-	<xacro:arg name="gazebo_ignition" default="false"/>
-    <xacro:rbvogui prefix="$(arg prefix)" hq="${hq}"/>
+    <xacro:arg name="namespace" default="robot" />
+    <xacro:arg name="prefix" default="robot_" />
+    <xacro:arg name="gazebo_classic" default="false" />
+    <xacro:arg name="gazebo_ignition" default="false" />
+    <xacro:rbvogui prefix="$(arg prefix)" hq="${hq}" />
     <!-- SENSORS see robotnik_sensors for the specific configuration -->
     <!-- IMU -->
     <xacro:sensor_vectornav
-    frame_prefix="$(arg prefix)vectornav_"
-    parent="$(arg prefix)base_link"
-    node_namespace="$(arg namespace)"
-    gazebo_classic="$(arg gazebo_classic)"
-    gazebo_ignition="$(arg gazebo_ignition)">
-    <origin xyz="${imu_offset_x} ${imu_offset_y} ${imu_offset_z}" rpy="0 0 0"/>
+        frame_prefix="$(arg prefix)vectornav_"
+        parent="$(arg prefix)base_link"
+        node_namespace="$(arg namespace)"
+        gazebo_classic="$(arg gazebo_classic)"
+        gazebo_ignition="$(arg gazebo_ignition)">
+        <origin xyz="${imu_offset_x} ${imu_offset_y} ${imu_offset_z}" rpy="0 0 0" />
     </xacro:sensor_vectornav>
-    <!-- SENSORS -->
+    <!-- LASERS -->
     <xacro:sensor_sick_s300
-    frame_prefix="$(arg prefix)front_laser_"
-    parent="$(arg prefix)base_link"
-    node_namespace="$(arg namespace)"
-    node_name="front_laser"
-    gazebo_classic="$(arg gazebo_classic)"
-    gazebo_ignition="$(arg gazebo_ignition)">
-    <origin xyz="${front_laser_offset_x} ${front_laser_offset_y} ${front_laser_offset_z}" rpy="0 ${-PI} ${3/4*PI}"/>
+        frame_prefix="$(arg prefix)front_laser_"
+        parent="$(arg prefix)base_link"
+        node_namespace="$(arg namespace)"
+        node_name="front_laser"
+        gazebo_classic="$(arg gazebo_classic)"
+        gazebo_ignition="$(arg gazebo_ignition)">
+        <origin xyz="${front_laser_offset_x} ${front_laser_offset_y} ${front_laser_offset_z}"
+            rpy="0 ${-PI} ${-3/4*PI}" />
     </xacro:sensor_sick_s300>
     <xacro:sensor_sick_s300
-    frame_prefix="$(arg prefix)rear_laser_"
-    parent="$(arg prefix)base_link"
-    node_namespace="$(arg namespace)"
-    node_name="rear_laser"
-    gazebo_classic="$(arg gazebo_classic)"
-    gazebo_ignition="$(arg gazebo_ignition)">
-    <origin xyz="${rear_laser_offset_x} ${rear_laser_offset_y} ${rear_laser_offset_z}" rpy="0 ${-PI} ${-1/4*PI}"/>
+        frame_prefix="$(arg prefix)rear_laser_"
+        parent="$(arg prefix)base_link"
+        node_namespace="$(arg namespace)"
+        node_name="rear_laser"
+        gazebo_classic="$(arg gazebo_classic)"
+        gazebo_ignition="$(arg gazebo_ignition)">
+        <origin xyz="${rear_laser_offset_x} ${rear_laser_offset_y} ${rear_laser_offset_z}"
+            rpy="0 ${-PI} ${1/4*PI}" />
     </xacro:sensor_sick_s300>
     <!-- Front Camera -->
     <xacro:sensor_intel_realsense_d435
-    frame_prefix="$(arg prefix)front_rgbd_camera_"
-    parent="$(arg prefix)base_link"
-    node_namespace="$(arg namespace)"
-    node_name="front_camera"
-    gazebo_classic="$(arg gazebo_classic)"
-    gazebo_ignition="$(arg gazebo_ignition)">
-    <origin xyz="${front_rgbd_camera_offset_x} ${front_rgbd_camera_offset_y} ${front_rgbd_camera_offset_z}" rpy="0 0 0"/>
+        frame_prefix="$(arg prefix)front_rgbd_camera_"
+        parent="$(arg prefix)base_link"
+        node_namespace="$(arg namespace)"
+        node_name="front_camera"
+        gazebo_classic="$(arg gazebo_classic)"
+        gazebo_ignition="$(arg gazebo_ignition)">
+        <origin
+            xyz="${front_rgbd_camera_offset_x} ${front_rgbd_camera_offset_y} ${front_rgbd_camera_offset_z}"
+            rpy="0 0 0" />
     </xacro:sensor_intel_realsense_d435>
     <!-- Rear Camera -->
     <xacro:sensor_intel_realsense_d435
-    frame_prefix="$(arg prefix)rear_rgbd_camera_"
-    parent="$(arg prefix)base_link"
-    node_namespace="$(arg namespace)"
-    node_name="rear_camera"
-    gazebo_classic="$(arg gazebo_classic)"
-    gazebo_ignition="$(arg gazebo_ignition)">
-    <origin xyz="${rear_rgbd_camera_offset_x} ${rear_rgbd_camera_offset_y} ${rear_rgbd_camera_offset_z}" rpy="0 0 -${PI}"/>
+        frame_prefix="$(arg prefix)rear_rgbd_camera_"
+        parent="$(arg prefix)base_link"
+        node_namespace="$(arg namespace)"
+        node_name="rear_camera"
+        gazebo_classic="$(arg gazebo_classic)"
+        gazebo_ignition="$(arg gazebo_ignition)">
+        <origin
+            xyz="${rear_rgbd_camera_offset_x} ${rear_rgbd_camera_offset_y} ${rear_rgbd_camera_offset_z}"
+            rpy="0 0 -${PI}" />
     </xacro:sensor_intel_realsense_d435>
-	<!-- Controllers -->
-	<xacro:if value="$(arg gazebo_classic)">
-		<xacro:rbvogui_gz_classic_control namespace="$(arg namespace)" prefix="$(arg prefix)"/>
-        <xacro:ros_planar_move_gazebo_classic/>
-	</xacro:if>
-	<xacro:if value="$(arg gazebo_ignition)">
-		<xacro:rbvogui_gz_ignition_control namespace="$(arg namespace)" prefix="$(arg prefix)"/>
-	</xacro:if>
+    <!-- Controllers -->
+    <xacro:if value="$(arg gazebo_classic)">
+        <xacro:rbvogui_gz_classic_control namespace="$(arg namespace)" prefix="$(arg prefix)" />
+        <xacro:ros_planar_move_gazebo_classic />
+    </xacro:if>
+    <xacro:if value="$(arg gazebo_ignition)">
+        <xacro:rbvogui_gz_ignition_control namespace="$(arg namespace)" prefix="$(arg prefix)" />
+    </xacro:if>
     <xacro:unless value="$(arg gazebo_classic)">
         <xacro:unless value="$(arg gazebo_ignition)">
-            <xacro:rbvogui_base_hw_controller/>
+            <xacro:rbvogui_base_hw_controller />
         </xacro:unless>
     </xacro:unless>

File: robots/rbvogui/rbvogui_plus.urdf.xacro (robot description, xacro)
@@ -1,54 +1,62 @@
 <?xml version="1.0"?>
 <robot name="rbvogui" xmlns:xacro="http://wiki.ros.org/xacro">
-  <!-- ***************** -->
-  <!-- Imported elements -->
-  <!-- ***************** -->
-  <!-- Import all posible elements defined in the urdf.xacro files. All these elements are defined as macro:xacros -->
-  <xacro:include filename="$(find robotnik_description)/urdf/bases/rbvogui/rbvogui_base.urdf.xacro" />
-  <xacro:include filename="$(find robotnik_description)/urdf/base_hw/rbvogui.ros2_control.urdf" />
-  <xacro:include filename="$(find robotnik_description)/simulators/gazebo_classic/rbvogui/rbvogui_control.urdf.xacro" />
-  <xacro:include filename="$(find robotnik_description)/simulators/gazebo_ignition/rbvogui/rbvogui_control.urdf.xacro" />
-  <xacro:include filename="$(find robotnik_sensors)/urdf/all_sensors.urdf.xacro" />
-  <xacro:include filename="$(find ur_description)/urdf/ur_macro.xacro" />
-  <!-- Properties and Arguments -->
-  <xacro:arg name="namespace" default="robot"/>
-  <xacro:arg name="prefix" default="robot_"/>
-  <xacro:arg name="gazebo_classic" default="false"/>
-  <xacro:arg name="gazebo_ignition" default="false"/>
-  <xacro:arg name="ur_type" default="ur5e"/>
-  <xacro:arg name="joint_limit_params" default="$(find ur_description)/config/$(arg ur_type)/joint_limits.yaml"/>
-  <xacro:arg name="kinematics_params" default="$(find ur_description)/config/$(arg ur_type)/default_kinematics.yaml"/>
-  <xacro:arg name="physical_params" default="$(find ur_description)/config/$(arg ur_type)/physical_parameters.yaml"/>
-  <xacro:arg name="visual_params" default="$(find ur_description)/config/$(arg ur_type)/visual_parameters.yaml"/>
-  <xacro:property name="front_laser_offset_x" value="0.53"/>
-  <xacro:property name="front_laser_offset_y" value="0.33"/>
-  <xacro:property name="front_laser_offset_z" value="0.1145"/>
-  <xacro:property name="rear_laser_offset_x" value="-0.53"/>
-  <xacro:property name="rear_laser_offset_y" value="-0.33"/>
-  <xacro:property name="rear_laser_offset_z" value="0.1145"/>
-  <xacro:property name="imu_offset_x" value="0.3"/>
-  <xacro:property name="imu_offset_y" value="-0.3"/>
-  <xacro:property name="imu_offset_z" value="0.0725"/>
-  <xacro:property name="front_rgbd_camera_offset_x" value="0.46462"/>
-  <xacro:property name="front_rgbd_camera_offset_y" value="0.0"/>
-  <xacro:property name="front_rgbd_camera_offset_z" value="0.18258"/>
-  <xacro:property name="rear_rgbd_camera_offset_x" value="-0.503"/>
-  <xacro:property name="rear_rgbd_camera_offset_y" value="0.0"/>
-  <xacro:property name="rear_rgbd_camera_offset_z" value="0.29"/>
-  <!-- Vogui -->
-  <xacro:rbvogui prefix="$(arg prefix)"/>
-  <!-- Import UR arm -->
-  <xacro:ur_robot
-      tf_prefix="$(arg prefix)arm_"
-      name="$(arg ur_type)"
-      parent="$(arg prefix)base_link"
-      joint_limits_parameters_file="$(arg joint_limit_params)"
-      kinematics_parameters_file="$(arg kinematics_params)"
-      physical_parameters_file="$(arg physical_params)"
-      visual_parameters_file="$(arg visual_params)"
-      sim_gazebo="$(arg gazebo_classic)">
-      <origin xyz="0 0 0.3995" rpy="0 0 0"/>
-  </xacro:ur_robot>
-  <!-- IMU -->
+    <!-- ***************** -->
+    <!-- Imported elements -->
+    <!-- ***************** -->
+    <!-- Import all posible elements defined in the urdf.xacro files. All these elements are defined
+  as macro:xacros -->
+    <xacro:include
+        filename="$(find robotnik_description)/urdf/bases/rbvogui/rbvogui_base.urdf.xacro" />
+    <xacro:include filename="$(find robotnik_description)/urdf/base_hw/rbvogui.ros2_control.urdf" />
+    <xacro:include
+        filename="$(find robotnik_description)/simulators/gazebo_classic/rbvogui/rbvogui_control.urdf.xacro" />
+    <xacro:include
+        filename="$(find robotnik_description)/simulators/gazebo_ignition/rbvogui/rbvogui_control.urdf.xacro" />
+    <xacro:include filename="$(find robotnik_sensors)/urdf/all_sensors.urdf.xacro" />
+    <xacro:include filename="$(find ur_description)/urdf/ur_macro.xacro" />
+    <!-- Properties and Arguments -->
+    <xacro:arg name="namespace" default="robot" />
+    <xacro:arg name="prefix" default="robot_" />
+    <xacro:arg name="gazebo_classic" default="false" />
+    <xacro:arg name="gazebo_ignition" default="false" />
+    <xacro:arg name="ur_type" default="ur5e" />
+    <xacro:arg name="joint_limit_params"
+        default="$(find ur_description)/config/$(arg ur_type)/joint_limits.yaml" />
+    <xacro:arg name="kinematics_params"
+        default="$(find ur_description)/config/$(arg ur_type)/default_kinematics.yaml" />
+    <xacro:arg name="physical_params"
+        default="$(find ur_description)/config/$(arg ur_type)/physical_parameters.yaml" />
+    <xacro:arg name="visual_params"
+        default="$(find ur_description)/config/$(arg ur_type)/visual_parameters.yaml" />
+    <xacro:property name="front_laser_offset_x" value="0.53" />
+    <xacro:property name="front_laser_offset_y" value="0.33" />
+    <xacro:property name="front_laser_offset_z" value="0.1145" />
+    <xacro:property name="rear_laser_offset_x" value="-0.53" />
+    <xacro:property name="rear_laser_offset_y" value="-0.33" />
+    <xacro:property name="rear_laser_offset_z" value="0.1145" />
+    <xacro:property name="imu_offset_x" value="0.127" />
+    <xacro:property name="imu_offset_y" value="-0.129" />
+    <xacro:property name="imu_offset_z" value="0.212" />
+    <xacro:property name="front_rgbd_camera_offset_x" value="0.46462" />
+    <xacro:property name="front_rgbd_camera_offset_y" value="0.0" />
+    <xacro:property name="front_rgbd_camera_offset_z" value="0.18258" />
+    <xacro:property name="rear_rgbd_camera_offset_x" value="-0.515" />
+    <xacro:property name="rear_rgbd_camera_offset_y" value="0.0" />
+    <xacro:property name="rear_rgbd_camera_offset_z" value="0.29" />
+    <!-- Vogui -->
+    <xacro:rbvogui prefix="$(arg prefix)" />
+    <!-- Import UR arm -->
+    <xacro:ur_robot
+        tf_prefix="$(arg prefix)arm_"
+        name="$(arg ur_type)"
+        parent="$(arg prefix)base_link"
+        joint_limits_parameters_file="$(arg joint_limit_params)"
+        kinematics_parameters_file="$(arg kinematics_params)"
+        physical_parameters_file="$(arg physical_params)"
+        visual_parameters_file="$(arg visual_params)"
+        sim_gazebo="$(arg gazebo_classic)">
+        <origin xyz="0 0 0.3995" rpy="0 0 0" />
+    </xacro:ur_robot>
+    <!-- IMU -->
     <xacro:sensor_vectornav
         frame_prefix="$(arg prefix)vectornav_"
@@ -57,7 +65,7 @@
         gazebo_classic="$(arg gazebo_classic)"
         gazebo_ignition="$(arg gazebo_ignition)">
-        <origin xyz="${imu_offset_x} ${imu_offset_y} ${imu_offset_z}" rpy="0 0 0"/>
+        <origin xyz="${imu_offset_x} ${imu_offset_y} ${imu_offset_z}" rpy="0 0 0" />
     </xacro:sensor_vectornav>
-  <!-- SENSORS -->
+    <!-- LASERS -->
     <xacro:sensor_sick_s300
         frame_prefix="$(arg prefix)front_laser_"
@@ -67,5 +75,6 @@
         gazebo_classic="$(arg gazebo_classic)"
         gazebo_ignition="$(arg gazebo_ignition)">
-        <origin xyz="${front_laser_offset_x} ${front_laser_offset_y} ${front_laser_offset_z}" rpy="0 ${-PI} ${3/4*PI}"/>
+        <origin xyz="${front_laser_offset_x} ${front_laser_offset_y} ${front_laser_offset_z}"
+            rpy="0 ${-PI} ${-3/4*PI}" />
     </xacro:sensor_sick_s300>
     <xacro:sensor_sick_s300
@@ -76,5 +85,6 @@
         gazebo_classic="$(arg gazebo_classic)"
         gazebo_ignition="$(arg gazebo_ignition)">
-        <origin xyz="${rear_laser_offset_x} ${rear_laser_offset_y} ${rear_laser_offset_z}" rpy="0 ${-PI} ${-1/4*PI}"/>
+        <origin xyz="${rear_laser_offset_x} ${rear_laser_offset_y} ${rear_laser_offset_z}"
+            rpy="0 ${-PI} ${1/4*PI}" />
     </xacro:sensor_sick_s300>
     <!-- Front Camera -->
@@ -86,5 +96,7 @@
         gazebo_classic="$(arg gazebo_classic)"
         gazebo_ignition="$(arg gazebo_ignition)">
-        <origin xyz="${front_rgbd_camera_offset_x} ${front_rgbd_camera_offset_y} ${front_rgbd_camera_offset_z}" rpy="0 0 0"/>
+        <origin
+            xyz="${front_rgbd_camera_offset_x} ${front_rgbd_camera_offset_y} ${front_rgbd_camera_offset_z}"
+            rpy="0 0 0" />
     </xacro:sensor_intel_realsense_d435>
     <!-- Rear Camera -->
@@ -96,18 +108,20 @@
         gazebo_classic="$(arg gazebo_classic)"
         gazebo_ignition="$(arg gazebo_ignition)">
-        <origin xyz="${rear_rgbd_camera_offset_x} ${rear_rgbd_camera_offset_y} ${rear_rgbd_camera_offset_z}" rpy="0 0 -${PI}"/>
+        <origin
+            xyz="${rear_rgbd_camera_offset_x} ${rear_rgbd_camera_offset_y} ${rear_rgbd_camera_offset_z}"
+            rpy="0 0 -${PI}" />
     </xacro:sensor_intel_realsense_d435>
     <!-- Controllers -->
     <xacro:if value="$(arg gazebo_classic)">
-      <xacro:rbvogui_gz_classic_control namespace="$(arg namespace)" prefix="$(arg prefix)"/>
-      <xacro:ros_planar_move_gazebo_classic/>
+        <xacro:rbvogui_gz_classic_control namespace="$(arg namespace)" prefix="$(arg prefix)" />
+        <xacro:ros_planar_move_gazebo_classic />
     </xacro:if>
     <xacro:if value="$(arg gazebo_ignition)">
-      <xacro:rbvogui_gz_ignition_control namespace="$(arg namespace)" prefix="$(arg prefix)"/>
+        <xacro:rbvogui_gz_ignition_control namespace="$(arg namespace)" prefix="$(arg prefix)" />
     </xacro:if>
     <xacro:unless value="$(arg gazebo_classic)">
-      <xacro:unless value="$(arg gazebo_ignition)">
-        <xacro:rbvogui_base_hw_controller/>
-      </xacro:unless>
+        <xacro:unless value="$(arg gazebo_ignition)">
+            <xacro:rbvogui_base_hw_controller />
+        </xacro:unless>
     </xacro:unless>
 </robot>
