Commit message: Cambios varios
Se ha añadido soporte para los prefijos y el control, además de otros cambios, como la edición de los urdfs del vogui y theron con el fin de sacar el PROTO y el FBX para Webots y Ubuntu

File: robots/rbvogui/rbvogui.urdf.xacro (robot description, xacro)
@@ -5,28 +5,70 @@
     <!-- Imported elements -->
     <!-- ***************** -->
-    <!-- First we import all posible elements defined in the urdf.xacro files. All these elements are defined as macro:xacros -->
+    <!-- First we import all posible elements defined in the urdf.xacro files. All these elements
+    are defined as macro:xacros -->
     <!-- Import rbvogui base elements-->
-    <xacro:include filename="$(find robot_description)/urdf/bases/rbvogui/rbvogui_base.urdf.xacro" />
+    <xacro:include
+        filename="$(find robot_description)/urdf/bases/rbvogui/rbvogui_base.urdf.xacro" />
     <xacro:include filename="$(find robot_description)/urdf/base_hw/rbvogui.ros2_control.urdf" />
-    <xacro:include filename="$(find robot_description)/simulators/gazebo_classic/rbvogui/rbvogui_control.urdf.xacro" />
+    <xacro:include
+        filename="$(find robot_description)/simulators/gazebo_classic/rbvogui/rbvogui_control.urdf.xacro" />
+    <xacro:include
+        filename="$(find robot_description)/simulators/gazebo_ignition/rbvogui/rbvogui_control.urdf.xacro" />
     <!-- Import all available sensors -->
     <xacro:include filename="$(find robotnik_sensors)/urdf/all_sensors.urdf.xacro" />
-    <xacro:include filename="$(find robot_description)/urdf/structures/sensor_support/gps_mast.urdf.xacro" />
     <!-- Flag to select the high or low quality model -->
     <xacro:property name="hq" value="true" />
+    <xacro:property name="front_laser_offset_x" value="0.53" />
+    <xacro:property name="front_laser_offset_y" value="0.33" />
+    <xacro:property name="front_laser_offset_z" value="0.1145" />
+    <xacro:property name="rear_laser_offset_x" value="-0.53" />
+    <xacro:property name="rear_laser_offset_y" value="-0.33" />
+    <xacro:property name="rear_laser_offset_z" value="0.1145" />
+    <xacro:property name="imu_offset_x" value="0.127" />
+    <xacro:property name="imu_offset_y" value="-0.129" />
+    <xacro:property name="imu_offset_z" value="0.212" />
+    <xacro:property name="front_rgbd_camera_offset_x" value="0.46462" />
+    <xacro:property name="front_rgbd_camera_offset_y" value="0.0" />
+    <xacro:property name="front_rgbd_camera_offset_z" value="0.18258" />
+    <xacro:property name="rear_rgbd_camera_offset_x" value="-0.515" />
+    <xacro:property name="rear_rgbd_camera_offset_y" value="0.0" />
+    <xacro:property name="rear_rgbd_camera_offset_z" value="0.29" />
     <!-- Launch Arguments -->
-	<xacro:arg name="namespace" default="robot"/>
-	<xacro:arg name="prefix" default="robot_"/>
-	<xacro:arg name="gazebo_classic" default="false"/>
-    <xacro:rbvogui prefix="$(arg prefix)" hq="${hq}"/>
+    <xacro:arg name="namespace" default="robot" />
+    <xacro:arg name="prefix" default="robot_" />
+    <xacro:arg name="gazebo_classic" default="true" />
+    <xacro:arg name="gazebo_ignition" default="false" />
+    <xacro:rbvogui prefix="$(arg prefix)" hq="${hq}" />
     <!-- SENSORS see robotnik_sensors for the specific configuration -->
-    <!-- IMU -->
+  <!-- IMU -->
     <xacro:sensor_vectornav
         frame_prefix="$(arg prefix)vectornav_"
-        parent="$(arg prefix)chassis_link"
+        parent="$(arg prefix)base_link"
         node_namespace="$(arg namespace)"
-        simulation="$(arg gazebo_classic)">
-        <origin xyz="0.3 -0.3 0.0725" rpy="0 0 0"/>
+        gazebo_classic="$(arg gazebo_classic)"
+        gazebo_ignition="$(arg gazebo_ignition)">
+        <origin xyz="${imu_offset_x} ${imu_offset_y} ${imu_offset_z}" rpy="0 0 0"/>
     </xacro:sensor_vectornav>
+    <!-- LASERS -->
+    <xacro:sensor_sick_s300
+        frame_prefix="$(arg prefix)front_laser_"
+        parent="$(arg prefix)base_link"
+        node_namespace="$(arg namespace)"
+        node_name="front_laser"
+        gazebo_classic="$(arg gazebo_classic)"
+        gazebo_ignition="$(arg gazebo_ignition)">
+        <origin xyz="${front_laser_offset_x} ${front_laser_offset_y} ${front_laser_offset_z}"
+            rpy="0 ${-PI} ${-3/4*PI}" />
+    </xacro:sensor_sick_s300>
+    <xacro:sensor_sick_s300
+        frame_prefix="$(arg prefix)rear_laser_"
+        parent="$(arg prefix)base_link"
+        node_namespace="$(arg namespace)"
+        node_name="rear_laser"
+        gazebo_classic="$(arg gazebo_classic)"
+        gazebo_ignition="$(arg gazebo_ignition)">
+        <origin xyz="${rear_laser_offset_x} ${rear_laser_offset_y} ${rear_laser_offset_z}"
+            rpy="0 ${-PI} ${1/4*PI}" />
+    </xacro:sensor_sick_s300>
     <!-- Front Camera -->
     <xacro:sensor_intel_realsense_d435
@@ -35,40 +77,34 @@
         node_namespace="$(arg namespace)"
         node_name="front_camera"
-        simulation="$(arg gazebo_classic)">
-        <origin xyz="0.46462 0.0 0.18258" rpy="0 0 0"/>
+        gazebo_classic="$(arg gazebo_classic)"
+        gazebo_ignition="$(arg gazebo_ignition)">
+        <origin
+            xyz="${front_rgbd_camera_offset_x} ${front_rgbd_camera_offset_y} ${front_rgbd_camera_offset_z}"
+            rpy="0 0 0" />
     </xacro:sensor_intel_realsense_d435>
     <!-- Rear Camera -->
-    <!-- <xacro:sensor_intel_realsense_d435
+    <xacro:sensor_intel_realsense_d435
         frame_prefix="$(arg prefix)rear_rgbd_camera_"
-        parent="$(arg prefix)chassis_link"
+        parent="$(arg prefix)base_link"
         node_namespace="$(arg namespace)"
         node_name="rear_camera"
-        simulation="$(arg gazebo_classic)">
-        <origin xyz="-0.503 0.0 0.29" rpy="0 0 -${PI}"/>
-    </xacro:sensor_intel_realsense_d435> -->
-    <!-- 2d laser -->
-    <xacro:sensor_sick_s300
-        frame_prefix="$(arg prefix)front_laser_"
-        parent="$(arg prefix)chassis_link"
-        node_namespace="$(arg namespace)"
-        node_name="front_laser"
-        simulation="$(arg gazebo_classic)">
-        <origin xyz="0.53 0.33 0.1145" rpy="${PI} 0 ${PI/4}"/>
-    </xacro:sensor_sick_s300>
-    <xacro:sensor_sick_s300
-        frame_prefix="$(arg prefix)rear_laser_"
-        parent="$(arg prefix)chassis_link"
-        node_namespace="$(arg namespace)"
-        node_name="rear_laser"
-        simulation="$(arg gazebo_classic)">
-        <origin xyz="-0.53 -0.33 0.1145" rpy="${PI} 0 ${-PI*3/4}"/>
-    </xacro:sensor_sick_s300>
-	<!-- Controllers -->
-	<xacro:if value="$(arg gazebo_classic)">
-		<xacro:rbvogui_gz_classic_control namespace="$(arg namespace)" prefix="$(arg prefix)"/>
-        <xacro:ros_planar_move_gazebo_classic/>
-	</xacro:if>
+        gazebo_classic="$(arg gazebo_classic)"
+        gazebo_ignition="$(arg gazebo_ignition)">
+        <origin
+            xyz="${rear_rgbd_camera_offset_x} ${rear_rgbd_camera_offset_y} ${rear_rgbd_camera_offset_z}"
+            rpy="0 0 -${PI}" />
+    </xacro:sensor_intel_realsense_d435>
+    <!-- Controllers -->
+    <xacro:if value="$(arg gazebo_classic)">
+        <xacro:rbvogui_gz_classic_control namespace="$(arg namespace)" prefix="$(arg prefix)" />
+        <xacro:ros_planar_move_gazebo_classic />
+    </xacro:if>
+    <xacro:if value="$(arg gazebo_ignition)">
+        <xacro:rbvogui_gz_ignition_control namespace="$(arg namespace)" prefix="$(arg prefix)" />
+    </xacro:if>
     <xacro:unless value="$(arg gazebo_classic)">
-        <xacro:rbvogui_base_hw_controller/>
+        <xacro:unless value="$(arg gazebo_ignition)">
+            <xacro:rbvogui_base_hw_controller />
+        </xacro:unless>
     </xacro:unless>
 </robot>

File: simulators/gazebo_ignition/rbtheron/rbtheron_control.urdf.xacro (robot description, xacro)
@@ -1,10 +1,10 @@
 <?xml version="1.0"?>
 <robot xmlns:xacro="http://wiki.ros.org/xacro">
-    <xacro:macro name="rbrobout_gz_ignition_control"  params="namespace prefix">
+    <xacro:macro name="rbtheron_gz_ignition_control" params="namespace prefix">
         <gazebo>
-          <plugin name="ign_ros2_control::IgnitionROS2ControlPlugin" filename="ign_ros2_control-system">
+            <plugin name="ign_ros2_control::IgnitionROS2ControlPlugin" filename="ign_ros2_control-system">
             <robot_param>robot_description</robot_param>
             <robot_param_node>robot_state_publisher</robot_param_node>
-            <parameters>$(find robot_description)/simulators/gazebo_ignition/rbrobout/rbrobout_controller_params.yaml</parameters>
+            <parameters>$(find robot_description)/simulators/gazebo_ignition/rbtheron/rbtheron_controller_params.yaml</parameters>
             <ros>
                 <namespace>/${namespace}</namespace>
@@ -25,11 +25,8 @@
         <ros2_control name="IgnitionSystem" type="system">
           <hardware>
-              <plugin>ign_ros2_control/IgnitionSystem</plugin>
+            <plugin>ign_ros2_control/IgnitionSystem</plugin>
           </hardware>
-          <xacro:ros2_joint interface="velocity" jmin="-10" jmax="10" name="robot_front_left_wheel_joint"/>
-          <xacro:ros2_joint interface="velocity" jmin="-10" jmax="10" name="robot_front_right_wheel_joint"/>
-          <xacro:ros2_joint interface="velocity" jmin="-20" jmax="20" name="robot_back_left_wheel_joint"/>
-          <xacro:ros2_joint interface="velocity" jmin="-20" jmax="20" name="robot_back_right_wheel_joint"/>
-          <xacro:ros2_joint interface="position" jmin="-20" jmax="20" name="robot_lift_ewellix_lift_top_joint"/>
+          <xacro:ros2_joint interface="velocity" jmin="-10" jmax="10" name="robot_left_wheel_joint"/>
+          <xacro:ros2_joint interface="velocity" jmin="-10" jmax="10" name="robot_right_wheel_joint"/>
         </ros2_control>
     </xacro:macro>

File: urdf/wheels/rubber_wheel/rbwatcher_rubber_wheel.urdf.xacro (robot description, xacro)
@@ -7,10 +7,10 @@
               izz="${m*(3*r*r+h*h)/12}" />
   </xacro:macro>
-  <xacro:macro name="rubber_wheel" params="prefix parent *origin reflect hq rubber_wheel_radius:=0.11 rubber_wheel_width:=0.15 rubber_wheel_mass:=6.5
+  <xacro:macro name="rubber_wheel" params="prefix1 prefix2 parent *origin reflect hq rubber_wheel_radius:=0.11 rubber_wheel_width:=0.15 rubber_wheel_mass:=6.5
                                           mesh_file:=robot_description/meshes/wheels/rubber_wheel/rubber_wheel_right">
 <!--WHEEL TIRE -->
-    <joint name="${prefix}_wheel_joint" type="continuous">
+    <joint name="robot_${prefix2}_wheel_joint" type="continuous">
       <parent link="${parent}"/>
-      <child link="${prefix}_wheel"/>
+      <child link="${prefix1}${prefix2}_wheel"/>
       <xacro:insert_block name="origin" />
       <axis xyz="0 1 0" rpy="0 0 0" />
@@ -18,5 +18,5 @@
       <joint_properties damping="0.0" friction="0.0"/>
     </joint>
-    <link name="${prefix}_wheel">
+    <link name="${prefix1}${prefix2}_wheel">
       <visual>
         <!-- HIGH RESOLUTION WHEELS -->
@@ -58,15 +58,15 @@
     </link>
     <!-- Transmission is important to link the joints and the controller (see summit_xl_control/config/summit_xl_control.yaml)-->
-    <transmission name="${prefix}_wheel_joint_trans">
+    <transmission name="${prefix1}${prefix2}_wheel_joint_trans">
       <type>transmission_interface/SimpleTransmission</type>
-      <joint name="${prefix}_wheel_joint">
+      <joint name="robot_${prefix2}_wheel_joint">
         <hardwareInterface>hardware_interface/VelocityJointInterface</hardwareInterface>
       </joint>
-      <actuator name="${prefix}_wheel_joint_motor">
+      <actuator name="${prefix1}${prefix2}_wheel_joint_motor">
         <mechanicalReduction>1</mechanicalReduction>
         <motorTorqueConstant>20</motorTorqueConstant>
       </actuator>
      </transmission>
-    <gazebo reference="${prefix}_wheel">
+    <gazebo reference="${prefix1}${prefix2}_wheel">
 			<material>Gazebo/Black</material>
 			<turnGravityOff>false</turnGravityOff>
