Commit message: feat(rbvogui): add kinematics arg to rbvogui macro for swerve/mecanum switching
  - Add vogui_wheel macro with always-present red fork and parametric joint type
  - kinematics=swerve: revolute steering joint + rubber wheel
  - kinematics=mecanum: fixed steering joint + mecanum wheel

File: robots/rbvogui/rbvogui.urdf.xacro (robot description, xacro)
@@ -17,9 +17,13 @@
     name="gazebo_ignition"
     default="false" />
+  <xacro:arg
+    name="kinematics"
+    default="swerve" />
   <!-- RB-VOGUI -->
   <xacro:rbvogui
     prefix="$(arg prefix)"
     gazebo_ignition="$(arg gazebo_ignition)"
-    namespace="$(arg namespace)" />
+    namespace="$(arg namespace)"
+    kinematics="$(arg kinematics)" />
   <!-- IMU -->
   <xacro:sensor_vectornav

File: urdf/bases/rbvogui/rbvogui_base.urdf.xacro (robot description, xacro)
@@ -8,15 +8,112 @@
     filename="$(find robotnik_description)/urdf/wheels/steering_wheel/steering_wheel.urdf.xacro" />
   <xacro:include
+    filename="$(find robotnik_description)/urdf/wheels/mecanum_wheel/rbkairos_mecanum_wheel.urdf.xacro" />
+  <xacro:include
     filename="$(find robotnik_description)/simulators/gazebo_ignition/rbvogui/rbvogui_control.urdf.xacro" />
   <!-- WHEELS PROPERTIES -->
-  <xacro:property
-    name="wheel_offset_x"
-    value="0.368" />
-  <xacro:property
-    name="wheel_offset_y"
-    value="0.235" />
-  <xacro:property
-    name="wheel_offset_z"
-    value="0.0" />
+  <xacro:property name="wheel_offset_x" value="0.368" />
+  <xacro:property name="wheel_offset_y" value="0.235" />
+  <xacro:property name="wheel_offset_z" value="0.0" />
+  <!--
+    Unified vogui wheel macro - always mounts the red fork (base_wheel link).
+    kinematics=swerve: steering_joint is revolute (rotates) + rubber wheel mesh.
+    kinematics=mecanum: steering_joint is fixed (no rotation) + mecanum wheel mesh.
+    The fork position and color are identical in both modes.
+  -->
+  <xacro:macro
+    name="vogui_wheel"
+    params="prefix parent xyz reflect hq kinematics">
+    <xacro:property name="steer_joint_damping" value="1.0" />
+    <xacro:property name="steer_joint_friction" value="1.0" />
+    <xacro:property name="steer_joint_effort_limit" value="200.0" />
+    <xacro:property name="steer_joint_velocity_limit" value="100.0" />
+    <xacro:property name="steering_support_mass" value="2.5" />
+    <xacro:property name="steering_support_width" value="0.1" />
+    <xacro:macro name="cylinder_inertia" params="m r h">
+      <inertia
+        ixx="${m*(3*r*r+h*h)/12}" ixy="0" ixz="0"
+        iyy="${m*(3*r*r+h*h)/12}" iyz="0"
+        izz="${m*r*r/2}" />
+    </xacro:macro>
+    <!-- Steering joint: revolute for swerve, fixed for mecanum -->
+    <xacro:if value="${kinematics == 'swerve'}">
+      <joint name="${prefix}steering_joint" type="revolute">
+        <parent link="${parent}" />
+        <child link="${prefix}base_wheel" />
+        <origin xyz="${xyz}" rpy="0 0 0" />
+        <axis xyz="0 0 1" />
+        <limit effort="${steer_joint_effort_limit}"
+               velocity="${steer_joint_velocity_limit}"
+               lower="-3.00" upper="3.00" />
+        <dynamics damping="${steer_joint_damping}" friction="${steer_joint_friction}" />
+      </joint>
+    </xacro:if>
+    <xacro:unless value="${kinematics == 'swerve'}">
+      <joint name="${prefix}steering_joint" type="fixed">
+        <parent link="${parent}" />
+        <child link="${prefix}base_wheel" />
+        <origin xyz="${xyz}" rpy="0 0 0" />
+      </joint>
+    </xacro:unless>
+    <!-- Fork (base_wheel): always present, always red -->
+    <link name="${prefix}base_wheel">
+      <visual>
+        <xacro:if value="${reflect}">
+          <origin xyz="0 0 0" rpy="0 0 0" />
+        </xacro:if>
+        <xacro:unless value="${reflect}">
+          <origin xyz="0 0 0" rpy="0 0 ${pi}" />
+        </xacro:unless>
+        <geometry>
+          <mesh filename="package://robotnik_description/meshes/wheels/steering_wheel/mw_frame_stl_color.dae" />
+        </geometry>
+        <material name="red">
+          <color rgba="0.9 0.1 0.1 1" />
+        </material>
+      </visual>
+      <collision>
+        <xacro:if value="${reflect}">
+          <origin xyz="0 0 0" rpy="0 0 0" />
+        </xacro:if>
+        <xacro:unless value="${reflect}">
+          <origin xyz="0 0 0" rpy="0 0 ${pi}" />
+        </xacro:unless>
+        <geometry>
+          <mesh filename="package://robotnik_description/meshes/wheels/steering_wheel/mw_frame_stl_color.dae" />
+        </geometry>
+      </collision>
+      <inertial>
+        <mass value="${steering_support_mass}" />
+        <xacro:if value="${reflect}">
+          <origin xyz="0 0 ${wheel_radius/1.5}" rpy="${pi/2.0} ${pi/2.0} 0" />
+        </xacro:if>
+        <xacro:unless value="${reflect}">
+          <origin xyz="0 0 ${wheel_radius/1.5}" rpy="${pi/2.0} ${pi/2.0} ${pi/2.0}" />
+        </xacro:unless>
+        <xacro:cylinder_inertia m="${steering_support_mass}" r="${wheel_radius}" h="${steering_support_width}" />
+      </inertial>
+    </link>
+    <!-- Wheel: rubber (swerve) or mecanum, both attached to the fork -->
+    <xacro:if value="${kinematics == 'swerve'}">
+      <xacro:rubber_wheel
+        prefix="${prefix}"
+        parent="${prefix}base_wheel"
+        reflect="${reflect}"
+        hq="${hq}"
+        rubber_wheel_radius="${wheel_radius}"
+        rubber_wheel_width="${wheel_width}"
+        rubber_wheel_mass="${wheel_mass}">
+        <origin xyz="0 0 0" rpy="0 0 0" />
+      </xacro:rubber_wheel>
+    </xacro:if>
+    <xacro:unless value="${kinematics == 'swerve'}">
+      <xacro:rbkairos_mecanum_wheel
+        prefix="${prefix}"
+        parent="${prefix}base_wheel"
+        reflect="${reflect}"
+        hq="${hq}"
+        xyz="0 0 0" />
+    </xacro:unless>
+  </xacro:macro>
   <xacro:macro
     name="rbvogui"
@@ -25,51 +122,22 @@
       gazebo_ignition:=false
       namespace:=''
+      kinematics:=swerve
       ">
-    <xacro:property
-      name="hq"
-      value="true" />
-    <xacro:rbvogui_body
-      prefix="${prefix}"
-      hq="${hq}" />
-    <xacro:steering_wheel
-      prefix="${prefix}front_right_"
-      parent="${prefix}base_link"
-      reflect="false"
-      hq="${hq}">
-      <origin
-        xyz="${wheel_offset_x} -${wheel_offset_y} ${wheel_offset_z}"
-        rpy="0 0 0" />
-    </xacro:steering_wheel>
-    <xacro:steering_wheel
-      prefix="${prefix}front_left_"
-      parent="${prefix}base_link"
-      reflect="true"
-      hq="${hq}">
-      <origin
-        xyz="${wheel_offset_x} ${wheel_offset_y} ${wheel_offset_z}"
-        rpy="0 0 0" />
-    </xacro:steering_wheel>
-    <xacro:steering_wheel
-      prefix="${prefix}back_left_"
-      parent="${prefix}base_link"
-      reflect="true"
-      hq="${hq}">
-      <origin
-        xyz="-${wheel_offset_x} ${wheel_offset_y} ${wheel_offset_z}"
-        rpy="0 0 0" />
-    </xacro:steering_wheel>
-    <xacro:steering_wheel
-      prefix="${prefix}back_right_"
-      parent="${prefix}base_link"
-      reflect="false"
-      hq="${hq}">
-      <origin
-        xyz="-${wheel_offset_x} -${wheel_offset_y} ${wheel_offset_z}"
-        rpy="0 0 0" />
-    </xacro:steering_wheel>
+    <xacro:property name="hq" value="true" />
+    <xacro:rbvogui_body prefix="${prefix}" hq="${hq}" />
+    <xacro:vogui_wheel prefix="${prefix}front_right_" parent="${prefix}base_link"
+      xyz="${wheel_offset_x} -${wheel_offset_y} ${wheel_offset_z}"
+      reflect="false" hq="${hq}" kinematics="${kinematics}" />
+    <xacro:vogui_wheel prefix="${prefix}front_left_" parent="${prefix}base_link"
+      xyz="${wheel_offset_x} ${wheel_offset_y} ${wheel_offset_z}"
+      reflect="true" hq="${hq}" kinematics="${kinematics}" />
+    <xacro:vogui_wheel prefix="${prefix}back_left_" parent="${prefix}base_link"
+      xyz="-${wheel_offset_x} ${wheel_offset_y} ${wheel_offset_z}"
+      reflect="true" hq="${hq}" kinematics="${kinematics}" />
+    <xacro:vogui_wheel prefix="${prefix}back_right_" parent="${prefix}base_link"
+      xyz="-${wheel_offset_x} -${wheel_offset_y} ${wheel_offset_z}"
+      reflect="false" hq="${hq}" kinematics="${kinematics}" />
     <xacro:if value="$(arg gazebo_ignition)">
-      <xacro:rbvogui_gz_ignition_control
-        namespace="${namespace}"
-        prefix="${prefix}" />
+      <xacro:rbvogui_gz_ignition_control namespace="${namespace}" prefix="${prefix}" />
     </xacro:if>
   </xacro:macro>
