Commit message: change sensors

File: robots/rbvogui/rbvogui_xl.urdf.xacro (robot description, xacro)
@@ -48,23 +48,13 @@
     <xacro:sensor_intel_realsense_d435
         frame_prefix="$(arg prefix)front_rgbd_camera_"
-        parent="$(arg prefix)base_link"
+        parent="$(arg prefix)chassis_link"
         node_namespace="$(arg namespace)"
         node_name="front_camera"
         gazebo_classic="$(arg gazebo_classic)"
         gazebo_ignition="$(arg gazebo_ignition)">
-        <origin xyz="${front_rgbd_camera_offset_x} ${front_rgbd_camera_offset_y} ${front_rgbd_camera_offset_z}" rpy="0 0 0"/>
-    </xacro:sensor_intel_realsense_d435>
-    <!-- Rear Camera -->
-    <xacro:sensor_intel_realsense_d435
-        frame_prefix="$(arg prefix)rear_rgbd_camera_"
-        parent="$(arg prefix)base_link"
-        node_namespace="$(arg namespace)"
-        node_name="rear_camera"
-        gazebo_classic="$(arg gazebo_classic)"
-        gazebo_ignition="$(arg gazebo_ignition)">
-        <origin xyz="${rear_rgbd_camera_offset_x} ${rear_rgbd_camera_offset_y} ${rear_rgbd_camera_offset_z}" rpy="0 0 -${PI}" />
+        <origin xyz="0.541 0.0 0.18258" rpy="0 0 0"/>
     </xacro:sensor_intel_realsense_d435>
     <!-- LASERS -->
-    <xacro:sensor_sick_s300
+    <xacro:sensor_sick_tim571
         frame_prefix="$(arg prefix)front_laser_"
         parent="$(arg prefix)chassis_link"
@@ -73,7 +63,7 @@
         gazebo_classic="$(arg gazebo_classic)"
         gazebo_ignition="$(arg gazebo_ignition)">
-        <origin xyz="${front_laser_offset_x} ${front_laser_offset_y} ${front_laser_offset_z}" rpy="0 ${-PI} ${-3/4*PI}" />
-    </xacro:sensor_sick_s300>
-    <xacro:sensor_sick_s300
+        <origin xyz="0.64555 0.39595 0.1145" rpy="${PI} 0 0.775398" />
+    </xacro:sensor_sick_tim571>
+    <xacro:sensor_sick_tim571
         frame_prefix="$(arg prefix)rear_laser_"
         parent="$(arg prefix)chassis_link"
@@ -82,6 +72,6 @@
         gazebo_classic="$(arg gazebo_classic)"
         gazebo_ignition="$(arg gazebo_ignition)">
-        <origin xyz="${rear_laser_offset_x} ${rear_laser_offset_y} ${rear_laser_offset_z}" rpy="0 ${-PI} ${1/4*PI}" />
-    </xacro:sensor_sick_s300>
+        <origin xyz="-0.64555 -0.39595 0.1145" rpy="${PI} 0 -2.35219"/>
+    </xacro:sensor_sick_tim571>
     <!-- Controllers
     <xacro:if value="$(arg gazebo_classic)">
