Commit message: Update simulation config files

File: simulators/gazebo_classic/rbkairos/rbkairos_control.urdf.xacro (robot description, xacro)
@@ -6,5 +6,5 @@
             <robot_param>robot_description</robot_param>
             <robot_param_node>robot_state_publisher</robot_param_node>
-            <parameters>$(find robotnik_description)/simulators/gazebo_classic/rbkairos/rbkairos_controller_params.yaml</parameters>
+            <parameters>$(find robotnik_gazebo_classic)/config/rbkairos/rbkairos_controller_params.yaml</parameters>
             <ros>
                 <namespace>/${namespace}</namespace>
@@ -38,5 +38,5 @@
             <ros>
               <!-- Remap the default topic -->
-              <remapping>cmd_vel:=/robot/robotnik_base_controller/cmd_vel</remapping>
+              <remapping>cmd_vel:=/robot/robotnik_base_controller/cmd_vel_unstamped</remapping>
             </ros>
             <update_rate>100</update_rate>

File: simulators/gazebo_classic/rbrobout/rbrobout_control.urdf.xacro (robot description, xacro)
@@ -6,5 +6,5 @@
             <robot_param>robot_description</robot_param>
             <robot_param_node>robot_state_publisher</robot_param_node>
-            <parameters>$(find robotnik_description)/simulators/gazebo_classic/rbrobout/rbrobout_controller_params.yaml</parameters>
+            <parameters>$(find robotnik_gazebo_classic)/config/rbrobout/rbrobout_controller_params.yaml</parameters>
             <ros>
                 <namespace>/${namespace}</namespace>
@@ -39,5 +39,5 @@
             <ros>
               <!-- Remap the default topic -->
-              <remapping>cmd_vel:=/robot/robotnik_base_controller/cmd_vel</remapping>
+              <remapping>cmd_vel:=/robot/robotnik_base_controller/cmd_vel_unstamped</remapping>
             </ros>
             <update_rate>100</update_rate>

File: simulators/gazebo_classic/rbsummit/rbsummit_control.urdf.xacro (robot description, xacro)
@@ -6,5 +6,5 @@
             <robot_param>robot_description</robot_param>
             <robot_param_node>robot_state_publisher</robot_param_node>
-            <parameters>$(find robotnik_description)/simulators/gazebo_classic/rbsummit/rbsummit_controller_params.yaml</parameters>
+            <parameters>$(find robotnik_gazebo_classic)/config/rbsummit/rbsummit_controller_params.yaml</parameters>
             <ros>
                 <namespace>/${namespace}</namespace>
@@ -38,5 +38,5 @@
             <ros>
               <!-- Remap the default topic -->
-              <remapping>cmd_vel:=/robot/robotnik_base_controller/cmd_vel</remapping>
+              <remapping>cmd_vel:=/robot/robotnik_base_controller/cmd_vel_unstamped</remapping>
             </ros>
             <update_rate>100</update_rate>

File: simulators/gazebo_classic/rbtheron/rbtheron_control.urdf.xacro (robot description, xacro)
@@ -6,5 +6,5 @@
             <robot_param>robot_description</robot_param>
             <robot_param_node>robot_state_publisher</robot_param_node>
-            <parameters>$(find robotnik_description)/simulators/gazebo_classic/rbtheron/rbtheron_controller_params.yaml</parameters>
+            <parameters>$(find robotnik_gazebo_classic)/config/rbtheron/rbtheron_controller_params.yaml</parameters>
             <ros>
                 <namespace>/${namespace}</namespace>
@@ -36,5 +36,5 @@
             <ros>
               <!-- Remap the default topic -->
-              <remapping>cmd_vel:=/robot/robotnik_base_controller/cmd_vel</remapping>
+              <remapping>cmd_vel:=/robot/robotnik_base_controller/cmd_vel_unstamped</remapping>
             </ros>
             <update_rate>100</update_rate>

File: simulators/gazebo_classic/rbvogui/rbvogui_control.urdf.xacro (robot description, xacro)
@@ -4,7 +4,7 @@
         <gazebo>
           <plugin name="ros_control" filename="libgazebo_ros2_control.so">
-            <robot_param>robotnik_description</robot_param>
+            <robot_param>robot_description</robot_param>
             <robot_param_node>robot_state_publisher</robot_param_node>
-            <parameters>$(find robotnik_description)/simulators/gazebo_classic/rbvogui/rbvogui_controller_params.yaml</parameters>
+            <parameters>$(find robotnik_gazebo_classic)/config/rbvogui/rbvogui_controller_params.yaml</parameters>
             <ros>
                 <namespace>/${namespace}</namespace>
@@ -37,20 +37,3 @@
         </ros2_control>
     </xacro:macro>
-    <xacro:macro name="ros_planar_move_gazebo_classic">
-        <gazebo>
-          <plugin name="planar_move" filename="libgazebo_ros_planar_move.so">
-            <ros>
-              <!-- Remap the default topic -->
-              <remapping>cmd_vel:=/robot/robotnik_base_controller/cmd_vel</remapping>
-            </ros>
-            <update_rate>100</update_rate>
-            <publish_rate>10</publish_rate>
-            <!-- output -->
-            <publish_odom>true</publish_odom>
-            <publish_odom_tf>true</publish_odom_tf>
-            <odometry_frame>robot_odom</odometry_frame>
-            <robot_base_frame>robot_base_footprint</robot_base_frame>
-          </plugin>
-        </gazebo>
-    </xacro:macro>
 </robot>

File: simulators/gazebo_ignition/rbkairos/rbkairos_control.urdf.xacro (robot description, xacro)
@@ -6,5 +6,5 @@
           <robot_param>robot_description</robot_param>
           <robot_param_node>robot_state_publisher</robot_param_node>
-          <parameters>$(find robotnik_description)/simulators/gazebo_ignition/rbkairos/rbkairos_controller_params.yaml</parameters>
+          <parameters>$(find robotnik_gazebo_ignition)/config/rbkairos/rbkairos_controller_params.yaml</parameters>
           <ros>
               <namespace>/${namespace}</namespace>

File: simulators/gazebo_ignition/rbrobout/rbrobout_control.urdf.xacro (robot description, xacro)
@@ -6,5 +6,5 @@
             <robot_param>robot_description</robot_param>
             <robot_param_node>robot_state_publisher</robot_param_node>
-            <parameters>$(find robotnik_description)/simulators/gazebo_ignition/rbrobout/rbrobout_controller_params.yaml</parameters>
+            <parameters>$(find robotnik_gazebo_ignition)/config/rbrobout/rbrobout_controller_params.yaml</parameters>
             <ros>
                 <namespace>/${namespace}</namespace>

File: simulators/gazebo_ignition/rbsummit/rbsummit_control.urdf.xacro (robot description, xacro)
@@ -6,5 +6,5 @@
             <robot_param>robot_description</robot_param>
             <robot_param_node>robot_state_publisher</robot_param_node>
-            <parameters>$(find robotnik_description)/simulators/gazebo_ignition/rbsummit/rbsummit_controller_params.yaml</parameters>
+            <parameters>$(find robotnik_gazebo_ignition)/config/rbsummit/rbsummit_controller_params.yaml</parameters>
             <ros>
                 <namespace>/${namespace}</namespace>

File: simulators/gazebo_ignition/rbtheron/rbtheron_control.urdf.xacro (robot description, xacro)
@@ -6,5 +6,5 @@
             <robot_param>robot_description</robot_param>
             <robot_param_node>robot_state_publisher</robot_param_node>
-            <parameters>$(find robotnik_description)/simulators/gazebo_ignition/rbtheron/rbtheron_controller_params.yaml</parameters>
+            <parameters>$(find robotnik_gazebo_ignition)/config/rbtheron/rbtheron_controller_params.yaml</parameters>
             <ros>
                 <namespace>/${namespace}</namespace>

File: simulators/gazebo_ignition/rbvogui/rbvogui_control.urdf.xacro (robot description, xacro)
@@ -6,5 +6,5 @@
             <robot_param>robot_description</robot_param>
             <robot_param_node>robot_state_publisher</robot_param_node>
-            <parameters>$(find robotnik_description)/simulators/gazebo_ignition/rbvogui/rbvogui_controller_params.yaml</parameters>
+            <parameters>$(find robotnik_gazebo_ignition)/config/rbvogui/rbvogui_controller_params.yaml</parameters>
             <ros>
                 <namespace>/${namespace}</namespace>
