Commit message: Add pearl to rbtheron_plus

File: robots/rbtheron/rbtheron_plus.urdf.xacro (robot description, xacro)
@@ -85,4 +85,7 @@
 	<xacro:property name="rear_laser_offset_y" value="0.215"/>
 	<xacro:property name="rear_laser_offset_z" value="0.1613"/>
+	<xacro:property name="top_lidar_offset_x" value="0.26"/>
+	<xacro:property name="top_lidar_offset_y" value="0.0"/>
+	<xacro:property name="top_lidar_offset_z" value="0.51"/>
 	<!-- IMU -->
     <xacro:sensor_vectornav
@@ -132,4 +135,14 @@
         <origin xyz="${rear_rgbd_camera_offset_x} ${rear_rgbd_camera_offset_y} ${rear_rgbd_camera_offset_z}" rpy="0 0 ${PI}"/>
     </xacro:sensor_intel_realsense_d435>
+    <!-- 3D LiDAR -->
+    <xacro:sensor_robosense_bpearl
+        frame_prefix="$(arg prefix)top_lidar_"
+        parent="$(arg prefix)top_chassis"
+        node_namespace="$(arg namespace)"
+        node_name="top_lidar"
+        gazebo_classic="$(arg gazebo_classic)"
+        gazebo_ignition="$(arg gazebo_ignition)">
+        <origin xyz="${top_lidar_offset_x} ${top_lidar_offset_y} ${top_lidar_offset_z}" rpy="0 ${PI/2} 0"/>
+    </xacro:sensor_robosense_bpearl>
 	<!-- Controllers -->
 	<xacro:if value="$(arg gazebo_classic)">

Commit message: use mesh as collision

File: robots/rbtheron/rbtheron_plus.urdf.xacro (robot description, xacro)
@@ -48,5 +48,5 @@
         <collision>
             <geometry>
-                <box size="0.624 0.544 0.629"/>
+                <mesh filename="package://robotnik_description/meshes/bases/rbtheron/rbtheron_plus_top_chassis.stl"/>
             </geometry>
         </collision>

Commit message: rbtheron_plus: Fix rbpearl position

File: robots/rbtheron/rbtheron_plus.urdf.xacro (robot description, xacro)
@@ -136,12 +136,19 @@
     </xacro:sensor_intel_realsense_d435>
     <!-- 3D LiDAR -->
+    <joint name="$(arg prefix)top_lidar_aux_joint" type="fixed">
+        <origin xyz="${top_lidar_offset_x} ${top_lidar_offset_y} ${top_lidar_offset_z}" rpy="0 ${PI/2}  0"/>
+        <parent link="$(arg prefix)top_chassis"/>
+        <child link="$(arg prefix)top_lidar_aux"/>
+    </joint>
+    <link name="$(arg prefix)top_lidar_aux">
+    </link>
     <xacro:sensor_robosense_bpearl
         frame_prefix="$(arg prefix)top_lidar_"
-        parent="$(arg prefix)top_chassis"
+        parent="$(arg prefix)top_lidar_aux"
         node_namespace="$(arg namespace)"
         node_name="top_lidar"
         gazebo_classic="$(arg gazebo_classic)"
         gazebo_ignition="$(arg gazebo_ignition)">
-        <origin xyz="${top_lidar_offset_x} ${top_lidar_offset_y} ${top_lidar_offset_z}" rpy="0 ${PI/2} 0"/>
+        <origin xyz="0 0 0" rpy="0 0 ${PI/3}"/>
     </xacro:sensor_robosense_bpearl>
 	<!-- Controllers -->

Commit message: fix rear camera position rbtheron_plus

File: robots/rbtheron/rbtheron_plus.urdf.xacro (robot description, xacro)
@@ -78,5 +78,5 @@
 	<xacro:property name="rear_rgbd_camera_offset_x" value="-0.3045"/>
 	<xacro:property name="rear_rgbd_camera_offset_y" value="0.0"/>
-	<xacro:property name="rear_rgbd_camera_offset_z" value="0.1158"/>
+	<xacro:property name="rear_rgbd_camera_offset_z" value="0.1598"/>
 	<xacro:property name="front_laser_offset_x" value="0.2675"/>
 	<xacro:property name="front_laser_offset_y" value="-0.215"/>
