Commit message: Remove robot_id and substituted by prefix (#16)

File: robots/rbtheron/rbtheron.urdf.xacro (robot description, xacro)
@@ -36,5 +36,5 @@
 	<!-- ELEVATOR_PLATFORM -->
 	<!-- <xacro:if value="$(arg has_elevator)">
-		<xacro:elevator_platform robot_id="rbtheron_elevator" parent="rbtheron_base_link" hq="${hq}">
+		<xacro:elevator_platform prefix="rbtheron_elevator" parent="rbtheron_base_link" hq="${hq}">
 			<origin xyz="${elevator_x} -${elevator_y} ${elevator_z}" rpy="1.5708 0 1.5708"/>
 		</xacro:elevator_platform>

File: robots/rbvogui/rbvogui_cart.urdf.xacro (robot description, xacro)
@@ -15,31 +15,31 @@
     <xacro:property name="hq" value="true" />
     <xacro:property name="publish_bf" value="true" />
-    <xacro:arg name="robot_id" default="robot" />
+    <xacro:arg name="prefix" default="robot" />
     <xacro:arg name="namespace" default="robot" />
     <xacro:arg name="gpu" default="true" />
     <xacro:arg name="hardware" default="omni" />
     <xacro:arg name="controllers" default="$(find rbvogui_gazebo)/config/omni_controller.yaml" />
-    <xacro:rbvogui robot_id="$(arg robot_id)_" hardware="$(arg hardware)" gpu="$(arg gpu)" publish_bf="${publish_bf}" hq="${hq}"/>
+    <xacro:rbvogui prefix="$(arg prefix)_" hardware="$(arg hardware)" gpu="$(arg gpu)" publish_bf="${publish_bf}" hq="${hq}"/>
     <!-- SENSORS see robotnik_sensors for the specific configuration -->
     <!-- IMU -->
-    <!-- <xacro:sensor_vectornav prefix="${prefix}" parent="${prefix}chassis_link" topic="${robot_id}/imu/data">
+    <!-- <xacro:sensor_vectornav prefix="${prefix}" parent="${prefix}chassis_link" topic="${prefix}/imu/data">
         <origin xyz="0.3 -0.3 0.0725" rpy="0 0 0"/>
     </xacro:sensor_vectornav> -->
     <!-- Front Camera -->
-    <!-- <xacro:sensor_intel_d435 prefix="${prefix}front_rgbd_camera" parent="${prefix}chassis_link" prefix_topic="${robot_id}/front_rgbd_camera" use_nominal_extrinsics="true">
+    <!-- <xacro:sensor_intel_d435 prefix="${prefix}front_rgbd_camera" parent="${prefix}chassis_link" prefix_topic="${prefix}/front_rgbd_camera" use_nominal_extrinsics="true">
         <origin xyz="0.46462 0.0 0.18258" rpy="0 0 0"/>
     </xacro:sensor_intel_d435> -->
     <!-- Rear Camera -->
-    <!-- <xacro:sensor_intel_d435 prefix="${prefix}rear_rgbd_camera" parent="${prefix}base_link" prefix_topic="${robot_id}/rear_rgbd_camera" use_nominal_extrinsics="true">
+    <!-- <xacro:sensor_intel_d435 prefix="${prefix}rear_rgbd_camera" parent="${prefix}base_link" prefix_topic="${prefix}/rear_rgbd_camera" use_nominal_extrinsics="true">
         <origin xyz="-0.503 0.0 0.29" rpy="0 0 -${PI}"/>
     </xacro:sensor_intel_d435> -->
     <!-- 2d laser -->
-    <!-- <xacro:sensor_sick_s300 prefix="${prefix}front_laser" parent="${prefix}chassis_link" gpu="${gpu}" prefix_topic="${robot_id}/front_laser">
+    <!-- <xacro:sensor_sick_s300 prefix="${prefix}front_laser" parent="${prefix}chassis_link" gpu="${gpu}" prefix_topic="${prefix}/front_laser">
         <origin xyz="0.53 0.33 0.1145" rpy="${PI} 0 ${PI/4}"/>
     </xacro:sensor_sick_s300>
-    <xacro:sensor_sick_s300 prefix="${prefix}rear_laser" parent="${prefix}chassis_link" gpu="${gpu}" prefix_topic="${robot_id}/rear_laser">
+    <xacro:sensor_sick_s300 prefix="${prefix}rear_laser" parent="${prefix}chassis_link" gpu="${gpu}" prefix_topic="${prefix}/rear_laser">
         <origin xyz="-0.53 -0.33 0.1145" rpy="${PI} 0 ${-PI*3/4}"/>
     </xacro:sensor_sick_s300> -->
-    <xacro:ros2_control namespace="$(arg namespace)" robot_id="$(arg robot_id)_" controllers="$(arg controllers)"/>
+    <xacro:ros2_control namespace="$(arg namespace)" prefix="$(arg prefix)_" controllers="$(arg controllers)"/>
     <!-- Cart -->
     <!-- <xacro:include filename="$(find robotnik_description)/urdf/cart/robot_cart_connection.urdf.xacro" />
@@ -51,5 +51,5 @@
         </xacro:cart_connection>
         <xacro:if value="$(arg connected)">
-            <xacro:cart_base prefix="$(arg prefix)cart_" connected="$(arg connected)" namespace="$(arg robot_id)">
+            <xacro:cart_base prefix="$(arg prefix)cart_" connected="$(arg connected)" namespace="$(arg prefix)">
             </xacro:cart_base>
         </xacro:if>

File: urdf/bases/rbkairos/rbkairos_base.urdf.xacro (robot description, xacro)
@@ -19,14 +19,14 @@
   		<!-- Here we create the robot elements using the xacro:macros imported at the beggining of this file -->
   		<xacro:rbkairos_plus_body prefix="${prefix}"/>
-  		<xacro:omni_wheel robot_id="${prefix}front_right" parent="${prefix}base_link" reflect="false" hq="true">
+  		<xacro:omni_wheel prefix="${prefix}front_right_" parent="${prefix}base_link" reflect="false" hq="true">
   			<origin xyz="${wheel_offset_x} -${wheel_offset_y} ${wheel_offset_z}" rpy="0 0 ${PI/4}"/>
   		</xacro:omni_wheel>
-  		<xacro:omni_wheel robot_id="${prefix}front_left" parent="${prefix}base_link" reflect="true" hq="true">
+  		<xacro:omni_wheel prefix="${prefix}front_left_" parent="${prefix}base_link" reflect="true" hq="true">
   			<origin xyz="${wheel_offset_x} ${wheel_offset_y} ${wheel_offset_z}" rpy="0 0 ${-PI/4}"/>
   		</xacro:omni_wheel>
-  		<xacro:omni_wheel robot_id="${prefix}back_left" parent="${prefix}base_link" reflect="false" hq="true">
+  		<xacro:omni_wheel prefix="${prefix}back_left_" parent="${prefix}base_link" reflect="false" hq="true">
   			<origin xyz="-${wheel_offset_x} ${wheel_offset_y} ${wheel_offset_z}" rpy="0 0 ${PI/4}"/>
   		</xacro:omni_wheel>
-  		<xacro:omni_wheel robot_id="${prefix}back_right" parent="${prefix}base_link" reflect="true" hq="true">
+  		<xacro:omni_wheel prefix="${prefix}back_right_" parent="${prefix}base_link" reflect="true" hq="true">
   			<origin xyz="-${wheel_offset_x} -${wheel_offset_y} ${wheel_offset_z}" rpy="0 0 ${-PI/4}"/>
   		</xacro:omni_wheel>

File: urdf/bases/rbrobout/rbrobout_base.urdf.xacro (robot description, xacro)
@@ -25,14 +25,14 @@
 		<xacro:rbrobout_body prefix="${prefix}" />
 		<!-- Wheels -->
-		<xacro:rbrobout_omni_wheel prefix="${prefix}front_right" parent="${prefix}base_link" reflect="false" hq="${hq}">
+		<xacro:rbrobout_omni_wheel prefix="${prefix}front_right_" parent="${prefix}base_link" reflect="false" hq="${hq}">
 			<origin xyz="${wheel_offset_x} -${wheel_offset_y} ${wheel_offset_z}" rpy="0 0 ${PI/4}"/>
 		</xacro:rbrobout_omni_wheel>
-		<xacro:rbrobout_omni_wheel prefix="${prefix}front_left" parent="${prefix}base_link" reflect="true" hq="${hq}">
+		<xacro:rbrobout_omni_wheel prefix="${prefix}front_left_" parent="${prefix}base_link" reflect="true" hq="${hq}">
 			<origin xyz="${wheel_offset_x} ${wheel_offset_y} ${wheel_offset_z}" rpy="0 0 ${-PI/4}"/>
 		</xacro:rbrobout_omni_wheel>
-		<xacro:rbrobout_omni_wheel prefix="${prefix}back_left" parent="${prefix}base_link" reflect="false" hq="${hq}">
+		<xacro:rbrobout_omni_wheel prefix="${prefix}back_left_" parent="${prefix}base_link" reflect="false" hq="${hq}">
 			<origin xyz="-${wheel_offset_x} ${wheel_offset_y} ${wheel_offset_z}" rpy="0 0 ${PI/4}"/>
 		</xacro:rbrobout_omni_wheel>
-		<xacro:rbrobout_omni_wheel prefix="${prefix}back_right" parent="${prefix}base_link" reflect="true" hq="${hq}">
+		<xacro:rbrobout_omni_wheel prefix="${prefix}back_right_" parent="${prefix}base_link" reflect="true" hq="${hq}">
 			<origin xyz="-${wheel_offset_x} -${wheel_offset_y} ${wheel_offset_z}" rpy="0 0 ${-PI/4}"/>
 		</xacro:rbrobout_omni_wheel>

File: urdf/bases/rbsteel/rbsteel_base.urdf.xacro (robot description, xacro)
@@ -21,14 +21,14 @@
   		<!-- Here we create the robot elements using the xacro:macros imported at the beggining of this file -->
   		<xacro:rbkairos_body prefix="robot_"/>
-  		<xacro:omni_wheel robot_id="${prefix}front_right" parent="${prefix}base_link" reflect="false" hq="true">
+  		<xacro:omni_wheel prefix="${prefix}front_right_" parent="${prefix}base_link" reflect="false" hq="true">
   			<origin xyz="${wheel_offset_x} -${wheel_offset_y} ${wheel_offset_z}" rpy="0 0 0"/>
   		</xacro:omni_wheel>
-  		<xacro:omni_wheel robot_id="${prefix}front_left" parent="${prefix}base_link" reflect="true" hq="true">
+  		<xacro:omni_wheel prefix="${prefix}front_left_" parent="${prefix}base_link" reflect="true" hq="true">
   			<origin xyz="${wheel_offset_x} ${wheel_offset_y} ${wheel_offset_z}" rpy="0 0 0"/>
   		</xacro:omni_wheel>
-  		<xacro:omni_wheel robot_id="${prefix}back_left" parent="${prefix}base_link" reflect="true" hq="true">
+  		<xacro:omni_wheel prefix="${prefix}back_left_" parent="${prefix}base_link" reflect="true" hq="true">
   			<origin xyz="-${wheel_offset_x} ${wheel_offset_y} ${wheel_offset_z}" rpy="0 0 0"/>
   		</xacro:omni_wheel>
-  		<xacro:omni_wheel robot_id="${prefix}back_right" parent="${prefix}base_link" reflect="false" hq="true">
+  		<xacro:omni_wheel prefix="${prefix}back_right_" parent="${prefix}base_link" reflect="false" hq="true">
   			<origin xyz="-${wheel_offset_x} -${wheel_offset_y} ${wheel_offset_z}" rpy="0 0 0"/>
   		</xacro:omni_wheel>

File: urdf/bases/rbsummit/rbsummit_base.xacro (robot description, xacro)
@@ -19,14 +19,14 @@
 		<xacro:rbsummit_body prefix="${prefix}" hq="${hq}" />
 		<!-- Summit XL wheels -->
-		<xacro:rubber_wheel robot_id="${prefix}front_right" parent="${prefix}base_link" reflect="false" hq="${hq}" mesh_file="${mesh_file_right}">
+		<xacro:rubber_wheel prefix="${prefix}front_right_" parent="${prefix}base_link" reflect="false" hq="${hq}" mesh_file="${mesh_file_right}">
 			<origin xyz="${wheel_offset_x} -${wheel_offset_y} ${wheel_offset_z}" rpy="0 0 0"/>
 		</xacro:rubber_wheel>
-		<xacro:rubber_wheel robot_id="${prefix}front_left" parent="${prefix}base_link" reflect="false" hq="${hq}" mesh_file="${mesh_file_left}">
+		<xacro:rubber_wheel prefix="${prefix}front_left_" parent="${prefix}base_link" reflect="false" hq="${hq}" mesh_file="${mesh_file_left}">
 			<origin xyz="${wheel_offset_x} ${wheel_offset_y} ${wheel_offset_z}" rpy="0 0 0"/>
 		</xacro:rubber_wheel>
-		<xacro:rubber_wheel robot_id="${prefix}back_left" parent="${prefix}base_link" reflect="false" hq="${hq}" mesh_file="${mesh_file_left}">
+		<xacro:rubber_wheel prefix="${prefix}back_left_" parent="${prefix}base_link" reflect="false" hq="${hq}" mesh_file="${mesh_file_left}">
 			<origin xyz="-${wheel_offset_x} ${wheel_offset_y} ${wheel_offset_z}" rpy="0 0 0"/>
 		</xacro:rubber_wheel>
-		<xacro:rubber_wheel robot_id="${prefix}back_right" parent="${prefix}base_link" reflect="false" hq="${hq}" mesh_file="${mesh_file_right}">
+		<xacro:rubber_wheel prefix="${prefix}back_right_" parent="${prefix}base_link" reflect="false" hq="${hq}" mesh_file="${mesh_file_right}">
 			<origin xyz="-${wheel_offset_x} -${wheel_offset_y} ${wheel_offset_z}" rpy="0 0 0"/>
 		</xacro:rubber_wheel>

File: urdf/bases/rbtheron/rbtheron_base.xacro (robot description, xacro)
@@ -23,21 +23,21 @@
 		<xacro:rbtheron_body prefix="${prefix}" hq="${hq}" />
 		<!-- WHEELS -->
-		<xacro:rubber_wheel robot_id="${prefix}right" parent="${prefix}base_link" hq="${hq}">
+		<xacro:rubber_wheel prefix="${prefix}right_" parent="${prefix}base_link" hq="${hq}">
 			<origin xyz="${wheel_offset_x} ${-wheel_offset_y} ${wheel_offset_z}" rpy="0 0 0"/>
 		</xacro:rubber_wheel>
-		<xacro:rubber_wheel robot_id="${prefix}left" parent="${prefix}base_link" hq="${hq}">
+		<xacro:rubber_wheel prefix="${prefix}left_" parent="${prefix}base_link" hq="${hq}">
 			<origin xyz="${wheel_offset_x} ${wheel_offset_y} ${wheel_offset_z}" rpy="0 0 0"/>
 		</xacro:rubber_wheel>
 		<!-- Castor wheels-->
-		<xacro:caster robot_id="${prefix}front_left" parent="${prefix}base_link" hq="${hq}" use_sim="true">
+		<xacro:caster prefix="${prefix}front_left_" parent="${prefix}base_link" hq="${hq}" use_sim="true">
 			<origin xyz="${castor_offset_x} ${castor_offset_y} ${castor_offset_z}" rpy="0 0 0"/>
 		</xacro:caster>
-		<xacro:caster robot_id="${prefix}front_right" parent="${prefix}base_link" hq="${hq}" use_sim="true">
+		<xacro:caster prefix="${prefix}front_right_" parent="${prefix}base_link" hq="${hq}" use_sim="true">
 			<origin xyz="${castor_offset_x} ${-castor_offset_y} ${castor_offset_z}" rpy="0 0 0"/>
 		</xacro:caster>
-		<xacro:caster robot_id="${prefix}rear_left" parent="${prefix}base_link" hq="${hq}" use_sim="true">
+		<xacro:caster prefix="${prefix}rear_left_" parent="${prefix}base_link" hq="${hq}" use_sim="true">
 			<origin xyz="${-castor_offset_x} ${castor_offset_y} ${castor_offset_z}" rpy="0 0 0"/>
 		</xacro:caster>
-		<xacro:caster robot_id="${prefix}rear_right" parent="${prefix}base_link" hq="${hq}" use_sim="true">
+		<xacro:caster prefix="${prefix}rear_right_" parent="${prefix}base_link" hq="${hq}" use_sim="true">
 			<origin xyz="${-castor_offset_x} ${-castor_offset_y} ${castor_offset_z}" rpy="0 0 0"/>
 		</xacro:caster>

File: urdf/bases/rbvogui/rbvogui_base.urdf.xacro (robot description, xacro)
@@ -23,14 +23,14 @@
         <!-- Here we create the robot elements using the xacro:macros imported at the beggining of this file -->
         <xacro:rbvogui_body prefix="${prefix}" hq="${hq}"/>
-        <xacro:steering_wheel robot_id="${prefix}front_right" parent="${prefix}base_link" reflect="false" hq="${hq}">
+        <xacro:steering_wheel prefix="${prefix}front_right_" parent="${prefix}base_link" reflect="false" hq="${hq}">
             <origin xyz="${wheel_offset_x} -${wheel_offset_y} ${wheel_offset_z}" rpy="0 0 0"/>
         </xacro:steering_wheel>
-        <xacro:steering_wheel robot_id="${prefix}front_left" parent="${prefix}base_link" reflect="true" hq="${hq}">
+        <xacro:steering_wheel prefix="${prefix}front_left_" parent="${prefix}base_link" reflect="true" hq="${hq}">
             <origin xyz="${wheel_offset_x} ${wheel_offset_y} ${wheel_offset_z}" rpy="0 0 0"/>
         </xacro:steering_wheel>
-        <xacro:steering_wheel robot_id="${prefix}back_left" parent="${prefix}base_link" reflect="true" hq="${hq}">
+        <xacro:steering_wheel prefix="${prefix}back_left_" parent="${prefix}base_link" reflect="true" hq="${hq}">
             <origin xyz="-${wheel_offset_x} ${wheel_offset_y} ${wheel_offset_z}" rpy="0 0 0"/>
         </xacro:steering_wheel>
-        <xacro:steering_wheel robot_id="${prefix}back_right" parent="${prefix}base_link" reflect="false" hq="${hq}">
+        <xacro:steering_wheel prefix="${prefix}back_right_" parent="${prefix}base_link" reflect="false" hq="${hq}">
             <origin xyz="-${wheel_offset_x} -${wheel_offset_y} ${wheel_offset_z}" rpy="0 0 0"/>
         </xacro:steering_wheel>

File: urdf/structures/container/structure_chair.urdf.xacro (robot description, xacro)
@@ -2,11 +2,11 @@
 <robot name="structure" xmlns:xacro="http://wiki.ros.org/xacro">
   <xacro:macro name="structure_chair" params="prefix parent *origin">
-	  <joint name="${prefix}_joint" type="fixed">
+	  <joint name="${prefix}joint" type="fixed">
 	    <axis xyz="0 1 0"/>
 	    <xacro:insert_block name="origin"/>
 	    <parent link="${parent}"/>
-	    <child link="${prefix}_link"/>
+	    <child link="${prefix}link"/>
 	  </joint>
-	  <link name="${prefix}_link">
+	  <link name="${prefix}link">
 	    <inertial>
 	      <mass value="0.001"/>
@@ -30,5 +30,5 @@
 	    </collision>
 	  </link>
-	  <gazebo reference="${prefix}_link">
+	  <gazebo reference="${prefix}link">
 	    <material>Gazebo/Black</material>
 	    <gravity>true</gravity>

File: urdf/structures/elevator/rb1_base_elevator.gazebo.xacro (robot description, xacro)
@@ -2,5 +2,5 @@
 <robot xmlns:xacro="http://www.ros.org/wiki/xacro">
 	<xacro:macro name="elevator_gazebo" params="prefix">
-		<gazebo reference="${prefix}_platform_link">
+		<gazebo reference="${prefix}platform_link">
 			<mu1 value="5.0"/>
 			<mu2 value="0.5"/>

File: urdf/structures/elevator/rb1_base_elevator.transmission.xacro (robot description, xacro)
@@ -4,7 +4,7 @@
 	<xacro:macro name="elevator_transmission" params="prefix">
 	<!-- Transmission is important to link the joints and the controller (see rb1_control/config/rb1_control.yaml)-->
-		<transmission name="${prefix}_platform_trans">
+		<transmission name="${prefix}platform_trans">
 			<type>transmission_interface/SimpleTransmission</type>
-			<joint name="${prefix}_platform_joint">
+			<joint name="${prefix}platform_joint">
 				<!-- for the gazebo plugin -->
 				<!--hardwareInterface>EffortJointInterface</hardwareInterface-->
@@ -12,5 +12,5 @@
 				<hardwareInterface>hardware_interface/EffortJointInterface</hardwareInterface>
 			</joint>
-			<actuator name="${prefix}_platform_joint_motor">
+			<actuator name="${prefix}platform_joint_motor">
 				<hardwareInterface>EffortJointInterface</hardwareInterface>
 				<mechanicalReduction>1</mechanicalReduction>

File: urdf/structures/elevator/rb1_base_elevator.urdf.xacro (robot description, xacro)
@@ -14,10 +14,10 @@
     </xacro:macro>
 	<!-- ELEVATOR_BASE_LINK -->
-	<joint name="${prefix}_base_joint" type="fixed">
+	<joint name="${prefix}base_joint" type="fixed">
 		<parent link="${parent}"/>
-		<child link="${prefix}_base_link"/>
+		<child link="${prefix}base_link"/>
 		<xacro:insert_block name="origin" />
 	</joint>
-	<link name="${prefix}_base_link">
+	<link name="${prefix}base_link">
 		<!--inertial>
 			<mass value="0.1" />
@@ -56,12 +56,12 @@
 	</link>
 	<!-- ELEVATOR PLATFORM -->
-	<joint name="${prefix}_platform_joint" type="prismatic">
+	<joint name="${prefix}platform_joint" type="prismatic">
 			<origin xyz="0.0 0.0 0.041" rpy="0 0 0 " />
-			<parent link="${prefix}_base_link"/>
-			<child link="${prefix}_platform_link" />
+			<parent link="${prefix}base_link"/>
+			<child link="${prefix}platform_link" />
 			<axis xyz="0 0 1"/>
 			<limit effort="10.0" lower="0.0" upper="0.034" velocity="0.5"/>
 	</joint>
-	<link name="${prefix}_platform_link">
+	<link name="${prefix}platform_link">
 		<!--inertial>
 			<mass value="0.05" />

File: urdf/structures/elevator/rb_theron_elevator.transmission.xacro (robot description, xacro)
@@ -4,7 +4,7 @@
 	<xacro:macro name="elevator_transmission" params="prefix">
 	<!-- Transmission is important to link the joints and the controller (see rb_theron_control/config/rb_theron_control.yaml)-->
-		<transmission name="${prefix}_platform_trans">
+		<transmission name="${prefix}platform_trans">
 			<type>transmission_interface/SimpleTransmission</type>
-			<joint name="${prefix}_platform_joint">
+			<joint name="${prefix}platform_joint">
 				<!-- for the gazebo plugin -->
 				<!--hardwareInterface>EffortJointInterface</hardwareInterface-->
@@ -12,5 +12,5 @@
 				<hardwareInterface>hardware_interface/EffortJointInterface</hardwareInterface>
 			</joint>
-			<actuator name="${prefix}_platform_joint_motor">
+			<actuator name="${prefix}platform_joint_motor">
 				<hardwareInterface>EffortJointInterface</hardwareInterface>
 				<mechanicalReduction>1</mechanicalReduction>

File: urdf/structures/elevator/rb_theron_elevator.urdf.xacro (robot description, xacro)
@@ -14,10 +14,10 @@
     </xacro:macro>
 	<!-- ELEVATOR_BASE_LINK -->
-	<joint name="${prefix}_base_joint" type="fixed">
+	<joint name="${prefix}base_joint" type="fixed">
 		<parent link="${parent}"/>
-		<child link="${prefix}_base_link"/>
+		<child link="${prefix}base_link"/>
 		<xacro:insert_block name="origin" />
 	</joint>
-	<link name="${prefix}_base_link">
+	<link name="${prefix}base_link">
 		<!--inertial>
 			<mass value="0.1" />
@@ -56,12 +56,12 @@
 	</link>
 	<!-- ELEVATOR PLATFORM -->
-	<joint name="${prefix}_platform_joint" type="prismatic">
+	<joint name="${prefix}platform_joint" type="prismatic">
 			<origin xyz="0.0 0.0 0.0" rpy="0 0 0 " />
-			<parent link="${prefix}_base_link"/>
-			<child link="${prefix}_platform_link" />
+			<parent link="${prefix}base_link"/>
+			<child link="${prefix}platform_link" />
 			<axis xyz="0 1 0"/>
 			<limit effort="10.0" lower="0.0" upper="0.03" velocity="0.5"/>
 	</joint>
-	<link name="${prefix}_platform_link">
+	<link name="${prefix}platform_link">
 		<!--inertial>
 			<mass value="0.05" />

File: urdf/structures/rbkairos_chassis/sick_microscan3_support.urdf.xacro (robot description, xacro)
@@ -3,10 +3,10 @@
   <xacro:macro name="sick_microscan3_support" params="prefix parent *origin">
     <!--CONTAINER -->
-    <joint name="${prefix}_support_joint" type="fixed">
+    <joint name="${prefix}support_joint" type="fixed">
       <xacro:insert_block name="origin"/>
       <parent link="${parent}"/>
-      <child link="${prefix}_support_link"/>
+      <child link="${prefix}support_link"/>
     </joint>
-    <link name="${prefix}_support_link">
+    <link name="${prefix}support_link">
 	       <visual>
 	      <geometry>

File: urdf/structures/rbkairos_chassis/structure_hokuyo.urdf.xacro (robot description, xacro)
@@ -2,11 +2,11 @@
 <robot name="structure" xmlns:xacro="http://wiki.ros.org/xacro">
   <xacro:macro name="structure_laser" params="prefix parent *origin">
-	  <joint name="${prefix}_joint" type="fixed">
+	  <joint name="${prefix}joint" type="fixed">
 	    <axis xyz="0 1 0"/>
 	    <xacro:insert_block name="origin"/>
 	    <parent link="${parent}"/>
-	    <child link="${prefix}_link"/>
+	    <child link="${prefix}link"/>
 	  </joint>
-	  <link name="${prefix}_link">
+	  <link name="${prefix}link">
 	    <inertial>
 	      <mass value="0.001"/>
@@ -30,5 +30,5 @@
 	    </collision>
 	  </link>
-	  <gazebo reference="${prefix}_link">
+	  <gazebo reference="${prefix}link">
 	    <material>Gazebo/White</material>
 	    <gravity>true</gravity>

File: urdf/structures/rbvogui_chassis/m1_mount.urdf.xacro (robot description, xacro)
@@ -2,10 +2,10 @@
 <robot name="m1_mount" xmlns:xacro="http://wiki.ros.org/xacro">
   <xacro:macro name="m1_mount" params="prefix parent *origin">
-	 <joint name="${prefix}_base_joint" type="fixed">
+	 <joint name="${prefix}base_joint" type="fixed">
            <xacro:insert_block name="origin" />
            <parent link="${parent}"/>
-           <child link="${prefix}_base_link" />
+           <child link="${prefix}base_link" />
          </joint>
-	  <link name="${prefix}_base_link">
+	  <link name="${prefix}base_link">
 	    <visual>
 	      <origin rpy="0 0 0" xyz="0 0 0"/>

File: urdf/structures/rbvogui_chassis/rigid_cover.urdf.xacro (robot description, xacro)
@@ -2,10 +2,10 @@
 <robot name="rigid_cover" xmlns:xacro="http://wiki.ros.org/xacro">
   <xacro:macro name="rigid_cover" params="prefix parent *origin">
-	 <joint name="${prefix}_base_joint" type="fixed">
+	 <joint name="${prefix}base_joint" type="fixed">
            <xacro:insert_block name="origin" />
            <parent link="${parent}"/>
-           <child link="${prefix}_base_link" />
+           <child link="${prefix}base_link" />
          </joint>
-	  <link name="${prefix}_base_link">
+	  <link name="${prefix}base_link">
 	    <visual>
 	      <origin rpy="0 0 0" xyz="0 0 0"/>
