Commit message: Remove robot_id and substituted by prefix (#16)

File: urdf/structures/rbvogui_chassis/top_cover.urdf.xacro (robot description, xacro)
@@ -2,10 +2,10 @@
 <robot name="top_cover" xmlns:xacro="http://wiki.ros.org/xacro">
   <xacro:macro name="structure_top_cover" params="prefix parent *origin">
-	 <joint name="${prefix}_base_joint" type="fixed">
+	 <joint name="${prefix}base_joint" type="fixed">
            <xacro:insert_block name="origin" />
            <parent link="${parent}"/>
-           <child link="${prefix}_top_cover_link" />
+           <child link="${prefix}top_cover_link" />
          </joint>
-	  <link name="${prefix}_top_cover_link">
+	  <link name="${prefix}top_cover_link">
 	    <visual>
 	      <origin rpy="0 0 0" xyz="0 0 0"/>
@@ -24,5 +24,5 @@
 	    </collision>
 	  </link>
-    <gazebo reference="${prefix}_top_cover_link">
+    <gazebo reference="${prefix}top_cover_link">
 		<visual>
 		  <material>

File: urdf/structures/rbvogui_chassis/zed_support.urdf.xacro (robot description, xacro)
@@ -2,10 +2,10 @@
 <robot name="zed_support" xmlns:xacro="http://wiki.ros.org/xacro">
   <xacro:macro name="zed_support" params="prefix parent *origin">
-	 <joint name="${prefix}_base_joint" type="fixed">
+	 <joint name="${prefix}base_joint" type="fixed">
            <xacro:insert_block name="origin" />
            <parent link="${parent}"/>
-           <child link="${prefix}_base_link" />
+           <child link="${prefix}base_link" />
          </joint>
-	  <link name="${prefix}_base_link">
+	  <link name="${prefix}base_link">
 	    <visual>
 	      <origin rpy="0 0 0" xyz="0 0 0"/>

Commit message: rbtheron_plus: Update UR arm, add positions arguments

File: robots/rbtheron/rbtheron.urdf.xacro (robot description, xacro)
@@ -13,4 +13,10 @@
 	<!-- Import all available sensors -->
 	<xacro:include filename="$(find robotnik_sensors)/urdf/all_sensors.urdf.xacro" />
+    <xacro:include filename="$(find ur_description)/urdf/ur_macro.xacro" />
+    <xacro:arg name="ur_type" default="ur5e"/>
+    <xacro:arg name="joint_limit_params" default="$(find ur_description)/config/$(arg ur_type)/joint_limits.yaml"/>
+    <xacro:arg name="kinematics_params" default="$(find ur_description)/config/$(arg ur_type)/default_kinematics.yaml"/>
+    <xacro:arg name="physical_params" default="$(find ur_description)/config/$(arg ur_type)/physical_parameters.yaml"/>
+    <xacro:arg name="visual_params" default="$(find ur_description)/config/$(arg ur_type)/visual_parameters.yaml"/>
 	<!-- ***************** -->
 	<!-- Global parameters -->
@@ -26,8 +32,61 @@
 	<!-- Here we create the robot using the xacro:macro imported at the beggining of this file -->
 	<xacro:rbtheron prefix="$(arg prefix)" hq="${hq}"/>
+    <joint name="$(arg prefix)top_chassis_joint" type="fixed">
+        <origin xyz="0.0 0.0 0.26" rpy="0.0 0.0 0.0"/>
+        <parent link="$(arg prefix)base_link"/>
+        <child link="$(arg prefix)top_chassis"/>
+    </joint>
+    <link name="$(arg prefix)top_chassis">
+        <visual>
+            <geometry>
+                <mesh filename="package://robotnik_description/meshes/bases/rbtheron/rbtheron_plus_top_chassis.stl"/>
+            </geometry>
+            <material name="grey">
+                <color rgba="0.2 0.2 0.2 1"/>
+            </material>
+        </visual>
+        <collision>
+            <geometry>
+                <mesh filename="package://robotnik_description/meshes/bases/rbtheron/rbtheron_plus_top_chassis.stl"/>
+            </geometry>
+        </collision>
+        <inertial>
+            <mass value="10.0"/>
+            <xacro:solid_cuboid_inertia w="0.544" h="0.629" d="0.624" m="10.0"/>
+        </inertial>
+    </link>
+    <!-- Import UR arm -->
+    <xacro:ur_robot
+        tf_prefix="$(arg prefix)arm_"
+        name="$(arg ur_type)"
+        parent="$(arg prefix)top_chassis"
+        joint_limits_parameters_file="$(arg joint_limit_params)"
+        kinematics_parameters_file="$(arg kinematics_params)"
+        physical_parameters_file="$(arg physical_params)"
+        visual_parameters_file="$(arg visual_params)"
+        sim_gazebo="$(arg gazebo_classic)"
+        sim_ignition="$(arg gazebo_ignition)">
+        <origin xyz="-0.2 0 0.6" rpy="0 0 0"/>
+    </xacro:ur_robot>
 	<!-- SENSORS -->
     <xacro:property name="imu_offset_x" value="-0.1975"/>
     <xacro:property name="imu_offset_y" value="0.0"/>
     <xacro:property name="imu_offset_z" value="0.1598"/>
+	<xacro:property name="front_rgbd_camera_offset_x" value="0.3045"/>
+	<xacro:property name="front_rgbd_camera_offset_y" value="0.0"/>
+	<xacro:property name="front_rgbd_camera_offset_z" value="0.1898"/>
+	<xacro:property name="rear_rgbd_camera_offset_x" value="-0.3045"/>
+	<xacro:property name="rear_rgbd_camera_offset_y" value="0.0"/>
+	<xacro:property name="rear_rgbd_camera_offset_z" value="0.1158"/>
+	<xacro:property name="front_laser_offset_x" value="0.2675"/>
+	<xacro:property name="front_laser_offset_y" value="-0.215"/>
+	<xacro:property name="front_laser_offset_z" value="0.1613"/>
+	<xacro:property name="rear_laser_offset_x" value="-0.2675"/>
+	<xacro:property name="rear_laser_offset_y" value="0.215"/>
+	<xacro:property name="rear_laser_offset_z" value="0.1613"/>
+	<xacro:property name="top_lidar_offset_x" value="0.26"/>
+	<xacro:property name="top_lidar_offset_y" value="0.0"/>
+	<xacro:property name="top_lidar_offset_z" value="0.51"/>
+	<!-- IMU -->
     <xacro:sensor_vectornav
         frame_prefix="$(arg prefix)vectornav_"
@@ -38,4 +97,59 @@
         <origin xyz="${imu_offset_x} ${imu_offset_y} ${imu_offset_z}" rpy="0 0 0"/>
     </xacro:sensor_vectornav>
+	<!-- 2D LASER -->
+    <xacro:sensor_hokuyo_ust20lx
+        frame_prefix="$(arg prefix)front_laser_"
+        parent="$(arg prefix)base_link"
+        node_namespace="$(arg namespace)"
+        node_name="front_laser"
+        gazebo_classic="$(arg gazebo_classic)"
+        gazebo_ignition="$(arg gazebo_ignition)">
+        <origin xyz="${front_laser_offset_x} ${front_laser_offset_y} ${front_laser_offset_z}" rpy="0 ${-PI} ${3/4*PI}"/>
+    </xacro:sensor_hokuyo_ust20lx>
+    <xacro:sensor_hokuyo_ust20lx
+        frame_prefix="$(arg prefix)rear_laser_"
+        parent="$(arg prefix)base_link"
+        node_namespace="$(arg namespace)"
+        node_name="rear_laser"
+        gazebo_classic="$(arg gazebo_classic)"
+        gazebo_ignition="$(arg gazebo_ignition)">
+        <origin xyz="${rear_laser_offset_x} ${rear_laser_offset_y} ${rear_laser_offset_z}" rpy="0 ${-PI} ${-1/4*PI}"/>
+    </xacro:sensor_hokuyo_ust20lx>
+  	<!-- CAMERAS -->
+    <xacro:sensor_intel_realsense_d435
+        frame_prefix="$(arg prefix)front_rgbd_camera_"
+        parent="$(arg prefix)base_link"
+        node_namespace="$(arg namespace)"
+        node_name="front_camera"
+        gazebo_classic="$(arg gazebo_classic)"
+        gazebo_ignition="$(arg gazebo_ignition)">
+        <origin xyz="${front_rgbd_camera_offset_x} ${front_rgbd_camera_offset_y} ${front_rgbd_camera_offset_z}" rpy="0 0 0"/>
+    </xacro:sensor_intel_realsense_d435>
+    <xacro:sensor_intel_realsense_d435
+        frame_prefix="$(arg prefix)rear_rgbd_camera_"
+        parent="$(arg prefix)base_link"
+        node_namespace="$(arg namespace)"
+        node_name="rear_camera"
+        gazebo_classic="$(arg gazebo_classic)"
+        gazebo_ignition="$(arg gazebo_ignition)">
+        <origin xyz="${rear_rgbd_camera_offset_x} ${rear_rgbd_camera_offset_y} ${rear_rgbd_camera_offset_z}" rpy="0 0 ${PI}"/>
+    </xacro:sensor_intel_realsense_d435>
+    <!-- 3D LiDAR -->
+    <joint name="$(arg prefix)top_lidar_aux_joint" type="fixed">
+        <origin xyz="${top_lidar_offset_x} ${top_lidar_offset_y} ${top_lidar_offset_z}" rpy="0 ${PI/2}  0"/>
+        <parent link="$(arg prefix)top_chassis"/>
+        <child link="$(arg prefix)top_lidar_aux"/>
+    </joint>
+    <link name="$(arg prefix)top_lidar_aux">
+    </link>
+    <xacro:sensor_robosense_bpearl
+        frame_prefix="$(arg prefix)top_lidar_"
+        parent="$(arg prefix)top_lidar_aux"
+        node_namespace="$(arg namespace)"
+        node_name="top_lidar"
+        gazebo_classic="$(arg gazebo_classic)"
+        gazebo_ignition="$(arg gazebo_ignition)">
+        <origin xyz="0 0 0" rpy="0 0 ${PI/3}"/>
+    </xacro:sensor_robosense_bpearl>
 	<!-- Controllers -->
 	<xacro:if value="$(arg gazebo_classic)">

Commit message: fix: remove rbtheron_plus objects from rbtheron

File: robots/rbtheron/rbtheron.urdf.xacro (robot description, xacro)
@@ -13,10 +13,4 @@
 	<!-- Import all available sensors -->
 	<xacro:include filename="$(find robotnik_sensors)/urdf/all_sensors.urdf.xacro" />
-    <xacro:include filename="$(find ur_description)/urdf/ur_macro.xacro" />
-    <xacro:arg name="ur_type" default="ur5e"/>
-    <xacro:arg name="joint_limit_params" default="$(find ur_description)/config/$(arg ur_type)/joint_limits.yaml"/>
-    <xacro:arg name="kinematics_params" default="$(find ur_description)/config/$(arg ur_type)/default_kinematics.yaml"/>
-    <xacro:arg name="physical_params" default="$(find ur_description)/config/$(arg ur_type)/physical_parameters.yaml"/>
-    <xacro:arg name="visual_params" default="$(find ur_description)/config/$(arg ur_type)/visual_parameters.yaml"/>
 	<!-- ***************** -->
 	<!-- Global parameters -->
@@ -32,41 +26,4 @@
 	<!-- Here we create the robot using the xacro:macro imported at the beggining of this file -->
 	<xacro:rbtheron prefix="$(arg prefix)" hq="${hq}"/>
-    <joint name="$(arg prefix)top_chassis_joint" type="fixed">
-        <origin xyz="0.0 0.0 0.26" rpy="0.0 0.0 0.0"/>
-        <parent link="$(arg prefix)base_link"/>
-        <child link="$(arg prefix)top_chassis"/>
-    </joint>
-    <link name="$(arg prefix)top_chassis">
-        <visual>
-            <geometry>
-                <mesh filename="package://robotnik_description/meshes/bases/rbtheron/rbtheron_plus_top_chassis.stl"/>
-            </geometry>
-            <material name="grey">
-                <color rgba="0.2 0.2 0.2 1"/>
-            </material>
-        </visual>
-        <collision>
-            <geometry>
-                <mesh filename="package://robotnik_description/meshes/bases/rbtheron/rbtheron_plus_top_chassis.stl"/>
-            </geometry>
-        </collision>
-        <inertial>
-            <mass value="10.0"/>
-            <xacro:solid_cuboid_inertia w="0.544" h="0.629" d="0.624" m="10.0"/>
-        </inertial>
-    </link>
-    <!-- Import UR arm -->
-    <xacro:ur_robot
-        tf_prefix="$(arg prefix)arm_"
-        name="$(arg ur_type)"
-        parent="$(arg prefix)top_chassis"
-        joint_limits_parameters_file="$(arg joint_limit_params)"
-        kinematics_parameters_file="$(arg kinematics_params)"
-        physical_parameters_file="$(arg physical_params)"
-        visual_parameters_file="$(arg visual_params)"
-        sim_gazebo="$(arg gazebo_classic)"
-        sim_ignition="$(arg gazebo_ignition)">
-        <origin xyz="-0.2 0 0.6" rpy="0 0 0"/>
-    </xacro:ur_robot>
 	<!-- SENSORS -->
     <xacro:property name="imu_offset_x" value="-0.1975"/>
@@ -78,9 +35,9 @@
 	<xacro:property name="rear_rgbd_camera_offset_x" value="-0.3045"/>
 	<xacro:property name="rear_rgbd_camera_offset_y" value="0.0"/>
-	<xacro:property name="rear_rgbd_camera_offset_z" value="0.1158"/>
-	<xacro:property name="front_laser_offset_x" value="0.2675"/>
+	<xacro:property name="rear_rgbd_camera_offset_z" value="0.1598"/>
+	<xacro:property name="front_laser_offset_x" value="0.268"/>
 	<xacro:property name="front_laser_offset_y" value="-0.215"/>
 	<xacro:property name="front_laser_offset_z" value="0.1613"/>
-	<xacro:property name="rear_laser_offset_x" value="-0.2675"/>
+	<xacro:property name="rear_laser_offset_x" value="-0.268"/>
 	<xacro:property name="rear_laser_offset_y" value="0.215"/>
 	<xacro:property name="rear_laser_offset_z" value="0.1613"/>
@@ -135,21 +92,4 @@
         <origin xyz="${rear_rgbd_camera_offset_x} ${rear_rgbd_camera_offset_y} ${rear_rgbd_camera_offset_z}" rpy="0 0 ${PI}"/>
     </xacro:sensor_intel_realsense_d435>
-    <!-- 3D LiDAR -->
-    <joint name="$(arg prefix)top_lidar_aux_joint" type="fixed">
-        <origin xyz="${top_lidar_offset_x} ${top_lidar_offset_y} ${top_lidar_offset_z}" rpy="0 ${PI/2}  0"/>
-        <parent link="$(arg prefix)top_chassis"/>
-        <child link="$(arg prefix)top_lidar_aux"/>
-    </joint>
-    <link name="$(arg prefix)top_lidar_aux">
-    </link>
-    <xacro:sensor_robosense_bpearl
-        frame_prefix="$(arg prefix)top_lidar_"
-        parent="$(arg prefix)top_lidar_aux"
-        node_namespace="$(arg namespace)"
-        node_name="top_lidar"
-        gazebo_classic="$(arg gazebo_classic)"
-        gazebo_ignition="$(arg gazebo_ignition)">
-        <origin xyz="0 0 0" rpy="0 0 ${PI/3}"/>
-    </xacro:sensor_robosense_bpearl>
 	<!-- Controllers -->
 	<xacro:if value="$(arg gazebo_classic)">

Commit message: fix: remove rear RGB-D camera from RB-THERON configuration - Only one camera is more standard

File: robots/rbtheron/rbtheron.urdf.xacro (robot description, xacro)
@@ -68,13 +68,3 @@
       rpy="0 0 0" />
   </xacro:sensor_intel_realsense_d435>
-  <xacro:sensor_intel_realsense_d435
-    frame_prefix="$(arg prefix)rear_rgbd_camera_"
-    parent="$(arg prefix)base_link"
-    node_namespace="$(arg namespace)"
-    node_name="rear_camera"
-    gazebo_ignition="$(arg gazebo_ignition)">
-    <origin
-      xyz="-0.3045 0 0.1358"
-      rpy="0 0 ${pi}" />
-  </xacro:sensor_intel_realsense_d435>
 </robot>
