Commit message: Fix antena_std urdf mesh_file

File: urdf/structures/sensor_support/antena_std.urdf.xacro (robot description, xacro)
@@ -2,5 +2,5 @@
 <robot name="sensor_antena_std" xmlns:xacro="http://wiki.ros.org/xacro">
   <!-- if no latitude/longitud is specified, then use Fuente del Jarro as default -->
-  <xacro:macro name="sensor_antena_std" params="prefix parent *origin mesh_file:=robot_description/meshes/others/antena_wifi_antena_wifi_2J7A747Bc
+  <xacro:macro name="sensor_antena_std" params="prefix parent *origin mesh_file:=robot_description/meshes/others/antena_wifi_2J7A747Bc
   												gazebo_color:=Gazebo/Gray">
 	  <!-- ANTENNA GPS -->
