Commit message: Remove gazebo files and ros2_control, add kairos with ur arm

File: robots/rbkairos/rbkairos.urdf.xacro (robot description, xacro)
@@ -5,5 +5,4 @@
   <!-- ***************** -->
   <!-- First we import all posible elements defined in the urdf.xacro files. All these elements are defined as macro:xacros -->
-  <xacro:arg name="controllers" default="$(find robot_gazebo)/config/rbkairos_control_gazebo.yaml"/>
   <xacro:include filename="$(find robot_description)/macros/rbkairos_macro.urdf.xacro" />
   <!-- Import all available sensors -->
@@ -32,5 +31,4 @@
   <xacro:property name="gps_offset_z" value="0.302"/>
   <xacro:rbkairos/>
-  <xacro:include filename="$(find robot_description)/urdf/ros2_control/rbkairos_control.urdf.xacro" />
   <!-- IMU -->
 	<xacro:sensor_vectornav prefix="rbkairos_" parent="rbkairos_base_link" topic="imu/data">
@@ -56,5 +54,3 @@
     <origin xyz="${gps_offset_x} ${gps_offset_y} ${gps_offset_z}" rpy="0 0 0"/>
   </xacro:sensor_gps-->
-  <xacro:ros2_control controllers="$(arg controllers)"/>
-  <xacro:ros_planar_move/>
 </robot>

File: robots/rbkairos/rbkairos_ur.urdf.xacro (robot description, xacro)
@@ -46,7 +46,4 @@
   <xacro:property name="gps_offset_z" value="0.302"/>
   <xacro:rbkairos/>
-  <xacro:include filename="$(find robot_description)/urdf/ros2_control/rbkairos_control.urdf.xacro" />
-  <!-- UR arm -->
-  <!-- <xacro:ur tf_prefix="rbkairos" ur_type="${ur_type}"/> -->
   <!-- IMU -->
 	<xacro:sensor_vectornav prefix="rbkairos_" parent="rbkairos_base_link" topic="imu/data">
@@ -72,5 +69,3 @@
     <origin xyz="${gps_offset_x} ${gps_offset_y} ${gps_offset_z}" rpy="0 0 0"/>
   </xacro:sensor_gps-->
-  <xacro:ros2_control controllers="$(arg controllers)"/>
-  <xacro:ros_planar_move/>
 </robot>

File: robots/rbsteel/rbsteel.urdf.xacro (robot description, xacro)
@@ -5,5 +5,4 @@
   <!-- ***************** -->
   <!-- First we import all posible elements defined in the urdf.xacro files. All these elements are defined as macro:xacros -->
-  <xacro:arg name="controllers" default="$(find robot_gazebo)/config/rbkairos_control_gazebo.yaml"/>
   <xacro:include filename="$(find robot_description)/macros/rbsteel_macro.urdf.xacro" />
   <!-- Import all available sensors -->

File: robots/rbsummit/rbsummit.urdf.xacro (robot description, xacro)
@@ -9,8 +9,9 @@
 	<!-- Import all available sensors -->
 	<xacro:include filename="$(find robotnik_sensors)/urdf/all_sensors.urdf.xacro" />
+	<xacro:include filename="$(find robotnik_sensors)/urdf/axis_m5013.urdf.xacro" />
+	<xacro:include filename="$(find robotnik_sensors)/urdf/rslidar.urdf.xacro" />
 	<!-- Import antenna -->
 	<xacro:include filename="$(find robot_description)/urdf/structures/sensor_support/structure_teltonika.urdf.xacro" />
-	<xacro:include filename="$(find robot_description)/gazebo/classic/rbsummit_control.urdf.xacro"/>
-	<xacro:include filename="$(find robot_description)/gazebo/ignition/rbsummit_control.urdf.xacro"/>
+	<xacro:include filename="$(find robot_description)/urdf/structures/sensor_support/antena-combo-5G-teltonika.urdf.xacro" />
 	<!-- ***************** -->
 	<!-- Sensor parameters -->
@@ -20,25 +21,21 @@
 	<xacro:property name="imu_offset_y" value="0.132"/>
 	<xacro:property name="imu_offset_z" value="0.158"/>
-	<xacro:property name="top_laser_offset_x" value="-0.11808"/>
+	<xacro:property name="top_laser_offset_x" value="-0.01924"/>
 	<xacro:property name="top_laser_offset_y" value="0.0"/>
-	<xacro:property name="top_laser_offset_z" value="0.38509"/>
+	<xacro:property name="top_laser_offset_z" value="0.35642"/>
 	<xacro:property name="front_rgbd_camera_offset_x" value="0.324"/>
 	<xacro:property name="front_rgbd_camera_offset_y" value="0.012"/>
 	<xacro:property name="front_rgbd_camera_offset_z" value="0.172"/>
-	<xacro:property name="front_ptz_camera_offset_x" value="0.19"/>
+	<xacro:property name="front_ptz_camera_offset_x" value="0.22151"/>
 	<xacro:property name="front_ptz_camera_offset_y" value="0.0"/>
-	<xacro:property name="front_ptz_camera_offset_z" value="0.26"/>
+	<xacro:property name="front_ptz_camera_offset_z" value="0.24022"/>
+	<xacro:property name="front_ptz_camera_offset_t" value="-1.308996939"/>
 	<xacro:property name="gps_offset_x" value="-0.22528"/>
 	<xacro:property name="gps_offset_y" value="0.095"/>
 	<xacro:property name="gps_offset_z" value="0.275"/>
 	<!-- Other elements -->
-	<!--
-	<xacro:property name="antenna_offset_x" value="-0.22528"/>
-	<xacro:property name="antenna_offset_y" value="-0.095"/>
-	<xacro:property name="antenna_offset_z" value="0.23325"/>
-	-->
-	<xacro:property name="antenna_offset_x" value="-0.25528"/>
+	<xacro:property name="antenna_offset_x" value="-0.18324"/>
 	<xacro:property name="antenna_offset_y" value="0.0"/>
-	<xacro:property name="antenna_offset_z" value="0.23325"/>
+	<xacro:property name="antenna_offset_z" value="0.27488"/>
 	<!-- ***************** -->
 	<!-- Global parameters -->
@@ -49,6 +46,4 @@
 	<xacro:property name="hq" value="true" />
 	<!-- Launch Arguments -->
-	<xacro:arg name="use_gazebo_classic" default="false" />
-	<xacro:arg name="use_gazebo_ignition" default="false" />
 	<xacro:arg name="gpu" default="true" />
 	<xacro:arg name="namespace" default="robot" />
@@ -69,5 +64,5 @@
 	</xacro:sensor_vectornav>
 	<!-- 3d laser -->
-	<xacro:sensor_robosense_helios
+	<xacro:sensor_robosense_rslidar_16
 		frame_prefix="rbsummit_top_3d_laser_"
 		parent="rbsummit_base_link"
@@ -78,42 +73,16 @@
 			rpy="0 0 0"
 		/>
-	</xacro:sensor_robosense_helios>
+	</xacro:sensor_robosense_rslidar_16>
 	<!-- ptz camera -->
-	<!--
-	<xacro:sensor_axis
-		prefix="rbsummit_front_ptz_camera"
+	<xacro:sensor_axis_m5013
+		frame_prefix="rbsummit_front_ptz_camera_"
 		parent="rbsummit_base_link"
 	>
 		<origin
-			xyz="0.19 0 0.26"
-			rpy="0 ${15*PI/180} 0"
+			xyz="${front_ptz_camera_offset_x} ${front_ptz_camera_offset_y} ${front_ptz_camera_offset_z}"
+			rpy="0 ${front_ptz_camera_offset_t} 0"
 		/>
-	</xacro:sensor_axis>
-	-->
-	<!-- RGBD -->
-	<xacro:sensor_intel_realsense_d435
-		frame_prefix="rbsummit_front_rgbd_camera_"
-		parent="rbsummit_base_link"
-		topic_prefix="front_rgbd_camera"
-	>
-		<origin
-			xyz="${front_rgbd_camera_offset_x} ${front_rgbd_camera_offset_y} ${front_rgbd_camera_offset_z}"
-			rpy="0 0 0"
-		/>
-	</xacro:sensor_intel_realsense_d435>
-	<!-- GPS -->
-	<xacro:sensor_gps
-		frame_prefix="rbsummit_gps_"
-		parent="rbsummit_base_link"
-		update_rate="5"
-	>
-		<origin
-			xyz="${gps_offset_x} ${gps_offset_y} ${gps_offset_z}"
-			rpy="0 0 0"
-		/>
-	</xacro:sensor_gps>
-	<!-- Other Elements -->
-	<!-- Antenna -->
-	<xacro:structure_mastil_teltonika
+	</xacro:sensor_axis_m5013>
+	<xacro:sensor_antena_combo_5G_teltonika
 		prefix="rbsummit_antenna"
 		parent="rbsummit_base_link"
@@ -123,10 +92,4 @@
 			rpy="0 0 0"
 		/>
-	</xacro:structure_mastil_teltonika>
-	<xacro:if value="$(arg use_gazebo_classic)">
-		<xacro:rbsummit_gz_classic_control namespace="$(arg namespace)"/>
-	</xacro:if>
-	<xacro:if value="$(arg use_gazebo_ignition)">
-		<xacro:rbsummit_gz_ignition_control namespace="$(arg namespace)"/>
-	</xacro:if>
+	</xacro:sensor_antena_combo_5G_teltonika>
 </robot>

File: robots/rbtheron/rbtheron.urdf.xacro (robot description, xacro)
@@ -14,6 +14,4 @@
 	<!-- Import Elevator -->
 	<xacro:include filename="$(find robot_description)/urdf/structures/elevator/rb_theron_elevator.urdf.xacro"/>
-    <xacro:include filename="$(find robot_description)/gazebo/classic/rbtheron_control.urdf.xacro"/>
-    <xacro:include filename="$(find robot_description)/gazebo/ignition/rbtheron_control.urdf.xacro"/>
 	<!-- ***************** -->
 	<!-- Global parameters -->
@@ -27,6 +25,4 @@
 	<xacro:property name="elevator_y" value="0.0" />
 	<xacro:property name="elevator_z" value="0.2238" />
-    <xacro:arg name="use_gazebo_classic" default="false" />
-    <xacro:arg name="use_gazebo_ignition" default="false" />
     <xacro:arg name="gpu" default="true" />
   	<xacro:arg name="namespace" default="robot" />
@@ -44,9 +40,3 @@
 		<origin xyz="-0.1975 0.0 0.1598" rpy="0 0 0"/>
     </xacro:sensor_vectornav>
-    <xacro:if value="$(arg use_gazebo_classic)">
-        <xacro:rbtheron_gz_classic_control namespace="$(arg namespace)"/>
-    </xacro:if>
-    <xacro:if value="$(arg use_gazebo_ignition)">
-        <xacro:rbtheron_gz_ignition_control namespace="$(arg namespace)"/>
-    </xacro:if>
 </robot>

File: robots/rbvogui/rbvogui.urdf.xacro (robot description, xacro)
@@ -8,6 +8,4 @@
     <!-- Import rbvogui base elements-->
     <xacro:include filename="$(find robot_description)/macros/rbvogui_macro.urdf.xacro" />
-    <xacro:include filename="$(find robot_description)/gazebo/classic/rbvogui_control.urdf.xacro"/>
-    <xacro:include filename="$(find robot_description)/gazebo/ignition/rbvogui_control.urdf.xacro"/>
     <!-- Import all available sensors -->
     <xacro:include filename="$(find robotnik_sensors)/urdf/all_sensors.urdf.xacro" />
@@ -16,6 +14,4 @@
     <xacro:property name="hq" value="true" />
     <!-- Launch Arguments -->
-    <xacro:arg name="use_gazebo_classic" default="false" />
-    <xacro:arg name="use_gazebo_ignition" default="false" />
     <xacro:arg name="gpu" default="true" />
     <xacro:arg name="namespace" default="robot" />
@@ -41,9 +37,3 @@
         <origin xyz="-0.53 -0.33 0.1145" rpy="${PI} 0 ${-PI*3/4}"/>
     </xacro:sensor_sick_s300>
-    <xacro:if value="$(arg use_gazebo_classic)">
-        <xacro:rbvogui_gz_classic_control namespace="$(arg namespace)"/>
-    </xacro:if>
-    <xacro:if value="$(arg use_gazebo_ignition)">
-        <xacro:rbvogui_gz_ignition_control namespace="$(arg namespace)"/>
-    </xacro:if>
 </robot>

File: urdf/bases/rbsummit/rbsummit_base.urdf.xacro (robot description, xacro)
@@ -1,5 +1,4 @@
 <?xml version="1.0"?>
 <robot name="summit_xl" xmlns:xacro="http://wiki.ros.org/xacro">
-  <xacro:include filename="$(find robot_description)/urdf/bases/gazebo/rbsummit_xl_base.gazebo.xacro" />
   <xacro:include filename="$(find robot_description)/urdf/structures/inertia.urdf.xacro" />
   <xacro:macro name="rbsummit_base" params="hq">

File: urdf/bases/rbtheron/rbtheron_base.urdf.xacro (robot description, xacro)
@@ -66,5 +66,5 @@
   </link>
   <joint name="rbtheron_base_logo_left_joint" type="fixed">
-    <origin xyz="0.0 0.28931 0.29062" rpy="0 0 0" />
+    <origin xyz="0.0 0.28931 0.19062" rpy="0 0 0" />
     <parent link="rbtheron_base_link"/>
     <child link="rbtheron_base_logo_left" />
@@ -83,5 +83,5 @@
   </link>
   <joint name="rbtheron_base_logo_right_joint" type="fixed">
-    <origin xyz="0.0 -0.28931 0.29062" rpy="0 0 ${PI}" />
+    <origin xyz="0.0 -0.28931 0.19062" rpy="0 0 ${PI}" />
     <parent link="rbtheron_base_link"/>
     <child link="rbtheron_base_logo_right" />

Commit message: refactor ros2_control and urdf

File: robots/rbkairos/rbkairos.urdf.xacro (robot description, xacro)
@@ -5,6 +5,6 @@
   <!-- ***************** -->
   <!-- Import all posible elements defined in the urdf.xacro files. All these elements are defined as macro:xacros -->
-  <xacro:include filename="$(find robot_description)/bases/rbkairos/rbkairos_base.urdf.xacro" />
-  <xacro:include filename="$(find robot_description)/gazebo/classic/rbkairos/rbkairos_control.urdf.xacro" />
+  <xacro:include filename="$(find robot_description)/urdf/bases/rbkairos/rbkairos_base.urdf.xacro" />
+  <xacro:include filename="$(find robot_description)/simulators/gazebo_classic/rbkairos/rbkairos_control.urdf.xacro" />
   <xacro:include filename="$(find robotnik_sensors)/urdf/all_sensors.urdf.xacro" />
   <!-- Properties and Arguments -->

File: robots/rbkairos/rbkairos_ur.urdf.xacro (robot description, xacro)
@@ -5,6 +5,6 @@
   <!-- ***************** -->
   <!-- Import all posible elements defined in the urdf.xacro files. All these elements are defined as macro:xacros -->
-  <xacro:include filename="$(find robot_description)/bases/rbkairos/rbkairos_base.urdf.xacro" />
-  <xacro:include filename="$(find robot_description)/gazebo/classic/rbkairos/rbkairos_control.urdf.xacro" />
+  <xacro:include filename="$(find robot_description)/urdf/bases/rbkairos/rbkairos_base.urdf.xacro" />
+  <xacro:include filename="$(find robot_description)/simulators/gazebo_classic/rbkairos/rbkairos_control.urdf.xacro" />
   <xacro:include filename="$(find robotnik_sensors)/urdf/all_sensors.urdf.xacro" />
   <xacro:include filename="$(find robot_description)/urdf/structures/rbkairos_chassis/structure_hokuyo.urdf.xacro" />

File: robots/rbrobout/rbrobout.urdf.xacro (robot description, xacro)
@@ -5,6 +5,6 @@
   <!-- ***************** -->
   <!-- Import all posible elements defined in the urdf.xacro files. All these elements are defined as macro:xacros -->
-  <xacro:include filename="$(find robot_description)/bases/rbrobout/rbrobout_base.urdf.xacro" />
-  <!-- <xacro:include filename="$(find robot_description)/gazebo/classic/rbkairos/rbkairos_control.urdf.xacro" /> -->
+  <xacro:include filename="$(find robot_description)/urdf/bases/rbrobout/rbrobout_base.urdf.xacro" />
+  <xacro:include filename="$(find robot_description)/simulators/gazebo_classic/rbrobout/rbrobout_control.urdf.xacro" />
   <xacro:include filename="$(find robotnik_sensors)/urdf/all_sensors.urdf.xacro" />
   <!-- Properties and Arguments -->

File: robots/rbrobout/rbrobout_boeing.urdf.xacro (robot description, xacro)
@@ -5,6 +5,6 @@
   <!-- ***************** -->
   <!-- Import all posible elements defined in the urdf.xacro files. All these elements are defined as macro:xacros -->
-  <xacro:include filename="$(find robot_description)/bases/rbrobout/rbrobout_base.urdf.xacro" />
-  <xacro:include filename="$(find robot_description)/gazebo/classic/rbrobout/rbrobout_control.urdf.xacro" />
+  <xacro:include filename="$(find robot_description)/urdf/bases/rbrobout/rbrobout_base.urdf.xacro" />
+  <xacro:include filename="$(find robot_description)/simulators/gazebo_classic/rbrobout/rbrobout_control.urdf.xacro" />
   <xacro:include filename="$(find robotnik_sensors)/urdf/all_sensors.urdf.xacro" />
   <xacro:include filename="$(find robot_description)/urdf/structures/rbrobout/top_cover.urdf.xacro" />

File: robots/rbsteel/rbsteel.urdf.xacro (robot description, xacro)
@@ -5,6 +5,6 @@
   <!-- ***************** -->
   <!-- First we import all posible elements defined in the urdf.xacro files. All these elements are defined as macro:xacros -->
-  <xacro:include filename="$(find robot_description)/bases/rbsteel/rbsteel_base.urdf.xacro" />
-  <xacro:include filename="$(find robot_description)/gazebo/classic/rbkairos/rbkairos_control.urdf.xacro" />
+  <xacro:include filename="$(find robot_description)/urdf/bases/rbsteel/rbsteel_base.urdf.xacro" />
+  <xacro:include filename="$(find robot_description)/simulators/gazebo_classic/rbkairos/rbkairos_control.urdf.xacro" />
   <!-- Import all available sensors -->
   <xacro:include filename="$(find robotnik_sensors)/urdf/all_sensors.urdf.xacro" />

File: robots/rbsummit/rbsummit.urdf.xacro (robot description, xacro)
@@ -6,6 +6,6 @@
 	<!-- First we import the robot and all the sensors. All these elements are defined as macro:xacros -->
 	<!-- Import summit XL macro -->
-	<xacro:include filename="$(find robot_description)/bases/rbsummit/rbsummit_base.xacro"/>
-	<xacro:include filename="$(find robot_description)/gazebo/classic/rbsummit/rbsummit_control.urdf.xacro"/>
+	<xacro:include filename="$(find robot_description)/urdf/bases/rbsummit/rbsummit_base.xacro"/>
+	<xacro:include filename="$(find robot_description)/simulators/gazebo_classic/rbsummit/rbsummit_control.urdf.xacro"/>
 	<!-- Import all available sensors -->
 	<xacro:include filename="$(find robotnik_sensors)/urdf/all_sensors.urdf.xacro" />

File: robots/rbtheron/rbtheron.urdf.xacro (robot description, xacro)
@@ -7,6 +7,6 @@
 	<!-- First we import all posible elements defined in the urdf.xacro files. All these elements are defined as macro:xacros -->
 	<!-- Import rbtheron macro -->
-	<xacro:include filename="$(find robot_description)/bases/rbtheron/rbtheron_base.xacro"/>
-	<xacro:include filename="$(find robot_description)/gazebo/classic/rbtheron/rbtheron_control.urdf.xacro"/>
+	<xacro:include filename="$(find robot_description)/urdf/bases/rbtheron/rbtheron_base.xacro"/>
+	<xacro:include filename="$(find robot_description)/simulators/gazebo_classic/rbtheron/rbtheron_control.urdf.xacro"/>
 	<!-- Import all available sensors -->
 	<xacro:include filename="$(find robotnik_sensors)/urdf/all_sensors.urdf.xacro" />

File: robots/rbvogui/rbvogui.urdf.xacro (robot description, xacro)
@@ -7,6 +7,6 @@
     <!-- First we import all posible elements defined in the urdf.xacro files. All these elements are defined as macro:xacros -->
     <!-- Import rbvogui base elements-->
-    <xacro:include filename="$(find robot_description)/bases/rbvogui/rbvogui_base.urdf.xacro" />
-    <xacro:include filename="$(find robot_description)/gazebo/classic/rbvogui/rbvogui_control.urdf.xacro" />
+    <xacro:include filename="$(find robot_description)/urdf/bases/rbvogui/rbvogui_base.urdf.xacro" />
+    <xacro:include filename="$(find robot_description)/simulators/gazebo_classic/rbvogui/rbvogui_control.urdf.xacro" />
     <!-- Import all available sensors -->
     <xacro:include filename="$(find robotnik_sensors)/urdf/all_sensors.urdf.xacro" />
@@ -19,25 +19,48 @@
 	<xacro:arg name="gazebo_classic" default="false"/>
     <xacro:rbvogui prefix="$(arg prefix)" hq="${hq}"/>
-    <!-- PENDIENTE DE ACTUALIZAR ROBOTNIK_SENSORS -->
     <!-- SENSORS see robotnik_sensors for the specific configuration -->
     <!-- IMU -->
-    <!-- <xacro:sensor_vectornav prefix="rbvogui_" parent="rbvogui_chassis_link" topic="imu/data">
+    <xacro:sensor_vectornav
+        frame_prefix="$(arg prefix)vectornav_"
+        parent="$(arg prefix)chassis_link"
+        node_namespace="$(arg namespace)"
+        simulation="$(arg gazebo_classic)">
         <origin xyz="0.3 -0.3 0.0725" rpy="0 0 0"/>
-    </xacro:sensor_vectornav> -->
+    </xacro:sensor_vectornav>
     <!-- Front Camera -->
-    <!-- <xacro:sensor_intel_d435 prefix="rbvogui_front_rgbd_camera" parent="rbvogui_chassis_link" prefix_topic="front_rgbd_camera" use_nominal_extrinsics="true">
+    <xacro:sensor_intel_realsense_d435
+        frame_prefix="$(arg prefix)front_rgbd_camera_"
+        parent="$(arg prefix)base_link"
+        node_namespace="$(arg namespace)"
+        node_name="front_camera"
+        simulation="$(arg gazebo_classic)">
         <origin xyz="0.46462 0.0 0.18258" rpy="0 0 0"/>
-    </xacro:sensor_intel_d435> -->
+    </xacro:sensor_intel_realsense_d435>
     <!-- Rear Camera -->
-    <!-- <xacro:sensor_intel_d435 prefix="rbvogui_rear_rgbd_camera" parent="rbvogui_base_link" prefix_topic="rear_rgbd_camera" use_nominal_extrinsics="true">
+    <!-- <xacro:sensor_intel_realsense_d435
+        frame_prefix="$(arg prefix)rear_rgbd_camera_"
+        parent="$(arg prefix)chassis_link"
+        node_namespace="$(arg namespace)"
+        node_name="rear_camera"
+        simulation="$(arg gazebo_classic)">
         <origin xyz="-0.503 0.0 0.29" rpy="0 0 -${PI}"/>
-    </xacro:sensor_intel_d435> -->
+    </xacro:sensor_intel_realsense_d435> -->
     <!-- 2d laser -->
-    <!-- <xacro:sensor_sick_s300 prefix="rbvogui_front_laser" parent="rbvogui_chassis_link" gpu="$(arg gpu)" prefix_topic="front_laser">
+    <xacro:sensor_sick_s300
+        frame_prefix="$(arg prefix)front_laser_"
+        parent="$(arg prefix)chassis_link"
+        node_namespace="$(arg namespace)"
+        node_name="front_laser"
+        simulation="$(arg gazebo_classic)">
         <origin xyz="0.53 0.33 0.1145" rpy="${PI} 0 ${PI/4}"/>
     </xacro:sensor_sick_s300>
-    <xacro:sensor_sick_s300 prefix="rbvogui_rear_laser" parent="rbvogui_chassis_link" gpu="$(arg gpu)" prefix_topic="rear_laser">
+    <xacro:sensor_sick_s300
+        frame_prefix="$(arg prefix)rear_laser_"
+        parent="$(arg prefix)chassis_link"
+        node_namespace="$(arg namespace)"
+        node_name="rear_laser"
+        simulation="$(arg gazebo_classic)">
         <origin xyz="-0.53 -0.33 0.1145" rpy="${PI} 0 ${-PI*3/4}"/>
-    </xacro:sensor_sick_s300> -->
+    </xacro:sensor_sick_s300>
 	<!-- Controllers -->
 	<xacro:if value="$(arg gazebo_classic)">

File: robots/rbvogui/rbvogui_cart.urdf.xacro (robot description, xacro)
@@ -7,5 +7,5 @@
     <!-- First we import all posible elements defined in the urdf.xacro files. All these elements are defined as macro:xacros -->
     <!-- Import rbvogui base elements-->
-    <xacro:include filename="$(find robot_description)/robots/bases/rbvogui_base.urdf.xacro" />
+    <xacro:include filename="$(find robot_description)/robots/urdf/bases/rbvogui_base.urdf.xacro" />
     <xacro:include filename="$(find robot_description)/urdf/ros2_control/rbvogui_control.urdf.xacro"/>
     <!-- Import all available sensors -->

File: robots/robot_template.urdf.xacro (robot description, xacro)
@@ -5,5 +5,5 @@
   <!-- ***************** -->
   <!-- Import all posible elements defined in the urdf.xacro files. All these elements are defined as macro:xacros -->
-  <xacro:include filename="$(find robot_description)/bases/rbvogui/rbvogui_base.urdf.xacro" />
+  <xacro:include filename="$(find robot_description)/urdf/bases/rbvogui/rbvogui_base.urdf.xacro" />
   <xacro:include filename="$(find robotnik_sensors)/urdf/all_sensors.urdf.xacro" />
   <!-- Args -->
@@ -21,7 +21,12 @@
   <xacro:rbvogui prefix="$(arg prefix)" hq="${hq}"/>
   <!-- Sensors -->
-  <!-- <xacro:sensor_sick_s300 prefix="rbkairos_front_laser" parent="rbkairos_base_link" prefix_topic="front_laser" gpu="true"> -->
-    <!-- <origin xyz="${front_laser_offset_x} ${front_laser_offset_y} ${front_laser_offset_z}" rpy="0 ${-PI} ${3/4*PI}" /> -->
-  <!-- </xacro:sensor_sick_s300> -->
+  <xacro:sensor_sick_s300
+      frame_prefix="$(arg prefix)front_laser_"
+      parent="$(arg prefix)chassis_link"
+      node_namespace="$(arg namespace)"
+      node_name="front_laser"
+      simulation="$(arg gazebo_classic)">
+      <origin xyz="0.53 0.33 0.1145" rpy="${PI} 0 ${PI/4}"/>
+  </xacro:sensor_sick_s300>
   <!-- Arm -->
   <xacro:if value="$(arg has_arm)">
@@ -39,5 +44,5 @@
   </xacro:if>
   <!-- Control -->
-  <xacro:include filename="$(find robot_description)/gazebo/classic/rbvogui/rbvogui_control.urdf.xacro" />
+  <xacro:include filename="$(find robot_description)/simulators/gazebo_classic/rbvogui/rbvogui_control.urdf.xacro" />
   <!-- <xacro:if value="$(arg gazebo_classic)">
     <xacro:rbvogui_gz_classic_control namespace="$(arg namespace)" prefix="$(arg prefix)"/>
