Commit message: update files for ros2_control

File: robots/rbkairos/rbkairos.urdf.xacro (robot description, xacro)
@@ -25,14 +25,28 @@
   <!-- PENDIENTE DE ACTUALIZAR ROBOTNIK_SENSORS -->
   <!-- IMU -->
-	<!-- <xacro:sensor_vectornav prefix="rbkairos_" parent="rbkairos_base_link" topic="imu/data">
-    <origin xyz="${imu_offset_x} ${imu_offset_y} ${imu_offset_z}" rpy="0 0 0"/>
-  </xacro:sensor_vectornav> -->
+    <xacro:sensor_vectornav
+        frame_prefix="$(arg prefix)vectornav_"
+        parent="$(arg prefix)base_link"
+        node_namespace="$(arg namespace)"
+        simulation="$(arg gazebo_classic)">
+        <origin xyz="${imu_offset_x} ${imu_offset_y} ${imu_offset_z}" rpy="0 0 0"/>
+    </xacro:sensor_vectornav>
   <!-- SENSORS -->
-  <!-- <xacro:sensor_sick_s300 prefix="rbkairos_front_laser" parent="rbkairos_base_link" prefix_topic="front_laser" gpu="true">
-    <origin xyz="${front_laser_offset_x} ${front_laser_offset_y} ${front_laser_offset_z}" rpy="0 ${-PI} ${3/4*PI}" />
-  </xacro:sensor_sick_s300>
-  <xacro:sensor_sick_s300 prefix="rbkairos_rear_laser" parent="rbkairos_base_link" prefix_topic="rear_laser" gpu="true">
-    <origin xyz="${rear_laser_offset_x} ${rear_laser_offset_y} ${rear_laser_offset_z}" rpy="0 ${-PI} ${-1/4*PI}" />
-  </xacro:sensor_sick_s300> -->
+    <xacro:sensor_sick_s300
+        frame_prefix="$(arg prefix)front_laser_"
+        parent="$(arg prefix)base_link"
+        node_namespace="$(arg namespace)"
+        node_name="front_laser"
+        simulation="$(arg gazebo_classic)">
+        <origin xyz="${front_laser_offset_x} ${front_laser_offset_y} ${front_laser_offset_z}" rpy="0 ${-PI} ${3/4*PI}"/>
+    </xacro:sensor_sick_s300>
+    <xacro:sensor_sick_s300
+        frame_prefix="$(arg prefix)rear_laser_"
+        parent="$(arg prefix)base_link"
+        node_namespace="$(arg namespace)"
+        node_name="rear_laser"
+        simulation="$(arg gazebo_classic)">
+        <origin xyz="${rear_laser_offset_x} ${rear_laser_offset_y} ${rear_laser_offset_z}" rpy="0 ${-PI} ${-1/4*PI}"/>
+    </xacro:sensor_sick_s300>
   <!-- Controllers -->
   <xacro:if value="$(arg gazebo_classic)">
@@ -41,5 +55,5 @@
   </xacro:if>
   <xacro:unless value="$(arg gazebo_classic)">
-    <xacro:base_hw_controller/>
+    <xacro:rbkairos_base_hw_controller/>
   </xacro:unless>
 </robot>

File: robots/rbkairos/rbkairos_ur.urdf.xacro (robot description, xacro)
@@ -10,8 +10,14 @@
   <xacro:include filename="$(find robotnik_sensors)/urdf/all_sensors.urdf.xacro" />
   <xacro:include filename="$(find robot_description)/urdf/structures/rbkairos_chassis/structure_hokuyo.urdf.xacro" />
+  <xacro:include filename="$(find ur_description)/urdf/ur_macro.xacro" />
   <!-- Properties and Arguments -->
   <xacro:arg name="namespace" default="robot"/>
   <xacro:arg name="prefix" default="robot_"/>
   <xacro:arg name="gazebo_classic" default="false"/>
+  <xacro:arg name="ur_type" default="ur5e"/>
+  <xacro:arg name="joint_limit_params" default="$(find ur_description)/config/$(arg ur_type)/joint_limits.yaml"/>
+  <xacro:arg name="kinematics_params" default="$(find ur_description)/config/$(arg ur_type)/default_kinematics.yaml"/>
+  <xacro:arg name="physical_params" default="$(find ur_description)/config/$(arg ur_type)/physical_parameters.yaml"/>
+  <xacro:arg name="visual_params" default="$(find ur_description)/config/$(arg ur_type)/visual_parameters.yaml"/>
   <xacro:property name="front_laser_offset_x" value="0.2865"/>
   <xacro:property name="front_laser_offset_y" value="-0.20894"/>
@@ -38,28 +44,41 @@
   <xacro:rbkairos prefix="$(arg prefix)"/>
   <!-- Import UR arm -->
-  <!-- <xacro:include filename="$(find ur_description)/urdf/ur.urdf.xacro" /> -->
-  <xacro:arg name="ur_type" default="ur5e"/>
-  <xacro:arg name="name" default="$(arg ur_type)"/>
-  <xacro:arg name="joint_limit_params" default="$(find ur_description)/config/$(arg ur_type)/joint_limits.yaml"/>
-  <xacro:arg name="kinematics_params" default="$(find ur_description)/config/$(arg ur_type)/default_kinematics.yaml"/>
-  <xacro:arg name="physical_params" default="$(find ur_description)/config/$(arg ur_type)/physical_parameters.yaml"/>
-  <xacro:arg name="visual_params" default="$(find ur_description)/config/$(arg ur_type)/visual_parameters.yaml"/>
-  <xacro:arg name="use_fake_hardware" default="false" />
-  <xacro:arg name="fake_sensor_commands" default="false" />
-  <xacro:arg name="sim_gazebo" default="true" />
-  <xacro:arg name="sim_ignition" default="false" />
-  <xacro:include filename="$(find robot_description)/urdf/arms/ur/ur.urdf.xacro"/>
+  <xacro:ur_robot
+      tf_prefix="$(arg prefix)arm_"
+      name="$(arg ur_type)"
+      parent="$(arg prefix)base_link"
+      joint_limits_parameters_file="$(arg joint_limit_params)"
+      kinematics_parameters_file="$(arg kinematics_params)"
+      physical_parameters_file="$(arg physical_params)"
+      visual_parameters_file="$(arg visual_params)"
+      sim_gazebo="$(arg gazebo_classic)">
+      <origin xyz="0 0 0" rpy="0 0 0"/>
+  </xacro:ur_robot>
   <!-- PENDIENTE DE ACTUALIZAR ROBOTNIK_SENSORS -->
   <!-- IMU -->
-	<!-- <xacro:sensor_vectornav prefix="rbkairos_" parent="rbkairos_base_link" topic="imu/data">
-    <origin xyz="${imu_offset_x} ${imu_offset_y} ${imu_offset_z}" rpy="0 0 0"/>
-  </xacro:sensor_vectornav> -->
+    <xacro:sensor_vectornav
+        frame_prefix="$(arg prefix)vectornav_"
+        parent="$(arg prefix)base_link"
+        node_namespace="$(arg namespace)"
+        simulation="$(arg gazebo_classic)">
+        <origin xyz="${imu_offset_x} ${imu_offset_y} ${imu_offset_z}" rpy="0 0 0"/>
+    </xacro:sensor_vectornav>
   <!-- SENSORS -->
-  <!-- <xacro:sensor_sick_s300 prefix="rbkairos_front_laser" parent="rbkairos_base_link" prefix_topic="front_laser" gpu="true">
-    <origin xyz="${front_laser_offset_x} ${front_laser_offset_y} ${front_laser_offset_z}" rpy="0 ${-PI} ${3/4*PI}" />
-  </xacro:sensor_sick_s300>
-  <xacro:sensor_sick_s300 prefix="rbkairos_rear_laser" parent="rbkairos_base_link" prefix_topic="rear_laser" gpu="true">
-    <origin xyz="${rear_laser_offset_x} ${rear_laser_offset_y} ${rear_laser_offset_z}" rpy="0 ${-PI} ${-1/4*PI}" />
-  </xacro:sensor_sick_s300> -->
+    <xacro:sensor_sick_s300
+        frame_prefix="$(arg prefix)front_laser_"
+        parent="$(arg prefix)base_link"
+        node_namespace="$(arg namespace)"
+        node_name="front_laser"
+        simulation="$(arg gazebo_classic)">
+        <origin xyz="${front_laser_offset_x} ${front_laser_offset_y} ${front_laser_offset_z}" rpy="0 ${-PI} ${3/4*PI}"/>
+    </xacro:sensor_sick_s300>
+    <xacro:sensor_sick_s300
+        frame_prefix="$(arg prefix)rear_laser_"
+        parent="$(arg prefix)base_link"
+        node_namespace="$(arg namespace)"
+        node_name="rear_laser"
+        simulation="$(arg gazebo_classic)">
+        <origin xyz="${rear_laser_offset_x} ${rear_laser_offset_y} ${rear_laser_offset_z}" rpy="0 ${-PI} ${-1/4*PI}"/>
+    </xacro:sensor_sick_s300>
   <!-- Controllers -->
   <xacro:if value="$(arg gazebo_classic)">
@@ -68,5 +87,5 @@
   </xacro:if>
   <xacro:unless value="$(arg gazebo_classic)">
-    <xacro:base_hw_controller/>
+    <xacro:rbkairos_base_hw_controller/>
   </xacro:unless>
 </robot>

File: robots/rbrobout/rbrobout.urdf.xacro (robot description, xacro)
@@ -22,6 +22,37 @@
   <xacro:property name="imu_offset_z" value="0.212"/>
   <xacro:rbrobout prefix="$(arg prefix)"/>
-  <xacro:unless value="$(arg gazebo_classic)">
-    <xacro:base_hw_controller/>
-  </xacro:unless>
+  <!-- IMU -->
+    <xacro:sensor_vectornav
+        frame_prefix="$(arg prefix)vectornav_"
+        parent="$(arg prefix)base_link"
+        node_namespace="$(arg namespace)"
+        simulation="$(arg gazebo_classic)">
+        <origin xyz="${imu_offset_x} ${imu_offset_y} ${imu_offset_z}" rpy="0 0 0"/>
+    </xacro:sensor_vectornav>
+  <!-- 2d laser -->
+    <xacro:sensor_sick_microscan3
+        frame_prefix="$(arg prefix)front_laser_"
+        parent="$(arg prefix)base_link"
+        node_namespace="$(arg namespace)"
+        node_name="front_laser"
+        simulation="$(arg gazebo_classic)">
+        <origin xyz="${front_laser_offset_x} ${front_laser_offset_y} ${front_laser_offset_z}" rpy="0 0 ${1/4*PI}"/>
+    </xacro:sensor_sick_microscan3>
+    <!-- 2d laser -->
+    <xacro:sensor_sick_microscan3
+        frame_prefix="$(arg prefix)rear_laser_"
+        parent="$(arg prefix)base_link"
+        node_namespace="$(arg namespace)"
+        node_name="rear_laser"
+        simulation="$(arg gazebo_classic)">
+        <origin xyz="${rear_laser_offset_x} ${rear_laser_offset_y} ${rear_laser_offset_z}" rpy="0 0 ${-3/4*PI}"/>
+    </xacro:sensor_sick_microscan3>
+    <!-- Controllers -->
+    <xacro:if value="$(arg gazebo_classic)">
+        <xacro:rbrobout_gz_classic_control namespace="$(arg namespace)" prefix="$(arg prefix)"/>
+        <xacro:ros_planar_move_gazebo_classic/>
+    </xacro:if>
+    <xacro:unless value="$(arg gazebo_classic)">
+        <xacro:rbrobout_base_hw_controller/>
+    </xacro:unless>
 </robot>

File: robots/rbrobout/rbrobout_boeing.urdf.xacro (robot description, xacro)
@@ -13,10 +13,4 @@
   <xacro:include filename="$(find ur_description)/urdf/ur_macro.xacro" />
   <xacro:include filename="$(find ewellix_description)/urdf/ewellix_lift_900mm.urdf.xacro" />
-  <xacro:property name="lift_position_x" value="0.72328"/>
-  <xacro:property name="lift_position_y" value="0"/>
-  <xacro:property name="lift_position_z" value="0.38"/>
-  <xacro:property name="lift_orientation_r" value="0"/>
-  <xacro:property name="lift_orientation_p" value="0"/>
-  <xacro:property name="lift_orientation_y" value="0"/>
   <!-- Properties and Arguments -->
   <xacro:arg name="namespace" default="robot"/>
@@ -34,7 +28,7 @@
   <xacro:property name="rear_laser_offset_y" value="-0.366"/>
   <xacro:property name="rear_laser_offset_z" value="-0.06"/>
-  <xacro:property name="imu_offset_x" value="0.242"/>
-  <xacro:property name="imu_offset_y" value="-0.053"/>
-  <xacro:property name="imu_offset_z" value="0.028"/>
+  <xacro:property name="imu_offset_x" value="0.3"/>
+  <xacro:property name="imu_offset_y" value="-0.3"/>
+  <xacro:property name="imu_offset_z" value="0.0725"/>
   <xacro:property name="front_rgbd_camera_offset_x" value="0.883"/>
   <xacro:property name="front_rgbd_camera_offset_y" value="0.0"/>
@@ -55,4 +49,10 @@
   <xacro:property name="rear_left_rgbd_camera_offset_y" value="0.399"/>
   <xacro:property name="rear_left_rgbd_camera_offset_z" value="0.994"/>
+  <xacro:property name="lift_position_x" value="0.72328"/>
+  <xacro:property name="lift_position_y" value="0"/>
+  <xacro:property name="lift_position_z" value="0.38"/>
+  <xacro:property name="lift_orientation_r" value="0"/>
+  <xacro:property name="lift_orientation_p" value="0"/>
+  <xacro:property name="lift_orientation_y" value="0"/>
   <xacro:rbrobout prefix="$(arg prefix)"/>
   <xacro:top_cover prefix="$(arg prefix)" parent="$(arg prefix)base_link">
@@ -64,5 +64,5 @@
   <xacro:ur_robot
       tf_prefix="$(arg prefix)arm_"
-      name="ur10"
+      name="$(arg ur_type)"
       parent="$(arg prefix)lift_ewellix_lift_top_link"
       joint_limits_parameters_file="$(arg joint_limit_params)"
@@ -79,5 +79,5 @@
         node_namespace="$(arg namespace)"
         simulation="$(arg gazebo_classic)">
-        <origin xyz="0.3 -0.3 0.0725" rpy="0 0 0"/>
+        <origin xyz="${imu_offset_x} ${imu_offset_y} ${imu_offset_z}" rpy="0 0 0"/>
     </xacro:sensor_vectornav>
     <!-- Front Camera -->
@@ -153,11 +153,11 @@
         <origin xyz="${rear_laser_offset_x} ${rear_laser_offset_y} ${rear_laser_offset_z}" rpy="0 0 ${-3/4*PI}"/>
     </xacro:sensor_sick_microscan3>
-  <!-- Controllers -->
-  <xacro:if value="$(arg gazebo_classic)">
-    <xacro:rbrobout_gz_classic_control namespace="$(arg namespace)" prefix="$(arg prefix)"/>
-    <xacro:ros_planar_move_gazebo_classic/>
-  </xacro:if>
-  <xacro:unless value="$(arg gazebo_classic)">
-    <xacro:base_hw_controller/>
-  </xacro:unless>
+    <!-- Controllers -->
+    <xacro:if value="$(arg gazebo_classic)">
+        <xacro:rbrobout_gz_classic_control namespace="$(arg namespace)" prefix="$(arg prefix)"/>
+        <xacro:ros_planar_move_gazebo_classic/>
+    </xacro:if>
+    <xacro:unless value="$(arg gazebo_classic)">
+        <xacro:rbrobout_base_hw_controller/>
+    </xacro:unless>
 </robot>

File: robots/rbsummit/rbsummit.urdf.xacro (robot description, xacro)
@@ -7,4 +7,5 @@
 	<!-- Import summit XL macro -->
 	<xacro:include filename="$(find robot_description)/urdf/bases/rbsummit/rbsummit_base.xacro"/>
+    <xacro:include filename="$(find robot_description)/urdf/base_hw/rbsummit.ros2_control.urdf" />
 	<xacro:include filename="$(find robot_description)/simulators/gazebo_classic/rbsummit/rbsummit_control.urdf.xacro"/>
 	<!-- Import all available sensors -->
@@ -99,5 +100,5 @@
   </xacro:if>
   <xacro:unless value="$(arg gazebo_classic)">
-    <xacro:base_hw_controller/>
+    <xacro:rbsummit_base_hw_controller/>
   </xacro:unless>
 </robot>

File: robots/rbtheron/rbtheron.urdf.xacro (robot description, xacro)
@@ -8,4 +8,5 @@
 	<!-- Import rbtheron macro -->
 	<xacro:include filename="$(find robot_description)/urdf/bases/rbtheron/rbtheron_base.xacro"/>
+    <xacro:include filename="$(find robot_description)/urdf/base_hw/rbtheron.ros2_control.urdf" />
 	<xacro:include filename="$(find robot_description)/simulators/gazebo_classic/rbtheron/rbtheron_control.urdf.xacro"/>
 	<!-- Import all available sensors -->
@@ -46,5 +47,5 @@
 	</xacro:if>
   <xacro:unless value="$(arg gazebo_classic)">
-    <xacro:base_hw_controller/>
+    <xacro:rbtheron_base_hw_controller/>
   </xacro:unless>
 </robot>

File: robots/rbvogui/rbvogui.urdf.xacro (robot description, xacro)
@@ -8,4 +8,5 @@
     <!-- Import rbvogui base elements-->
     <xacro:include filename="$(find robot_description)/urdf/bases/rbvogui/rbvogui_base.urdf.xacro" />
+    <xacro:include filename="$(find robot_description)/urdf/base_hw/rbvogui.ros2_control.urdf" />
     <xacro:include filename="$(find robot_description)/simulators/gazebo_classic/rbvogui/rbvogui_control.urdf.xacro" />
     <!-- Import all available sensors -->
@@ -68,5 +69,5 @@
 	</xacro:if>
     <xacro:unless value="$(arg gazebo_classic)">
-        <xacro:base_hw_controller/>
+        <xacro:rbvogui_base_hw_controller/>
     </xacro:unless>
 </robot>

File: simulators/gazebo_classic/rbrobout/rbrobout_control.urdf.xacro (robot description, xacro)
@@ -3,5 +3,5 @@
     <xacro:macro name="rbrobout_gz_classic_control"  params="namespace prefix">
         <gazebo>
-          <plugin name="ros_control" filename="libgazebo_ros2_control.so">
+          <plugin name="ros2_control" filename="libgazebo_ros2_control.so">
             <robot_param>robot_description</robot_param>
             <robot_param_node>robot_state_publisher</robot_param_node>
