Commit message: Add gazebo ignition control files and arguments, update sensors, fix mecanum wheels physics

File: robots/rbkairos/rbkairos.urdf.xacro (robot description, xacro)
@@ -8,4 +8,5 @@
   <xacro:include filename="$(find robot_description)/urdf/base_hw/rbkairos.ros2_control.urdf" />
   <xacro:include filename="$(find robot_description)/simulators/gazebo_classic/rbkairos/rbkairos_control.urdf.xacro" />
+  <xacro:include filename="$(find robot_description)/simulators/gazebo_ignition/rbkairos/rbkairos_control.urdf.xacro" />
   <xacro:include filename="$(find robotnik_sensors)/urdf/all_sensors.urdf.xacro" />
   <!-- Properties and Arguments -->
@@ -13,4 +14,5 @@
   <xacro:arg name="prefix" default="robot_"/>
   <xacro:arg name="gazebo_classic" default="false"/>
+  <xacro:arg name="gazebo_ignition" default="false"/>
   <xacro:property name="front_laser_offset_x" value="0.2865"/>
   <xacro:property name="front_laser_offset_y" value="-0.20894"/>
@@ -29,5 +31,6 @@
         parent="$(arg prefix)base_link"
         node_namespace="$(arg namespace)"
-        simulation="$(arg gazebo_classic)">
+        gazebo_classic="$(arg gazebo_classic)"
+        gazebo_ignition="$(arg gazebo_ignition)">
         <origin xyz="${imu_offset_x} ${imu_offset_y} ${imu_offset_z}" rpy="0 0 0"/>
     </xacro:sensor_vectornav>
@@ -38,5 +41,6 @@
         node_namespace="$(arg namespace)"
         node_name="front_laser"
-        simulation="$(arg gazebo_classic)">
+        gazebo_classic="$(arg gazebo_classic)"
+        gazebo_ignition="$(arg gazebo_ignition)">
         <origin xyz="${front_laser_offset_x} ${front_laser_offset_y} ${front_laser_offset_z}" rpy="0 ${-PI} ${3/4*PI}"/>
     </xacro:sensor_sick_s300>
@@ -46,5 +50,6 @@
         node_namespace="$(arg namespace)"
         node_name="rear_laser"
-        simulation="$(arg gazebo_classic)">
+        gazebo_classic="$(arg gazebo_classic)"
+        gazebo_ignition="$(arg gazebo_ignition)">
         <origin xyz="${rear_laser_offset_x} ${rear_laser_offset_y} ${rear_laser_offset_z}" rpy="0 ${-PI} ${-1/4*PI}"/>
     </xacro:sensor_sick_s300>
@@ -54,6 +59,11 @@
     <xacro:ros_planar_move_gazebo_classic/>
   </xacro:if>
+  <xacro:if value="$(arg gazebo_ignition)">
+    <xacro:rbkairos_gz_ignition_control namespace="$(arg namespace)" prefix="$(arg prefix)"/>
+  </xacro:if>
   <xacro:unless value="$(arg gazebo_classic)">
-    <xacro:rbkairos_base_hw_controller/>
+    <xacro:unless value="$(arg gazebo_ignition)">
+      <xacro:rbkairos_base_hw_controller/>
+    </xacro:unless>
   </xacro:unless>
 </robot>

File: robots/rbkairos/rbkairos_plus.urdf.xacro (robot description, xacro)
@@ -8,4 +8,5 @@
   <xacro:include filename="$(find robot_description)/urdf/base_hw/rbkairos.ros2_control.urdf" />
   <xacro:include filename="$(find robot_description)/simulators/gazebo_classic/rbkairos/rbkairos_control.urdf.xacro" />
+  <xacro:include filename="$(find robot_description)/simulators/gazebo_ignition/rbkairos/rbkairos_control.urdf.xacro" />
   <xacro:include filename="$(find robotnik_sensors)/urdf/all_sensors.urdf.xacro" />
   <xacro:include filename="$(find robot_description)/urdf/structures/rbkairos_chassis/structure_hokuyo.urdf.xacro" />
@@ -15,4 +16,5 @@
   <xacro:arg name="prefix" default="robot_"/>
   <xacro:arg name="gazebo_classic" default="false"/>
+  <xacro:arg name="gazebo_ignition" default="false"/>
   <xacro:arg name="ur_type" default="ur5e"/>
   <xacro:arg name="joint_limit_params" default="$(find ur_description)/config/$(arg ur_type)/joint_limits.yaml"/>
@@ -61,5 +63,6 @@
         parent="$(arg prefix)base_link"
         node_namespace="$(arg namespace)"
-        simulation="$(arg gazebo_classic)">
+        gazebo_classic="$(arg gazebo_classic)"
+        gazebo_ignition="$(arg gazebo_ignition)">
         <origin xyz="${imu_offset_x} ${imu_offset_y} ${imu_offset_z}" rpy="0 0 0"/>
     </xacro:sensor_vectornav>
@@ -70,5 +73,6 @@
         node_namespace="$(arg namespace)"
         node_name="front_laser"
-        simulation="$(arg gazebo_classic)">
+        gazebo_classic="$(arg gazebo_classic)"
+        gazebo_ignition="$(arg gazebo_ignition)">
         <origin xyz="${front_laser_offset_x} ${front_laser_offset_y} ${front_laser_offset_z}" rpy="0 ${-PI} ${3/4*PI}"/>
     </xacro:sensor_sick_s300>
@@ -78,5 +82,6 @@
         node_namespace="$(arg namespace)"
         node_name="rear_laser"
-        simulation="$(arg gazebo_classic)">
+        gazebo_classic="$(arg gazebo_classic)"
+        gazebo_ignition="$(arg gazebo_ignition)">
         <origin xyz="${rear_laser_offset_x} ${rear_laser_offset_y} ${rear_laser_offset_z}" rpy="0 ${-PI} ${-1/4*PI}"/>
     </xacro:sensor_sick_s300>
@@ -86,6 +91,11 @@
     <xacro:ros_planar_move_gazebo_classic/>
   </xacro:if>
+  <xacro:if value="$(arg gazebo_ignition)">
+    <xacro:rbkairos_gz_ignition_control namespace="$(arg namespace)" prefix="$(arg prefix)"/>
+  </xacro:if>
   <xacro:unless value="$(arg gazebo_classic)">
-    <xacro:rbkairos_base_hw_controller/>
+    <xacro:unless value="$(arg gazebo_ignition)">
+      <xacro:rbkairos_base_hw_controller/>
+    </xacro:unless>
   </xacro:unless>
 </robot>

File: robots/rbrobout/rbrobout.urdf.xacro (robot description, xacro)
@@ -7,4 +7,5 @@
   <xacro:include filename="$(find robot_description)/urdf/bases/rbrobout/rbrobout_base.urdf.xacro" />
   <xacro:include filename="$(find robot_description)/simulators/gazebo_classic/rbrobout/rbrobout_control.urdf.xacro" />
+  <xacro:include filename="$(find robot_description)/simulators/gazebo_ignition/rbrobout/rbrobout_control.urdf.xacro" />
   <xacro:include filename="$(find robotnik_sensors)/urdf/all_sensors.urdf.xacro" />
   <!-- Properties and Arguments -->
@@ -12,4 +13,5 @@
   <xacro:arg name="prefix" default="robot_"/>
   <xacro:arg name="gazebo_classic" default="false"/>
+  <xacro:arg name="gazebo_ignition" default="false"/>
   <xacro:property name="front_laser_offset_x" value="0.8"/>
   <xacro:property name="front_laser_offset_y" value="0.366"/>
@@ -27,5 +29,6 @@
         parent="$(arg prefix)base_link"
         node_namespace="$(arg namespace)"
-        simulation="$(arg gazebo_classic)">
+        gazebo_classic="$(arg gazebo_classic)"
+        gazebo_ignition="$(arg gazebo_ignition)">
         <origin xyz="${imu_offset_x} ${imu_offset_y} ${imu_offset_z}" rpy="0 0 0"/>
     </xacro:sensor_vectornav>
@@ -36,5 +39,6 @@
         node_namespace="$(arg namespace)"
         node_name="front_laser"
-        simulation="$(arg gazebo_classic)">
+        gazebo_classic="$(arg gazebo_classic)"
+        gazebo_ignition="$(arg gazebo_ignition)">
         <origin xyz="${front_laser_offset_x} ${front_laser_offset_y} ${front_laser_offset_z}" rpy="0 0 ${1/4*PI}"/>
     </xacro:sensor_sick_microscan3>
@@ -45,5 +49,6 @@
         node_namespace="$(arg namespace)"
         node_name="rear_laser"
-        simulation="$(arg gazebo_classic)">
+        gazebo_classic="$(arg gazebo_classic)"
+        gazebo_ignition="$(arg gazebo_ignition)">
         <origin xyz="${rear_laser_offset_x} ${rear_laser_offset_y} ${rear_laser_offset_z}" rpy="0 0 ${-3/4*PI}"/>
     </xacro:sensor_sick_microscan3>
@@ -53,6 +58,11 @@
         <xacro:ros_planar_move_gazebo_classic/>
     </xacro:if>
+    <xacro:if value="$(arg gazebo_ignition)">
+        <xacro:rbrobout_gz_ignition_control namespace="$(arg namespace)" prefix="$(arg prefix)"/>
+    </xacro:if>
     <xacro:unless value="$(arg gazebo_classic)">
-        <xacro:rbrobout_base_hw_controller/>
+        <xacro:unless value="$(arg gazebo_ignition)">
+            <xacro:rbrobout_base_hw_controller/>
+        </xacro:unless>
     </xacro:unless>
 </robot>

File: robots/rbrobout/rbrobout_plus.urdf.xacro (robot description, xacro)
@@ -78,5 +78,6 @@
         parent="$(arg prefix)base_link"
         node_namespace="$(arg namespace)"
-        simulation="$(arg gazebo_classic)">
+        gazebo_classic="$(arg gazebo_classic)"
+        gazebo_ignition="$(arg gazebo_ignition)">
         <origin xyz="${imu_offset_x} ${imu_offset_y} ${imu_offset_z}" rpy="0 0 0"/>
     </xacro:sensor_vectornav>
@@ -87,5 +88,6 @@
         node_namespace="$(arg namespace)"
         node_name="front_camera"
-        simulation="$(arg gazebo_classic)">
+        gazebo_classic="$(arg gazebo_classic)"
+        gazebo_ignition="$(arg gazebo_ignition)">
         <origin xyz="${front_rgbd_camera_offset_x} ${front_rgbd_camera_offset_y} ${front_rgbd_camera_offset_z}" rpy="0 1.0472 0"/>
     </xacro:sensor_intel_realsense_d435>
@@ -96,5 +98,6 @@
         node_namespace="$(arg namespace)"
         node_name="front_right_camera"
-        simulation="$(arg gazebo_classic)">
+        gazebo_classic="$(arg gazebo_classic)"
+        gazebo_ignition="$(arg gazebo_ignition)">
         <origin xyz="${front_right_rgbd_camera_offset_x} ${front_right_rgbd_camera_offset_y} ${front_right_rgbd_camera_offset_z}" rpy="0 1.0472 -${PI/2}"/>
     </xacro:sensor_intel_realsense_d435>
@@ -105,5 +108,6 @@
         node_namespace="$(arg namespace)"
         node_name="front_left_camera"
-        simulation="$(arg gazebo_classic)">
+        gazebo_classic="$(arg gazebo_classic)"
+        gazebo_ignition="$(arg gazebo_ignition)">
         <origin xyz="${front_left_rgbd_camera_offset_x} ${front_left_rgbd_camera_offset_y} ${front_left_rgbd_camera_offset_z}" rpy="0 1.0472 ${PI/2}"/>
     </xacro:sensor_intel_realsense_d435>
@@ -114,5 +118,6 @@
         node_namespace="$(arg namespace)"
         node_name="rear_camera"
-        simulation="$(arg gazebo_classic)">
+        gazebo_classic="$(arg gazebo_classic)"
+        gazebo_ignition="$(arg gazebo_ignition)">
         <origin xyz="${rear_rgbd_camera_offset_x} ${rear_rgbd_camera_offset_y} ${rear_rgbd_camera_offset_z}" rpy="0 1.0472 ${PI}"/>
     </xacro:sensor_intel_realsense_d435>
@@ -123,5 +128,6 @@
         node_namespace="$(arg namespace)"
         node_name="rear_right_camera"
-        simulation="$(arg gazebo_classic)">
+        gazebo_classic="$(arg gazebo_classic)"
+        gazebo_ignition="$(arg gazebo_ignition)">
         <origin xyz="${rear_right_rgbd_camera_offset_x} ${rear_right_rgbd_camera_offset_y} ${rear_right_rgbd_camera_offset_z}" rpy="0 1.0472 -${PI/2}"/>
     </xacro:sensor_intel_realsense_d435>
@@ -132,5 +138,6 @@
         node_namespace="$(arg namespace)"
         node_name="rear_left_camera"
-        simulation="$(arg gazebo_classic)">
+        gazebo_classic="$(arg gazebo_classic)"
+        gazebo_ignition="$(arg gazebo_ignition)">
         <origin xyz="${rear_left_rgbd_camera_offset_x} ${rear_left_rgbd_camera_offset_y} ${rear_left_rgbd_camera_offset_z}" rpy="0 1.0472 ${PI/2}"/>
     </xacro:sensor_intel_realsense_d435>
@@ -141,5 +148,6 @@
         node_namespace="$(arg namespace)"
         node_name="front_laser"
-        simulation="$(arg gazebo_classic)">
+        gazebo_classic="$(arg gazebo_classic)"
+        gazebo_ignition="$(arg gazebo_ignition)">
         <origin xyz="${front_laser_offset_x} ${front_laser_offset_y} ${front_laser_offset_z}" rpy="0 0 ${1/4*PI}"/>
     </xacro:sensor_sick_microscan3>
@@ -150,5 +158,6 @@
         node_namespace="$(arg namespace)"
         node_name="rear_laser"
-        simulation="$(arg gazebo_classic)">
+        gazebo_classic="$(arg gazebo_classic)"
+        gazebo_ignition="$(arg gazebo_ignition)">
         <origin xyz="${rear_laser_offset_x} ${rear_laser_offset_y} ${rear_laser_offset_z}" rpy="0 0 ${-3/4*PI}"/>
     </xacro:sensor_sick_microscan3>
@@ -158,6 +167,11 @@
         <xacro:ros_planar_move_gazebo_classic/>
     </xacro:if>
+    <xacro:if value="$(arg gazebo_ignition)">
+        <xacro:rbrobout_gz_ignition_control namespace="$(arg namespace)" prefix="$(arg prefix)"/>
+    </xacro:if>
     <xacro:unless value="$(arg gazebo_classic)">
-        <xacro:rbrobout_base_hw_controller/>
+        <xacro:unless value="$(arg gazebo_ignition)">
+            <xacro:rbrobout_base_hw_controller/>
+        </xacro:unless>
     </xacro:unless>
 </robot>

File: robots/rbsummit/rbsummit.urdf.xacro (robot description, xacro)
@@ -9,4 +9,5 @@
     <xacro:include filename="$(find robot_description)/urdf/base_hw/rbsummit.ros2_control.urdf" />
 	<xacro:include filename="$(find robot_description)/simulators/gazebo_classic/rbsummit/rbsummit_control.urdf.xacro"/>
+	<xacro:include filename="$(find robot_description)/simulators/gazebo_ignition/rbsummit/rbsummit_control.urdf.xacro"/>
 	<!-- Import all available sensors -->
 	<xacro:include filename="$(find robotnik_sensors)/urdf/all_sensors.urdf.xacro" />
@@ -21,4 +22,5 @@
 	<xacro:arg name="prefix" default="robot_"/>
 	<xacro:arg name="gazebo_classic" default="false"/>
+	<xacro:arg name="gazebo_ignition" default="false"/>
 	<xacro:property name="imu_offset_x" value="0.0385"/>
 	<xacro:property name="imu_offset_y" value="0.132"/>
@@ -66,8 +68,10 @@
 	</xacro:sensor_vectornav>
 	<!-- 3d laser -->
-	<!-- <xacro:sensor_robosense_rslidar_16
+	<xacro:sensor_robosense_rslidar_16
 		frame_prefix="rbsummit_top_3d_laser_"
 		parent="rbsummit_base_link"
 		gpu="$(arg gpu)"
+        gazebo_classic="$(arg gazebo_classic)"
+        gazebo_ignition="$(arg gazebo_ignition)"
 	>
 		<origin
@@ -75,5 +79,5 @@
 			rpy="0 0 0"
 		/>
-	</xacro:sensor_robosense_rslidar_16> -->
+	</xacro:sensor_robosense_rslidar_16>
 	<!-- ptz camera -->
 	<!-- <xacro:sensor_axis_m5013
@@ -100,6 +104,11 @@
         <xacro:ros_planar_move_gazebo_classic/>
   </xacro:if>
-  <xacro:unless value="$(arg gazebo_classic)">
-    <xacro:rbsummit_base_hw_controller/>
-  </xacro:unless>
+  <xacro:if value="$(arg gazebo_ignition)">
+    <xacro:rbsummit_gz_ignition_control namespace="$(arg namespace)" prefix="$(arg prefix)"/>
+  </xacro:if>
+    <xacro:unless value="$(arg gazebo_classic)">
+        <xacro:unless value="$(arg gazebo_ignition)">
+            <xacro:rbsummit_base_hw_controller/>
+        </xacro:unless>
+    </xacro:unless>
 </robot>

File: robots/rbtheron/rbtheron.urdf.xacro (robot description, xacro)
@@ -10,4 +10,5 @@
     <xacro:include filename="$(find robot_description)/urdf/base_hw/rbtheron.ros2_control.urdf" />
 	<xacro:include filename="$(find robot_description)/simulators/gazebo_classic/rbtheron/rbtheron_control.urdf.xacro"/>
+	<xacro:include filename="$(find robot_description)/simulators/gazebo_ignition/rbtheron/rbtheron_control.urdf.xacro"/>
 	<!-- Import all available sensors -->
 	<xacro:include filename="$(find robotnik_sensors)/urdf/all_sensors.urdf.xacro" />
@@ -28,4 +29,5 @@
 	<xacro:arg name="prefix" default="robot_"/>
 	<xacro:arg name="gazebo_classic" default="false"/>
+	<xacro:arg name="gazebo_ignition" default="false"/>
     <!-- <xacro:arg name="has_elevator" default="false" /> -->
 	<!-- Here we create the robot using the xacro:macro imported at the beggining of this file -->
@@ -47,6 +49,11 @@
         <xacro:ros_planar_move_gazebo_classic/>
 	</xacro:if>
-  <xacro:unless value="$(arg gazebo_classic)">
-    <xacro:rbtheron_base_hw_controller/>
-  </xacro:unless>
+	<xacro:if value="$(arg gazebo_ignition)">
+		<xacro:rbtheron_gz_ignition_control namespace="$(arg namespace)" prefix="$(arg prefix)"/>
+	</xacro:if>
+    <xacro:unless value="$(arg gazebo_classic)">
+        <xacro:unless value="$(arg gazebo_ignition)">
+            <xacro:rbtheron_base_hw_controller/>
+        </xacro:unless>
+    </xacro:unless>
 </robot>

File: robots/rbvogui/rbvogui.urdf.xacro (robot description, xacro)
@@ -9,5 +9,5 @@
     <xacro:include filename="$(find robot_description)/urdf/bases/rbvogui/rbvogui_base.urdf.xacro" />
     <xacro:include filename="$(find robot_description)/urdf/base_hw/rbvogui.ros2_control.urdf" />
-    <xacro:include filename="$(find robot_description)/simulators/gazebo_classic/rbvogui/rbvogui_control.urdf.xacro" />
+    <xacro:include filename="$(find robot_description)/simulators/gazebo_ignition/rbvogui/rbvogui_control.urdf.xacro" />
     <!-- Import all available sensors -->
     <xacro:include filename="$(find robotnik_sensors)/urdf/all_sensors.urdf.xacro" />
@@ -19,4 +19,5 @@
 	<xacro:arg name="prefix" default="robot_"/>
 	<xacro:arg name="gazebo_classic" default="false"/>
+	<xacro:arg name="gazebo_ignition" default="false"/>
     <xacro:rbvogui prefix="$(arg prefix)" hq="${hq}"/>
     <!-- SENSORS see robotnik_sensors for the specific configuration -->
@@ -26,5 +27,6 @@
         parent="$(arg prefix)chassis_link"
         node_namespace="$(arg namespace)"
-        simulation="$(arg gazebo_classic)">
+        gazebo_classic="$(arg gazebo_classic)"
+        gazebo_ignition="$(arg gazebo_ignition)">
         <origin xyz="0.3 -0.3 0.0725" rpy="0 0 0"/>
     </xacro:sensor_vectornav>
@@ -35,16 +37,18 @@
         node_namespace="$(arg namespace)"
         node_name="front_camera"
-        simulation="$(arg gazebo_classic)">
+        gazebo_classic="$(arg gazebo_classic)"
+        gazebo_ignition="$(arg gazebo_ignition)">
         <origin xyz="0.46462 0.0 0.18258" rpy="0 0 0"/>
     </xacro:sensor_intel_realsense_d435>
     <!-- Rear Camera -->
-    <!-- <xacro:sensor_intel_realsense_d435
+    <xacro:sensor_intel_realsense_d435
         frame_prefix="$(arg prefix)rear_rgbd_camera_"
-        parent="$(arg prefix)chassis_link"
+        parent="$(arg prefix)base_link"
         node_namespace="$(arg namespace)"
         node_name="rear_camera"
-        simulation="$(arg gazebo_classic)">
+        gazebo_classic="$(arg gazebo_classic)"
+        gazebo_ignition="$(arg gazebo_ignition)">
         <origin xyz="-0.503 0.0 0.29" rpy="0 0 -${PI}"/>
-    </xacro:sensor_intel_realsense_d435> -->
+    </xacro:sensor_intel_realsense_d435>
     <!-- 2d laser -->
     <xacro:sensor_sick_s300
@@ -53,5 +57,6 @@
         node_namespace="$(arg namespace)"
         node_name="front_laser"
-        simulation="$(arg gazebo_classic)">
+        gazebo_classic="$(arg gazebo_classic)"
+        gazebo_ignition="$(arg gazebo_ignition)">
         <origin xyz="0.53 0.33 0.1145" rpy="${PI} 0 ${PI/4}"/>
     </xacro:sensor_sick_s300>
@@ -61,5 +66,6 @@
         node_namespace="$(arg namespace)"
         node_name="rear_laser"
-        simulation="$(arg gazebo_classic)">
+        gazebo_classic="$(arg gazebo_classic)"
+        gazebo_ignition="$(arg gazebo_ignition)">
         <origin xyz="-0.53 -0.33 0.1145" rpy="${PI} 0 ${-PI*3/4}"/>
     </xacro:sensor_sick_s300>
@@ -69,6 +75,11 @@
         <xacro:ros_planar_move_gazebo_classic/>
 	</xacro:if>
+	<xacro:if value="$(arg gazebo_ignition)">
+		<xacro:rbvogui_gz_ignition_control namespace="$(arg namespace)" prefix="$(arg prefix)"/>
+	</xacro:if>
     <xacro:unless value="$(arg gazebo_classic)">
-        <xacro:rbvogui_base_hw_controller/>
+        <xacro:unless value="$(arg gazebo_ignition)">
+            <xacro:rbvogui_base_hw_controller/>
+        </xacro:unless>
     </xacro:unless>
 </robot>

File: urdf/bases/rbkairos/rbkairos_base.urdf.xacro (robot description, xacro)
@@ -20,14 +20,14 @@
   		<xacro:rbkairos_plus_body prefix="${prefix}"/>
   		<xacro:omni_wheel robot_id="${prefix}front_right" parent="${prefix}base_link" reflect="false" hq="true">
-  			<origin xyz="${wheel_offset_x} -${wheel_offset_y} ${wheel_offset_z}" rpy="0 0 0"/>
+  			<origin xyz="${wheel_offset_x} -${wheel_offset_y} ${wheel_offset_z}" rpy="0 0 ${PI/4}"/>
   		</xacro:omni_wheel>
   		<xacro:omni_wheel robot_id="${prefix}front_left" parent="${prefix}base_link" reflect="true" hq="true">
-  			<origin xyz="${wheel_offset_x} ${wheel_offset_y} ${wheel_offset_z}" rpy="0 0 0"/>
+  			<origin xyz="${wheel_offset_x} ${wheel_offset_y} ${wheel_offset_z}" rpy="0 0 ${-PI/4}"/>
   		</xacro:omni_wheel>
-  		<xacro:omni_wheel robot_id="${prefix}back_left" parent="${prefix}base_link" reflect="true" hq="true">
-  			<origin xyz="-${wheel_offset_x} ${wheel_offset_y} ${wheel_offset_z}" rpy="0 0 0"/>
+  		<xacro:omni_wheel robot_id="${prefix}back_left" parent="${prefix}base_link" reflect="false" hq="true">
+  			<origin xyz="-${wheel_offset_x} ${wheel_offset_y} ${wheel_offset_z}" rpy="0 0 ${PI/4}"/>
   		</xacro:omni_wheel>
-  		<xacro:omni_wheel robot_id="${prefix}back_right" parent="${prefix}base_link" reflect="false" hq="true">
-  			<origin xyz="-${wheel_offset_x} -${wheel_offset_y} ${wheel_offset_z}" rpy="0 0 0"/>
+  		<xacro:omni_wheel robot_id="${prefix}back_right" parent="${prefix}base_link" reflect="true" hq="true">
+  			<origin xyz="-${wheel_offset_x} -${wheel_offset_y} ${wheel_offset_z}" rpy="0 0 ${-PI/4}"/>
   		</xacro:omni_wheel>
      </xacro:macro>

File: urdf/bases/rbrobout/rbrobout_base.urdf.xacro (robot description, xacro)
@@ -26,14 +26,14 @@
 		<!-- Wheels -->
 		<xacro:rbrobout_omni_wheel prefix="${prefix}front_right" parent="${prefix}base_link" reflect="false" hq="${hq}">
-			<origin xyz="${wheel_offset_x} -${wheel_offset_y} ${wheel_offset_z}" rpy="0 0 0"/>
+			<origin xyz="${wheel_offset_x} -${wheel_offset_y} ${wheel_offset_z}" rpy="0 0 ${PI/4}"/>
 		</xacro:rbrobout_omni_wheel>
 		<xacro:rbrobout_omni_wheel prefix="${prefix}front_left" parent="${prefix}base_link" reflect="true" hq="${hq}">
-			<origin xyz="${wheel_offset_x} ${wheel_offset_y} ${wheel_offset_z}" rpy="0 0 0"/>
+			<origin xyz="${wheel_offset_x} ${wheel_offset_y} ${wheel_offset_z}" rpy="0 0 ${-PI/4}"/>
 		</xacro:rbrobout_omni_wheel>
-		<xacro:rbrobout_omni_wheel prefix="${prefix}back_left" parent="${prefix}base_link" reflect="true" hq="${hq}">
-			<origin xyz="-${wheel_offset_x} ${wheel_offset_y} ${wheel_offset_z}" rpy="0 0 0"/>
+		<xacro:rbrobout_omni_wheel prefix="${prefix}back_left" parent="${prefix}base_link" reflect="false" hq="${hq}">
+			<origin xyz="-${wheel_offset_x} ${wheel_offset_y} ${wheel_offset_z}" rpy="0 0 ${PI/4}"/>
 		</xacro:rbrobout_omni_wheel>
-		<xacro:rbrobout_omni_wheel prefix="${prefix}back_right" parent="${prefix}base_link" reflect="false" hq="${hq}">
-			<origin xyz="-${wheel_offset_x} -${wheel_offset_y} ${wheel_offset_z}" rpy="0 0 0"/>
+		<xacro:rbrobout_omni_wheel prefix="${prefix}back_right" parent="${prefix}base_link" reflect="true" hq="${hq}">
+			<origin xyz="-${wheel_offset_x} -${wheel_offset_y} ${wheel_offset_z}" rpy="0 0 ${-PI/4}"/>
 		</xacro:rbrobout_omni_wheel>
    </xacro:macro>
