Commit message: Add gazebo ignition control files and arguments, update sensors, fix mecanum wheels physics

File: urdf/wheels/omni_wheel/omni_wheel.urdf.xacro (robot description, xacro)
@@ -1,67 +1,112 @@
 <?xml version="1.0"?>
-<robot name="wheel" xmlns:xacro="http://wiki.ros.org/xacro">
-  <xacro:property name="M_PI" value="3.1415926535897931" />
-  <!-- Wheels -->
-  <xacro:property name="omni_wheel_radius" value="0.127" />
-  <xacro:property name="omni_wheel_height" value="0.087" />
-  <xacro:property name="omni_wheel_mass" value="6.5" /> <!-- in kg-->
-  <xacro:macro name="cylinder_inertia" params="m r h">
-    <inertia  ixx="${m*(3*r*r+h*h)/12}" ixy = "0" ixz = "0"
-              iyy="${m*r*r/2}" iyz = "0"
-              izz="${m*(3*r*r+h*h)/12}" />
-  </xacro:macro>
-  <xacro:macro name="omni_wheel" params="robot_id parent *origin reflect hq">
-    <joint name="${robot_id}_wheel_joint" type="continuous">
-      <parent link="${parent}"/>
-      <child link="${robot_id}_wheel_link"/>
-      <xacro:insert_block name="origin" />
-      <axis xyz="0 1 0" rpy="0 0 0" />
-      <limit effort="100" velocity="100"/>
-      <joint_properties damping="1.0" friction="1.0"/>
-    </joint>
-    <link name="${robot_id}_wheel_link">
-      <visual>
-        <xacro:if value="${hq}">
-          <origin xyz="0 0 0" rpy="0 0 0" />
-          <xacro:if value="${reflect}">
-            <geometry>
-              <mesh filename="package://robot_description/meshes/wheels/omni_wheel/omni_wheel_1.dae" />
-            </geometry>
-          </xacro:if>
-          <xacro:unless value="${reflect}">
-            <geometry>
-              <mesh filename="package://robot_description/meshes/wheels/omni_wheel/omni_wheel_2.dae" />
-            </geometry>
-		  </xacro:unless>
-        </xacro:if>
-        <xacro:unless value="${hq}">
-          <origin xyz="0 0 0" rpy="0 0 0" />
-          <geometry>
-            <sphere radius="${omni_wheel_radius}" />
-          </geometry>
-        </xacro:unless>
-        <material name="darkgrey">
-           <color rgba="0.2 0.2 0.2 1"/>
-        </material>
-      </visual>
-      <collision>
-				<origin xyz="0 0 0" rpy="${PI/2} 0 0" />
-        <geometry>
-					<cylinder length="${omni_wheel_height}" radius="${omni_wheel_radius}" />
-        </geometry>
-      </collision>
-      <inertial>
-        <mass value="${omni_wheel_mass}" />
-        <origin xyz="0 0 0" />
-        <xacro:cylinder_inertia  m="${omni_wheel_mass}" r="${omni_wheel_radius}" h="${omni_wheel_height}" />
-      </inertial>
-    </link>
-    <gazebo reference="${robot_id}_wheel_link">
-      <mu1>0.90</mu1>
-      <mu2>0.85</mu2>
-      <kp>2.75e6</kp>
-      <kd>8.25e1</kd>
-      <fdir1>0 0 0</fdir1>
-    </gazebo>
-  </xacro:macro>
+<robot name="wheel" xmlns:xacro="http://wiki.ros.org/xacro" xmlns:gz="http://gazebosim.org/schema">
+    <xacro:property name="M_PI" value="3.1415926535897931" />
+    <!-- Wheels -->
+    <xacro:property name="omni_wheel_radius" value="0.127" />
+    <xacro:property name="omni_wheel_height" value="0.087" />
+    <xacro:property name="omni_wheel_mass" value="6.5" /> <!-- in kg-->
+    <xacro:macro name="cylinder_inertia" params="m r h">
+        <inertia ixx="${m*(3*r*r+h*h)/12}" ixy="0" ixz="0"
+            iyy="${m*r*r/2}" iyz="0"
+            izz="${m*(3*r*r+h*h)/12}" />
+    </xacro:macro>
+    <xacro:macro name="omni_wheel" params="robot_id parent *origin reflect hq">
+        <joint name="${robot_id}_wheel_joint" type="continuous">
+            <parent link="${parent}" />
+            <child link="${robot_id}_wheel_link" />
+            <xacro:insert_block name="origin" />
+            <axis xyz="0 1 0" rpy="0 0 0" />
+            <limit effort="100000" velocity="100" />
+            <!-- <joint_properties damping="1.0" friction="1.0"/> -->
+        </joint>
+        <link name="${robot_id}_wheel_link">
+            <visual>
+                <origin xyz="0 0 0" rpy="0 0 0" />
+                <geometry>
+                    <box size="0.01 0.01 0.01"/>
+                </geometry>
+                <material name="darkgrey">
+                    <color rgba="0.2 0.2 0.2 1" />
+                </material>
+            </visual>
+            <collision>
+                <origin xyz="0 0 0" rpy="0 0 0" />
+                <geometry>
+                    <sphere radius="${omni_wheel_radius}" />
+                </geometry>
+            </collision>
+            <inertial>
+                <mass value="${omni_wheel_mass}" />
+                <origin xyz="0 0 0" />
+                <xacro:cylinder_inertia m="${omni_wheel_mass}" r="${omni_wheel_radius}"
+                    h="${omni_wheel_height}" />
+            </inertial>
+        </link>
+        <gazebo reference="${robot_id}_wheel_link">
+            <collision>
+                <surface>
+                    <friction>
+                        <ode>
+                            <mu>1.0</mu>
+                            <mu2>0.0</mu2>
+                            <!-- <slip1>0.2</slip1>
+              <slip2>0.2</slip2> -->
+                            <xacro:if value="${reflect}">
+                                <fdir1 gz:expressed_in="${parent}">1 0 0</fdir1>
+                            </xacro:if>
+                            <xacro:unless value="${reflect}">
+                                <fdir1 gz:expressed_in="${parent}">1 0 0</fdir1>
+                            </xacro:unless>
+                        </ode>
+                    </friction>
+                </surface>
+            </collision>
+        </gazebo>
+        <joint name="${robot_id}_visual_wheel_joint" type="fixed">
+            <parent link="${parent}" />
+            <child link="${robot_id}_visual_wheel_link" />
+            <xacro:insert_block name="origin" />
+        </joint>
+        <link name="${robot_id}_visual_wheel_link">
+            <visual>
+                <xacro:if value="${hq}">
+                    <xacro:if value="${reflect}">
+                    <origin xyz="0 0 0" rpy="0 0 ${PI/4}" />
+                        <geometry>
+                            <mesh
+                                filename="package://robot_description/meshes/wheels/omni_wheel/omni_wheel_1.dae" />
+                        </geometry>
+                    </xacro:if>
+                    <xacro:unless value="${reflect}">
+                    <origin xyz="0 0 0" rpy="0 0 ${-PI/4}" />
+                        <geometry>
+                            <mesh
+                                filename="package://robot_description/meshes/wheels/omni_wheel/omni_wheel_2.dae" />
+                        </geometry>
+                    </xacro:unless>
+                </xacro:if>
+                <xacro:unless value="${hq}">
+                    <origin xyz="0 0 0" rpy="0 0 0" />
+                    <geometry>
+                        <sphere radius="${omni_wheel_radius}" />
+                    </geometry>
+                </xacro:unless>
+                <material name="darkgrey">
+                    <color rgba="0.2 0.2 0.2 1" />
+                </material>
+            </visual>
+            <collision>
+                <origin xyz="0 0 0" rpy="0 0 0" />
+                <geometry>
+                    <box size="0.01 0.01 0.01"/>
+                </geometry>
+            </collision>
+            <inertial>
+                <mass value="${omni_wheel_mass}" />
+                <origin xyz="0 0 0" />
+                <xacro:cylinder_inertia m="${omni_wheel_mass}" r="${omni_wheel_radius}"
+                    h="${omni_wheel_height}" />
+            </inertial>
+        </link>
+    </xacro:macro>
 </robot>
