Commit message: Mecanum wheels joints adapted to simulation or real robot

File: robots/rbkairos/rbkairos.urdf.xacro (robot description, xacro)
@@ -24,5 +24,5 @@
   <xacro:property name="imu_offset_y" value="-0.129"/>
   <xacro:property name="imu_offset_z" value="0.212"/>
-  <xacro:rbkairos prefix="$(arg prefix)"/>
+  <xacro:rbkairos prefix="$(arg prefix)" gazebo_classic="$(arg gazebo_classic)" gazebo_ignition="$(arg gazebo_ignition)"/>
   <!-- PENDIENTE DE ACTUALIZAR ROBOTNIK_SENSORS -->
   <!-- IMU -->

File: robots/rbkairos/rbkairos_plus.urdf.xacro (robot description, xacro)
@@ -43,5 +43,5 @@
   <xacro:property name="gps_offset_z" value="0.302"/>
   <!-- Kairos -->
-  <xacro:rbkairos prefix="$(arg prefix)"/>
+  <xacro:rbkairos prefix="$(arg prefix)" gazebo_classic="$(arg gazebo_classic)" gazebo_ignition="$(arg gazebo_ignition)"/>
   <!-- Import UR arm -->
   <xacro:ur_robot

File: robots/rbrobout/rbrobout.urdf.xacro (robot description, xacro)
@@ -24,5 +24,5 @@
   <xacro:property name="imu_offset_y" value="-0.3"/>
   <xacro:property name="imu_offset_z" value="0.0725"/>
-  <xacro:rbrobout prefix="$(arg prefix)"/>
+  <xacro:rbrobout prefix="$(arg prefix)" gazebo_classic="$(arg gazebo_classic)" gazebo_ignition="$(arg gazebo_ignition)"/>
   <!-- IMU -->
     <xacro:sensor_vectornav

File: robots/rbrobout/rbrobout_plus.urdf.xacro (robot description, xacro)
@@ -56,5 +56,5 @@
   <xacro:property name="lift_orientation_p" value="0"/>
   <xacro:property name="lift_orientation_y" value="0"/>
-  <xacro:rbrobout prefix="$(arg prefix)"/>
+  <xacro:rbrobout prefix="$(arg prefix)"  gazebo_classic="$(arg gazebo_classic)" gazebo_ignition="$(arg gazebo_ignition)"/>
   <xacro:top_cover prefix="$(arg prefix)" parent="$(arg prefix)base_link">
       <origin xyz="0 0 0" rpy="0 0 0"/>

File: urdf/bases/rbkairos/rbkairos_base.urdf.xacro (robot description, xacro)
@@ -13,5 +13,5 @@
   	<xacro:property name="wheel_offset_y" value="0.2590" />
   	<xacro:property name="wheel_offset_z" value="0.0" />
-    <xacro:macro name="rbkairos" params="prefix:=robot_">
+    <xacro:macro name="rbkairos" params="prefix:=robot_ gazebo_classic:=false gazebo_ignition:=false">
   		<!-- *************** -->
   		<!-- Robots Elements -->
@@ -19,15 +19,15 @@
   		<!-- Here we create the robot elements using the xacro:macros imported at the beggining of this file -->
   		<xacro:rbkairos_plus_body prefix="${prefix}"/>
-  		<xacro:mecanum_wheel prefix="${prefix}front_right_" parent="${prefix}base_link" reflect="false" hq="true">
-  			<origin xyz="${wheel_offset_x} -${wheel_offset_y} ${wheel_offset_z}" rpy="0 0 ${PI/4}"/>
+  		<xacro:mecanum_wheel prefix="${prefix}front_right_" parent="${prefix}base_link" reflect="false" hq="true" gazebo_classic="${gazebo_classic}" gazebo_ignition="${gazebo_ignition}"
+			xyz="${wheel_offset_x} -${wheel_offset_y} ${wheel_offset_z}">
   		</xacro:mecanum_wheel>
-  		<xacro:mecanum_wheel prefix="${prefix}front_left_" parent="${prefix}base_link" reflect="true" hq="true">
-  			<origin xyz="${wheel_offset_x} ${wheel_offset_y} ${wheel_offset_z}" rpy="0 0 ${-PI/4}"/>
+  		<xacro:mecanum_wheel prefix="${prefix}front_left_" parent="${prefix}base_link" reflect="true" hq="true" gazebo_classic="${gazebo_classic}" gazebo_ignition="${gazebo_ignition}"
+			xyz="${wheel_offset_x} ${wheel_offset_y} ${wheel_offset_z}">
   		</xacro:mecanum_wheel>
-  		<xacro:mecanum_wheel prefix="${prefix}back_left_" parent="${prefix}base_link" reflect="false" hq="true">
-  			<origin xyz="-${wheel_offset_x} ${wheel_offset_y} ${wheel_offset_z}" rpy="0 0 ${PI/4}"/>
+  		<xacro:mecanum_wheel prefix="${prefix}back_left_" parent="${prefix}base_link" reflect="false" hq="true" gazebo_classic="${gazebo_classic}" gazebo_ignition="${gazebo_ignition}"
+			xyz="-${wheel_offset_x} ${wheel_offset_y} ${wheel_offset_z}">
   		</xacro:mecanum_wheel>
-  		<xacro:mecanum_wheel prefix="${prefix}back_right_" parent="${prefix}base_link" reflect="true" hq="true">
-  			<origin xyz="-${wheel_offset_x} -${wheel_offset_y} ${wheel_offset_z}" rpy="0 0 ${-PI/4}"/>
+  		<xacro:mecanum_wheel prefix="${prefix}back_right_" parent="${prefix}base_link" reflect="true" hq="true" gazebo_classic="${gazebo_classic}" gazebo_ignition="${gazebo_ignition}"
+			xyz="-${wheel_offset_x} -${wheel_offset_y} ${wheel_offset_z}">
   		</xacro:mecanum_wheel>
      </xacro:macro>

File: urdf/bases/rbrobout/rbrobout_base.urdf.xacro (robot description, xacro)
@@ -18,5 +18,5 @@
 	<!-- Flag to select the high or low quality model -->
 	<xacro:property name="hq" value="true" />
-    <xacro:macro name="rbrobout" params="prefix:=robot_">
+    <xacro:macro name="rbrobout" params="prefix:=robot_ gazebo_classic:=false gazebo_ignition:=false">
 		<!-- *************** -->
 		<!-- Robots Elements -->
@@ -25,15 +25,15 @@
 		<xacro:rbrobout_body prefix="${prefix}" />
 		<!-- Wheels -->
-		<xacro:rbrobout_mecanum_wheel prefix="${prefix}front_right_" parent="${prefix}base_link" reflect="false" hq="${hq}">
-			<origin xyz="${wheel_offset_x} -${wheel_offset_y} ${wheel_offset_z}" rpy="0 0 ${PI/4}"/>
+		<xacro:rbrobout_mecanum_wheel prefix="${prefix}front_right_" parent="${prefix}base_link" reflect="false" hq="${hq}" gazebo_classic="${gazebo_classic}" gazebo_ignition="${gazebo_ignition}"
+			xyz="${wheel_offset_x} -${wheel_offset_y} ${wheel_offset_z}">
 		</xacro:rbrobout_mecanum_wheel>
-		<xacro:rbrobout_mecanum_wheel prefix="${prefix}front_left_" parent="${prefix}base_link" reflect="true" hq="${hq}">
-			<origin xyz="${wheel_offset_x} ${wheel_offset_y} ${wheel_offset_z}" rpy="0 0 ${-PI/4}"/>
+		<xacro:rbrobout_mecanum_wheel prefix="${prefix}front_left_" parent="${prefix}base_link" reflect="true" hq="${hq}" gazebo_classic="${gazebo_classic}" gazebo_ignition="${gazebo_ignition}"
+			xyz="${wheel_offset_x} ${wheel_offset_y} ${wheel_offset_z}">
 		</xacro:rbrobout_mecanum_wheel>
-		<xacro:rbrobout_mecanum_wheel prefix="${prefix}back_left_" parent="${prefix}base_link" reflect="false" hq="${hq}">
-			<origin xyz="-${wheel_offset_x} ${wheel_offset_y} ${wheel_offset_z}" rpy="0 0 ${PI/4}"/>
+		<xacro:rbrobout_mecanum_wheel prefix="${prefix}back_left_" parent="${prefix}base_link" reflect="false" hq="${hq}" gazebo_classic="${gazebo_classic}" gazebo_ignition="${gazebo_ignition}"
+			xyz="-${wheel_offset_x} ${wheel_offset_y} ${wheel_offset_z}">
 		</xacro:rbrobout_mecanum_wheel>
-		<xacro:rbrobout_mecanum_wheel prefix="${prefix}back_right_" parent="${prefix}base_link" reflect="true" hq="${hq}">
-			<origin xyz="-${wheel_offset_x} -${wheel_offset_y} ${wheel_offset_z}" rpy="0 0 ${-PI/4}"/>
+		<xacro:rbrobout_mecanum_wheel prefix="${prefix}back_right_" parent="${prefix}base_link" reflect="true" hq="${hq}" gazebo_classic="${gazebo_classic}" gazebo_ignition="${gazebo_ignition}"
+			xyz="-${wheel_offset_x} -${wheel_offset_y} ${wheel_offset_z}">
 		</xacro:rbrobout_mecanum_wheel>
    </xacro:macro>

File: urdf/wheels/mecanum_wheel/rbkairos_mecanum_wheel.urdf.xacro (robot description, xacro)
@@ -11,23 +11,52 @@
             izz="${m*(3*r*r+h*h)/12}" />
     </xacro:macro>
-    <xacro:macro name="mecanum_wheel" params="prefix parent *origin reflect hq">
+    <xacro:macro name="mecanum_wheel" params="prefix parent xyz reflect hq gazebo_classic:=false gazebo_ignition:=false">
         <joint name="${prefix}wheel_joint" type="continuous">
             <parent link="${parent}" />
             <child link="${prefix}wheel_link" />
-            <xacro:insert_block name="origin" />
-            <axis xyz="0 1 0" />
+            <xacro:if value="${gazebo_classic or gazebo_ignition}">
+                <xacro:if value="${reflect}">
+                    <origin xyz="${xyz}" rpy="0.0 0.0 -${PI/4}"/>
+                </xacro:if>
+                <xacro:unless value="${reflect}">
+                    <origin xyz="${xyz}" rpy="0.0 0.0 ${PI/4}"/>
+                </xacro:unless>
+            </xacro:if>
+            <xacro:unless value="${gazebo_classic or gazebo_ignition}">
+                <origin xyz="${xyz}" rpy="0.0 0.0 0.0"/>
+            </xacro:unless>
             <limit effort="100000" velocity="100" />
-            <!-- <joint_properties damping="1.0" friction="1.0"/> -->
+            <axis xyz="0 1 0"/>
         </joint>
         <link name="${prefix}wheel_link">
-            <visual>
-                <origin xyz="0 0 0" rpy="0 0 0" />
-                <geometry>
-                    <box size="0.01 0.01 0.01"/>
-                </geometry>
-                <material name="darkgrey">
-                    <color rgba="0.2 0.2 0.2 1" />
-                </material>
-            </visual>
+            <xacro:unless value="${gazebo_classic or gazebo_ignition}">
+                <visual>
+                    <xacro:if value="${hq}">
+                        <xacro:if value="${reflect}">
+                        <origin xyz="0 0 0" rpy="0 0 0" />
+                            <geometry>
+                                <mesh
+                                    filename="package://robotnik_description/meshes/wheels/mecanum_wheel/mecanum_wheel_1.dae" />
+                            </geometry>
+                        </xacro:if>
+                        <xacro:unless value="${reflect}">
+                        <origin xyz="0 0 0" rpy="0 0 0" />
+                            <geometry>
+                                <mesh
+                                    filename="package://robotnik_description/meshes/wheels/mecanum_wheel/mecanum_wheel_2.dae" />
+                            </geometry>
+                        </xacro:unless>
+                    </xacro:if>
+                    <xacro:unless value="${hq}">
+                        <origin xyz="0 0 0" rpy="0 0 0" />
+                        <geometry>
+                            <sphere radius="${mecanum_wheel_radius}" />
+                        </geometry>
+                    </xacro:unless>
+                    <material name="darkgrey">
+                        <color rgba="0.2 0.2 0.2 1" />
+                    </material>
+                </visual>
+            </xacro:unless>
             <collision>
                 <origin xyz="0 0 0" rpy="0 0 0" />
@@ -43,70 +72,60 @@
             </inertial>
         </link>
-        <gazebo reference="${prefix}wheel_link">
-            <collision>
-                <surface>
-                    <friction>
-                        <ode>
-                            <mu>1.0</mu>
-                            <mu2>0.0</mu2>
-                            <!-- <slip1>0.2</slip1>
-              <slip2>0.2</slip2> -->
-                            <xacro:if value="${reflect}">
-                                <fdir1 gz:expressed_in="${parent}">1 0 0</fdir1>
-                            </xacro:if>
-                            <xacro:unless value="${reflect}">
-                                <fdir1 gz:expressed_in="${parent}">1 0 0</fdir1>
-                            </xacro:unless>
-                        </ode>
-                    </friction>
-                </surface>
-            </collision>
-        </gazebo>
-        <joint name="${prefix}visual_wheel_joint" type="fixed">
-            <parent link="${parent}" />
-            <child link="${prefix}visual_wheel_link" />
-            <xacro:insert_block name="origin" />
-        </joint>
-        <link name="${prefix}visual_wheel_link">
-            <visual>
-                <xacro:if value="${hq}">
-                    <xacro:if value="${reflect}">
-                    <origin xyz="0 0 0" rpy="0 0 ${PI/4}" />
+        <xacro:if value="${gazebo_classic or gazebo_ignition}">
+            <gazebo reference="${prefix}wheel_link">
+                <collision>
+                    <surface>
+                        <friction>
+                            <ode>
+                                <mu>1.0</mu>
+                                <mu2>0.0</mu2>
+                                <!-- <slip1>0.2</slip1>
+                <slip2>0.2</slip2> -->
+                                <xacro:if value="${reflect}">
+                                    <fdir1 gz:expressed_in="${parent}">1 0 0</fdir1>
+                                </xacro:if>
+                                <xacro:unless value="${reflect}">
+                                    <fdir1 gz:expressed_in="${parent}">1 0 0</fdir1>
+                                </xacro:unless>
+                            </ode>
+                        </friction>
+                    </surface>
+                </collision>
+            </gazebo>
+            <joint name="${prefix}visual_wheel_joint" type="fixed">
+                <parent link="${parent}" />
+                <child link="${prefix}visual_wheel_link" />
+                <origin xyz="${xyz}"/>
+            </joint>
+            <link name="${prefix}visual_wheel_link">
+                <visual>
+                    <xacro:if value="${hq}">
+                        <xacro:if value="${reflect}">
+                        <origin xyz="0 0 0" rpy="0 0 0" />
+                            <geometry>
+                                <mesh
+                                    filename="package://robotnik_description/meshes/wheels/mecanum_wheel/mecanum_wheel_1.dae" />
+                            </geometry>
+                        </xacro:if>
+                        <xacro:unless value="${reflect}">
+                        <origin xyz="0 0 0" rpy="0 0 0" />
+                            <geometry>
+                                <mesh
+                                    filename="package://robotnik_description/meshes/wheels/mecanum_wheel/mecanum_wheel_2.dae" />
+                            </geometry>
+                        </xacro:unless>
+                    </xacro:if>
+                    <xacro:unless value="${hq}">
+                        <origin xyz="0 0 0" rpy="0 0 0" />
                         <geometry>
-                            <mesh
-                                filename="package://robotnik_description/meshes/wheels/mecanum_wheel/mecanum_wheel_1.dae" />
-                        </geometry>
-                    </xacro:if>
-                    <xacro:unless value="${reflect}">
-                    <origin xyz="0 0 0" rpy="0 0 ${-PI/4}" />
-                        <geometry>
-                            <mesh
-                                filename="package://robotnik_description/meshes/wheels/mecanum_wheel/mecanum_wheel_2.dae" />
+                            <sphere radius="${mecanum_wheel_radius}" />
                         </geometry>
                     </xacro:unless>
-                </xacro:if>
-                <xacro:unless value="${hq}">
-                    <origin xyz="0 0 0" rpy="0 0 0" />
-                    <geometry>
-                        <sphere radius="${mecanum_wheel_radius}" />
-                    </geometry>
-                </xacro:unless>
-                <material name="darkgrey">
-                    <color rgba="0.2 0.2 0.2 1" />
-                </material>
-            </visual>
-            <collision>
-                <origin xyz="0 0 0" rpy="0 0 0" />
-                <geometry>
-                    <box size="0.01 0.01 0.01"/>
-                </geometry>
-            </collision>
-            <inertial>
-                <mass value="${mecanum_wheel_mass}" />
-                <origin xyz="0 0 0" />
-                <xacro:cylinder_inertia m="${mecanum_wheel_mass}" r="${mecanum_wheel_radius}"
-                    h="${mecanum_wheel_height}" />
-            </inertial>
-        </link>
+                    <material name="darkgrey">
+                        <color rgba="0.2 0.2 0.2 1" />
+                    </material>
+                </visual>
+            </link>
+        </xacro:if>
     </xacro:macro>
 </robot>
