Commit message: Mecanum wheels joints adapted to simulation or real robot

File: urdf/wheels/mecanum_wheel/rbrobout_mecanum_wheel.urdf.xacro (robot description, xacro)
@@ -11,23 +11,52 @@
             izz="${m*(3*r*r+h*h)/12}" />
     </xacro:macro>
-    <xacro:macro name="rbrobout_mecanum_wheel" params="prefix parent *origin reflect hq">
+    <xacro:macro name="rbrobout_mecanum_wheel" params="prefix parent xyz reflect hq gazebo_classic:=false gazebo_ignition:=false">
         <joint name="${prefix}wheel_joint" type="continuous">
             <parent link="${parent}" />
             <child link="${prefix}wheel_link" />
-            <xacro:insert_block name="origin" />
-            <axis xyz="0 1 0" />
+            <xacro:if value="${gazebo_classic or gazebo_ignition}">
+                <xacro:if value="${reflect}">
+                    <origin xyz="${xyz}" rpy="0.0 0.0 -${PI/4}"/>
+                </xacro:if>
+                <xacro:unless value="${reflect}">
+                    <origin xyz="${xyz}" rpy="0.0 0.0 ${PI/4}"/>
+                </xacro:unless>
+            </xacro:if>
+            <xacro:unless value="${gazebo_classic or gazebo_ignition}">
+                <origin xyz="${xyz}" rpy="0.0 0.0 0.0"/>
+            </xacro:unless>
             <limit effort="100000" velocity="100" />
-            <!-- <joint_properties damping="1.0" friction="1.0"/> -->
+            <axis xyz="0 1 0"/>
         </joint>
         <link name="${prefix}wheel_link">
-            <visual>
-                <origin xyz="0 0 0" rpy="0 0 0" />
-                <geometry>
-                    <box size="0.01 0.01 0.01"/>
-                </geometry>
-                <material name="darkgrey">
-                    <color rgba="0.2 0.2 0.2 1" />
-                </material>
-            </visual>
+            <xacro:unless value="${gazebo_classic or gazebo_ignition}">
+                <visual>
+                    <xacro:if value="${hq}">
+                        <xacro:if value="${reflect}">
+                        <origin xyz="0 0 0" rpy="${PI/2} 0 0" />
+                            <geometry>
+                                <mesh
+                                    filename="package://robotnik_description/meshes/wheels/mecanum_wheel/robout_wheel.stl" />
+                            </geometry>
+                        </xacro:if>
+                        <xacro:unless value="${reflect}">
+                        <origin xyz="0 0 0" rpy="${-PI/2} 0 0" />
+                            <geometry>
+                                <mesh
+                                    filename="package://robotnik_description/meshes/wheels/mecanum_wheel/robout_wheel.stl" />
+                            </geometry>
+                        </xacro:unless>
+                    </xacro:if>
+                    <xacro:unless value="${hq}">
+                        <origin xyz="0 0 0" rpy="0 0 0" />
+                        <geometry>
+                            <sphere radius="${mecanum_wheel_radius}" />
+                        </geometry>
+                    </xacro:unless>
+                    <material name="darkgrey">
+                        <color rgba="0.2 0.2 0.2 1" />
+                    </material>
+                </visual>
+            </xacro:unless>
             <collision>
                 <origin xyz="0 0 0" rpy="0 0 0" />
@@ -43,70 +72,58 @@
             </inertial>
         </link>
-        <gazebo reference="${prefix}wheel_link">
-            <collision>
-                <surface>
-                    <friction>
-                        <ode>
-                            <mu>1.0</mu>
-                            <mu2>0.0</mu2>
-                            <!-- <slip1>0.2</slip1>
-              <slip2>0.2</slip2> -->
-                            <xacro:if value="${reflect}">
-                                <fdir1 gz:expressed_in="${parent}">1 0 0</fdir1>
-                            </xacro:if>
-                            <xacro:unless value="${reflect}">
-                                <fdir1 gz:expressed_in="${parent}">1 0 0</fdir1>
-                            </xacro:unless>
-                        </ode>
-                    </friction>
-                </surface>
-            </collision>
-        </gazebo>
-        <joint name="${prefix}visual_wheel_joint" type="fixed">
-            <parent link="${parent}" />
-            <child link="${prefix}visual_wheel_link" />
-            <xacro:insert_block name="origin" />
-        </joint>
-        <link name="${prefix}visual_wheel_link">
-            <visual>
-                <xacro:if value="${hq}">
-                    <xacro:if value="${reflect}">
-                    <origin xyz="0 0 0" rpy="${PI/2} 0 ${PI/4}" />
+        <xacro:if value="${gazebo_classic or gazebo_ignition}">
+            <gazebo reference="${prefix}wheel_link">
+                <collision>
+                    <surface>
+                        <friction>
+                            <ode>
+                                <mu>1.0</mu>
+                                <mu2>0.0</mu2>
+                                <xacro:if value="${reflect}">
+                                    <fdir1 gz:expressed_in="${parent}">1 0 0</fdir1>
+                                </xacro:if>
+                                <xacro:unless value="${reflect}">
+                                    <fdir1 gz:expressed_in="${parent}">1 0 0</fdir1>
+                                </xacro:unless>
+                            </ode>
+                        </friction>
+                    </surface>
+                </collision>
+            </gazebo>
+            <joint name="${prefix}visual_wheel_joint" type="fixed">
+                <parent link="${parent}" />
+                <child link="${prefix}visual_wheel_link" />
+                <origin xyz="${xyz}"/>
+            </joint>
+            <link name="${prefix}visual_wheel_link">
+                <visual>
+                    <xacro:if value="${hq}">
+                        <xacro:if value="${reflect}">
+                        <origin xyz="0 0 0" rpy="${PI/2} 0 0" />
+                            <geometry>
+                                <mesh
+                                    filename="package://robotnik_description/meshes/wheels/mecanum_wheel/robout_wheel.stl" />
+                            </geometry>
+                        </xacro:if>
+                        <xacro:unless value="${reflect}">
+                        <origin xyz="0 0 0" rpy="${-PI/2} 0 0" />
+                            <geometry>
+                                <mesh
+                                    filename="package://robotnik_description/meshes/wheels/mecanum_wheel/robout_wheel.stl" />
+                            </geometry>
+                        </xacro:unless>
+                    </xacro:if>
+                    <xacro:unless value="${hq}">
+                        <origin xyz="0 0 0" rpy="0 0 0" />
                         <geometry>
-                            <mesh
-                                filename="package://robotnik_description/meshes/wheels/mecanum_wheel/robout_wheel.stl" />
-                        </geometry>
-                    </xacro:if>
-                    <xacro:unless value="${reflect}">
-                    <origin xyz="0 0 0" rpy="${-PI/2} 0 ${-PI/4}" />
-                        <geometry>
-                            <mesh
-                                filename="package://robotnik_description/meshes/wheels/mecanum_wheel/robout_wheel.stl" />
+                            <sphere radius="${mecanum_wheel_radius}" />
                         </geometry>
                     </xacro:unless>
-                </xacro:if>
-                <xacro:unless value="${hq}">
-                    <origin xyz="0 0 0" rpy="0 0 0" />
-                    <geometry>
-                        <sphere radius="${mecanum_wheel_radius}" />
-                    </geometry>
-                </xacro:unless>
-                <material name="darkgrey">
-                    <color rgba="0.2 0.2 0.2 1" />
-                </material>
-            </visual>
-            <collision>
-                <origin xyz="0 0 0" rpy="0 0 0" />
-                <geometry>
-                    <box size="0.01 0.01 0.01"/>
-                </geometry>
-            </collision>
-            <inertial>
-                <mass value="${mecanum_wheel_mass}" />
-                <origin xyz="0 0 0" />
-                <xacro:cylinder_inertia m="${mecanum_wheel_mass}" r="${mecanum_wheel_radius}"
-                    h="${mecanum_wheel_height}" />
-            </inertial>
-        </link>
+                    <material name="darkgrey">
+                        <color rgba="0.2 0.2 0.2 1" />
+                    </material>
+                </visual>
+            </link>
+        </xacro:if>
     </xacro:macro>
 </robot>

Commit message: Add basic sensors to robots

File: robots/rbkairos/rbkairos.urdf.xacro (robot description, xacro)
@@ -15,13 +15,16 @@
   <xacro:arg name="gazebo_classic" default="false"/>
   <xacro:arg name="gazebo_ignition" default="false"/>
-  <xacro:property name="front_laser_offset_x" value="0.2865"/>
-  <xacro:property name="front_laser_offset_y" value="-0.20894"/>
-  <xacro:property name="front_laser_offset_z" value="0.2973"/>
-  <xacro:property name="rear_laser_offset_x" value="-0.2865"/>
-  <xacro:property name="rear_laser_offset_y" value="0.20894"/>
-  <xacro:property name="rear_laser_offset_z" value="0.2973"/>
+  <xacro:property name="front_laser_offset_x" value="0.42109"/>
+  <xacro:property name="front_laser_offset_y" value="-0.32737"/>
+  <xacro:property name="front_laser_offset_z" value="0.16037"/>
+  <xacro:property name="rear_laser_offset_x" value="-0.42109"/>
+  <xacro:property name="rear_laser_offset_y" value="0.32737"/>
+  <xacro:property name="rear_laser_offset_z" value="0.16037"/>
   <xacro:property name="imu_offset_x" value="0.127"/>
   <xacro:property name="imu_offset_y" value="-0.129"/>
   <xacro:property name="imu_offset_z" value="0.212"/>
+  <xacro:property name="front_rgbd_camera_offset_x" value="0.35850"/>
+  <xacro:property name="front_rgbd_camera_offset_y" value="0.0"/>
+  <xacro:property name="front_rgbd_camera_offset_z" value="0.25062"/>
   <xacro:rbkairos prefix="$(arg prefix)" gazebo_classic="$(arg gazebo_classic)" gazebo_ignition="$(arg gazebo_ignition)"/>
   <!-- PENDIENTE DE ACTUALIZAR ROBOTNIK_SENSORS -->
@@ -54,4 +57,14 @@
         <origin xyz="${rear_laser_offset_x} ${rear_laser_offset_y} ${rear_laser_offset_z}" rpy="0 ${-PI} ${-1/4*PI}"/>
     </xacro:sensor_sick_s300>
+  <!-- CAMERA -->
+    <xacro:sensor_intel_realsense_d435
+        frame_prefix="$(arg prefix)front_rgbd_camera_"
+        parent="$(arg prefix)base_link"
+        node_namespace="$(arg namespace)"
+        node_name="front_camera"
+        gazebo_classic="$(arg gazebo_classic)"
+        gazebo_ignition="$(arg gazebo_ignition)">
+        <origin xyz="${front_rgbd_camera_offset_x} ${front_rgbd_camera_offset_y} ${front_rgbd_camera_offset_z}" rpy="0 0 0"/>
+    </xacro:sensor_intel_realsense_d435>
   <!-- Controllers -->
   <xacro:if value="$(arg gazebo_classic)">

File: robots/rbkairos/rbkairos_plus.urdf.xacro (robot description, xacro)
@@ -27,10 +27,4 @@
   <xacro:property name="rear_laser_offset_y" value="0.20894"/>
   <xacro:property name="rear_laser_offset_z" value="0.2973"/>
-  <xacro:property name="front_ptz_camera_offset_x" value="0.308"/>
-  <xacro:property name="front_ptz_camera_offset_y" value="0.141"/>
-  <xacro:property name="front_ptz_camera_offset_z" value="0.195"/>
-  <xacro:property name="rear_ptz_camera_offset_x" value="-0.308"/>
-  <xacro:property name="rear_ptz_camera_offset_y" value="-0.141"/>
-  <xacro:property name="rear_ptz_camera_offset_z" value="0.195"/>
   <xacro:property name="imu_offset_x" value="0.127"/>
   <xacro:property name="imu_offset_y" value="-0.129"/>
@@ -39,7 +33,4 @@
   <xacro:property name="front_rgbd_camera_offset_y" value="0.0"/>
   <xacro:property name="front_rgbd_camera_offset_z" value="0.25062"/>
-  <xacro:property name="gps_offset_x" value="-0.365"/>
-  <xacro:property name="gps_offset_y" value="-0.167"/>
-  <xacro:property name="gps_offset_z" value="0.302"/>
   <!-- Kairos -->
   <xacro:rbkairos prefix="$(arg prefix)" gazebo_classic="$(arg gazebo_classic)" gazebo_ignition="$(arg gazebo_ignition)"/>
@@ -86,4 +77,14 @@
         <origin xyz="${rear_laser_offset_x} ${rear_laser_offset_y} ${rear_laser_offset_z}" rpy="0 ${-PI} ${-1/4*PI}"/>
     </xacro:sensor_sick_s300>
+  <!-- CAMERA -->
+    <xacro:sensor_intel_realsense_d435
+        frame_prefix="$(arg prefix)front_rgbd_camera_"
+        parent="$(arg prefix)base_link"
+        node_namespace="$(arg namespace)"
+        node_name="front_camera"
+        gazebo_classic="$(arg gazebo_classic)"
+        gazebo_ignition="$(arg gazebo_ignition)">
+        <origin xyz="${front_rgbd_camera_offset_x} ${front_rgbd_camera_offset_y} ${front_rgbd_camera_offset_z}" rpy="0 0 0"/>
+    </xacro:sensor_intel_realsense_d435>
   <!-- Controllers -->
   <xacro:if value="$(arg gazebo_classic)">

File: robots/rbsummit/rbsummit.urdf.xacro (robot description, xacro)
@@ -25,30 +25,14 @@
 	<xacro:property name="top_laser_offset_x" value="-0.01924"/>
 	<xacro:property name="top_laser_offset_y" value="0.0"/>
-	<xacro:property name="top_laser_offset_z" value="0.35642"/>
+	<xacro:property name="top_laser_offset_z" value="0.27642"/>
 	<xacro:property name="front_rgbd_camera_offset_x" value="0.324"/>
 	<xacro:property name="front_rgbd_camera_offset_y" value="0.012"/>
 	<xacro:property name="front_rgbd_camera_offset_z" value="0.172"/>
-	<xacro:property name="front_ptz_camera_offset_x" value="0.22151"/>
-	<xacro:property name="front_ptz_camera_offset_y" value="0.0"/>
-	<xacro:property name="front_ptz_camera_offset_z" value="0.24022"/>
-	<xacro:property name="front_ptz_camera_offset_t" value="-1.308996939"/>
 	<xacro:property name="gps_offset_x" value="-0.22528"/>
 	<xacro:property name="gps_offset_y" value="0.095"/>
-	<xacro:property name="gps_offset_z" value="0.275"/>
-	<!-- Other elements -->
-	<xacro:property name="antenna_offset_x" value="-0.18324"/>
-	<xacro:property name="antenna_offset_y" value="0.0"/>
-	<xacro:property name="antenna_offset_z" value="0.27488"/>
-	<!-- ***************** -->
-	<!-- Global parameters -->
-	<!-- ***************** -->
-	<!-- Second we define all the parameters and arguments to customize the robot characteristics -->
+	<xacro:property name="gps_offset_z" value="0.48"/>
 	<xacro:property name="PI" value="3.1415926535897931"/>
 	<!-- Flag to select the high or low quality model -->
 	<xacro:property name="hq" value="true" />
-	<!-- Launch Arguments -->
-	<xacro:arg name="gpu" default="true" />
-	<xacro:arg name="gps_latitude" default="0"/>
-	<xacro:arg name="gps_longitude" default="0"/>
 	<!-- Here we create the robot using the xacro:macro imported at the beggining of this file -->
 	<xacro:rbsummit prefix="$(arg prefix)" hq="${hq}"/>
@@ -63,4 +47,42 @@
         <origin xyz="${imu_offset_x} ${imu_offset_y} ${imu_offset_z}" rpy="0 0 0"/>
     </xacro:sensor_vectornav>
+	<!-- 3D LIDAR -->
+	<xacro:sensor_robosense_helios_16p
+		frame_prefix="$(arg prefix)top_3d_laser_"
+		parent="$(arg prefix)base_link"
+        node_namespace="$(arg namespace)"
+        gazebo_classic="$(arg gazebo_classic)"
+        gazebo_ignition="$(arg gazebo_ignition)">
+		<origin
+			xyz="${top_laser_offset_x} ${top_laser_offset_y} ${top_laser_offset_z}"
+			rpy="0 0 0"
+		/>
+	</xacro:sensor_robosense_helios_16p>
+	<!-- CAMERA -->
+	<xacro:sensor_intel_realsense_d435
+		frame_prefix="$(arg prefix)front_rgbd_camera_"
+		parent="$(arg prefix)base_link"
+		topic_prefix="front_rgbd_camera"
+        node_namespace="$(arg namespace)"
+        gazebo_classic="$(arg gazebo_classic)"
+        gazebo_ignition="$(arg gazebo_ignition)">
+		<origin
+			xyz="${front_rgbd_camera_offset_x} ${front_rgbd_camera_offset_y} ${front_rgbd_camera_offset_z}"
+			rpy="0 0 0"
+		/>
+	</xacro:sensor_intel_realsense_d435>
+	<!-- GPS -->
+	<xacro:sensor_ublox_with_mast
+		frame_prefix="$(arg prefix)gps_"
+		parent="$(arg prefix)base_link"
+		update_rate="5"
+        node_namespace="$(arg namespace)"
+        gazebo_classic="$(arg gazebo_classic)"
+        gazebo_ignition="$(arg gazebo_ignition)">
+		<origin
+			xyz="${gps_offset_x} ${gps_offset_y} ${gps_offset_z}"
+			rpy="0 0 0"
+		/>
+	</xacro:sensor_ublox_with_mast>
 	<!-- Controllers -->
     <xacro:if value="$(arg gazebo_classic)">

File: robots/rbtheron/rbtheron.urdf.xacro (robot description, xacro)
@@ -30,4 +30,17 @@
     <xacro:property name="imu_offset_y" value="0.0"/>
     <xacro:property name="imu_offset_z" value="0.1598"/>
+	<xacro:property name="front_rgbd_camera_offset_x" value="0.3045"/>
+	<xacro:property name="front_rgbd_camera_offset_y" value="0.0"/>
+	<xacro:property name="front_rgbd_camera_offset_z" value="0.1898"/>
+	<xacro:property name="rear_rgbd_camera_offset_x" value="-0.3045"/>
+	<xacro:property name="rear_rgbd_camera_offset_y" value="0.0"/>
+	<xacro:property name="rear_rgbd_camera_offset_z" value="0.1158"/>
+	<xacro:property name="front_laser_offset_x" value="0.2675"/>
+	<xacro:property name="front_laser_offset_y" value="-0.215"/>
+	<xacro:property name="front_laser_offset_z" value="0.1613"/>
+	<xacro:property name="rear_laser_offset_x" value="-0.2675"/>
+	<xacro:property name="rear_laser_offset_y" value="0.215"/>
+	<xacro:property name="rear_laser_offset_z" value="0.1613"/>
+	<!-- IMU -->
     <xacro:sensor_vectornav
         frame_prefix="$(arg prefix)vectornav_"
@@ -38,4 +51,42 @@
         <origin xyz="${imu_offset_x} ${imu_offset_y} ${imu_offset_z}" rpy="0 0 0"/>
     </xacro:sensor_vectornav>
+	<!-- 2D LASER -->
+    <xacro:sensor_hokuyo_ust20lx
+        frame_prefix="$(arg prefix)front_laser_"
+        parent="$(arg prefix)base_link"
+        node_namespace="$(arg namespace)"
+        node_name="front_laser"
+        gazebo_classic="$(arg gazebo_classic)"
+        gazebo_ignition="$(arg gazebo_ignition)">
+        <origin xyz="${front_laser_offset_x} ${front_laser_offset_y} ${front_laser_offset_z}" rpy="0 ${-PI} ${3/4*PI}"/>
+    </xacro:sensor_hokuyo_ust20lx>
+    <xacro:sensor_hokuyo_ust20lx
+        frame_prefix="$(arg prefix)rear_laser_"
+        parent="$(arg prefix)base_link"
+        node_namespace="$(arg namespace)"
+        node_name="rear_laser"
+        gazebo_classic="$(arg gazebo_classic)"
+        gazebo_ignition="$(arg gazebo_ignition)">
+        <origin xyz="${rear_laser_offset_x} ${rear_laser_offset_y} ${rear_laser_offset_z}" rpy="0 ${-PI} ${-1/4*PI}"/>
+    </xacro:sensor_hokuyo_ust20lx>
+  	<!-- CAMERAS -->
+    <xacro:sensor_intel_realsense_d435
+        frame_prefix="$(arg prefix)front_rgbd_camera_"
+        parent="$(arg prefix)base_link"
+        node_namespace="$(arg namespace)"
+        node_name="front_camera"
+        gazebo_classic="$(arg gazebo_classic)"
+        gazebo_ignition="$(arg gazebo_ignition)">
+        <origin xyz="${front_rgbd_camera_offset_x} ${front_rgbd_camera_offset_y} ${front_rgbd_camera_offset_z}" rpy="0 0 0"/>
+    </xacro:sensor_intel_realsense_d435>
+    <xacro:sensor_intel_realsense_d435
+        frame_prefix="$(arg prefix)rear_rgbd_camera_"
+        parent="$(arg prefix)base_link"
+        node_namespace="$(arg namespace)"
+        node_name="rear_camera"
+        gazebo_classic="$(arg gazebo_classic)"
+        gazebo_ignition="$(arg gazebo_ignition)">
+        <origin xyz="${rear_rgbd_camera_offset_x} ${rear_rgbd_camera_offset_y} ${rear_rgbd_camera_offset_z}" rpy="0 0 ${PI}"/>
+    </xacro:sensor_intel_realsense_d435>
 	<!-- Controllers -->
 	<xacro:if value="$(arg gazebo_classic)">
