Commit message: Feat/ros2/standard robots (#40)
* Fix issues with ur meshes and position of arms

* change plugins for gazebo simulation ignition

* Fix issues with ur meshes and position of arms

* Add basic sensors to robots

* fix issue with rbsummit sensors

* Update rbkairos.urdf.xacro

---------

Co-authored-by: Rafael Martin <rmartin@robotnik.es>

File: robots/rbkairos/rbkairos.urdf.xacro (robot description, xacro)
@@ -15,15 +15,17 @@
   <xacro:arg name="gazebo_classic" default="false"/>
   <xacro:arg name="gazebo_ignition" default="false"/>
-  <xacro:property name="front_laser_offset_x" value="0.2865"/>
-  <xacro:property name="front_laser_offset_y" value="-0.20894"/>
-  <xacro:property name="front_laser_offset_z" value="0.2973"/>
-  <xacro:property name="rear_laser_offset_x" value="-0.2865"/>
-  <xacro:property name="rear_laser_offset_y" value="0.20894"/>
-  <xacro:property name="rear_laser_offset_z" value="0.2973"/>
+  <xacro:property name="front_laser_offset_x" value="0.42109"/>
+  <xacro:property name="front_laser_offset_y" value="-0.32737"/>
+  <xacro:property name="front_laser_offset_z" value="0.16037"/>
+  <xacro:property name="rear_laser_offset_x" value="-0.42109"/>
+  <xacro:property name="rear_laser_offset_y" value="0.32737"/>
+  <xacro:property name="rear_laser_offset_z" value="0.16037"/>
   <xacro:property name="imu_offset_x" value="0.127"/>
   <xacro:property name="imu_offset_y" value="-0.129"/>
   <xacro:property name="imu_offset_z" value="0.212"/>
+  <xacro:property name="front_rgbd_camera_offset_x" value="0.35850"/>
+  <xacro:property name="front_rgbd_camera_offset_y" value="0.0"/>
+  <xacro:property name="front_rgbd_camera_offset_z" value="0.25062"/>
   <xacro:rbkairos prefix="$(arg prefix)" gazebo_classic="$(arg gazebo_classic)" gazebo_ignition="$(arg gazebo_ignition)"/>
-  <!-- PENDIENTE DE ACTUALIZAR ROBOTNIK_SENSORS -->
   <!-- IMU -->
     <xacro:sensor_vectornav
@@ -54,4 +56,14 @@
         <origin xyz="${rear_laser_offset_x} ${rear_laser_offset_y} ${rear_laser_offset_z}" rpy="0 ${-PI} ${-1/4*PI}"/>
     </xacro:sensor_sick_s300>
+  <!-- CAMERA -->
+    <xacro:sensor_intel_realsense_d435
+        frame_prefix="$(arg prefix)front_rgbd_camera_"
+        parent="$(arg prefix)base_link"
+        node_namespace="$(arg namespace)"
+        node_name="front_camera"
+        gazebo_classic="$(arg gazebo_classic)"
+        gazebo_ignition="$(arg gazebo_ignition)">
+        <origin xyz="${front_rgbd_camera_offset_x} ${front_rgbd_camera_offset_y} ${front_rgbd_camera_offset_z}" rpy="0 0 0"/>
+    </xacro:sensor_intel_realsense_d435>
   <!-- Controllers -->
   <xacro:if value="$(arg gazebo_classic)">

File: robots/rbsummit/rbsummit.urdf.xacro (robot description, xacro)
@@ -25,30 +25,14 @@
 	<xacro:property name="top_laser_offset_x" value="-0.01924"/>
 	<xacro:property name="top_laser_offset_y" value="0.0"/>
-	<xacro:property name="top_laser_offset_z" value="0.35642"/>
+	<xacro:property name="top_laser_offset_z" value="0.27642"/>
 	<xacro:property name="front_rgbd_camera_offset_x" value="0.324"/>
 	<xacro:property name="front_rgbd_camera_offset_y" value="0.012"/>
 	<xacro:property name="front_rgbd_camera_offset_z" value="0.172"/>
-	<xacro:property name="front_ptz_camera_offset_x" value="0.22151"/>
-	<xacro:property name="front_ptz_camera_offset_y" value="0.0"/>
-	<xacro:property name="front_ptz_camera_offset_z" value="0.24022"/>
-	<xacro:property name="front_ptz_camera_offset_t" value="-1.308996939"/>
 	<xacro:property name="gps_offset_x" value="-0.22528"/>
 	<xacro:property name="gps_offset_y" value="0.095"/>
-	<xacro:property name="gps_offset_z" value="0.275"/>
-	<!-- Other elements -->
-	<xacro:property name="antenna_offset_x" value="-0.18324"/>
-	<xacro:property name="antenna_offset_y" value="0.0"/>
-	<xacro:property name="antenna_offset_z" value="0.27488"/>
-	<!-- ***************** -->
-	<!-- Global parameters -->
-	<!-- ***************** -->
-	<!-- Second we define all the parameters and arguments to customize the robot characteristics -->
+	<xacro:property name="gps_offset_z" value="0.48"/>
 	<xacro:property name="PI" value="3.1415926535897931"/>
 	<!-- Flag to select the high or low quality model -->
 	<xacro:property name="hq" value="true" />
-	<!-- Launch Arguments -->
-	<xacro:arg name="gpu" default="true" />
-	<xacro:arg name="gps_latitude" default="0"/>
-	<xacro:arg name="gps_longitude" default="0"/>
 	<!-- Here we create the robot using the xacro:macro imported at the beggining of this file -->
 	<xacro:rbsummit prefix="$(arg prefix)" hq="${hq}"/>
@@ -63,4 +47,40 @@
         <origin xyz="${imu_offset_x} ${imu_offset_y} ${imu_offset_z}" rpy="0 0 0"/>
     </xacro:sensor_vectornav>
+	<!-- 3D LIDAR -->
+	<xacro:sensor_robosense_helios_16p
+		frame_prefix="$(arg prefix)top_3d_laser_"
+		parent="$(arg prefix)base_link"
+        node_namespace="$(arg namespace)"
+        node_name="top_lidar"
+        gazebo_classic="$(arg gazebo_classic)"
+        gazebo_ignition="$(arg gazebo_ignition)">
+		<origin
+			xyz="${top_laser_offset_x} ${top_laser_offset_y} ${top_laser_offset_z}"
+			rpy="0 0 0"
+		/>
+	</xacro:sensor_robosense_helios_16p>
+	<!-- CAMERA -->
+    <xacro:sensor_intel_realsense_d435
+        frame_prefix="$(arg prefix)front_rgbd_camera_"
+        parent="$(arg prefix)base_link"
+        node_namespace="$(arg namespace)"
+        node_name="front_camera"
+        gazebo_classic="$(arg gazebo_classic)"
+        gazebo_ignition="$(arg gazebo_ignition)">
+        <origin xyz="${front_rgbd_camera_offset_x} ${front_rgbd_camera_offset_y} ${front_rgbd_camera_offset_z}" rpy="0 0 0"/>
+    </xacro:sensor_intel_realsense_d435>
+	<!-- GPS -->
+	<xacro:sensor_ublox_with_mast
+		frame_prefix="$(arg prefix)gps_"
+		parent="$(arg prefix)base_link"
+		update_rate="5"
+        node_namespace="$(arg namespace)"
+        gazebo_classic="$(arg gazebo_classic)"
+        gazebo_ignition="$(arg gazebo_ignition)">
+		<origin
+			xyz="${gps_offset_x} ${gps_offset_y} ${gps_offset_z}"
+			rpy="0 0 0"
+		/>
+	</xacro:sensor_ublox_with_mast>
 	<!-- Controllers -->
     <xacro:if value="$(arg gazebo_classic)">

Commit message: fix: compat between humble to jazzy

File: robots/rbkairos/rbkairos.urdf.xacro (robot description, xacro)
@@ -30,5 +30,5 @@
   <!-- IMU -->
     <xacro:sensor_vectornav
-        frame_prefix="$(arg prefix)vectornav_"
+        frame_prefix="$(arg prefix)imu_"
         parent="$(arg prefix)base_link"
         node_namespace="$(arg namespace)"

File: robots/rbkairos/rbkairos_plus.urdf.xacro (robot description, xacro)
@@ -36,19 +36,18 @@
   <xacro:rbkairos prefix="$(arg prefix)" gazebo_classic="$(arg gazebo_classic)" gazebo_ignition="$(arg gazebo_ignition)"/>
   <!-- Import UR arm -->
+  <!-- TODO: Restore simulation functionality, removed jazzy -->
   <xacro:ur_robot
+      name="$(arg ur_type)"
       tf_prefix="$(arg prefix)arm_"
-      name="$(arg ur_type)"
       parent="$(arg prefix)top_cover"
       joint_limits_parameters_file="$(arg joint_limit_params)"
       kinematics_parameters_file="$(arg kinematics_params)"
       physical_parameters_file="$(arg physical_params)"
-      visual_parameters_file="$(arg visual_params)"
-      sim_gazebo="$(arg gazebo_classic)"
-      sim_ignition="$(arg gazebo_ignition)">
+      visual_parameters_file="$(arg visual_params)">
       <origin xyz="0 0 0" rpy="0 0 0"/>
   </xacro:ur_robot>
   <!-- IMU -->
     <xacro:sensor_vectornav
-        frame_prefix="$(arg prefix)vectornav_"
+        frame_prefix="$(arg prefix)imu_"
         parent="$(arg prefix)base_link"
         node_namespace="$(arg namespace)"

File: robots/rbrobout/rbrobout.urdf.xacro (robot description, xacro)
@@ -27,5 +27,5 @@
   <!-- IMU -->
     <xacro:sensor_vectornav
-        frame_prefix="$(arg prefix)vectornav_"
+        frame_prefix="$(arg prefix)imu_"
         parent="$(arg prefix)base_link"
         node_namespace="$(arg namespace)"

File: robots/rbrobout/rbrobout_plus.urdf.xacro (robot description, xacro)
@@ -45,19 +45,19 @@
       <origin xyz="${lift_position_x} 0 ${lift_position_z}" rpy="0 0 0"/>
   </xacro:ewellix_lift_900mm>
+  <!-- Import UR arm -->
+  <!-- TODO: Restore simulation functionality, removed jazzy -->
   <xacro:ur_robot
+      name="$(arg ur_type)"
       tf_prefix="$(arg prefix)arm_"
-      name="$(arg ur_type)"
       parent="$(arg prefix)lift_ewellix_lift_top_link"
       joint_limits_parameters_file="$(arg joint_limit_params)"
       kinematics_parameters_file="$(arg kinematics_params)"
       physical_parameters_file="$(arg physical_params)"
-      visual_parameters_file="$(arg visual_params)"
-      sim_gazebo="$(arg gazebo_classic)"
-      sim_ignition="$(arg gazebo_ignition)">
+      visual_parameters_file="$(arg visual_params)">
       <origin xyz="0 0 0" rpy="0 0 0"/>
   </xacro:ur_robot>
   <!-- IMU -->
     <xacro:sensor_vectornav
-        frame_prefix="$(arg prefix)vectornav_"
+        frame_prefix="$(arg prefix)imu_"
         parent="$(arg prefix)base_link"
         node_namespace="$(arg namespace)"

File: robots/rbsummit/rbsummit.urdf.xacro (robot description, xacro)
@@ -40,5 +40,5 @@
 	<!-- IMU -->
     <xacro:sensor_vectornav
-        frame_prefix="$(arg prefix)vectornav_"
+        frame_prefix="$(arg prefix)imu_"
         parent="$(arg prefix)base_link"
         node_namespace="$(arg namespace)"

File: robots/rbtheron/rbtheron.urdf.xacro (robot description, xacro)
@@ -35,17 +35,15 @@
 	<xacro:property name="rear_rgbd_camera_offset_x" value="-0.3045"/>
 	<xacro:property name="rear_rgbd_camera_offset_y" value="0.0"/>
-	<xacro:property name="rear_rgbd_camera_offset_z" value="0.1598"/>
-	<xacro:property name="front_laser_offset_x" value="0.268"/>
+	<!-- rear camera offset_z rb_theron chassis type v3: 0.1598 v4 (default): 0.1158 -->
+	<xacro:property name="rear_rgbd_camera_offset_z" value="0.1158"/>
+	<xacro:property name="front_laser_offset_x" value="0.2675"/>
 	<xacro:property name="front_laser_offset_y" value="-0.215"/>
 	<xacro:property name="front_laser_offset_z" value="0.1613"/>
-	<xacro:property name="rear_laser_offset_x" value="-0.268"/>
+	<xacro:property name="rear_laser_offset_x" value="-0.2675"/>
 	<xacro:property name="rear_laser_offset_y" value="0.215"/>
 	<xacro:property name="rear_laser_offset_z" value="0.1613"/>
-	<xacro:property name="top_lidar_offset_x" value="0.26"/>
-	<xacro:property name="top_lidar_offset_y" value="0.0"/>
-	<xacro:property name="top_lidar_offset_z" value="0.51"/>
 	<!-- IMU -->
     <xacro:sensor_vectornav
-        frame_prefix="$(arg prefix)vectornav_"
+        frame_prefix="$(arg prefix)imu_"
         parent="$(arg prefix)base_link"
         node_namespace="$(arg namespace)"

File: robots/rbtheron/rbtheron_plus.urdf.xacro (robot description, xacro)
@@ -57,14 +57,13 @@
     </link>
     <!-- Import UR arm -->
+    <!-- TODO: Restore simulation functionality, removed jazzy -->
     <xacro:ur_robot
+        name="$(arg ur_type)"
         tf_prefix="$(arg prefix)arm_"
-        name="$(arg ur_type)"
         parent="$(arg prefix)top_chassis"
         joint_limits_parameters_file="$(arg joint_limit_params)"
         kinematics_parameters_file="$(arg kinematics_params)"
         physical_parameters_file="$(arg physical_params)"
-        visual_parameters_file="$(arg visual_params)"
-        sim_gazebo="$(arg gazebo_classic)"
-        sim_ignition="$(arg gazebo_ignition)">
+        visual_parameters_file="$(arg visual_params)">
         <origin xyz="-0.2 0 0.6" rpy="0 0 0"/>
     </xacro:ur_robot>
@@ -78,5 +77,6 @@
 	<xacro:property name="rear_rgbd_camera_offset_x" value="-0.3045"/>
 	<xacro:property name="rear_rgbd_camera_offset_y" value="0.0"/>
-	<xacro:property name="rear_rgbd_camera_offset_z" value="0.1598"/>
+	<!-- rear camera offset_z rb_theron chassis type v3: 0.1598 v4 (default): 0.1158 -->
+	<xacro:property name="rear_rgbd_camera_offset_z" value="0.1158"/>
 	<xacro:property name="front_laser_offset_x" value="0.2675"/>
 	<xacro:property name="front_laser_offset_y" value="-0.215"/>
@@ -90,5 +90,5 @@
 	<!-- IMU -->
     <xacro:sensor_vectornav
-        frame_prefix="$(arg prefix)vectornav_"
+        frame_prefix="$(arg prefix)imu_"
         parent="$(arg prefix)base_link"
         node_namespace="$(arg namespace)"
@@ -137,5 +137,5 @@
     <!-- 3D LiDAR -->
     <joint name="$(arg prefix)top_lidar_aux_joint" type="fixed">
-        <origin xyz="${top_lidar_offset_x} ${top_lidar_offset_y} ${top_lidar_offset_z}" rpy="0 ${PI/2}  0"/>
+        <origin xyz="${top_lidar_offset_x} ${top_lidar_offset_y} ${top_lidar_offset_z}" rpy="0 ${PI/2} 0"/>
         <parent link="$(arg prefix)top_chassis"/>
         <child link="$(arg prefix)top_lidar_aux"/>
@@ -149,5 +149,5 @@
         gazebo_classic="$(arg gazebo_classic)"
         gazebo_ignition="$(arg gazebo_ignition)">
-        <origin xyz="${top_lidar_offset_x} ${top_lidar_offset_y} ${top_lidar_offset_z}" rpy="0 ${PI/2} 0"/>
+        <origin xyz="0 0 0" rpy="0 0 ${PI/3}"/>
     </xacro:sensor_robosense_bpearl>
 	<!-- Controllers -->

File: robots/rbvogui/rbvogui.urdf.xacro (robot description, xacro)
@@ -5,18 +5,12 @@
     <!-- Imported elements -->
     <!-- ***************** -->
-    <!-- First we import all posible elements defined in the urdf.xacro files. All these elements
-    are defined as macro:xacros -->
+    <!-- First we import all posible elements defined in the urdf.xacro files. All these elements are defined as macro:xacros -->
     <!-- Import rbvogui base elements-->
-    <xacro:include
-        filename="$(find robotnik_description)/urdf/bases/rbvogui/rbvogui_base.urdf.xacro" />
+    <xacro:include filename="$(find robotnik_description)/urdf/bases/rbvogui/rbvogui_base.urdf.xacro" />
     <xacro:include filename="$(find robotnik_description)/urdf/base_hw/rbvogui.ros2_control.urdf" />
-    <xacro:include
-        filename="$(find robotnik_description)/simulators/gazebo_classic/rbvogui/rbvogui_control.urdf.xacro" />
-    <xacro:include
-        filename="$(find robotnik_description)/simulators/gazebo_ignition/rbvogui/rbvogui_control.urdf.xacro" />
+    <xacro:include filename="$(find robotnik_description)/simulators/gazebo_classic/rbvogui/rbvogui_control.urdf.xacro" />
+    <xacro:include filename="$(find robotnik_description)/simulators/gazebo_ignition/rbvogui/rbvogui_control.urdf.xacro" />
     <!-- Import all available sensors -->
     <xacro:include filename="$(find robotnik_sensors)/urdf/all_sensors.urdf.xacro" />
-    <!-- Flag to select the high or low quality model -->
-    <xacro:property name="hq" value="true" />
     <xacro:property name="front_laser_offset_x" value="0.53" />
     <xacro:property name="front_laser_offset_y" value="0.33" />
@@ -34,15 +28,17 @@
     <xacro:property name="rear_rgbd_camera_offset_y" value="0.0" />
     <xacro:property name="rear_rgbd_camera_offset_z" value="0.29" />
+    <!-- Flag to select the high or low quality model -->
+    <xacro:property name="hq" value="true" />
     <!-- Launch Arguments -->
-    <xacro:arg name="namespace" default="robot" />
-    <xacro:arg name="prefix" default="robot_" />
-    <xacro:arg name="gazebo_classic" default="false" />
-    <xacro:arg name="gazebo_ignition" default="false" />
+	<xacro:arg name="namespace" default="robot"/>
+	<xacro:arg name="prefix" default="robot_"/>
+	<xacro:arg name="gazebo_classic" default="false"/>
+	<xacro:arg name="gazebo_ignition" default="false"/>
     <xacro:rbvogui prefix="$(arg prefix)" hq="${hq}" />
     <!-- SENSORS see robotnik_sensors for the specific configuration -->
     <!-- IMU -->
     <xacro:sensor_vectornav
-        frame_prefix="$(arg prefix)vectornav_"
-        parent="$(arg prefix)base_link"
+        frame_prefix="$(arg prefix)imu_"
+        parent="$(arg prefix)chassis_link"
         node_namespace="$(arg namespace)"
         gazebo_classic="$(arg gazebo_classic)"
@@ -50,25 +46,4 @@
         <origin xyz="${imu_offset_x} ${imu_offset_y} ${imu_offset_z}" rpy="0 0 0" />
     </xacro:sensor_vectornav>
-    <!-- LASERS -->
-    <xacro:sensor_sick_s300
-        frame_prefix="$(arg prefix)front_laser_"
-        parent="$(arg prefix)base_link"
-        node_namespace="$(arg namespace)"
-        node_name="front_laser"
-        gazebo_classic="$(arg gazebo_classic)"
-        gazebo_ignition="$(arg gazebo_ignition)">
-        <origin xyz="${front_laser_offset_x} ${front_laser_offset_y} ${front_laser_offset_z}"
-            rpy="0 ${-PI} ${-3/4*PI}" />
-    </xacro:sensor_sick_s300>
-    <xacro:sensor_sick_s300
-        frame_prefix="$(arg prefix)rear_laser_"
-        parent="$(arg prefix)base_link"
-        node_namespace="$(arg namespace)"
-        node_name="rear_laser"
-        gazebo_classic="$(arg gazebo_classic)"
-        gazebo_ignition="$(arg gazebo_ignition)">
-        <origin xyz="${rear_laser_offset_x} ${rear_laser_offset_y} ${rear_laser_offset_z}"
-            rpy="0 ${-PI} ${1/4*PI}" />
-    </xacro:sensor_sick_s300>
     <!-- Front Camera -->
     <xacro:sensor_intel_realsense_d435
@@ -79,7 +54,5 @@
         gazebo_classic="$(arg gazebo_classic)"
         gazebo_ignition="$(arg gazebo_ignition)">
-        <origin
-            xyz="${front_rgbd_camera_offset_x} ${front_rgbd_camera_offset_y} ${front_rgbd_camera_offset_z}"
-            rpy="0 0 0" />
+        <origin xyz="${front_rgbd_camera_offset_x} ${front_rgbd_camera_offset_y} ${front_rgbd_camera_offset_z}" rpy="0 0 0"/>
     </xacro:sensor_intel_realsense_d435>
     <!-- Rear Camera -->
@@ -91,8 +64,25 @@
         gazebo_classic="$(arg gazebo_classic)"
         gazebo_ignition="$(arg gazebo_ignition)">
-        <origin
-            xyz="${rear_rgbd_camera_offset_x} ${rear_rgbd_camera_offset_y} ${rear_rgbd_camera_offset_z}"
-            rpy="0 0 -${PI}" />
+        <origin xyz="${rear_rgbd_camera_offset_x} ${rear_rgbd_camera_offset_y} ${rear_rgbd_camera_offset_z}" rpy="0 0 -${PI}" />
     </xacro:sensor_intel_realsense_d435>
+    <!-- LASERS -->
+    <xacro:sensor_sick_s300
+        frame_prefix="$(arg prefix)front_laser_"
+        parent="$(arg prefix)chassis_link"
+        node_namespace="$(arg namespace)"
+        node_name="front_laser"
+        gazebo_classic="$(arg gazebo_classic)"
+        gazebo_ignition="$(arg gazebo_ignition)">
+        <origin xyz="${front_laser_offset_x} ${front_laser_offset_y} ${front_laser_offset_z}" rpy="0 ${-PI} ${-3/4*PI}" />
+    </xacro:sensor_sick_s300>
+    <xacro:sensor_sick_s300
+        frame_prefix="$(arg prefix)rear_laser_"
+        parent="$(arg prefix)chassis_link"
+        node_namespace="$(arg namespace)"
+        node_name="rear_laser"
+        gazebo_classic="$(arg gazebo_classic)"
+        gazebo_ignition="$(arg gazebo_ignition)">
+        <origin xyz="${rear_laser_offset_x} ${rear_laser_offset_y} ${rear_laser_offset_z}" rpy="0 ${-PI} ${1/4*PI}" />
+    </xacro:sensor_sick_s300>
     <!-- Controllers -->
     <xacro:if value="$(arg gazebo_classic)">

File: robots/rbvogui/rbvogui_plus.urdf.xacro (robot description, xacro)
@@ -42,18 +42,17 @@
     <xacro:property name="rear_rgbd_camera_offset_z" value="0.29" />
     <!-- Import UR arm -->
+    <!-- TODO: Restore simulation functionality, removed jazzy -->
     <xacro:ur_robot
+        name="$(arg ur_type)"
         tf_prefix="$(arg prefix)arm_"
-        name="$(arg ur_type)"
         parent="$(arg prefix)chassis_link"
         joint_limits_parameters_file="$(arg joint_limit_params)"
         kinematics_parameters_file="$(arg kinematics_params)"
         physical_parameters_file="$(arg physical_params)"
-        visual_parameters_file="$(arg visual_params)"
-        sim_gazebo="$(arg gazebo_classic)"
-        sim_ignition="$(arg gazebo_ignition)">
+        visual_parameters_file="$(arg visual_params)">
         <origin xyz="0 0 0.235" rpy="0 0 0"/>
     </xacro:ur_robot>
     <xacro:sensor_vectornav
-        frame_prefix="$(arg prefix)vectornav_"
+        frame_prefix="$(arg prefix)imu_"
         parent="$(arg prefix)chassis_link"
         node_namespace="$(arg namespace)"
@@ -65,5 +64,5 @@
     <xacro:sensor_intel_realsense_d435
         frame_prefix="$(arg prefix)front_rgbd_camera_"
-        parent="$(arg prefix)base_link"
+        parent="$(arg prefix)chassis_link"
         node_namespace="$(arg namespace)"
         node_name="front_camera"
@@ -75,32 +74,28 @@
     <xacro:sensor_intel_realsense_d435
         frame_prefix="$(arg prefix)rear_rgbd_camera_"
-        parent="$(arg prefix)base_link"
+        parent="$(arg prefix)chassis_link"
         node_namespace="$(arg namespace)"
         node_name="rear_camera"
         gazebo_classic="$(arg gazebo_classic)"
         gazebo_ignition="$(arg gazebo_ignition)">
-        <origin
-            xyz="${rear_rgbd_camera_offset_x} ${rear_rgbd_camera_offset_y} ${rear_rgbd_camera_offset_z}"
-            rpy="0 0 -${PI}" />
+        <origin xyz="${rear_rgbd_camera_offset_x} ${rear_rgbd_camera_offset_y} ${rear_rgbd_camera_offset_z}" rpy="0 0 -${PI}" />
     </xacro:sensor_intel_realsense_d435>
     <xacro:sensor_sick_s300
         frame_prefix="$(arg prefix)front_laser_"
-        parent="$(arg prefix)base_link"
+        parent="$(arg prefix)chassis_link"
         node_namespace="$(arg namespace)"
         node_name="front_laser"
         gazebo_classic="$(arg gazebo_classic)"
         gazebo_ignition="$(arg gazebo_ignition)">
-        <origin xyz="${front_laser_offset_x} ${front_laser_offset_y} ${front_laser_offset_z}"
-            rpy="0 ${-PI} ${-3/4*PI}" />
+        <origin xyz="${front_laser_offset_x} ${front_laser_offset_y} ${front_laser_offset_z}" rpy="0 ${-PI} ${-3/4*PI}" />
     </xacro:sensor_sick_s300>
     <xacro:sensor_sick_s300
         frame_prefix="$(arg prefix)rear_laser_"
-        parent="$(arg prefix)base_link"
+        parent="$(arg prefix)chassis_link"
         node_namespace="$(arg namespace)"
         node_name="rear_laser"
         gazebo_classic="$(arg gazebo_classic)"
         gazebo_ignition="$(arg gazebo_ignition)">
-        <origin xyz="${rear_laser_offset_x} ${rear_laser_offset_y} ${rear_laser_offset_z}"
-            rpy="0 ${-PI} ${1/4*PI}" />
+        <origin xyz="${rear_laser_offset_x} ${rear_laser_offset_y} ${rear_laser_offset_z}" rpy="0 ${-PI} ${1/4*PI}" />
     </xacro:sensor_sick_s300>
 	<!-- Controllers -->
