Commit message: sync to prefix instead of frame_prefix

File: robots/rbkairos/rbkairos.urdf.xacro (robot description, xacro)
@@ -12,5 +12,5 @@
   <!-- Properties and Arguments -->
   <xacro:arg name="namespace" default="robot"/>
-  <xacro:arg name="frame_prefix" default=""/>
+  <xacro:arg name="prefix" default=""/>
   <xacro:arg name="gazebo_classic" default="false"/>
   <xacro:arg name="gazebo_ignition" default="false"/>
@@ -27,9 +27,9 @@
   <xacro:property name="front_rgbd_camera_offset_y" value="0.0"/>
   <xacro:property name="front_rgbd_camera_offset_z" value="0.25062"/>
-  <xacro:rbkairos prefix="$(arg frame_prefix)" gazebo_classic="$(arg gazebo_classic)" gazebo_ignition="$(arg gazebo_ignition)"/>
+  <xacro:rbkairos prefix="$(arg prefix)" gazebo_classic="$(arg gazebo_classic)" gazebo_ignition="$(arg gazebo_ignition)"/>
   <!-- IMU -->
     <xacro:sensor_vectornav
-        frame_prefix="$(arg frame_prefix)imu_"
-        parent="$(arg frame_prefix)base_link"
+        frame_prefix="$(arg prefix)imu_"
+        parent="$(arg prefix)base_link"
         node_namespace="$(arg namespace)"
         gazebo_classic="$(arg gazebo_classic)"
@@ -39,6 +39,6 @@
   <!-- SENSORS -->
     <xacro:sensor_sick_s300
-        frame_prefix="$(arg frame_prefix)front_laser_"
-        parent="$(arg frame_prefix)base_link"
+        frame_prefix="$(arg prefix)front_laser_"
+        parent="$(arg prefix)base_link"
         node_namespace="$(arg namespace)"
         node_name="front_laser"
@@ -48,6 +48,6 @@
     </xacro:sensor_sick_s300>
     <xacro:sensor_sick_s300
-        frame_prefix="$(arg frame_prefix)rear_laser_"
-        parent="$(arg frame_prefix)base_link"
+        frame_prefix="$(arg prefix)rear_laser_"
+        parent="$(arg prefix)base_link"
         node_namespace="$(arg namespace)"
         node_name="rear_laser"
@@ -58,6 +58,6 @@
   <!-- CAMERA -->
     <xacro:sensor_intel_realsense_d435
-        frame_prefix="$(arg frame_prefix)front_rgbd_camera_"
-        parent="$(arg frame_prefix)base_link"
+        frame_prefix="$(arg prefix)front_rgbd_camera_"
+        parent="$(arg prefix)base_link"
         node_namespace="$(arg namespace)"
         node_name="front_camera"
@@ -68,9 +68,9 @@
   <!-- Controllers -->
   <xacro:if value="$(arg gazebo_classic)">
-    <xacro:rbkairos_gz_classic_control namespace="$(arg namespace)" prefix="$(arg frame_prefix)"/>
+    <xacro:rbkairos_gz_classic_control namespace="$(arg namespace)" prefix="$(arg prefix)"/>
     <xacro:ros_planar_move_gazebo_classic/>
   </xacro:if>
   <xacro:if value="$(arg gazebo_ignition)">
-    <xacro:rbkairos_gz_ignition_control namespace="$(arg namespace)" prefix="$(arg frame_prefix)"/>
+    <xacro:rbkairos_gz_ignition_control namespace="$(arg namespace)" prefix="$(arg prefix)"/>
   </xacro:if>
   <xacro:unless value="$(arg gazebo_classic)">

File: robots/rbkairos/rbkairos_plus.urdf.xacro (robot description, xacro)
@@ -13,5 +13,5 @@
   <!-- Properties and Arguments -->
   <xacro:arg name="namespace" default="robot"/>
-  <xacro:arg name="frame_prefix" default=""/>
+  <xacro:arg name="prefix" default=""/>
   <xacro:arg name="gazebo_classic" default="false"/>
   <xacro:arg name="gazebo_ignition" default="false"/>
@@ -34,11 +34,11 @@
   <xacro:property name="front_rgbd_camera_offset_z" value="0.25062"/>
   <!-- Kairos -->
-  <xacro:rbkairos prefix="$(arg frame_prefix)" gazebo_classic="$(arg gazebo_classic)" gazebo_ignition="$(arg gazebo_ignition)"/>
+  <xacro:rbkairos prefix="$(arg prefix)" gazebo_classic="$(arg gazebo_classic)" gazebo_ignition="$(arg gazebo_ignition)"/>
   <!-- Import UR arm -->
   <!-- TODO: Restore simulation functionality, removed jazzy -->
   <xacro:ur_robot
       name="$(arg ur_type)"
-      tf_prefix="$(arg frame_prefix)arm_"
-      parent="$(arg frame_prefix)top_cover"
+      tf_prefix="$(arg prefix)arm_"
+      parent="$(arg prefix)top_cover"
       joint_limits_parameters_file="$(arg joint_limit_params)"
       kinematics_parameters_file="$(arg kinematics_params)"
@@ -49,6 +49,6 @@
   <!-- IMU -->
     <xacro:sensor_vectornav
-        frame_prefix="$(arg frame_prefix)imu_"
-        parent="$(arg frame_prefix)base_link"
+        frame_prefix="$(arg prefix)imu_"
+        parent="$(arg prefix)base_link"
         node_namespace="$(arg namespace)"
         gazebo_classic="$(arg gazebo_classic)"
@@ -58,6 +58,6 @@
   <!-- SENSORS -->
     <xacro:sensor_sick_s300
-        frame_prefix="$(arg frame_prefix)front_laser_"
-        parent="$(arg frame_prefix)base_link"
+        frame_prefix="$(arg prefix)front_laser_"
+        parent="$(arg prefix)base_link"
         node_namespace="$(arg namespace)"
         node_name="front_laser"
@@ -67,6 +67,6 @@
     </xacro:sensor_sick_s300>
     <xacro:sensor_sick_s300
-        frame_prefix="$(arg frame_prefix)rear_laser_"
-        parent="$(arg frame_prefix)base_link"
+        frame_prefix="$(arg prefix)rear_laser_"
+        parent="$(arg prefix)base_link"
         node_namespace="$(arg namespace)"
         node_name="rear_laser"
@@ -77,6 +77,6 @@
   <!-- CAMERA -->
     <xacro:sensor_intel_realsense_d435
-        frame_prefix="$(arg frame_prefix)front_rgbd_camera_"
-        parent="$(arg frame_prefix)base_link"
+        frame_prefix="$(arg prefix)front_rgbd_camera_"
+        parent="$(arg prefix)base_link"
         node_namespace="$(arg namespace)"
         node_name="front_camera"
@@ -87,9 +87,9 @@
   <!-- Controllers -->
   <xacro:if value="$(arg gazebo_classic)">
-    <xacro:rbkairos_gz_classic_control namespace="$(arg namespace)" prefix="$(arg frame_prefix)"/>
+    <xacro:rbkairos_gz_classic_control namespace="$(arg namespace)" prefix="$(arg prefix)"/>
     <xacro:ros_planar_move_gazebo_classic/>
   </xacro:if>
   <xacro:if value="$(arg gazebo_ignition)">
-    <xacro:rbkairos_gz_ignition_control namespace="$(arg namespace)" prefix="$(arg frame_prefix)"/>
+    <xacro:rbkairos_gz_ignition_control namespace="$(arg namespace)" prefix="$(arg prefix)"/>
   </xacro:if>
   <xacro:unless value="$(arg gazebo_classic)">

File: robots/rbrobout/rbrobout.urdf.xacro (robot description, xacro)
@@ -12,5 +12,5 @@
   <!-- Properties and Arguments -->
   <xacro:arg name="namespace" default="robot"/>
-  <xacro:arg name="frame_prefix" default=""/>
+  <xacro:arg name="prefix" default=""/>
   <xacro:arg name="gazebo_classic" default="false"/>
   <xacro:arg name="gazebo_ignition" default="false"/>
@@ -24,9 +24,9 @@
   <xacro:property name="imu_offset_y" value="-0.3"/>
   <xacro:property name="imu_offset_z" value="0.0725"/>
-  <xacro:rbrobout prefix="$(arg frame_prefix)" gazebo_classic="$(arg gazebo_classic)" gazebo_ignition="$(arg gazebo_ignition)"/>
+  <xacro:rbrobout prefix="$(arg prefix)" gazebo_classic="$(arg gazebo_classic)" gazebo_ignition="$(arg gazebo_ignition)"/>
   <!-- IMU -->
     <xacro:sensor_vectornav
-        frame_prefix="$(arg frame_prefix)imu_"
-        parent="$(arg frame_prefix)base_link"
+        frame_prefix="$(arg prefix)imu_"
+        parent="$(arg prefix)base_link"
         node_namespace="$(arg namespace)"
         gazebo_classic="$(arg gazebo_classic)"
@@ -36,6 +36,6 @@
   <!-- 2d laser -->
     <xacro:sensor_sick_microscan3
-        frame_prefix="$(arg frame_prefix)front_laser_"
-        parent="$(arg frame_prefix)base_link"
+        frame_prefix="$(arg prefix)front_laser_"
+        parent="$(arg prefix)base_link"
         node_namespace="$(arg namespace)"
         node_name="front_laser"
@@ -46,6 +46,6 @@
     <!-- 2d laser -->
     <xacro:sensor_sick_microscan3
-        frame_prefix="$(arg frame_prefix)rear_laser_"
-        parent="$(arg frame_prefix)base_link"
+        frame_prefix="$(arg prefix)rear_laser_"
+        parent="$(arg prefix)base_link"
         node_namespace="$(arg namespace)"
         node_name="rear_laser"
@@ -56,9 +56,9 @@
     <!-- Controllers -->
     <xacro:if value="$(arg gazebo_classic)">
-        <xacro:rbrobout_gz_classic_control namespace="$(arg namespace)" prefix="$(arg frame_prefix)"/>
+        <xacro:rbrobout_gz_classic_control namespace="$(arg namespace)" prefix="$(arg prefix)"/>
         <xacro:ros_planar_move_gazebo_classic/>
     </xacro:if>
     <xacro:if value="$(arg gazebo_ignition)">
-        <xacro:rbrobout_gz_ignition_control namespace="$(arg namespace)" prefix="$(arg frame_prefix)"/>
+        <xacro:rbrobout_gz_ignition_control namespace="$(arg namespace)" prefix="$(arg prefix)"/>
     </xacro:if>
     <xacro:unless value="$(arg gazebo_classic)">

File: robots/rbrobout/rbrobout_plus.urdf.xacro (robot description, xacro)
@@ -15,5 +15,5 @@
   <!-- Properties and Arguments -->
   <xacro:arg name="namespace" default="robot"/>
-  <xacro:arg name="frame_prefix" default=""/>
+  <xacro:arg name="prefix" default=""/>
   <xacro:arg name="gazebo_classic" default="false"/>
   <xacro:arg name="gazebo_ignition" default="false"/>
@@ -38,9 +38,9 @@
   <xacro:property name="lift_orientation_p" value="0"/>
   <xacro:property name="lift_orientation_y" value="0"/>
-  <xacro:rbrobout prefix="$(arg frame_prefix)"  gazebo_classic="$(arg gazebo_classic)" gazebo_ignition="$(arg gazebo_ignition)"/>
-  <xacro:top_cover prefix="$(arg frame_prefix)" parent="$(arg frame_prefix)base_link">
+  <xacro:rbrobout prefix="$(arg prefix)"  gazebo_classic="$(arg gazebo_classic)" gazebo_ignition="$(arg gazebo_ignition)"/>
+  <xacro:top_cover prefix="$(arg prefix)" parent="$(arg prefix)base_link">
       <origin xyz="0 0 -0.1" rpy="0 0 0"/>
   </xacro:top_cover>
-  <xacro:ewellix_lift_900mm prefix="$(arg frame_prefix)lift_" parent="$(arg frame_prefix)base_link">
+  <xacro:ewellix_lift_900mm prefix="$(arg prefix)lift_" parent="$(arg prefix)base_link">
       <origin xyz="${lift_position_x} 0 ${lift_position_z}" rpy="0 0 0"/>
   </xacro:ewellix_lift_900mm>
@@ -49,6 +49,6 @@
   <xacro:ur_robot
       name="$(arg ur_type)"
-      tf_prefix="$(arg frame_prefix)arm_"
-      parent="$(arg frame_prefix)lift_ewellix_lift_top_link"
+      tf_prefix="$(arg prefix)arm_"
+      parent="$(arg prefix)lift_ewellix_lift_top_link"
       joint_limits_parameters_file="$(arg joint_limit_params)"
       kinematics_parameters_file="$(arg kinematics_params)"
@@ -59,6 +59,6 @@
   <!-- IMU -->
     <xacro:sensor_vectornav
-        frame_prefix="$(arg frame_prefix)imu_"
-        parent="$(arg frame_prefix)base_link"
+        frame_prefix="$(arg prefix)imu_"
+        parent="$(arg prefix)base_link"
         node_namespace="$(arg namespace)"
         gazebo_classic="$(arg gazebo_classic)"
@@ -68,6 +68,6 @@
     <!-- 2d laser -->
     <xacro:sensor_sick_microscan3
-        frame_prefix="$(arg frame_prefix)front_laser_"
-        parent="$(arg frame_prefix)base_link"
+        frame_prefix="$(arg prefix)front_laser_"
+        parent="$(arg prefix)base_link"
         node_namespace="$(arg namespace)"
         node_name="front_laser"
@@ -78,6 +78,6 @@
     <!-- 2d laser -->
     <xacro:sensor_sick_microscan3
-        frame_prefix="$(arg frame_prefix)rear_laser_"
-        parent="$(arg frame_prefix)base_link"
+        frame_prefix="$(arg prefix)rear_laser_"
+        parent="$(arg prefix)base_link"
         node_namespace="$(arg namespace)"
         node_name="rear_laser"
@@ -88,9 +88,9 @@
     <!-- Controllers -->
     <xacro:if value="$(arg gazebo_classic)">
-        <xacro:rbrobout_gz_classic_control namespace="$(arg namespace)" prefix="$(arg frame_prefix)"/>
+        <xacro:rbrobout_gz_classic_control namespace="$(arg namespace)" prefix="$(arg prefix)"/>
         <xacro:ros_planar_move_gazebo_classic/>
     </xacro:if>
     <xacro:if value="$(arg gazebo_ignition)">
-        <xacro:rbrobout_gz_ignition_control namespace="$(arg namespace)" prefix="$(arg frame_prefix)"/>
+        <xacro:rbrobout_gz_ignition_control namespace="$(arg namespace)" prefix="$(arg prefix)"/>
     </xacro:if>
     <xacro:unless value="$(arg gazebo_classic)">

File: robots/rbsummit/rbsummit.urdf.xacro (robot description, xacro)
@@ -17,5 +17,5 @@
 	<!-- x,y,z in translation from base_link to the center of the sensor -->
 	<xacro:arg name="namespace" default="robot"/>
-	<xacro:arg name="frame_prefix" default=""/>
+	<xacro:arg name="prefix" default=""/>
 	<xacro:arg name="gazebo_classic" default="false"/>
 	<xacro:arg name="gazebo_ignition" default="false"/>
@@ -36,10 +36,10 @@
 	<xacro:property name="hq" value="true" />
 	<!-- Here we create the robot using the xacro:macro imported at the beggining of this file -->
-	<xacro:rbsummit prefix="$(arg frame_prefix)" hq="${hq}"/>
+	<xacro:rbsummit prefix="$(arg prefix)" hq="${hq}"/>
 	<!-- Custom Sensors -->
 	<!-- IMU -->
     <xacro:sensor_vectornav
-        frame_prefix="$(arg frame_prefix)imu_"
-        parent="$(arg frame_prefix)base_link"
+        frame_prefix="$(arg prefix)imu_"
+        parent="$(arg prefix)base_link"
         node_namespace="$(arg namespace)"
         gazebo_classic="$(arg gazebo_classic)"
@@ -49,6 +49,6 @@
 	<!-- 3D LIDAR -->
 	<xacro:sensor_robosense_helios_16p
-		frame_prefix="$(arg frame_prefix)top_3d_laser_"
-		parent="$(arg frame_prefix)base_link"
+		frame_prefix="$(arg prefix)top_3d_laser_"
+		parent="$(arg prefix)base_link"
         node_namespace="$(arg namespace)"
         node_name="top_lidar"
@@ -62,6 +62,6 @@
 	<!-- CAMERA -->
     <xacro:sensor_intel_realsense_d435
-        frame_prefix="$(arg frame_prefix)front_rgbd_camera_"
-        parent="$(arg frame_prefix)base_link"
+        frame_prefix="$(arg prefix)front_rgbd_camera_"
+        parent="$(arg prefix)base_link"
         node_namespace="$(arg namespace)"
         node_name="front_camera"
@@ -72,6 +72,6 @@
 	<!-- GPS -->
 	<xacro:sensor_ublox_with_mast
-		frame_prefix="$(arg frame_prefix)gps_"
-		parent="$(arg frame_prefix)base_link"
+		frame_prefix="$(arg prefix)gps_"
+		parent="$(arg prefix)base_link"
 		update_rate="5"
         node_namespace="$(arg namespace)"
@@ -85,9 +85,9 @@
 	<!-- Controllers -->
     <xacro:if value="$(arg gazebo_classic)">
-      <xacro:rbsummit_gz_classic_control namespace="$(arg namespace)" prefix="$(arg frame_prefix)"/>
+      <xacro:rbsummit_gz_classic_control namespace="$(arg namespace)" prefix="$(arg prefix)"/>
         <xacro:ros_planar_move_gazebo_classic/>
     </xacro:if>
     <xacro:if value="$(arg gazebo_ignition)">
-      <xacro:rbsummit_gz_ignition_control namespace="$(arg namespace)" prefix="$(arg frame_prefix)"/>
+      <xacro:rbsummit_gz_ignition_control namespace="$(arg namespace)" prefix="$(arg prefix)"/>
     </xacro:if>
     <xacro:unless value="$(arg gazebo_classic)">

File: robots/rbtheron/rbtheron.urdf.xacro (robot description, xacro)
@@ -21,9 +21,9 @@
 	<xacro:property name="hq" value="true" />
 	<xacro:arg name="namespace" default="robot"/>
-	<xacro:arg name="frame_prefix" default=""/>
+	<xacro:arg name="prefix" default=""/>
 	<xacro:arg name="gazebo_classic" default="false"/>
 	<xacro:arg name="gazebo_ignition" default="false"/>
 	<!-- Here we create the robot using the xacro:macro imported at the beggining of this file -->
-	<xacro:rbtheron prefix="$(arg frame_prefix)" hq="${hq}"/>
+	<xacro:rbtheron prefix="$(arg prefix)" hq="${hq}"/>
 	<!-- SENSORS -->
     <xacro:property name="imu_offset_x" value="-0.1975"/>
@@ -45,6 +45,6 @@
 	<!-- IMU -->
     <xacro:sensor_vectornav
-        frame_prefix="$(arg frame_prefix)imu_"
-        parent="$(arg frame_prefix)base_link"
+        frame_prefix="$(arg prefix)imu_"
+        parent="$(arg prefix)base_link"
         node_namespace="$(arg namespace)"
         gazebo_classic="$(arg gazebo_classic)"
@@ -54,6 +54,6 @@
 	<!-- 2D LASER -->
     <xacro:sensor_hokuyo_ust20lx
-        frame_prefix="$(arg frame_prefix)front_laser_"
-        parent="$(arg frame_prefix)base_link"
+        frame_prefix="$(arg prefix)front_laser_"
+        parent="$(arg prefix)base_link"
         node_namespace="$(arg namespace)"
         node_name="front_laser"
@@ -63,6 +63,6 @@
     </xacro:sensor_hokuyo_ust20lx>
     <xacro:sensor_hokuyo_ust20lx
-        frame_prefix="$(arg frame_prefix)rear_laser_"
-        parent="$(arg frame_prefix)base_link"
+        frame_prefix="$(arg prefix)rear_laser_"
+        parent="$(arg prefix)base_link"
         node_namespace="$(arg namespace)"
         node_name="rear_laser"
@@ -73,6 +73,6 @@
   	<!-- CAMERAS -->
     <xacro:sensor_intel_realsense_d435
-        frame_prefix="$(arg frame_prefix)front_rgbd_camera_"
-        parent="$(arg frame_prefix)base_link"
+        frame_prefix="$(arg prefix)front_rgbd_camera_"
+        parent="$(arg prefix)base_link"
         node_namespace="$(arg namespace)"
         node_name="front_camera"
@@ -82,6 +82,6 @@
     </xacro:sensor_intel_realsense_d435>
     <xacro:sensor_intel_realsense_d435
-        frame_prefix="$(arg frame_prefix)rear_rgbd_camera_"
-        parent="$(arg frame_prefix)base_link"
+        frame_prefix="$(arg prefix)rear_rgbd_camera_"
+        parent="$(arg prefix)base_link"
         node_namespace="$(arg namespace)"
         node_name="rear_camera"
@@ -92,9 +92,9 @@
 	<!-- Controllers -->
 	<xacro:if value="$(arg gazebo_classic)">
-		<xacro:rbtheron_gz_classic_control namespace="$(arg namespace)" prefix="$(arg frame_prefix)"/>
+		<xacro:rbtheron_gz_classic_control namespace="$(arg namespace)" prefix="$(arg prefix)"/>
         <xacro:ros_planar_move_gazebo_classic/>
 	</xacro:if>
 	<xacro:if value="$(arg gazebo_ignition)">
-		<xacro:rbtheron_gz_ignition_control namespace="$(arg namespace)" prefix="$(arg frame_prefix)"/>
+		<xacro:rbtheron_gz_ignition_control namespace="$(arg namespace)" prefix="$(arg prefix)"/>
 	</xacro:if>
     <xacro:unless value="$(arg gazebo_classic)">

File: robots/rbtheron/rbtheron_plus.urdf.xacro (robot description, xacro)
@@ -27,15 +27,15 @@
 	<xacro:property name="hq" value="true" />
 	<xacro:arg name="namespace" default="robot"/>
-	<xacro:arg name="frame_prefix" default=""/>
+	<xacro:arg name="prefix" default=""/>
 	<xacro:arg name="gazebo_classic" default="false"/>
 	<xacro:arg name="gazebo_ignition" default="false"/>
 	<!-- Here we create the robot using the xacro:macro imported at the beggining of this file -->
-	<xacro:rbtheron prefix="$(arg frame_prefix)" hq="${hq}"/>
-    <joint name="$(arg frame_prefix)top_chassis_joint" type="fixed">
+	<xacro:rbtheron prefix="$(arg prefix)" hq="${hq}"/>
+    <joint name="$(arg prefix)top_chassis_joint" type="fixed">
         <origin xyz="0.0 0.0 0.26" rpy="0.0 0.0 0.0"/>
-        <parent link="$(arg frame_prefix)base_link"/>
-        <child link="$(arg frame_prefix)top_chassis"/>
+        <parent link="$(arg prefix)base_link"/>
+        <child link="$(arg prefix)top_chassis"/>
     </joint>
-    <link name="$(arg frame_prefix)top_chassis">
+    <link name="$(arg prefix)top_chassis">
         <visual>
             <geometry>
@@ -60,6 +60,6 @@
     <xacro:ur_robot
         name="$(arg ur_type)"
-        tf_prefix="$(arg frame_prefix)arm_"
-        parent="$(arg frame_prefix)top_chassis"
+        tf_prefix="$(arg prefix)arm_"
+        parent="$(arg prefix)top_chassis"
         joint_limits_parameters_file="$(arg joint_limit_params)"
         kinematics_parameters_file="$(arg kinematics_params)"
@@ -90,6 +90,6 @@
 	<!-- IMU -->
     <xacro:sensor_vectornav
-        frame_prefix="$(arg frame_prefix)imu_"
-        parent="$(arg frame_prefix)base_link"
+        frame_prefix="$(arg prefix)imu_"
+        parent="$(arg prefix)base_link"
         node_namespace="$(arg namespace)"
         gazebo_classic="$(arg gazebo_classic)"
@@ -99,6 +99,6 @@
 	<!-- 2D LASER -->
     <xacro:sensor_hokuyo_ust20lx
-        frame_prefix="$(arg frame_prefix)front_laser_"
-        parent="$(arg frame_prefix)base_link"
+        frame_prefix="$(arg prefix)front_laser_"
+        parent="$(arg prefix)base_link"
         node_namespace="$(arg namespace)"
         node_name="front_laser"
@@ -108,6 +108,6 @@
     </xacro:sensor_hokuyo_ust20lx>
     <xacro:sensor_hokuyo_ust20lx
-        frame_prefix="$(arg frame_prefix)rear_laser_"
-        parent="$(arg frame_prefix)base_link"
+        frame_prefix="$(arg prefix)rear_laser_"
+        parent="$(arg prefix)base_link"
         node_namespace="$(arg namespace)"
         node_name="rear_laser"
@@ -118,6 +118,6 @@
   	<!-- CAMERAS -->
     <xacro:sensor_intel_realsense_d435
-        frame_prefix="$(arg frame_prefix)front_rgbd_camera_"
-        parent="$(arg frame_prefix)base_link"
+        frame_prefix="$(arg prefix)front_rgbd_camera_"
+        parent="$(arg prefix)base_link"
         node_namespace="$(arg namespace)"
         node_name="front_camera"
@@ -127,6 +127,6 @@
     </xacro:sensor_intel_realsense_d435>
     <xacro:sensor_intel_realsense_d435
-        frame_prefix="$(arg frame_prefix)rear_rgbd_camera_"
-        parent="$(arg frame_prefix)base_link"
+        frame_prefix="$(arg prefix)rear_rgbd_camera_"
+        parent="$(arg prefix)base_link"
         node_namespace="$(arg namespace)"
         node_name="rear_camera"
@@ -136,13 +136,13 @@
     </xacro:sensor_intel_realsense_d435>
     <!-- 3D LiDAR -->
-    <joint name="$(arg frame_prefix)top_lidar_aux_joint" type="fixed">
+    <joint name="$(arg prefix)top_lidar_aux_joint" type="fixed">
         <origin xyz="${top_lidar_offset_x} ${top_lidar_offset_y} ${top_lidar_offset_z}" rpy="0 ${PI/2} 0"/>
-        <parent link="$(arg frame_prefix)top_chassis"/>
-        <child link="$(arg frame_prefix)top_lidar_aux"/>
+        <parent link="$(arg prefix)top_chassis"/>
+        <child link="$(arg prefix)top_lidar_aux"/>
     </joint>
-    <link name="$(arg frame_prefix)top_lidar_aux" />
+    <link name="$(arg prefix)top_lidar_aux" />
     <xacro:sensor_robosense_bpearl
-        frame_prefix="$(arg frame_prefix)top_lidar_"
-        parent="$(arg frame_prefix)top_lidar_aux"
+        frame_prefix="$(arg prefix)top_lidar_"
+        parent="$(arg prefix)top_lidar_aux"
         node_namespace="$(arg namespace)"
         node_name="top_lidar"
@@ -153,9 +153,9 @@
 	<!-- Controllers -->
 	<xacro:if value="$(arg gazebo_classic)">
-		<xacro:rbtheron_gz_classic_control namespace="$(arg namespace)" prefix="$(arg frame_prefix)"/>
+		<xacro:rbtheron_gz_classic_control namespace="$(arg namespace)" prefix="$(arg prefix)"/>
         <xacro:ros_planar_move_gazebo_classic/>
 	</xacro:if>
 	<xacro:if value="$(arg gazebo_ignition)">
-		<xacro:rbtheron_gz_ignition_control namespace="$(arg namespace)" prefix="$(arg frame_prefix)"/>
+		<xacro:rbtheron_gz_ignition_control namespace="$(arg namespace)" prefix="$(arg prefix)"/>
 	</xacro:if>
     <xacro:unless value="$(arg gazebo_classic)">
