Commit message: sync to prefix instead of frame_prefix

File: robots/rbvogui/rbvogui.urdf.xacro (robot description, xacro)
@@ -32,13 +32,13 @@
     <!-- Launch Arguments -->
 	<xacro:arg name="namespace" default="robot"/>
-	<xacro:arg name="frame_prefix" default=""/>
+	<xacro:arg name="prefix" default=""/>
 	<xacro:arg name="gazebo_classic" default="false"/>
 	<xacro:arg name="gazebo_ignition" default="false"/>
-    <xacro:rbvogui prefix="$(arg frame_prefix)" hq="${hq}" />
+    <xacro:rbvogui prefix="$(arg prefix)" hq="${hq}" />
     <!-- SENSORS see robotnik_sensors for the specific configuration -->
     <!-- IMU -->
     <xacro:sensor_vectornav
-        frame_prefix="$(arg frame_prefix)imu_"
-        parent="$(arg frame_prefix)chassis_link"
+        frame_prefix="$(arg prefix)imu_"
+        parent="$(arg prefix)chassis_link"
         node_namespace="$(arg namespace)"
         gazebo_classic="$(arg gazebo_classic)"
@@ -48,6 +48,6 @@
     <!-- Front Camera -->
     <xacro:sensor_intel_realsense_d435
-        frame_prefix="$(arg frame_prefix)front_rgbd_camera_"
-        parent="$(arg frame_prefix)base_link"
+        frame_prefix="$(arg prefix)front_rgbd_camera_"
+        parent="$(arg prefix)base_link"
         node_namespace="$(arg namespace)"
         node_name="front_camera"
@@ -58,6 +58,6 @@
     <!-- Rear Camera -->
     <xacro:sensor_intel_realsense_d435
-        frame_prefix="$(arg frame_prefix)rear_rgbd_camera_"
-        parent="$(arg frame_prefix)base_link"
+        frame_prefix="$(arg prefix)rear_rgbd_camera_"
+        parent="$(arg prefix)base_link"
         node_namespace="$(arg namespace)"
         node_name="rear_camera"
@@ -68,6 +68,6 @@
     <!-- LASERS -->
     <xacro:sensor_sick_s300
-        frame_prefix="$(arg frame_prefix)front_laser_"
-        parent="$(arg frame_prefix)chassis_link"
+        frame_prefix="$(arg prefix)front_laser_"
+        parent="$(arg prefix)chassis_link"
         node_namespace="$(arg namespace)"
         node_name="front_laser"
@@ -77,6 +77,6 @@
     </xacro:sensor_sick_s300>
     <xacro:sensor_sick_s300
-        frame_prefix="$(arg frame_prefix)rear_laser_"
-        parent="$(arg frame_prefix)chassis_link"
+        frame_prefix="$(arg prefix)rear_laser_"
+        parent="$(arg prefix)chassis_link"
         node_namespace="$(arg namespace)"
         node_name="rear_laser"
@@ -87,9 +87,9 @@
     <!-- Controllers -->
     <xacro:if value="$(arg gazebo_classic)">
-        <xacro:rbvogui_gz_classic_control namespace="$(arg namespace)" prefix="$(arg frame_prefix)" />
+        <xacro:rbvogui_gz_classic_control namespace="$(arg namespace)" prefix="$(arg prefix)" />
         <xacro:ros_planar_move_gazebo_classic />
     </xacro:if>
     <xacro:if value="$(arg gazebo_ignition)">
-        <xacro:rbvogui_gz_ignition_control namespace="$(arg namespace)" prefix="$(arg frame_prefix)" />
+        <xacro:rbvogui_gz_ignition_control namespace="$(arg namespace)" prefix="$(arg prefix)" />
     </xacro:if>
     <xacro:unless value="$(arg gazebo_classic)">

File: robots/rbvogui/rbvogui_plus.urdf.xacro (robot description, xacro)
@@ -22,8 +22,8 @@
     <!-- Launch Arguments -->
     <xacro:arg name="namespace" default="robot"/>
-    <xacro:arg name="frame_prefix" default=""/>
+    <xacro:arg name="prefix" default=""/>
     <xacro:arg name="gazebo_classic" default="false"/>
     <xacro:arg name="gazebo_ignition" default="false"/>
-    <xacro:rbvogui prefix="$(arg frame_prefix)" hq="${hq}"/>
+    <xacro:rbvogui prefix="$(arg prefix)" hq="${hq}"/>
     <xacro:property name="front_laser_offset_x" value="0.53" />
     <xacro:property name="front_laser_offset_y" value="0.33" />
@@ -45,6 +45,6 @@
     <xacro:ur_robot
         name="$(arg ur_type)"
-        tf_prefix="$(arg frame_prefix)arm_"
-        parent="$(arg frame_prefix)chassis_link"
+        tf_prefix="$(arg prefix)arm_"
+        parent="$(arg prefix)chassis_link"
         joint_limits_parameters_file="$(arg joint_limit_params)"
         kinematics_parameters_file="$(arg kinematics_params)"
@@ -54,6 +54,6 @@
     </xacro:ur_robot>
     <xacro:sensor_vectornav
-        frame_prefix="$(arg frame_prefix)imu_"
-        parent="$(arg frame_prefix)chassis_link"
+        frame_prefix="$(arg prefix)imu_"
+        parent="$(arg prefix)chassis_link"
         node_namespace="$(arg namespace)"
         gazebo_classic="$(arg gazebo_classic)"
@@ -63,6 +63,6 @@
     <!-- Front Camera -->
     <xacro:sensor_intel_realsense_d435
-        frame_prefix="$(arg frame_prefix)front_rgbd_camera_"
-        parent="$(arg frame_prefix)chassis_link"
+        frame_prefix="$(arg prefix)front_rgbd_camera_"
+        parent="$(arg prefix)chassis_link"
         node_namespace="$(arg namespace)"
         node_name="front_camera"
@@ -73,6 +73,6 @@
     <!-- Rear Camera -->
     <xacro:sensor_intel_realsense_d435
-        frame_prefix="$(arg frame_prefix)rear_rgbd_camera_"
-        parent="$(arg frame_prefix)chassis_link"
+        frame_prefix="$(arg prefix)rear_rgbd_camera_"
+        parent="$(arg prefix)chassis_link"
         node_namespace="$(arg namespace)"
         node_name="rear_camera"
@@ -82,6 +82,6 @@
     </xacro:sensor_intel_realsense_d435>
     <xacro:sensor_sick_s300
-        frame_prefix="$(arg frame_prefix)front_laser_"
-        parent="$(arg frame_prefix)chassis_link"
+        frame_prefix="$(arg prefix)front_laser_"
+        parent="$(arg prefix)chassis_link"
         node_namespace="$(arg namespace)"
         node_name="front_laser"
@@ -91,6 +91,6 @@
     </xacro:sensor_sick_s300>
     <xacro:sensor_sick_s300
-        frame_prefix="$(arg frame_prefix)rear_laser_"
-        parent="$(arg frame_prefix)chassis_link"
+        frame_prefix="$(arg prefix)rear_laser_"
+        parent="$(arg prefix)chassis_link"
         node_namespace="$(arg namespace)"
         node_name="rear_laser"
@@ -101,9 +101,9 @@
 	<!-- Controllers -->
 	<xacro:if value="$(arg gazebo_classic)">
-		<xacro:rbvogui_gz_classic_control namespace="$(arg namespace)" prefix="$(arg frame_prefix)"/>
+		<xacro:rbvogui_gz_classic_control namespace="$(arg namespace)" prefix="$(arg prefix)"/>
         <xacro:ros_planar_move_gazebo_classic/>
 	</xacro:if>
 	<xacro:if value="$(arg gazebo_ignition)">
-		<xacro:rbvogui_gz_ignition_control namespace="$(arg namespace)" prefix="$(arg frame_prefix)"/>
+		<xacro:rbvogui_gz_ignition_control namespace="$(arg namespace)" prefix="$(arg prefix)"/>
 	</xacro:if>
     <xacro:unless value="$(arg gazebo_classic)">
