Commit message: removed references to gazebo classic

File: robots/rbkairos/rbkairos.urdf.xacro (robot description, xacro)
@@ -7,5 +7,4 @@
   <xacro:include filename="$(find robotnik_description)/urdf/bases/rbkairos/rbkairos_base.urdf.xacro" />
   <xacro:include filename="$(find robotnik_description)/urdf/base_hw/rbkairos.ros2_control.urdf" />
-  <xacro:include filename="$(find robotnik_description)/simulators/gazebo_classic/rbkairos/rbkairos_control.urdf.xacro" />
   <xacro:include filename="$(find robotnik_description)/simulators/gazebo_ignition/rbkairos/rbkairos_control.urdf.xacro" />
   <xacro:include filename="$(find robotnik_sensors)/urdf/all_sensors.urdf.xacro" />
@@ -13,5 +12,4 @@
   <xacro:arg name="namespace" default="robot"/>
   <xacro:arg name="prefix" default="robot_"/>
-  <xacro:arg name="gazebo_classic" default="false"/>
   <xacro:arg name="gazebo_ignition" default="false"/>
   <xacro:property name="front_laser_offset_x" value="0.42109"/>
@@ -27,5 +25,5 @@
   <xacro:property name="front_rgbd_camera_offset_y" value="0.0"/>
   <xacro:property name="front_rgbd_camera_offset_z" value="0.25062"/>
-  <xacro:rbkairos prefix="$(arg prefix)" gazebo_classic="$(arg gazebo_classic)" gazebo_ignition="$(arg gazebo_ignition)"/>
+  <xacro:rbkairos prefix="$(arg prefix)" gazebo_ignition="$(arg gazebo_ignition)"/>
   <!-- IMU -->
     <xacro:sensor_vectornav
@@ -33,5 +31,4 @@
         parent="$(arg prefix)base_link"
         node_namespace="$(arg namespace)"
-        gazebo_classic="$(arg gazebo_classic)"
         gazebo_ignition="$(arg gazebo_ignition)">
         <origin xyz="${imu_offset_x} ${imu_offset_y} ${imu_offset_z}" rpy="0 0 0"/>
@@ -43,5 +40,4 @@
         node_namespace="$(arg namespace)"
         node_name="front_laser"
-        gazebo_classic="$(arg gazebo_classic)"
         gazebo_ignition="$(arg gazebo_ignition)">
         <origin xyz="${front_laser_offset_x} ${front_laser_offset_y} ${front_laser_offset_z}" rpy="0 ${-PI} ${3/4*PI}"/>
@@ -52,5 +48,4 @@
         node_namespace="$(arg namespace)"
         node_name="rear_laser"
-        gazebo_classic="$(arg gazebo_classic)"
         gazebo_ignition="$(arg gazebo_ignition)">
         <origin xyz="${rear_laser_offset_x} ${rear_laser_offset_y} ${rear_laser_offset_z}" rpy="0 ${-PI} ${-1/4*PI}"/>
@@ -62,20 +57,13 @@
         node_namespace="$(arg namespace)"
         node_name="front_camera"
-        gazebo_classic="$(arg gazebo_classic)"
         gazebo_ignition="$(arg gazebo_ignition)">
         <origin xyz="${front_rgbd_camera_offset_x} ${front_rgbd_camera_offset_y} ${front_rgbd_camera_offset_z}" rpy="0 0 0"/>
     </xacro:sensor_intel_realsense_d435>
   <!-- Controllers -->
-  <xacro:if value="$(arg gazebo_classic)">
-    <xacro:rbkairos_gz_classic_control namespace="$(arg namespace)" prefix="$(arg prefix)"/>
-    <xacro:ros_planar_move_gazebo_classic/>
-  </xacro:if>
   <xacro:if value="$(arg gazebo_ignition)">
     <xacro:rbkairos_gz_ignition_control namespace="$(arg namespace)" prefix="$(arg prefix)"/>
   </xacro:if>
-  <xacro:unless value="$(arg gazebo_classic)">
-    <xacro:unless value="$(arg gazebo_ignition)">
-      <xacro:rbkairos_base_hw_controller/>
-    </xacro:unless>
+  <xacro:unless value="$(arg gazebo_ignition)">
+    <xacro:rbkairos_base_hw_controller/>
   </xacro:unless>
 </robot>

File: robots/rbkairos/rbkairos_plus.urdf.xacro (robot description, xacro)
@@ -7,5 +7,4 @@
   <xacro:include filename="$(find robotnik_description)/urdf/bases/rbkairos/rbkairos_base.urdf.xacro" />
   <xacro:include filename="$(find robotnik_description)/urdf/base_hw/rbkairos.ros2_control.urdf" />
-  <xacro:include filename="$(find robotnik_description)/simulators/gazebo_classic/rbkairos/rbkairos_control.urdf.xacro" />
   <xacro:include filename="$(find robotnik_description)/simulators/gazebo_ignition/rbkairos/rbkairos_control.urdf.xacro" />
   <xacro:include filename="$(find robotnik_sensors)/urdf/all_sensors.urdf.xacro" />
@@ -14,5 +13,4 @@
   <xacro:arg name="namespace" default="robot"/>
   <xacro:arg name="prefix" default="robot_"/>
-  <xacro:arg name="gazebo_classic" default="false"/>
   <xacro:arg name="gazebo_ignition" default="false"/>
   <xacro:arg name="ur_type" default="ur5e"/>
@@ -34,5 +32,5 @@
   <xacro:property name="front_rgbd_camera_offset_z" value="0.25062"/>
   <!-- Kairos -->
-  <xacro:rbkairos prefix="$(arg prefix)" gazebo_classic="$(arg gazebo_classic)" gazebo_ignition="$(arg gazebo_ignition)"/>
+  <xacro:rbkairos prefix="$(arg prefix)" gazebo_ignition="$(arg gazebo_ignition)"/>
   <!-- Import UR arm -->
   <xacro:ur_robot
@@ -44,5 +42,4 @@
       physical_parameters_file="$(arg physical_params)"
       visual_parameters_file="$(arg visual_params)"
-      sim_gazebo="$(arg gazebo_classic)"
       sim_ignition="$(arg gazebo_ignition)">
       <origin xyz="0 0 0" rpy="0 0 0"/>
@@ -54,5 +51,4 @@
         parent="$(arg prefix)base_link"
         node_namespace="$(arg namespace)"
-        gazebo_classic="$(arg gazebo_classic)"
         gazebo_ignition="$(arg gazebo_ignition)">
         <origin xyz="${imu_offset_x} ${imu_offset_y} ${imu_offset_z}" rpy="0 0 0"/>
@@ -64,5 +60,4 @@
         node_namespace="$(arg namespace)"
         node_name="front_laser"
-        gazebo_classic="$(arg gazebo_classic)"
         gazebo_ignition="$(arg gazebo_ignition)">
         <origin xyz="${front_laser_offset_x} ${front_laser_offset_y} ${front_laser_offset_z}" rpy="0 ${-PI} ${3/4*PI}"/>
@@ -73,5 +68,4 @@
         node_namespace="$(arg namespace)"
         node_name="rear_laser"
-        gazebo_classic="$(arg gazebo_classic)"
         gazebo_ignition="$(arg gazebo_ignition)">
         <origin xyz="${rear_laser_offset_x} ${rear_laser_offset_y} ${rear_laser_offset_z}" rpy="0 ${-PI} ${-1/4*PI}"/>
@@ -83,20 +77,13 @@
         node_namespace="$(arg namespace)"
         node_name="front_camera"
-        gazebo_classic="$(arg gazebo_classic)"
         gazebo_ignition="$(arg gazebo_ignition)">
         <origin xyz="${front_rgbd_camera_offset_x} ${front_rgbd_camera_offset_y} ${front_rgbd_camera_offset_z}" rpy="0 0 0"/>
     </xacro:sensor_intel_realsense_d435>
   <!-- Controllers -->
-  <xacro:if value="$(arg gazebo_classic)">
-    <xacro:rbkairos_gz_classic_control namespace="$(arg namespace)" prefix="$(arg prefix)"/>
-    <xacro:ros_planar_move_gazebo_classic/>
-  </xacro:if>
   <xacro:if value="$(arg gazebo_ignition)">
     <xacro:rbkairos_gz_ignition_control namespace="$(arg namespace)" prefix="$(arg prefix)"/>
   </xacro:if>
-  <xacro:unless value="$(arg gazebo_classic)">
-    <xacro:unless value="$(arg gazebo_ignition)">
-      <xacro:rbkairos_base_hw_controller/>
-    </xacro:unless>
+  <xacro:unless value="$(arg gazebo_ignition)">
+    <xacro:rbkairos_base_hw_controller/>
   </xacro:unless>
 </robot>

File: robots/rbrobout/rbrobout.urdf.xacro (robot description, xacro)
@@ -7,5 +7,4 @@
   <xacro:include filename="$(find robotnik_description)/urdf/bases/rbrobout/rbrobout_base.urdf.xacro" />
   <xacro:include filename="$(find robotnik_description)/urdf/base_hw/rbrobout.ros2_control.urdf" />
-  <xacro:include filename="$(find robotnik_description)/simulators/gazebo_classic/rbrobout/rbrobout_control.urdf.xacro" />
   <xacro:include filename="$(find robotnik_description)/simulators/gazebo_ignition/rbrobout/rbrobout_control.urdf.xacro" />
   <xacro:include filename="$(find robotnik_sensors)/urdf/all_sensors.urdf.xacro" />
@@ -13,5 +12,4 @@
   <xacro:arg name="namespace" default="robot"/>
   <xacro:arg name="prefix" default="robot_"/>
-  <xacro:arg name="gazebo_classic" default="false"/>
   <xacro:arg name="gazebo_ignition" default="false"/>
   <xacro:property name="front_laser_offset_x" value="0.8"/>
@@ -24,5 +22,5 @@
   <xacro:property name="imu_offset_y" value="-0.3"/>
   <xacro:property name="imu_offset_z" value="0.0725"/>
-  <xacro:rbrobout prefix="$(arg prefix)" gazebo_classic="$(arg gazebo_classic)" gazebo_ignition="$(arg gazebo_ignition)"/>
+  <xacro:rbrobout prefix="$(arg prefix)" gazebo_ignition="$(arg gazebo_ignition)"/>
   <!-- IMU -->
     <xacro:sensor_vectornav
@@ -30,5 +28,4 @@
         parent="$(arg prefix)base_link"
         node_namespace="$(arg namespace)"
-        gazebo_classic="$(arg gazebo_classic)"
         gazebo_ignition="$(arg gazebo_ignition)">
         <origin xyz="${imu_offset_x} ${imu_offset_y} ${imu_offset_z}" rpy="0 0 0"/>
@@ -40,5 +37,4 @@
         node_namespace="$(arg namespace)"
         node_name="front_laser"
-        gazebo_classic="$(arg gazebo_classic)"
         gazebo_ignition="$(arg gazebo_ignition)">
         <origin xyz="${front_laser_offset_x} ${front_laser_offset_y} ${front_laser_offset_z}" rpy="0 0 ${1/4*PI}"/>
@@ -50,20 +46,13 @@
         node_namespace="$(arg namespace)"
         node_name="rear_laser"
-        gazebo_classic="$(arg gazebo_classic)"
         gazebo_ignition="$(arg gazebo_ignition)">
         <origin xyz="${rear_laser_offset_x} ${rear_laser_offset_y} ${rear_laser_offset_z}" rpy="0 0 ${-3/4*PI}"/>
     </xacro:sensor_sick_microscan3>
     <!-- Controllers -->
-    <xacro:if value="$(arg gazebo_classic)">
-        <xacro:rbrobout_gz_classic_control namespace="$(arg namespace)" prefix="$(arg prefix)"/>
-        <xacro:ros_planar_move_gazebo_classic/>
-    </xacro:if>
     <xacro:if value="$(arg gazebo_ignition)">
         <xacro:rbrobout_gz_ignition_control namespace="$(arg namespace)" prefix="$(arg prefix)"/>
     </xacro:if>
-    <xacro:unless value="$(arg gazebo_classic)">
-        <xacro:unless value="$(arg gazebo_ignition)">
-            <xacro:rbrobout_base_hw_controller/>
-        </xacro:unless>
+    <xacro:unless value="$(arg gazebo_ignition)">
+        <xacro:rbrobout_base_hw_controller/>
     </xacro:unless>
 </robot>

File: robots/rbrobout/rbrobout_plus.urdf.xacro (robot description, xacro)
@@ -8,5 +8,4 @@
   <xacro:include filename="$(find robotnik_description)/urdf/bases/rbrobout/rbrobout_top_cover.urdf.xacro" />
   <xacro:include filename="$(find robotnik_description)/urdf/base_hw/rbrobout.ros2_control.urdf" />
-  <xacro:include filename="$(find robotnik_description)/simulators/gazebo_classic/rbrobout/rbrobout_control.urdf.xacro" />
   <xacro:include filename="$(find robotnik_description)/simulators/gazebo_ignition/rbrobout/rbrobout_control.urdf.xacro" />
   <xacro:include filename="$(find robotnik_sensors)/urdf/all_sensors.urdf.xacro" />
@@ -16,5 +15,4 @@
   <xacro:arg name="namespace" default="robot"/>
   <xacro:arg name="prefix" default="robot_"/>
-  <xacro:arg name="gazebo_classic" default="false"/>
   <xacro:arg name="gazebo_ignition" default="false"/>
   <xacro:arg name="ur_type" default="ur10e"/>
@@ -38,5 +36,5 @@
   <xacro:property name="lift_orientation_p" value="0"/>
   <xacro:property name="lift_orientation_y" value="0"/>
-  <xacro:rbrobout prefix="$(arg prefix)"  gazebo_classic="$(arg gazebo_classic)" gazebo_ignition="$(arg gazebo_ignition)"/>
+  <xacro:rbrobout prefix="$(arg prefix)" gazebo_ignition="$(arg gazebo_ignition)"/>
   <xacro:top_cover prefix="$(arg prefix)" parent="$(arg prefix)base_link">
       <origin xyz="0 0 -0.1" rpy="0 0 0"/>
@@ -53,5 +51,4 @@
       physical_parameters_file="$(arg physical_params)"
       visual_parameters_file="$(arg visual_params)"
-      sim_gazebo="$(arg gazebo_classic)"
       sim_ignition="$(arg gazebo_ignition)">
       <origin xyz="0 0 0" rpy="0 0 0"/>
@@ -62,5 +59,4 @@
         parent="$(arg prefix)base_link"
         node_namespace="$(arg namespace)"
-        gazebo_classic="$(arg gazebo_classic)"
         gazebo_ignition="$(arg gazebo_ignition)">
         <origin xyz="${imu_offset_x} ${imu_offset_y} ${imu_offset_z}" rpy="0 0 0"/>
@@ -72,5 +68,4 @@
         node_namespace="$(arg namespace)"
         node_name="front_laser"
-        gazebo_classic="$(arg gazebo_classic)"
         gazebo_ignition="$(arg gazebo_ignition)">
         <origin xyz="${front_laser_offset_x} ${front_laser_offset_y} ${front_laser_offset_z}" rpy="0 0 ${1/4*PI}"/>
@@ -82,20 +77,13 @@
         node_namespace="$(arg namespace)"
         node_name="rear_laser"
-        gazebo_classic="$(arg gazebo_classic)"
         gazebo_ignition="$(arg gazebo_ignition)">
         <origin xyz="${rear_laser_offset_x} ${rear_laser_offset_y} ${rear_laser_offset_z}" rpy="0 0 ${-3/4*PI}"/>
     </xacro:sensor_sick_microscan3>
     <!-- Controllers -->
-    <xacro:if value="$(arg gazebo_classic)">
-        <xacro:rbrobout_gz_classic_control namespace="$(arg namespace)" prefix="$(arg prefix)"/>
-        <xacro:ros_planar_move_gazebo_classic/>
-    </xacro:if>
     <xacro:if value="$(arg gazebo_ignition)">
         <xacro:rbrobout_gz_ignition_control namespace="$(arg namespace)" prefix="$(arg prefix)"/>
     </xacro:if>
-    <xacro:unless value="$(arg gazebo_classic)">
-        <xacro:unless value="$(arg gazebo_ignition)">
-            <xacro:rbrobout_base_hw_controller/>
-        </xacro:unless>
+    <xacro:unless value="$(arg gazebo_ignition)">
+        <xacro:rbrobout_base_hw_controller/>
     </xacro:unless>
 </robot>

File: robots/rbsummit/rbsummit.urdf.xacro (robot description, xacro)
@@ -8,5 +8,4 @@
 	<xacro:include filename="$(find robotnik_description)/urdf/bases/rbsummit/rbsummit_base.xacro"/>
     <xacro:include filename="$(find robotnik_description)/urdf/base_hw/rbsummit.ros2_control.urdf" />
-	<xacro:include filename="$(find robotnik_description)/simulators/gazebo_classic/rbsummit/rbsummit_control.urdf.xacro"/>
 	<xacro:include filename="$(find robotnik_description)/simulators/gazebo_ignition/rbsummit/rbsummit_control.urdf.xacro"/>
 	<!-- Import all available sensors -->
@@ -18,5 +17,4 @@
 	<xacro:arg name="namespace" default="robot"/>
 	<xacro:arg name="prefix" default="robot_"/>
-	<xacro:arg name="gazebo_classic" default="false"/>
 	<xacro:arg name="gazebo_ignition" default="false"/>
 	<xacro:property name="imu_offset_x" value="0.0385"/>
@@ -43,5 +41,4 @@
         parent="$(arg prefix)base_link"
         node_namespace="$(arg namespace)"
-        gazebo_classic="$(arg gazebo_classic)"
         gazebo_ignition="$(arg gazebo_ignition)">
         <origin xyz="${imu_offset_x} ${imu_offset_y} ${imu_offset_z}" rpy="0 0 0"/>
@@ -53,5 +50,4 @@
         node_namespace="$(arg namespace)"
         node_name="top_lidar"
-        gazebo_classic="$(arg gazebo_classic)"
         gazebo_ignition="$(arg gazebo_ignition)">
 		<origin
@@ -66,5 +62,4 @@
         node_namespace="$(arg namespace)"
         node_name="front_camera"
-        gazebo_classic="$(arg gazebo_classic)"
         gazebo_ignition="$(arg gazebo_ignition)">
         <origin xyz="${front_rgbd_camera_offset_x} ${front_rgbd_camera_offset_y} ${front_rgbd_camera_offset_z}" rpy="0 0 0"/>
@@ -76,5 +71,4 @@
 		update_rate="5"
         node_namespace="$(arg namespace)"
-        gazebo_classic="$(arg gazebo_classic)"
         gazebo_ignition="$(arg gazebo_ignition)">
 		<origin
@@ -84,15 +78,9 @@
 	</xacro:sensor_ublox_with_mast>
 	<!-- Controllers -->
-    <xacro:if value="$(arg gazebo_classic)">
-      <xacro:rbsummit_gz_classic_control namespace="$(arg namespace)" prefix="$(arg prefix)"/>
-        <xacro:ros_planar_move_gazebo_classic/>
-    </xacro:if>
     <xacro:if value="$(arg gazebo_ignition)">
       <xacro:rbsummit_gz_ignition_control namespace="$(arg namespace)" prefix="$(arg prefix)"/>
     </xacro:if>
-    <xacro:unless value="$(arg gazebo_classic)">
-      <xacro:unless value="$(arg gazebo_ignition)">
-        <xacro:rbsummit_base_hw_controller/>
-      </xacro:unless>
+    <xacro:unless value="$(arg gazebo_ignition)">
+      <xacro:rbsummit_base_hw_controller/>
     </xacro:unless>
 </robot>

File: robots/rbtheron/rbtheron.urdf.xacro (robot description, xacro)
@@ -9,5 +9,4 @@
 	<xacro:include filename="$(find robotnik_description)/urdf/bases/rbtheron/rbtheron_base.xacro"/>
     <xacro:include filename="$(find robotnik_description)/urdf/base_hw/rbtheron.ros2_control.urdf" />
-	<xacro:include filename="$(find robotnik_description)/simulators/gazebo_classic/rbtheron/rbtheron_control.urdf.xacro"/>
 	<xacro:include filename="$(find robotnik_description)/simulators/gazebo_ignition/rbtheron/rbtheron_control.urdf.xacro"/>
 	<!-- Import all available sensors -->
@@ -22,5 +21,4 @@
 	<xacro:arg name="namespace" default="robot"/>
 	<xacro:arg name="prefix" default="robot_"/>
-	<xacro:arg name="gazebo_classic" default="false"/>
 	<xacro:arg name="gazebo_ignition" default="false"/>
 	<!-- Here we create the robot using the xacro:macro imported at the beggining of this file -->
@@ -47,5 +45,4 @@
         parent="$(arg prefix)base_link"
         node_namespace="$(arg namespace)"
-        gazebo_classic="$(arg gazebo_classic)"
         gazebo_ignition="$(arg gazebo_ignition)">
         <origin xyz="${imu_offset_x} ${imu_offset_y} ${imu_offset_z}" rpy="0 0 0"/>
@@ -57,5 +54,4 @@
         node_namespace="$(arg namespace)"
         node_name="front_laser"
-        gazebo_classic="$(arg gazebo_classic)"
         gazebo_ignition="$(arg gazebo_ignition)">
         <origin xyz="${front_laser_offset_x} ${front_laser_offset_y} ${front_laser_offset_z}" rpy="0 ${-PI} ${3/4*PI}"/>
@@ -66,5 +62,4 @@
         node_namespace="$(arg namespace)"
         node_name="rear_laser"
-        gazebo_classic="$(arg gazebo_classic)"
         gazebo_ignition="$(arg gazebo_ignition)">
         <origin xyz="${rear_laser_offset_x} ${rear_laser_offset_y} ${rear_laser_offset_z}" rpy="0 ${-PI} ${-1/4*PI}"/>
@@ -76,5 +71,4 @@
         node_namespace="$(arg namespace)"
         node_name="front_camera"
-        gazebo_classic="$(arg gazebo_classic)"
         gazebo_ignition="$(arg gazebo_ignition)">
         <origin xyz="${front_rgbd_camera_offset_x} ${front_rgbd_camera_offset_y} ${front_rgbd_camera_offset_z}" rpy="0 0 0"/>
@@ -85,20 +79,13 @@
         node_namespace="$(arg namespace)"
         node_name="rear_camera"
-        gazebo_classic="$(arg gazebo_classic)"
         gazebo_ignition="$(arg gazebo_ignition)">
         <origin xyz="${rear_rgbd_camera_offset_x} ${rear_rgbd_camera_offset_y} ${rear_rgbd_camera_offset_z}" rpy="0 0 ${PI}"/>
     </xacro:sensor_intel_realsense_d435>
 	<!-- Controllers -->
-	<xacro:if value="$(arg gazebo_classic)">
-		<xacro:rbtheron_gz_classic_control namespace="$(arg namespace)" prefix="$(arg prefix)"/>
-        <xacro:ros_planar_move_gazebo_classic/>
-	</xacro:if>
 	<xacro:if value="$(arg gazebo_ignition)">
 		<xacro:rbtheron_gz_ignition_control namespace="$(arg namespace)" prefix="$(arg prefix)"/>
 	</xacro:if>
-    <xacro:unless value="$(arg gazebo_classic)">
-        <xacro:unless value="$(arg gazebo_ignition)">
-            <xacro:rbtheron_base_hw_controller/>
-        </xacro:unless>
+    <xacro:unless value="$(arg gazebo_ignition)">
+        <xacro:rbtheron_base_hw_controller/>
     </xacro:unless>
 </robot>

File: robots/rbtheron/rbtheron_plus.urdf.xacro (robot description, xacro)
@@ -9,5 +9,4 @@
 	<xacro:include filename="$(find robotnik_description)/urdf/bases/rbtheron/rbtheron_base.xacro"/>
     <xacro:include filename="$(find robotnik_description)/urdf/base_hw/rbtheron.ros2_control.urdf" />
-	<xacro:include filename="$(find robotnik_description)/simulators/gazebo_classic/rbtheron/rbtheron_control.urdf.xacro"/>
 	<xacro:include filename="$(find robotnik_description)/simulators/gazebo_ignition/rbtheron/rbtheron_control.urdf.xacro"/>
 	<!-- Import all available sensors -->
@@ -28,5 +27,4 @@
 	<xacro:arg name="namespace" default="robot"/>
 	<xacro:arg name="prefix" default="robot_"/>
-	<xacro:arg name="gazebo_classic" default="false"/>
 	<xacro:arg name="gazebo_ignition" default="false"/>
 	<!-- Here we create the robot using the xacro:macro imported at the beggining of this file -->
@@ -65,5 +63,4 @@
         physical_parameters_file="$(arg physical_params)"
         visual_parameters_file="$(arg visual_params)"
-        sim_gazebo="$(arg gazebo_classic)"
         sim_ignition="$(arg gazebo_ignition)">
         <origin xyz="-0.2 0 0.6" rpy="0 0 0"/>
@@ -93,5 +90,4 @@
         parent="$(arg prefix)base_link"
         node_namespace="$(arg namespace)"
-        gazebo_classic="$(arg gazebo_classic)"
         gazebo_ignition="$(arg gazebo_ignition)">
         <origin xyz="${imu_offset_x} ${imu_offset_y} ${imu_offset_z}" rpy="0 0 0"/>
@@ -103,5 +99,4 @@
         node_namespace="$(arg namespace)"
         node_name="front_laser"
-        gazebo_classic="$(arg gazebo_classic)"
         gazebo_ignition="$(arg gazebo_ignition)">
         <origin xyz="${front_laser_offset_x} ${front_laser_offset_y} ${front_laser_offset_z}" rpy="0 ${-PI} ${3/4*PI}"/>
@@ -112,5 +107,4 @@
         node_namespace="$(arg namespace)"
         node_name="rear_laser"
-        gazebo_classic="$(arg gazebo_classic)"
         gazebo_ignition="$(arg gazebo_ignition)">
         <origin xyz="${rear_laser_offset_x} ${rear_laser_offset_y} ${rear_laser_offset_z}" rpy="0 ${-PI} ${-1/4*PI}"/>
@@ -122,5 +116,4 @@
         node_namespace="$(arg namespace)"
         node_name="front_camera"
-        gazebo_classic="$(arg gazebo_classic)"
         gazebo_ignition="$(arg gazebo_ignition)">
         <origin xyz="${front_rgbd_camera_offset_x} ${front_rgbd_camera_offset_y} ${front_rgbd_camera_offset_z}" rpy="0 0 0"/>
@@ -131,5 +124,4 @@
         node_namespace="$(arg namespace)"
         node_name="rear_camera"
-        gazebo_classic="$(arg gazebo_classic)"
         gazebo_ignition="$(arg gazebo_ignition)">
         <origin xyz="${rear_rgbd_camera_offset_x} ${rear_rgbd_camera_offset_y} ${rear_rgbd_camera_offset_z}" rpy="0 0 ${PI}"/>
@@ -141,20 +133,13 @@
         node_namespace="$(arg namespace)"
         node_name="top_lidar"
-        gazebo_classic="$(arg gazebo_classic)"
         gazebo_ignition="$(arg gazebo_ignition)">
         <origin xyz="${top_lidar_offset_x} ${top_lidar_offset_y} ${top_lidar_offset_z}" rpy="0 ${PI/2} 0"/>
     </xacro:sensor_robosense_bpearl>
 	<!-- Controllers -->
-	<xacro:if value="$(arg gazebo_classic)">
-		<xacro:rbtheron_gz_classic_control namespace="$(arg namespace)" prefix="$(arg prefix)"/>
-        <xacro:ros_planar_move_gazebo_classic/>
-	</xacro:if>
 	<xacro:if value="$(arg gazebo_ignition)">
 		<xacro:rbtheron_gz_ignition_control namespace="$(arg namespace)" prefix="$(arg prefix)"/>
 	</xacro:if>
-    <xacro:unless value="$(arg gazebo_classic)">
-        <xacro:unless value="$(arg gazebo_ignition)">
-            <xacro:rbtheron_base_hw_controller/>
-        </xacro:unless>
+    <xacro:unless value="$(arg gazebo_ignition)">
+        <xacro:rbtheron_base_hw_controller/>
     </xacro:unless>
 </robot>
