Commit message: removed references to gazebo classic

File: robots/rbvogui/rbvogui.urdf.xacro (robot description, xacro)
@@ -9,5 +9,4 @@
     <xacro:include filename="$(find robotnik_description)/urdf/bases/rbvogui/rbvogui_base.urdf.xacro" />
     <xacro:include filename="$(find robotnik_description)/urdf/base_hw/rbvogui.ros2_control.urdf" />
-    <xacro:include filename="$(find robotnik_description)/simulators/gazebo_classic/rbvogui/rbvogui_control.urdf.xacro" />
     <xacro:include filename="$(find robotnik_description)/simulators/gazebo_ignition/rbvogui/rbvogui_control.urdf.xacro" />
     <!-- Import all available sensors -->
@@ -18,5 +17,4 @@
 	<xacro:arg name="namespace" default="robot"/>
 	<xacro:arg name="prefix" default="robot_"/>
-	<xacro:arg name="gazebo_classic" default="false"/>
 	<xacro:arg name="gazebo_ignition" default="false"/>
     <xacro:rbvogui prefix="$(arg prefix)" hq="${hq}"/>
@@ -27,5 +25,4 @@
         parent="$(arg prefix)chassis_link"
         node_namespace="$(arg namespace)"
-        gazebo_classic="$(arg gazebo_classic)"
         gazebo_ignition="$(arg gazebo_ignition)">
         <origin xyz="0.3 -0.3 0.0725" rpy="0 0 0"/>
@@ -37,5 +34,4 @@
         node_namespace="$(arg namespace)"
         node_name="front_camera"
-        gazebo_classic="$(arg gazebo_classic)"
         gazebo_ignition="$(arg gazebo_ignition)">
         <origin xyz="0.46462 0.0 0.18258" rpy="0 0 0"/>
@@ -47,5 +43,4 @@
         node_namespace="$(arg namespace)"
         node_name="rear_camera"
-        gazebo_classic="$(arg gazebo_classic)"
         gazebo_ignition="$(arg gazebo_ignition)">
         <origin xyz="-0.503 0.0 0.29" rpy="0 0 -${PI}"/>
@@ -57,5 +52,4 @@
         node_namespace="$(arg namespace)"
         node_name="front_laser"
-        gazebo_classic="$(arg gazebo_classic)"
         gazebo_ignition="$(arg gazebo_ignition)">
         <origin xyz="0.53 0.33 0.1145" rpy="${PI} 0 ${PI/4}"/>
@@ -66,20 +60,13 @@
         node_namespace="$(arg namespace)"
         node_name="rear_laser"
-        gazebo_classic="$(arg gazebo_classic)"
         gazebo_ignition="$(arg gazebo_ignition)">
         <origin xyz="-0.53 -0.33 0.1145" rpy="${PI} 0 ${-PI*3/4}"/>
     </xacro:sensor_sick_s300>
 	<!-- Controllers -->
-	<xacro:if value="$(arg gazebo_classic)">
-		<xacro:rbvogui_gz_classic_control namespace="$(arg namespace)" prefix="$(arg prefix)"/>
-        <xacro:ros_planar_move_gazebo_classic/>
-	</xacro:if>
 	<xacro:if value="$(arg gazebo_ignition)">
 		<xacro:rbvogui_gz_ignition_control namespace="$(arg namespace)" prefix="$(arg prefix)"/>
 	</xacro:if>
-    <xacro:unless value="$(arg gazebo_classic)">
-        <xacro:unless value="$(arg gazebo_ignition)">
-            <xacro:rbvogui_base_hw_controller/>
-        </xacro:unless>
+    <xacro:unless value="$(arg gazebo_ignition)">
+        <xacro:rbvogui_base_hw_controller/>
     </xacro:unless>
 </robot>

File: robots/rbvogui/rbvogui_plus.urdf.xacro (robot description, xacro)
@@ -9,5 +9,4 @@
     <xacro:include filename="$(find robotnik_description)/urdf/bases/rbvogui/rbvogui_base.urdf.xacro" />
     <xacro:include filename="$(find robotnik_description)/urdf/base_hw/rbvogui.ros2_control.urdf" />
-    <xacro:include filename="$(find robotnik_description)/simulators/gazebo_classic/rbvogui/rbvogui_control.urdf.xacro" />
     <xacro:include filename="$(find robotnik_description)/simulators/gazebo_ignition/rbvogui/rbvogui_control.urdf.xacro" />
     <!-- Import all available sensors -->
@@ -24,5 +23,4 @@
 	<xacro:arg name="namespace" default="robot"/>
 	<xacro:arg name="prefix" default="robot_"/>
-	<xacro:arg name="gazebo_classic" default="false"/>
 	<xacro:arg name="gazebo_ignition" default="false"/>
     <xacro:rbvogui prefix="$(arg prefix)" hq="${hq}"/>
@@ -36,5 +34,4 @@
         physical_parameters_file="$(arg physical_params)"
         visual_parameters_file="$(arg visual_params)"
-        sim_gazebo="$(arg gazebo_classic)"
         sim_ignition="$(arg gazebo_ignition)">
         <origin xyz="0 0 0.235" rpy="0 0 0"/>
@@ -46,5 +43,4 @@
         parent="$(arg prefix)chassis_link"
         node_namespace="$(arg namespace)"
-        gazebo_classic="$(arg gazebo_classic)"
         gazebo_ignition="$(arg gazebo_ignition)">
         <origin xyz="0.3 -0.3 0.0725" rpy="0 0 0"/>
@@ -56,5 +52,4 @@
         node_namespace="$(arg namespace)"
         node_name="front_camera"
-        gazebo_classic="$(arg gazebo_classic)"
         gazebo_ignition="$(arg gazebo_ignition)">
         <origin xyz="0.46462 0.0 0.18258" rpy="0 0 0"/>
@@ -66,5 +61,4 @@
         node_namespace="$(arg namespace)"
         node_name="rear_camera"
-        gazebo_classic="$(arg gazebo_classic)"
         gazebo_ignition="$(arg gazebo_ignition)">
         <origin xyz="-0.503 0.0 0.29" rpy="0 0 -${PI}"/>
@@ -76,5 +70,4 @@
         node_namespace="$(arg namespace)"
         node_name="front_laser"
-        gazebo_classic="$(arg gazebo_classic)"
         gazebo_ignition="$(arg gazebo_ignition)">
         <origin xyz="0.53 0.33 0.1145" rpy="${PI} 0 ${PI/4}"/>
@@ -85,20 +78,13 @@
         node_namespace="$(arg namespace)"
         node_name="rear_laser"
-        gazebo_classic="$(arg gazebo_classic)"
         gazebo_ignition="$(arg gazebo_ignition)">
         <origin xyz="-0.53 -0.33 0.1145" rpy="${PI} 0 ${-PI*3/4}"/>
     </xacro:sensor_sick_s300>
 	<!-- Controllers -->
-	<xacro:if value="$(arg gazebo_classic)">
-		<xacro:rbvogui_gz_classic_control namespace="$(arg namespace)" prefix="$(arg prefix)"/>
-        <xacro:ros_planar_move_gazebo_classic/>
-	</xacro:if>
 	<xacro:if value="$(arg gazebo_ignition)">
 		<xacro:rbvogui_gz_ignition_control namespace="$(arg namespace)" prefix="$(arg prefix)"/>
 	</xacro:if>
-    <xacro:unless value="$(arg gazebo_classic)">
-        <xacro:unless value="$(arg gazebo_ignition)">
-            <xacro:rbvogui_base_hw_controller/>
-        </xacro:unless>
+    <xacro:unless value="$(arg gazebo_ignition)">
+        <xacro:rbvogui_base_hw_controller/>
     </xacro:unless>
 </robot>

File: urdf/bases/rbkairos/rbkairos_base.urdf.xacro (robot description, xacro)
@@ -13,5 +13,5 @@
   	<xacro:property name="wheel_offset_y" value="0.2590" />
   	<xacro:property name="wheel_offset_z" value="0.0" />
-    <xacro:macro name="rbkairos" params="prefix:=robot_ gazebo_classic:=false gazebo_ignition:=false">
+    <xacro:macro name="rbkairos" params="prefix:=robot_ gazebo_ignition:=false">
   		<!-- *************** -->
   		<!-- Robots Elements -->
@@ -19,14 +19,14 @@
   		<!-- Here we create the robot elements using the xacro:macros imported at the beggining of this file -->
   		<xacro:rbkairos_plus_body prefix="${prefix}"/>
-  		<xacro:rbkairos_mecanum_wheel prefix="${prefix}front_right_" parent="${prefix}base_link" reflect="false" hq="true" gazebo_classic="${gazebo_classic}" gazebo_ignition="${gazebo_ignition}"
+  		<xacro:rbkairos_mecanum_wheel prefix="${prefix}front_right_" parent="${prefix}base_link" reflect="false" hq="true" gazebo_ignition="${gazebo_ignition}"
 			xyz="${wheel_offset_x} -${wheel_offset_y} ${wheel_offset_z}">
   		</xacro:rbkairos_mecanum_wheel>
-  		<xacro:rbkairos_mecanum_wheel prefix="${prefix}front_left_" parent="${prefix}base_link" reflect="true" hq="true" gazebo_classic="${gazebo_classic}" gazebo_ignition="${gazebo_ignition}"
+  		<xacro:rbkairos_mecanum_wheel prefix="${prefix}front_left_" parent="${prefix}base_link" reflect="true" hq="true" gazebo_ignition="${gazebo_ignition}"
 			xyz="${wheel_offset_x} ${wheel_offset_y} ${wheel_offset_z}">
   		</xacro:rbkairos_mecanum_wheel>
-  		<xacro:rbkairos_mecanum_wheel prefix="${prefix}back_left_" parent="${prefix}base_link" reflect="false" hq="true" gazebo_classic="${gazebo_classic}" gazebo_ignition="${gazebo_ignition}"
+  		<xacro:rbkairos_mecanum_wheel prefix="${prefix}back_left_" parent="${prefix}base_link" reflect="false" hq="true" gazebo_ignition="${gazebo_ignition}"
 			xyz="-${wheel_offset_x} ${wheel_offset_y} ${wheel_offset_z}">
   		</xacro:rbkairos_mecanum_wheel>
-  		<xacro:rbkairos_mecanum_wheel prefix="${prefix}back_right_" parent="${prefix}base_link" reflect="true" hq="true" gazebo_classic="${gazebo_classic}" gazebo_ignition="${gazebo_ignition}"
+  		<xacro:rbkairos_mecanum_wheel prefix="${prefix}back_right_" parent="${prefix}base_link" reflect="true" hq="true" gazebo_ignition="${gazebo_ignition}"
 			xyz="-${wheel_offset_x} -${wheel_offset_y} ${wheel_offset_z}">
   		</xacro:rbkairos_mecanum_wheel>

File: urdf/bases/rbrobout/rbrobout_base.urdf.xacro (robot description, xacro)
@@ -18,5 +18,5 @@
 	<!-- Flag to select the high or low quality model -->
 	<xacro:property name="hq" value="true" />
-    <xacro:macro name="rbrobout" params="prefix:=robot_ gazebo_classic:=false gazebo_ignition:=false">
+    <xacro:macro name="rbrobout" params="prefix:=robot_ gazebo_ignition:=false">
 		<!-- *************** -->
 		<!-- Robots Elements -->
@@ -25,14 +25,14 @@
 		<xacro:rbrobout_body prefix="${prefix}" />
 		<!-- Wheels -->
-		<xacro:rbrobout_mecanum_wheel prefix="${prefix}front_right_" parent="${prefix}base_link" reflect="false" hq="${hq}" gazebo_classic="${gazebo_classic}" gazebo_ignition="${gazebo_ignition}"
+		<xacro:rbrobout_mecanum_wheel prefix="${prefix}front_right_" parent="${prefix}base_link" reflect="false" hq="${hq}" gazebo_ignition="${gazebo_ignition}"
 			xyz="${wheel_offset_x} -${wheel_offset_y} ${wheel_offset_z}">
 		</xacro:rbrobout_mecanum_wheel>
-		<xacro:rbrobout_mecanum_wheel prefix="${prefix}front_left_" parent="${prefix}base_link" reflect="true" hq="${hq}" gazebo_classic="${gazebo_classic}" gazebo_ignition="${gazebo_ignition}"
+		<xacro:rbrobout_mecanum_wheel prefix="${prefix}front_left_" parent="${prefix}base_link" reflect="true" hq="${hq}" gazebo_ignition="${gazebo_ignition}"
 			xyz="${wheel_offset_x} ${wheel_offset_y} ${wheel_offset_z}">
 		</xacro:rbrobout_mecanum_wheel>
-		<xacro:rbrobout_mecanum_wheel prefix="${prefix}back_left_" parent="${prefix}base_link" reflect="false" hq="${hq}" gazebo_classic="${gazebo_classic}" gazebo_ignition="${gazebo_ignition}"
+		<xacro:rbrobout_mecanum_wheel prefix="${prefix}back_left_" parent="${prefix}base_link" reflect="false" hq="${hq}" gazebo_ignition="${gazebo_ignition}"
 			xyz="-${wheel_offset_x} ${wheel_offset_y} ${wheel_offset_z}">
 		</xacro:rbrobout_mecanum_wheel>
-		<xacro:rbrobout_mecanum_wheel prefix="${prefix}back_right_" parent="${prefix}base_link" reflect="true" hq="${hq}" gazebo_classic="${gazebo_classic}" gazebo_ignition="${gazebo_ignition}"
+		<xacro:rbrobout_mecanum_wheel prefix="${prefix}back_right_" parent="${prefix}base_link" reflect="true" hq="${hq}" gazebo_ignition="${gazebo_ignition}"
 			xyz="-${wheel_offset_x} -${wheel_offset_y} ${wheel_offset_z}">
 		</xacro:rbrobout_mecanum_wheel>

File: urdf/wheels/mecanum_wheel/rbkairos_mecanum_wheel.urdf.xacro (robot description, xacro)
@@ -11,9 +11,9 @@
             izz="${m*(3*r*r+h*h)/12}" />
     </xacro:macro>
-    <xacro:macro name="rbkairos_mecanum_wheel" params="prefix parent xyz reflect hq gazebo_classic:=false gazebo_ignition:=false">
+    <xacro:macro name="rbkairos_mecanum_wheel" params="prefix parent xyz reflect hq gazebo_ignition:=false">
         <joint name="${prefix}wheel_joint" type="continuous">
             <parent link="${parent}" />
             <child link="${prefix}wheel_link" />
-            <xacro:if value="${gazebo_classic or gazebo_ignition}">
+            <xacro:if value="${gazebo_ignition}">
                 <xacro:if value="${reflect}">
                     <origin xyz="${xyz}" rpy="0.0 0.0 -${PI/4}"/>
@@ -23,5 +23,5 @@
                 </xacro:unless>
             </xacro:if>
-            <xacro:unless value="${gazebo_classic or gazebo_ignition}">
+            <xacro:unless value="${gazebo_ignition}">
                 <origin xyz="${xyz}" rpy="0.0 0.0 0.0"/>
             </xacro:unless>
@@ -30,5 +30,5 @@
         </joint>
         <link name="${prefix}wheel_link">
-            <xacro:unless value="${gazebo_classic or gazebo_ignition}">
+            <xacro:unless value="${gazebo_ignition}">
                 <visual>
                     <xacro:if value="${hq}">
@@ -72,5 +72,5 @@
             </inertial>
         </link>
-        <xacro:if value="${gazebo_classic or gazebo_ignition}">
+        <xacro:if value="${gazebo_ignition}">
             <gazebo reference="${prefix}wheel_link">
                 <collision>

File: urdf/wheels/mecanum_wheel/rbrobout_mecanum_wheel.urdf.xacro (robot description, xacro)
@@ -11,9 +11,9 @@
             izz="${m*(3*r*r+h*h)/12}" />
     </xacro:macro>
-    <xacro:macro name="rbrobout_mecanum_wheel" params="prefix parent xyz reflect hq gazebo_classic:=false gazebo_ignition:=false">
+    <xacro:macro name="rbrobout_mecanum_wheel" params="prefix parent xyz reflect hq gazebo_ignition:=false">
         <joint name="${prefix}wheel_joint" type="continuous">
             <parent link="${parent}" />
             <child link="${prefix}wheel_link" />
-            <xacro:if value="${gazebo_classic or gazebo_ignition}">
+            <xacro:if value="${gazebo_ignition}">
                 <xacro:if value="${reflect}">
                     <origin xyz="${xyz}" rpy="0.0 0.0 -${PI/4}"/>
@@ -23,5 +23,5 @@
                 </xacro:unless>
             </xacro:if>
-            <xacro:unless value="${gazebo_classic or gazebo_ignition}">
+            <xacro:unless value="${gazebo_ignition}">
                 <origin xyz="${xyz}" rpy="0.0 0.0 0.0"/>
             </xacro:unless>
@@ -30,5 +30,5 @@
         </joint>
         <link name="${prefix}wheel_link">
-            <xacro:unless value="${gazebo_classic or gazebo_ignition}">
+            <xacro:unless value="${gazebo_ignition}">
                 <visual>
                     <xacro:if value="${hq}">
@@ -72,5 +72,5 @@
             </inertial>
         </link>
-        <xacro:if value="${gazebo_classic or gazebo_ignition}">
+        <xacro:if value="${gazebo_ignition}">
             <gazebo reference="${prefix}wheel_link">
                 <collision>
