Commit message: working basic robots after removing references

File: robots/rbkairos/rbkairos_plus.urdf.xacro (robot description, xacro)
@@ -10,5 +10,4 @@
   <xacro:include filename="$(find robotnik_description)/simulators/gazebo_ignition/rbkairos/rbkairos_control.urdf.xacro" />
   <xacro:include filename="$(find robotnik_sensors)/urdf/all_sensors.urdf.xacro" />
-  <xacro:include filename="$(find robotnik_description)/urdf/structures/rbkairos_chassis/structure_hokuyo.urdf.xacro" />
   <xacro:include filename="$(find ur_description)/urdf/ur_macro.xacro" />
   <!-- Properties and Arguments -->

File: robots/rbrobout/rbrobout.urdf.xacro (robot description, xacro)
@@ -6,4 +6,5 @@
   <!-- Import all posible elements defined in the urdf.xacro files. All these elements are defined as macro:xacros -->
   <xacro:include filename="$(find robotnik_description)/urdf/bases/rbrobout/rbrobout_base.urdf.xacro" />
+  <xacro:include filename="$(find robotnik_description)/urdf/base_hw/rbrobout.ros2_control.urdf" />
   <xacro:include filename="$(find robotnik_description)/simulators/gazebo_classic/rbrobout/rbrobout_control.urdf.xacro" />
   <xacro:include filename="$(find robotnik_description)/simulators/gazebo_ignition/rbrobout/rbrobout_control.urdf.xacro" />

File: robots/rbrobout/rbrobout_plus.urdf.xacro (robot description, xacro)
@@ -6,11 +6,12 @@
   <!-- Import all posible elements defined in the urdf.xacro files. All these elements are defined as macro:xacros -->
   <xacro:include filename="$(find robotnik_description)/urdf/bases/rbrobout/rbrobout_base.urdf.xacro" />
+  <xacro:include filename="$(find robotnik_description)/urdf/bases/rbrobout/rbrobout_top_cover.urdf.xacro" />
+  <xacro:include filename="$(find robotnik_description)/urdf/bases/rbrobout/rbrobout_cameras_cover.urdf.xacro" />
   <xacro:include filename="$(find robotnik_description)/urdf/base_hw/rbrobout.ros2_control.urdf" />
   <xacro:include filename="$(find robotnik_description)/simulators/gazebo_classic/rbrobout/rbrobout_control.urdf.xacro" />
+  <xacro:include filename="$(find robotnik_description)/simulators/gazebo_ignition/rbrobout/rbrobout_control.urdf.xacro" />
   <xacro:include filename="$(find robotnik_sensors)/urdf/all_sensors.urdf.xacro" />
-  <xacro:include filename="$(find robotnik_description)/urdf/structures/rbrobout/top_cover.urdf.xacro" />
-  <xacro:include filename="$(find robotnik_description)/urdf/structures/rbrobout/cameras_cover.urdf.xacro" />
   <xacro:include filename="$(find ur_description)/urdf/ur_macro.xacro" />
-  <xacro:include filename="$(find ewellix_description)/urdf/ewellix_lift_900mm.urdf.xacro" />
+  <!-- xacro:include filename="$(find ewellix_description)/urdf/ewellix_lift_900mm.urdf.xacro" / -->
   <!-- Properties and Arguments -->
   <xacro:arg name="namespace" default="robot"/>
@@ -59,11 +60,13 @@
       <origin xyz="0 0 0" rpy="0 0 0"/>
   </xacro:top_cover>
-  <xacro:ewellix_lift_900mm prefix="$(arg prefix)lift_" parent="$(arg prefix)base_link">
+  <!-- xacro:ewellix_lift_900mm prefix="$(arg prefix)lift_" parent="$(arg prefix)base_link">
       <origin xyz="${lift_position_x} 0 ${lift_position_z}" rpy="0 0 0"/>
-  </xacro:ewellix_lift_900mm>
+  </xacro:ewellix_lift_900mm-->
+<!-- parent="$(arg prefix)lift_ewellix_lift_top_link"
+      -->
   <xacro:ur_robot
       tf_prefix="$(arg prefix)arm_"
       name="$(arg ur_type)"
-      parent="$(arg prefix)lift_ewellix_lift_top_link"
+      parent="$(arg prefix)base_link"
       joint_limits_parameters_file="$(arg joint_limit_params)"
       kinematics_parameters_file="$(arg kinematics_params)"

File: robots/rbsummit/rbsummit.urdf.xacro (robot description, xacro)
@@ -12,7 +12,4 @@
 	<!-- Import all available sensors -->
 	<xacro:include filename="$(find robotnik_sensors)/urdf/all_sensors.urdf.xacro" />
-	<!-- Import antenna -->
-	<xacro:include filename="$(find robotnik_description)/urdf/structures/sensor_support/structure_teltonika.urdf.xacro" />
-	<xacro:include filename="$(find robotnik_description)/urdf/structures/sensor_support/antena-combo-5G-teltonika.urdf.xacro" />
 	<!-- ***************** -->
 	<!-- Sensor parameters -->
@@ -58,57 +55,24 @@
 	<!-- Custom Sensors -->
 	<!-- IMU -->
-	<xacro:sensor_vectornav
-		frame_prefix="$(arg prefix)imu_"
-		parent="$(arg prefix)base_link"
-	>
-		<origin
-			xyz="${imu_offset_x} ${imu_offset_y} ${imu_offset_z}"
-			rpy="0 0 0"
-		/>
-	</xacro:sensor_vectornav>
-	<!-- 3d laser -->
-	<!-- <xacro:sensor_robosense_rslidar_16
-		frame_prefix="rbsummit_top_3d_laser_"
-		parent="rbsummit_base_link"
-		gpu="$(arg gpu)"
+    <xacro:sensor_vectornav
+        frame_prefix="$(arg prefix)vectornav_"
+        parent="$(arg prefix)base_link"
+        node_namespace="$(arg namespace)"
         gazebo_classic="$(arg gazebo_classic)"
-        gazebo_ignition="$(arg gazebo_ignition)"
-	>
-		<origin
-			xyz="${top_laser_offset_x} ${top_laser_offset_y} ${top_laser_offset_z}"
-			rpy="0 0 0"
-		/>
-	</xacro:sensor_robosense_rslidar_16> -->
-	<!-- ptz camera -->
-	<!-- <xacro:sensor_axis_m5013
-		frame_prefix="rbsummit_front_ptz_camera_"
-		parent="rbsummit_base_link"
-	>
-		<origin
-			xyz="${front_ptz_camera_offset_x} ${front_ptz_camera_offset_y} ${front_ptz_camera_offset_z}"
-			rpy="0 ${front_ptz_camera_offset_t} 0"
-		/>
-	</xacro:sensor_axis_m5013> -->
-	<!-- <xacro:sensor_antena_combo_5G_teltonika
-		prefix="rbsummit_antenna"
-		parent="rbsummit_base_link"
-	>
-		<origin
-			xyz="${antenna_offset_x} ${antenna_offset_y} ${antenna_offset_z}"
-			rpy="0 0 0"
-		/>
-	</xacro:sensor_antena_combo_5G_teltonika> -->
+        gazebo_ignition="$(arg gazebo_ignition)">
+        <origin xyz="${imu_offset_x} ${imu_offset_y} ${imu_offset_z}" rpy="0 0 0"/>
+    </xacro:sensor_vectornav>
 	<!-- Controllers -->
-  <xacro:if value="$(arg gazebo_classic)">
-    <xacro:rbsummit_gz_classic_control namespace="$(arg namespace)" prefix="$(arg prefix)"/>
+    <xacro:if value="$(arg gazebo_classic)">
+      <xacro:rbsummit_gz_classic_control namespace="$(arg namespace)" prefix="$(arg prefix)"/>
         <xacro:ros_planar_move_gazebo_classic/>
-  </xacro:if>
-  <xacro:if value="$(arg gazebo_ignition)">
-    <xacro:rbsummit_gz_ignition_control namespace="$(arg namespace)" prefix="$(arg prefix)"/>
-  </xacro:if>
+    </xacro:if>
+    <xacro:if value="$(arg gazebo_ignition)">
+      <xacro:rbsummit_gz_ignition_control namespace="$(arg namespace)" prefix="$(arg prefix)"/>
+    </xacro:if>
     <xacro:unless value="$(arg gazebo_classic)">
-        <xacro:unless value="$(arg gazebo_ignition)">
-            <xacro:rbsummit_base_hw_controller/>
-        </xacro:unless>
+      <xacro:unless value="$(arg gazebo_ignition)">
+        <xacro:rbsummit_base_hw_controller/>
+      </xacro:unless>
     </xacro:unless>
 </robot>

File: robots/rbtheron/rbtheron.urdf.xacro (robot description, xacro)
@@ -13,6 +13,4 @@
 	<!-- Import all available sensors -->
 	<xacro:include filename="$(find robotnik_sensors)/urdf/all_sensors.urdf.xacro" />
-	<!-- Import Elevator -->
-	<xacro:include filename="$(find robotnik_description)/urdf/structures/elevator/rb_theron_elevator.urdf.xacro"/>
 	<!-- ***************** -->
 	<!-- Global parameters -->
@@ -22,26 +20,22 @@
 	<!-- Flag to select the high or low quality model -->
 	<xacro:property name="hq" value="true" />
-	<!-- ELEVATOR PARAMETERS -->
-	<xacro:property name="elevator_x" value="0.0" />
-	<xacro:property name="elevator_y" value="0.0" />
-	<xacro:property name="elevator_z" value="0.2238" />
 	<xacro:arg name="namespace" default="robot"/>
 	<xacro:arg name="prefix" default="robot_"/>
 	<xacro:arg name="gazebo_classic" default="false"/>
 	<xacro:arg name="gazebo_ignition" default="false"/>
-    <!-- <xacro:arg name="has_elevator" default="false" /> -->
 	<!-- Here we create the robot using the xacro:macro imported at the beggining of this file -->
 	<xacro:rbtheron prefix="$(arg prefix)" hq="${hq}"/>
-  	<!-- PENDIENTE DE ACTUALIZAR ROBOTNIK_SENSORS -->
-	<!-- ELEVATOR_PLATFORM -->
-	<!-- <xacro:if value="$(arg has_elevator)">
-		<xacro:elevator_platform robot_id="rbtheron_elevator" parent="rbtheron_base_link" hq="${hq}">
-			<origin xyz="${elevator_x} -${elevator_y} ${elevator_z}" rpy="1.5708 0 1.5708"/>
-		</xacro:elevator_platform>
-	</xacro:if> -->
 	<!-- SENSORS -->
-	<!-- <xacro:sensor_vectornav prefix="rbtheron_" parent="rbtheron_base_link" topic="imu/data">
-		<origin xyz="-0.1975 0.0 0.1598" rpy="0 0 0"/>
-    </xacro:sensor_vectornav> -->
+    <xacro:property name="imu_offset_x" value="-0.1975"/>
+    <xacro:property name="imu_offset_y" value="0.0"/>
+    <xacro:property name="imu_offset_z" value="0.1598"/>
+    <xacro:sensor_vectornav
+        frame_prefix="$(arg prefix)vectornav_"
+        parent="$(arg prefix)base_link"
+        node_namespace="$(arg namespace)"
+        gazebo_classic="$(arg gazebo_classic)"
+        gazebo_ignition="$(arg gazebo_ignition)">
+        <origin xyz="${imu_offset_x} ${imu_offset_y} ${imu_offset_z}" rpy="0 0 0"/>
+    </xacro:sensor_vectornav>
 	<!-- Controllers -->
 	<xacro:if value="$(arg gazebo_classic)">

File: robots/rbvogui/rbvogui.urdf.xacro (robot description, xacro)
@@ -9,8 +9,8 @@
     <xacro:include filename="$(find robotnik_description)/urdf/bases/rbvogui/rbvogui_base.urdf.xacro" />
     <xacro:include filename="$(find robotnik_description)/urdf/base_hw/rbvogui.ros2_control.urdf" />
+    <xacro:include filename="$(find robotnik_description)/simulators/gazebo_classic/rbvogui/rbvogui_control.urdf.xacro" />
     <xacro:include filename="$(find robotnik_description)/simulators/gazebo_ignition/rbvogui/rbvogui_control.urdf.xacro" />
     <!-- Import all available sensors -->
     <xacro:include filename="$(find robotnik_sensors)/urdf/all_sensors.urdf.xacro" />
-    <xacro:include filename="$(find robotnik_description)/urdf/structures/sensor_support/gps_mast.urdf.xacro" />
     <!-- Flag to select the high or low quality model -->
     <xacro:property name="hq" value="true" />

File: urdf/bases/rbkairos/rbkairos_base.urdf.xacro (robot description, xacro)
@@ -7,5 +7,5 @@
   	<!-- Import summit XL base elements -->
 	<xacro:include filename="$(find robotnik_description)/urdf/bodies/rbkairos/rbkairos_plus_body.urdf.xacro" />
-  	<xacro:include filename="$(find robotnik_description)/urdf/wheels/omni_wheel/omni_wheel.urdf.xacro" />
+  	<xacro:include filename="$(find robotnik_description)/urdf/wheels/omni_wheel/rbkairos_omni_wheel.urdf.xacro" />
   	<xacro:property name="PI" value="3.1415926535897931"/>
   	<!-- Wheel parameters -->
@@ -19,14 +19,14 @@
   		<!-- Here we create the robot elements using the xacro:macros imported at the beggining of this file -->
   		<xacro:rbkairos_plus_body prefix="${prefix}"/>
-  		<xacro:omni_wheel robot_id="${prefix}front_right" parent="${prefix}base_link" reflect="false" hq="true">
+  		<xacro:omni_wheel prefix="${prefix}front_right_" parent="${prefix}base_link" reflect="false" hq="true">
   			<origin xyz="${wheel_offset_x} -${wheel_offset_y} ${wheel_offset_z}" rpy="0 0 ${PI/4}"/>
   		</xacro:omni_wheel>
-  		<xacro:omni_wheel robot_id="${prefix}front_left" parent="${prefix}base_link" reflect="true" hq="true">
+  		<xacro:omni_wheel prefix="${prefix}front_left_" parent="${prefix}base_link" reflect="true" hq="true">
   			<origin xyz="${wheel_offset_x} ${wheel_offset_y} ${wheel_offset_z}" rpy="0 0 ${-PI/4}"/>
   		</xacro:omni_wheel>
-  		<xacro:omni_wheel robot_id="${prefix}back_left" parent="${prefix}base_link" reflect="false" hq="true">
+  		<xacro:omni_wheel prefix="${prefix}back_left_" parent="${prefix}base_link" reflect="false" hq="true">
   			<origin xyz="-${wheel_offset_x} ${wheel_offset_y} ${wheel_offset_z}" rpy="0 0 ${PI/4}"/>
   		</xacro:omni_wheel>
-  		<xacro:omni_wheel robot_id="${prefix}back_right" parent="${prefix}base_link" reflect="true" hq="true">
+  		<xacro:omni_wheel prefix="${prefix}back_right_" parent="${prefix}base_link" reflect="true" hq="true">
   			<origin xyz="-${wheel_offset_x} -${wheel_offset_y} ${wheel_offset_z}" rpy="0 0 ${-PI/4}"/>
   		</xacro:omni_wheel>

File: urdf/bases/rbrobout/rbrobout_base.urdf.xacro (robot description, xacro)
@@ -18,5 +18,5 @@
 	<!-- Flag to select the high or low quality model -->
 	<xacro:property name="hq" value="true" />
-  <xacro:macro name="rbrobout" params="prefix:=robot_">
+    <xacro:macro name="rbrobout" params="prefix:=robot_">
 		<!-- *************** -->
 		<!-- Robots Elements -->
@@ -25,14 +25,14 @@
 		<xacro:rbrobout_body prefix="${prefix}" />
 		<!-- Wheels -->
-		<xacro:rbrobout_omni_wheel prefix="${prefix}front_right" parent="${prefix}base_link" reflect="false" hq="${hq}">
+		<xacro:rbrobout_omni_wheel prefix="${prefix}front_right_" parent="${prefix}base_link" reflect="false" hq="${hq}">
 			<origin xyz="${wheel_offset_x} -${wheel_offset_y} ${wheel_offset_z}" rpy="0 0 ${PI/4}"/>
 		</xacro:rbrobout_omni_wheel>
-		<xacro:rbrobout_omni_wheel prefix="${prefix}front_left" parent="${prefix}base_link" reflect="true" hq="${hq}">
+		<xacro:rbrobout_omni_wheel prefix="${prefix}front_left_" parent="${prefix}base_link" reflect="true" hq="${hq}">
 			<origin xyz="${wheel_offset_x} ${wheel_offset_y} ${wheel_offset_z}" rpy="0 0 ${-PI/4}"/>
 		</xacro:rbrobout_omni_wheel>
-		<xacro:rbrobout_omni_wheel prefix="${prefix}back_left" parent="${prefix}base_link" reflect="false" hq="${hq}">
+		<xacro:rbrobout_omni_wheel prefix="${prefix}back_left_" parent="${prefix}base_link" reflect="false" hq="${hq}">
 			<origin xyz="-${wheel_offset_x} ${wheel_offset_y} ${wheel_offset_z}" rpy="0 0 ${PI/4}"/>
 		</xacro:rbrobout_omni_wheel>
-		<xacro:rbrobout_omni_wheel prefix="${prefix}back_right" parent="${prefix}base_link" reflect="true" hq="${hq}">
+		<xacro:rbrobout_omni_wheel prefix="${prefix}back_right_" parent="${prefix}base_link" reflect="true" hq="${hq}">
 			<origin xyz="-${wheel_offset_x} -${wheel_offset_y} ${wheel_offset_z}" rpy="0 0 ${-PI/4}"/>
 		</xacro:rbrobout_omni_wheel>

File: urdf/bases/rbsummit/rbsummit_base.xacro (robot description, xacro)
@@ -10,6 +10,4 @@
 	<xacro:property name="wheel_offset_z" value="0.0" />
     <xacro:macro name="rbsummit" params="prefix:=robot_ hq:=true">
-		<xacro:property name="mesh_file_left" value="robotnik_description/meshes/wheels/rubber_wheel/rubber_wheel_left" />
-		<xacro:property name="mesh_file_right" value="robotnik_description/meshes/wheels/rubber_wheel/rubber_wheel_right" />
 		<!-- *************** -->
 		<!-- Robots Elements -->
@@ -19,14 +17,14 @@
 		<xacro:rbsummit_body prefix="${prefix}" hq="${hq}" />
 		<!-- Summit XL wheels -->
-		<xacro:rubber_wheel robot_id="${prefix}front_right" parent="${prefix}base_link" reflect="false" hq="${hq}" mesh_file="${mesh_file_right}">
+		<xacro:rubber_wheel robot_id="${prefix}front_right" parent="${prefix}base_link" reflect="false" hq="${hq}">
 			<origin xyz="${wheel_offset_x} -${wheel_offset_y} ${wheel_offset_z}" rpy="0 0 0"/>
 		</xacro:rubber_wheel>
-		<xacro:rubber_wheel robot_id="${prefix}front_left" parent="${prefix}base_link" reflect="false" hq="${hq}" mesh_file="${mesh_file_left}">
+		<xacro:rubber_wheel robot_id="${prefix}front_left" parent="${prefix}base_link" reflect="true" hq="${hq}">
 			<origin xyz="${wheel_offset_x} ${wheel_offset_y} ${wheel_offset_z}" rpy="0 0 0"/>
 		</xacro:rubber_wheel>
-		<xacro:rubber_wheel robot_id="${prefix}back_left" parent="${prefix}base_link" reflect="false" hq="${hq}" mesh_file="${mesh_file_left}">
+		<xacro:rubber_wheel robot_id="${prefix}back_left" parent="${prefix}base_link" reflect="true" hq="${hq}">
 			<origin xyz="-${wheel_offset_x} ${wheel_offset_y} ${wheel_offset_z}" rpy="0 0 0"/>
 		</xacro:rubber_wheel>
-		<xacro:rubber_wheel robot_id="${prefix}back_right" parent="${prefix}base_link" reflect="false" hq="${hq}" mesh_file="${mesh_file_right}">
+		<xacro:rubber_wheel robot_id="${prefix}back_right" parent="${prefix}base_link" reflect="false" hq="${hq}">
 			<origin xyz="-${wheel_offset_x} -${wheel_offset_y} ${wheel_offset_z}" rpy="0 0 0"/>
 		</xacro:rubber_wheel>

File: urdf/bases/rbtheron/rbtheron_base.xacro (robot description, xacro)
@@ -6,5 +6,5 @@
 	<xacro:include filename="$(find robotnik_description)/urdf/wheels/rubber_wheel/rubber_wheel_150.urdf.xacro" />
 	<!-- Import casters -->
-	<xacro:include filename="$(find robotnik_description)/urdf/wheels/caster_wheel/rb_theron_caster.urdf.xacro" />
+	<xacro:include filename="$(find robotnik_description)/urdf/wheels/caster_wheel/rbtheron_caster.urdf.xacro" />
 	<!-- Wheel parameters -->
 	<xacro:property name="wheel_offset_x" value="0" />

File: urdf/bodies/rbrobout/rbrobout_body.urdf.xacro (robot description, xacro)
@@ -2,7 +2,7 @@
 <robot name="rbrobout" xmlns:xacro="http://wiki.ros.org/xacro">
   <xacro:macro name="rbrobout_body" params="prefix:=robot_">
-      <!-- Robot mechanical and motor parameters -->
-      <xacro:property name="PI" value="3.1415926535897931"/>
-     <xacro:property name="wheel_radius" value="0.127" />
+    <!-- Robot mechanical and motor parameters -->
+    <xacro:property name="PI" value="3.1415926535897931"/>
+    <xacro:property name="wheel_radius" value="0.127" />
       <!-- BASE FOOTPRINT -->
         <link name="${prefix}base_footprint">
@@ -29,5 +29,5 @@
         <origin xyz="0 0 0" rpy="0 0 0" />
         <geometry>
-        <mesh filename="package://robotnik_description/meshes/bases/rbrobout/robout_chassis.stl"/>
+        <mesh filename="package://robotnik_description/meshes/bases/rbrobout/rbrobout_chassis.stl"/>
         </geometry>
         <material name="darkgrey">
@@ -38,5 +38,5 @@
              <origin xyz="0 0 0" rpy="0 0 0 " />
              <geometry>
-               <mesh filename="package://robotnik_description/meshes/bases/rbrobout/robout_chassis.stl"/>
+               <mesh filename="package://robotnik_description/meshes/bases/rbrobout/rbrobout_chassis.stl"/>
              </geometry>
           </collision>

File: urdf/bodies/rbsummit/rbsummit_body.urdf.xacro (robot description, xacro)
@@ -1,5 +1,5 @@
 <?xml version="1.0"?>
 <robot name="summit_xl" xmlns:xacro="http://wiki.ros.org/xacro">
-  <xacro:include filename="$(find robotnik_description)/urdf/structures/inertia.urdf.xacro" />
+  <xacro:include filename="$(find robotnik_description)/urdf/inertia.urdf.xacro" />
   <xacro:macro name="rbsummit_body" params="prefix:=robot_ hq:=true">
 	  <!-- Robot mechanical and motor parameters -->
