Commit message: working basic robots after removing references

File: urdf/wheels/omni_wheel/rbrobout_omni_wheel.urdf.xacro (robot description, xacro)
@@ -1,60 +1,112 @@
 <?xml version="1.0"?>
-<robot name="wheel" xmlns:xacro="http://wiki.ros.org/xacro">
-  <xacro:property name="M_PI" value="3.1415926535897931" />
-  <!-- Wheels -->
-  <xacro:property name="omni_wheel_radius" value="0.127" />
-  <xacro:property name="omni_wheel_height" value="0.087" />
-  <xacro:property name="omni_wheel_mass" value="6.5" /> <!-- in kg-->
-  <xacro:macro name="cylinder_inertia" params="m r h">
-    <inertia  ixx="${m*(3*r*r+h*h)/12}" ixy = "0" ixz = "0"
-              iyy="${m*r*r/2}" iyz = "0"
-              izz="${m*(3*r*r+h*h)/12}" />
-  </xacro:macro>
-  <xacro:macro name="rbrobout_omni_wheel" params="prefix parent *origin reflect hq">
-    <joint name="${prefix}_wheel_joint" type="continuous">
-      <parent link="${parent}"/>
-      <child link="${prefix}_wheel_link"/>
-      <xacro:insert_block name="origin" />
-      <axis xyz="0 1 0" rpy="0 0 0" />
-      <limit effort="100" velocity="100"/>
-      <joint_properties damping="0.0" friction="0.0"/>
-    </joint>
-    <link name="${prefix}_wheel_link">
-      <visual>
-        <xacro:if value="${hq}">
-          <origin xyz="0 0 0" rpy="${PI/2} 0 0" />
-          <geometry>
-            <mesh filename="package://robotnik_description/meshes/wheels/omni_wheel/robout_wheel.stl" />
-          </geometry>
-        </xacro:if>
-        <xacro:unless value="${hq}">
-          <origin xyz="0 0 0" rpy="0 0 0" />
-          <geometry>
-            <sphere radius="${omni_wheel_radius}" />
-          </geometry>
-        </xacro:unless>
-        <material name="darkgrey">
-           <color rgba="0.2 0.2 0.2 1"/>
-        </material>
-      </visual>
-      <collision>
-				<origin xyz="0 0 0" rpy="${PI/2} 0 0" />
-        <geometry>
-					<cylinder length="${omni_wheel_height}" radius="${omni_wheel_radius}" />
-        </geometry>
-      </collision>
-      <inertial>
-        <mass value="${omni_wheel_mass}" />
-        <origin xyz="0 0 0" />
-        <xacro:cylinder_inertia  m="${omni_wheel_mass}" r="${omni_wheel_radius}" h="${omni_wheel_height}" />
-      </inertial>
-    </link>
-    <gazebo reference="${prefix}_wheel_link">
-      <mu1>0.0</mu1>
-      <mu2>0.0</mu2>
-      <kp>0</kp>
-      <kd>0</kd>
-      <fdir1>0 0 0</fdir1>
-    </gazebo>
-  </xacro:macro>
+<robot name="wheel" xmlns:xacro="http://wiki.ros.org/xacro" xmlns:gz="http://gazebosim.org/schema">
+    <xacro:property name="M_PI" value="3.1415926535897931" />
+    <!-- Wheels -->
+    <xacro:property name="omni_wheel_radius" value="0.127" />
+    <xacro:property name="omni_wheel_height" value="0.087" />
+    <xacro:property name="omni_wheel_mass" value="6.5" /> <!-- in kg-->
+    <xacro:macro name="cylinder_inertia" params="m r h">
+        <inertia ixx="${m*(3*r*r+h*h)/12}" ixy="0" ixz="0"
+            iyy="${m*r*r/2}" iyz="0"
+            izz="${m*(3*r*r+h*h)/12}" />
+    </xacro:macro>
+    <xacro:macro name="rbrobout_omni_wheel" params="prefix parent *origin reflect hq">
+        <joint name="${prefix}wheel_joint" type="continuous">
+            <parent link="${parent}" />
+            <child link="${prefix}wheel_link" />
+            <xacro:insert_block name="origin" />
+            <axis xyz="0 1 0" rpy="0 0 0" />
+            <limit effort="100000" velocity="100" />
+            <!-- <joint_properties damping="1.0" friction="1.0"/> -->
+        </joint>
+        <link name="${prefix}wheel_link">
+            <visual>
+                <origin xyz="0 0 0" rpy="0 0 0" />
+                <geometry>
+                    <box size="0.01 0.01 0.01"/>
+                </geometry>
+                <material name="darkgrey">
+                    <color rgba="0.2 0.2 0.2 1" />
+                </material>
+            </visual>
+            <collision>
+                <origin xyz="0 0 0" rpy="0 0 0" />
+                <geometry>
+                    <sphere radius="${omni_wheel_radius}" />
+                </geometry>
+            </collision>
+            <inertial>
+                <mass value="${omni_wheel_mass}" />
+                <origin xyz="0 0 0" />
+                <xacro:cylinder_inertia m="${omni_wheel_mass}" r="${omni_wheel_radius}"
+                    h="${omni_wheel_height}" />
+            </inertial>
+        </link>
+        <gazebo reference="${prefix}wheel_link">
+            <collision>
+                <surface>
+                    <friction>
+                        <ode>
+                            <mu>1.0</mu>
+                            <mu2>0.0</mu2>
+                            <!-- <slip1>0.2</slip1>
+              <slip2>0.2</slip2> -->
+                            <xacro:if value="${reflect}">
+                                <fdir1 gz:expressed_in="${parent}">1 0 0</fdir1>
+                            </xacro:if>
+                            <xacro:unless value="${reflect}">
+                                <fdir1 gz:expressed_in="${parent}">1 0 0</fdir1>
+                            </xacro:unless>
+                        </ode>
+                    </friction>
+                </surface>
+            </collision>
+        </gazebo>
+        <joint name="${prefix}visual_wheel_joint" type="fixed">
+            <parent link="${parent}" />
+            <child link="${prefix}visual_wheel_link" />
+            <xacro:insert_block name="origin" />
+        </joint>
+        <link name="${prefix}visual_wheel_link">
+            <visual>
+                <xacro:if value="${hq}">
+                    <xacro:if value="${reflect}">
+                    <origin xyz="0 0 0" rpy="${PI/2} 0 ${PI/4}" />
+                        <geometry>
+                            <mesh
+                                filename="package://robotnik_description/meshes/wheels/omni_wheel/robout_wheel.stl" />
+                        </geometry>
+                    </xacro:if>
+                    <xacro:unless value="${reflect}">
+                    <origin xyz="0 0 0" rpy="${-PI/2} 0 ${-PI/4}" />
+                        <geometry>
+                            <mesh
+                                filename="package://robotnik_description/meshes/wheels/omni_wheel/robout_wheel.stl" />
+                        </geometry>
+                    </xacro:unless>
+                </xacro:if>
+                <xacro:unless value="${hq}">
+                    <origin xyz="0 0 0" rpy="0 0 0" />
+                    <geometry>
+                        <sphere radius="${omni_wheel_radius}" />
+                    </geometry>
+                </xacro:unless>
+                <material name="darkgrey">
+                    <color rgba="0.2 0.2 0.2 1" />
+                </material>
+            </visual>
+            <collision>
+                <origin xyz="0 0 0" rpy="0 0 0" />
+                <geometry>
+                    <box size="0.01 0.01 0.01"/>
+                </geometry>
+            </collision>
+            <inertial>
+                <mass value="${omni_wheel_mass}" />
+                <origin xyz="0 0 0" />
+                <xacro:cylinder_inertia m="${omni_wheel_mass}" r="${omni_wheel_radius}"
+                    h="${omni_wheel_height}" />
+            </inertial>
+        </link>
+    </xacro:macro>
 </robot>

File: urdf/wheels/rubber_wheel/rubber_wheel.urdf.xacro (robot description, xacro)
@@ -7,6 +7,5 @@
               izz="${m*(3*r*r+h*h)/12}" />
   </xacro:macro>
-  <xacro:macro name="rubber_wheel" params="robot_id parent *origin reflect hq rubber_wheel_radius:=0.11 rubber_wheel_width:=0.15 rubber_wheel_mass:=6.5
-                                          mesh_file:=robotnik_description/meshes/wheels/rubber_wheel/rubber_wheel_right">
+  <xacro:macro name="rubber_wheel" params="robot_id parent *origin reflect hq rubber_wheel_radius:=0.11 rubber_wheel_width:=0.15 rubber_wheel_mass:=6.5">
 <!--WHEEL TIRE -->
     <joint name="${robot_id}_wheel_joint" type="continuous">
@@ -29,5 +28,5 @@
           </xacro:if>
           <geometry>
-							<mesh filename="package://${mesh_file}.dae" />
+							<mesh filename="package://robotnik_description/meshes/wheels/rubber_wheel/rubber_wheel.dae" />
           </geometry>
         </xacro:if>

Commit message: Fix issues with ur meshes and position of arms

File: robots/rbkairos/rbkairos_plus.urdf.xacro (robot description, xacro)
@@ -48,10 +48,11 @@
       tf_prefix="$(arg prefix)arm_"
       name="$(arg ur_type)"
-      parent="$(arg prefix)base_link"
+      parent="$(arg prefix)top_cover"
       joint_limits_parameters_file="$(arg joint_limit_params)"
       kinematics_parameters_file="$(arg kinematics_params)"
       physical_parameters_file="$(arg physical_params)"
       visual_parameters_file="$(arg visual_params)"
-      sim_gazebo="$(arg gazebo_classic)">
+      sim_gazebo="$(arg gazebo_classic)"
+      sim_ignition="$(arg gazebo_ignition)">
       <origin xyz="0 0 0" rpy="0 0 0"/>
   </xacro:ur_robot>

File: robots/rbrobout/rbrobout_plus.urdf.xacro (robot description, xacro)
@@ -71,5 +71,6 @@
       physical_parameters_file="$(arg physical_params)"
       visual_parameters_file="$(arg visual_params)"
-      sim_gazebo="$(arg gazebo_classic)">
+      sim_gazebo="$(arg gazebo_classic)"
+      sim_ignition="$(arg gazebo_ignition)">
       <origin xyz="0 0 0" rpy="0 0 0"/>
   </xacro:ur_robot>

File: urdf/bodies/rbkairos/rbkairos_plus_body.urdf.xacro (robot description, xacro)
@@ -45,10 +45,10 @@
     <material>Gazebo/Black</material>
   </gazebo>
-  <!-- CHAPAS INOX TAPAS -->
-  <link name="${prefix}base_chapa">
+  <!-- TOP COVER -->
+  <link name="${prefix}top_cover">
   <visual>
     <origin xyz="0 0 0" rpy="0 0 0" />
     <geometry>
-      <mesh filename="package://robotnik_description/meshes/bases/rbkairos/rbkairos_chapas_inox_tapas.stl"/>
+      <mesh filename="package://robotnik_description/meshes/bases/rbkairos/rbkairos_top_cover.stl"/>
     </geometry>
     <material name="darkgrey">
@@ -57,10 +57,10 @@
     </visual>
   </link>
-  <joint name="${prefix}base_tapa_joint" type="fixed">
+  <joint name="${prefix}top_cover_joint" type="fixed">
     <origin xyz="0.0 0 0.56162" rpy="0 0 0" />
     <parent link="${prefix}base_link"/>
-    <child link="${prefix}base_chapa" />
+    <child link="${prefix}top_cover" />
   </joint>
-  <!-- LOGO ROBOTNIK IZQUIERDO -->
+  <!-- LOGO ROBOTNIK LEFT -->
   <link name="${prefix}base_logo_left">
   <visual>
@@ -79,5 +79,5 @@
     <child link="${prefix}base_logo_left" />
   </joint>
-  <!-- LOGO ROBOTNIK DERECHO -->
+  <!-- LOGO ROBOTNIK RIGHT -->
   <link name="${prefix}base_logo_right">
   <visual>
@@ -96,5 +96,5 @@
     <child link="${prefix}base_logo_right" />
   </joint>
-  <!-- LOGO ROBOTNIK FRONTAL -->
+  <!-- LOGO ROBOTNIK FRONT -->
   <link name="${prefix}base_logo_front">
   <visual>
@@ -113,5 +113,5 @@
     <child link="${prefix}base_logo_front" />
   </joint>
-  <!-- LOGO ROBOTNIK TRASERO -->
+  <!-- LOGO ROBOTNIK REAR -->
   <link name="${prefix}base_logo_rear">
   <visual>

Commit message: Sets real Z for UR base in RB-KAIROS+

File: robots/rbkairos/rbkairos_plus.urdf.xacro (robot description, xacro)
@@ -54,5 +54,5 @@
       visual_parameters_file="$(arg visual_params)"
       sim_gazebo="$(arg gazebo_classic)">
-      <origin xyz="0 0 0" rpy="0 0 0"/>
+      <origin xyz="0 0 0.56362" rpy="0 0 0"/>
   </xacro:ur_robot>
   <!-- PENDIENTE DE ACTUALIZAR ROBOTNIK_SENSORS -->

Commit message: Sets real Z for UR in rbkairos plus model

File: robots/rbkairos/rbkairos_plus.urdf.xacro (robot description, xacro)
@@ -46,5 +46,5 @@
       sim_gazebo="$(arg gazebo_classic)"
       sim_ignition="$(arg gazebo_ignition)">
-      <origin xyz="0 0 0" rpy="0 0 0"/>
+      <origin xyz="0 0 0.56362" rpy="0 0 0"/>
   </xacro:ur_robot>
   <!-- PENDIENTE DE ACTUALIZAR ROBOTNIK_SENSORS -->

Commit message: Fix rbkairos_plus arm issues

File: robots/rbkairos/rbkairos_plus.urdf.xacro (robot description, xacro)
@@ -48,13 +48,13 @@
       tf_prefix="$(arg prefix)arm_"
       name="$(arg ur_type)"
-      parent="$(arg prefix)base_link"
+      parent="$(arg prefix)top_cover"
       joint_limits_parameters_file="$(arg joint_limit_params)"
       kinematics_parameters_file="$(arg kinematics_params)"
       physical_parameters_file="$(arg physical_params)"
       visual_parameters_file="$(arg visual_params)"
-      sim_gazebo="$(arg gazebo_classic)">
-      <origin xyz="0 0 0.56362" rpy="0 0 0"/>
+      sim_gazebo="$(arg gazebo_classic)"
+      sim_ignition="$(arg gazebo_ignition)">
+      <origin xyz="0 0 0" rpy="0 0 0"/>
   </xacro:ur_robot>
-  <!-- PENDIENTE DE ACTUALIZAR ROBOTNIK_SENSORS -->
   <!-- IMU -->
     <xacro:sensor_vectornav

Commit message: fix rbkairos_plus issue with arm position

File: robots/rbkairos/rbkairos_plus.urdf.xacro (robot description, xacro)
@@ -48,13 +48,13 @@
       tf_prefix="$(arg prefix)arm_"
       name="$(arg ur_type)"
-      parent="$(arg prefix)base_link"
+      parent="$(arg prefix)top_cover"
       joint_limits_parameters_file="$(arg joint_limit_params)"
       kinematics_parameters_file="$(arg kinematics_params)"
       physical_parameters_file="$(arg physical_params)"
       visual_parameters_file="$(arg visual_params)"
-      sim_gazebo="$(arg gazebo_classic)">
-      <origin xyz="0 0 0.56362" rpy="0 0 0"/>
+      sim_gazebo="$(arg gazebo_classic)"
+      sim_ignition="$(arg gazebo_ignition)">
+      <origin xyz="0 0 0.0" rpy="0 0 0"/>
   </xacro:ur_robot>
-  <!-- PENDIENTE DE ACTUALIZAR ROBOTNIK_SENSORS -->
   <!-- IMU -->
     <xacro:sensor_vectornav

Commit message: working version

File: robots/rbkairos/rbkairos_plus.urdf.xacro (robot description, xacro)
@@ -9,4 +9,8 @@
   <xacro:include
     filename="$(find robotnik_sensors)/urdf/all_sensors.urdf.xacro" />
+  <xacro:include
+    filename="$(find robotnik_sensors)/urdf/depth/intel_realsense_d435i.urdf.xacro" />
+  <xacro:include
+    filename="$(find robotnik_description)/urdf/grippers/suction_gripper/suction_gripper.urdf.xacro" />
   <!-- ARGUMENTS -->
   <xacro:arg
@@ -22,4 +26,7 @@
     name="ur_type"
     default="ur5e" />
+  <xacro:arg
+    name="world_name"
+    default="room_test_world" />
   <!-- RB-KAIROS -->
   <xacro:rbkairos
@@ -37,4 +44,20 @@
       rpy="0 0 0" />
   </xacro:arm_ur>
+  <!-- WRIST CAMERA -->
+  <xacro:sensor_intel_realsense_d435i
+    frame_prefix="$(arg prefix)wrist_rgbd_camera_"
+    parent="$(arg prefix)arm_tool0"
+    node_namespace="$(arg namespace)"
+    node_name="wrist_camera"
+    gazebo_ignition="$(arg gazebo_ignition)">
+    <origin xyz="0.0 -0.055 0.020" rpy="0 -1.5708 1.5708" />
+  </xacro:sensor_intel_realsense_d435i>
+  <!-- SUCTION GRIPPER -->
+  <xacro:suction_gripper
+    prefix="$(arg prefix)vacuum_"
+    parent="$(arg prefix)arm_tool0"
+    ns="$(arg namespace)">
+    <origin xyz="0 0 0" rpy="0 0 0" />
+  </xacro:suction_gripper>
   <!-- IMU -->
   <xacro:sensor_vectornav
@@ -83,3 +106,13 @@
       rpy="0 0 0" />
   </xacro:sensor_intel_realsense_d435>
+  <!-- VACUUM GRIPPER PLUGIN -->
+  <gazebo>
+    <plugin filename="libVacuumGripper.so"
+            name="vacuum_gripper_plugin::VacuumGripper">
+      <suction_link>$(arg prefix)vacuum_link_suction_gripper</suction_link>
+      <contact_topic>/world/$(arg world_name)/model/$(arg namespace)/link/$(arg prefix)vacuum_link_suction_gripper/sensor/$(arg prefix)vacuum_suction_contact_sensor/contact</contact_topic>
+      <cmd_topic>/$(arg namespace)/vacuum_on</cmd_topic>
+      <max_distance>0.15</max_distance>
+    </plugin>
+  </gazebo>
 </robot>

File: robots/rbrobout/rbrobout_plus.urdf.xacro (robot description, xacro)
@@ -23,5 +23,5 @@
   <xacro:arg name="prefix"         default="" />
   <xacro:arg name="gazebo_ignition" default="false" />
-  <xacro:arg name="ur_type"        default="ur5e" />
+  <xacro:arg name="ur_type"        default="ur20" />
   <xacro:arg name="world_name" default="room_test_world"/>
   <!-- RB-ROBOUT BASE -->
