Commit message: Sim working with kairos with snder and zivid camera

File: robots/rbkairos/centauro_rbkairos_plus.urdf.xacro (robot description, xacro)
@@ -70,4 +70,7 @@
     prefix="$(arg prefix)arm_tool_"
     parent="$(arg prefix)arm_tool0"
+    node_namespace="$(arg namespace)"
+    node_name="arm_tool_zivid2"
+    gazebo_ignition="$(arg gazebo_ignition)"
     >
     <origin

File: urdf/structures/tools/onrobot_sander_zivid2.urdf.xacro (robot description, xacro)
@@ -3,8 +3,36 @@
   name="onrobot_sander_zivid2"
   xmlns:xacro="http://www.ros.org/wiki/xacro">
+  <xacro:include
+    filename="$(find robotnik_sensors)/urdf/depth/depth_camera_plugin.urdf.xacro" />
+  <xacro:include
+    filename="$(find robotnik_sensors)/urdf/camera/camera_plugin.urdf.xacro" />
   <!-- ONROBOT SANDER ZIVID2 -->
   <xacro:macro
     name="onrobot_sander_zivid2"
-    params="prefix parent cut_model:=false *origin">
+    params="prefix
+            parent
+            cut_model:=false
+            *origin
+            gazebo_ignition:=false
+            node_name:=zivid2
+            node_namespace:=${None}
+            topic_prefix:=~/">
+    <xacro:if value="${node_namespace == None}">
+      <xacro:property
+        name="node_namespace"
+        value="${node_name}" />
+    </xacro:if>
+    <xacro:property
+      name="zivid2_depth_horizontal_fov"
+      value="52.71264861" />
+    <xacro:property
+      name="zivid2_depth_vertical_fov"
+      value="42.24943829" />
+    <xacro:property
+      name="zivid2_color_horizontal_fov"
+      value="52.71264861" />
+    <xacro:property
+      name="zivid2_color_vertical_fov"
+      value="42.24943829" />
     <!-- Lift base link -->
     <link name="${prefix}tool_link">
@@ -33,5 +61,5 @@
       </collision>
       <inertial>
-        <mass value="0" />
+        <mass value="0.001" />
         <origin
           xyz="0 0 0"
@@ -71,9 +99,79 @@
       <origin
         xyz="0 -0.1155 0.075 "
-        rpy="0.261799 0 0" /><!-- 15 deg 0 0 -->
+        rpy="0 0 0" />
       <parent link="${prefix}tool_link" />
       <child link="${prefix}zivid_link" />
     </joint>
     <link name="${prefix}zivid_link" />
+    <!-- zivid depth joints and links -->
+    <joint
+      name="${prefix}zivid_depth_joint"
+      type="fixed">
+      <origin
+        xyz="0 0 0"
+        rpy="0 0 0" />
+      <parent link="${prefix}zivid_link" />
+      <child link="${prefix}zivid_depth_frame" />
+    </joint>
+    <link name="${prefix}zivid_depth_frame" />
+    <joint
+      name="${prefix}zivid_depth_optical_joint"
+      type="fixed">
+      <origin
+        xyz="0 0 0"
+        rpy="0 0 0" />
+      <parent link="${prefix}zivid_depth_frame" />
+      <child link="${prefix}zivid_depth_optical_frame" />
+    </joint>
+    <link name="${prefix}zivid_depth_optical_frame" />
+    <!-- zivid color joints and links -->
+    <joint
+      name="${prefix}zivid_color_joint"
+      type="fixed">
+      <origin
+        xyz="0 0 0"
+        rpy="0 0 0" />
+      <parent link="${prefix}zivid_link" />
+      <child link="${prefix}zivid_color_frame" />
+    </joint>
+    <link name="${prefix}zivid_color_frame" />
+    <joint
+      name="${prefix}zivid_color_optical_joint"
+      type="fixed">
+      <origin
+        xyz="0 0 0"
+        rpy="0 0 0" />
+      <parent link="${prefix}zivid_color_frame" />
+      <child link="${prefix}zivid_color_optical_frame" />
+    </joint>
+    <link name="${prefix}zivid_color_optical_frame" />
+    <xacro:depth_camera_plugin
+      node_namespace="${node_namespace}"
+      node_name="${node_name}_depth"
+      topic_prefix="${topic_prefix}_depth"
+      gazebo_ignition="${gazebo_ignition}"
+      optical_frame="${prefix}zivid_depth_optical_frame"
+      reference_frame="${prefix}zivid_depth_frame"
+      horizontal_fov="${zivid2_depth_horizontal_fov}"
+      vertical_fov="${zivid2_depth_vertical_fov}"
+      video_width="1280"
+      video_height="720"
+      min_depth="0.700"
+      max_depth="1.700"
+      rate="30" />
+    <xacro:camera_plugin
+      node_namespace="${node_namespace}"
+      node_name="${node_name}_color"
+      topic_prefix="${topic_prefix}_color"
+      gazebo_ignition="${gazebo_ignition}"
+      optical_frame="${prefix}zivid_color_optical_frame"
+      reference_frame="${prefix}zivid_color_frame"
+      horizontal_fov="${zivid2_color_horizontal_fov}"
+      vertical_fov="${zivid2_color_vertical_fov}"
+      video_width="2448"
+      video_height="2048"
+      min_depth="0.700"
+      max_depth="1.700"
+      rate="30" />
     <gazebo reference="${prefix}tool_link">
       <material>Gazebo/Grey</material>

Commit message: centauro kairos URDF updated with photoneo camera in the tool

File: robots/rbkairos/centauro_rbkairos_plus.urdf.xacro (robot description, xacro)
@@ -8,5 +8,5 @@
     filename="$(find robotnik_description)/urdf/arms/ur_macro.urdf.xacro" />
   <xacro:include
-    filename="$(find robotnik_description)/urdf/structures/tools/onrobot_sander_zivid2.urdf.xacro" />
+    filename="$(find robotnik_description)/urdf/structures/tools/onrobot_sander_photoneo_motioncam.urdf.xacro" />
   <xacro:include
     filename="$(find robotnik_sensors)/urdf/all_sensors.urdf.xacro" />
@@ -20,5 +20,5 @@
   <xacro:arg
     name="gazebo_ignition"
-    default="false" />
+    default="true" />
   <xacro:arg
     name="ur_type"
@@ -67,9 +67,9 @@
   </xacro:arm_ur>
   <!-- TOOL -->
-  <xacro:onrobot_sander_zivid2
+  <xacro:onrobot_sander_photoneo_motioncam
     prefix="$(arg prefix)arm_tool_"
     parent="$(arg prefix)arm_tool0"
     node_namespace="$(arg namespace)"
-    node_name="arm_tool_zivid2"
+    node_name="arm_tool_photoneo_motioncam"
     gazebo_ignition="$(arg gazebo_ignition)"
     >
@@ -77,5 +77,5 @@
       xyz="0 0 0"
       rpy="0 0 0" />
-  </xacro:onrobot_sander_zivid2>
+  </xacro:onrobot_sander_photoneo_motioncam>
   <!-- IMU -->
   <xacro:sensor_vectornav
@@ -114,5 +114,5 @@
   </xacro:sensor_sick_microscan3>
   <!-- CAMERAS -->
-  <xacro:sensor_intel_realsense_d435
+  <xacro:sensor_intel_realsense_d435i
     frame_prefix="$(arg prefix)front_rgbd_camera_"
     parent="$(arg prefix)base_link"
@@ -123,4 +123,4 @@
       xyz="0.35850 0.0 0.25062"
       rpy="0 0 0" />
-  </xacro:sensor_intel_realsense_d435>
+  </xacro:sensor_intel_realsense_d435i>
 </robot>

File: urdf/structures/tools/onrobot_sander_photoneo_motioncam.urdf.xacro (robot description, xacro)
@@ -99,5 +99,5 @@
       <origin
         xyz="0 -0.1155 0.075 "
-        rpy="0 0 0" />
+        rpy="${radians(15)} 0 0" />
       <parent link="${prefix}tool_link" />
       <child link="${prefix}photoneo_motioncam_link" />
@@ -141,5 +141,5 @@
       <origin
         xyz="0 0 0"
-        rpy="0 0 0" />
+        rpy="${radians(0)} ${radians(-90)} ${radians(90)}" />
       <parent link="${prefix}photoneo_motioncam_color_frame" />
       <child link="${prefix}photoneo_motioncam_color_optical_frame" />
@@ -152,5 +152,5 @@
       gazebo_ignition="${gazebo_ignition}"
       optical_frame="${prefix}photoneo_motioncam_depth_optical_frame"
-      reference_frame="${prefix}photoneo_motioncam_depth_frame"
+      reference_frame="${prefix}photoneo_motioncam_depth_optical_frame"
       horizontal_fov="${photoneo_motioncam_depth_horizontal_fov}"
       vertical_fov="${photoneo_motioncam_depth_vertical_fov}"
@@ -158,5 +158,5 @@
       video_height="720"
       min_depth="0.700"
-      max_depth="1.700"
+      max_depth="201.700"
       rate="30" />
     <xacro:camera_plugin
@@ -166,5 +166,5 @@
       gazebo_ignition="${gazebo_ignition}"
       optical_frame="${prefix}photoneo_motioncam_color_optical_frame"
-      reference_frame="${prefix}photoneo_motioncam_color_frame"
+      reference_frame="${prefix}photoneo_motioncam_color_optical_frame"
       horizontal_fov="${photoneo_motioncam_color_horizontal_fov}"
       vertical_fov="${photoneo_motioncam_color_vertical_fov}"
@@ -172,43 +172,45 @@
       video_height="2048"
       min_depth="0.700"
-      max_depth="1.700"
+      max_depth="201.700"
       rate="30" />
-    <gazebo reference="${prefix}photoneo_motioncam_color_optical_frame">
-      <sensor name="${prefix}" type="depth">
-          <always_on>true</always_on>
-          <update_rate>15</update_rate>
-          <pose>0 0 0 0 0 0</pose>
-          <camera name="realsense_depth_camera">
-              <horizontal_fov>1.46608</horizontal_fov>
-              <image>
-                  <width>424</width>
-                  <height>240</height>
-                  <format>B8G8R8</format>
-              </image>
-              <clip>
-                  <near>0.05</near>
-                  <far>8</far>
-              </clip>
-          </camera>
-          <!-- https://github.com/mlherd/ros2_turtlebot3_waffle_intel_realsense -->
-          <plugin name="intel_realsense_d430_depth_driver" filename="libgazebo_ros_camera.so">
-              <ros>
-                  <namespace>d430</namespace>
-                  <remapping>${prefix}/image_raw:=color/image_raw</remapping>
-                  <remapping>${prefix}/depth/image_raw:=depth/image_rect_raw</remapping>
-                  <remapping>${prefix}/camera_info:=camera_info</remapping>
-                  <remapping>${prefix}/depth/camera_info:=depth/camera_info</remapping>
-                  <remapping>${prefix}/points:=depth/points</remapping>
-              </ros>
-              <camera_name>${prefix}</camera_name>
-              <frame_name>${prefix}photoneo_motioncam_color_optical_frame</frame_name>
-              <hack_baseline>0.07</hack_baseline>
-              <min_depth>0.05</min_depth>
-              <max_depth>8.0</max_depth>
-          </plugin>
-      </sensor>
-      <material>Gazebo/Grey</material>
-      <gravity>true</gravity>
-    </gazebo>
+    <xacro:unless value="${gazebo_ignition}">
+      <gazebo reference="${prefix}photoneo_motioncam_color_optical_frame">
+        <sensor name="${prefix}" type="depth">
+            <always_on>true</always_on>
+            <update_rate>15</update_rate>
+            <pose>0 0 0 0 0 0</pose>
+            <camera name="realsense_depth_camera">
+                <horizontal_fov>1.46608</horizontal_fov>
+                <image>
+                    <width>424</width>
+                    <height>240</height>
+                    <format>B8G8R8</format>
+                </image>
+                <clip>
+                    <near>0.05</near>
+                    <far>8</far>
+                </clip>
+            </camera>
+            <!-- https://github.com/mlherd/ros2_turtlebot3_waffle_intel_realsense
+            <plugin name="intel_realsense_d430_depth_driver" filename="libgazebo_ros_camera.so">
+                <ros>
+                    <namespace>d430</namespace>
+                    <remapping>${prefix}/image_raw:=color/image_raw</remapping>
+                    <remapping>${prefix}/depth/image_raw:=depth/image_rect_raw</remapping>
+                    <remapping>${prefix}/camera_info:=camera_info</remapping>
+                    <remapping>${prefix}/depth/camera_info:=depth/camera_info</remapping>
+                    <remapping>${prefix}/points:=depth/points</remapping>
+                </ros>
+                <camera_name>${prefix}</camera_name>
+                <frame_name>${prefix}photoneo_motioncam_color_optical_frame</frame_name>
+                <hack_baseline>0.07</hack_baseline>
+                <min_depth>0.05</min_depth>
+                <max_depth>8.0</max_depth>
+            </plugin> -->
+        </sensor>
+        <material>Gazebo/Grey</material>
+        <gravity>true</gravity>
+      </gazebo>
+    </xacro:unless>
   </xacro:macro>
 </robot>
