Commit message: moved vogui xl to its own folder

File: robots/rbvogui_xl/rbvogui_xl.urdf.xacro (robot description, xacro)
@@ -6,7 +6,7 @@
     <!-- First we import all posible elements defined in the urdf.xacro files. All these elements are defined as macro:xacros -->
     <!-- Import rbvogui_xl base elements-->
-    <xacro:include filename="$(find robotnik_description)/urdf/bases/rbvogui/rbvogui_xl_base.urdf.xacro" />
+    <xacro:include filename="$(find robotnik_description)/urdf/bases/rbvogui_xl/rbvogui_xl_base.urdf.xacro" />
     <xacro:include filename="$(find robotnik_description)/urdf/base_hw/rbvogui_xl.ros2_control.urdf" />
-    <xacro:include filename="$(find robotnik_description)/simulators/gazebo_ignition/rbvogui/rbvogui_xl_control.urdf.xacro" />
+    <xacro:include filename="$(find robotnik_description)/simulators/gazebo_ignition/rbvogui_xl/rbvogui_xl_control.urdf.xacro" />
     <!-- Import all available sensors -->
     <xacro:include filename="$(find robotnik_sensors)/urdf/all_sensors.urdf.xacro" />

File: simulators/gazebo_ignition/rbvogui_xl/rbvogui_xl_control.urdf.xacro (robot description, xacro)
@@ -6,5 +6,5 @@
             <robot_param>robot_description</robot_param>
             <robot_param_node>robot_state_publisher</robot_param_node>
-            <parameters>$(find robotnik_description)/simulators/gazebo_ignition/rbvogui/rbvogui_xl_controller_params.yaml</parameters>
+            <parameters>$(find robotnik_description)/simulators/gazebo_ignition/rbvogui_xl/rbvogui_xl_controller_params.yaml</parameters>
             <ros>
                 <namespace>/${namespace}</namespace>

File: urdf/bases/rbvogui_xl/rbvogui_xl_base.urdf.xacro (robot description, xacro)
@@ -7,5 +7,5 @@
     <!-- First we import all posible elements defined in the urdf.xacro files. All these elements are defined as macro:xacros -->
     <!-- Import rbvogui_xl base elements-->
-    <xacro:include filename="$(find robotnik_description)/urdf/bodies/rbvogui/rbvogui_xl_body.urdf.xacro" />
+    <xacro:include filename="$(find robotnik_description)/urdf/bodies/rbvogui_xl/rbvogui_xl_body.urdf.xacro" />
     <!-- Import rbvogui_xl wheels -->
     <xacro:include filename="$(find robotnik_description)/urdf/wheels/steering_wheel/steering_wheel_350.urdf.xacro" />

File: urdf/bodies/rbvogui_xl/rbvogui_xl_body.urdf.xacro (robot description, xacro)
@@ -1,5 +1,5 @@
 <?xml version="1.0"?>
 <robot xmlns:xacro="http://www.ros.org/wiki/xacro">
-  <xacro:include filename="$(find robotnik_description)/urdf/bodies/rbvogui/rbvogui_xl_base.gazebo.xacro" />
+  <xacro:include filename="$(find robotnik_description)/urdf/bodies/rbvogui_xl/rbvogui_xl_base.gazebo.xacro" />
   <xacro:macro name="rbvogui_xl_body" params="prefix:=robot_ hq:=true">
     <!-- Robot mechanical and motor parameters -->
@@ -32,10 +32,10 @@
         <xacro:if value="${hq}">
           <geometry>
-            <mesh filename="package://robotnik_description/meshes/bases/rbvogui/rbvogui_xl_chassis.stl"/>
+            <mesh filename="package://robotnik_description/meshes/bases/rbvogui_xl/rbvogui_xl_chassis.stl"/>
           </geometry>
         </xacro:if>
         <xacro:unless value="${hq}">
           <geometry>
-            <mesh filename="package://robotnik_description/meshes/bases/rbvogui/rbvogui_xl_chassis.stl"/>
+            <mesh filename="package://robotnik_description/meshes/bases/rbvogui_xl/rbvogui_xl_chassis.stl"/>
           </geometry>
         </xacro:unless>
@@ -47,5 +47,5 @@
         <origin xyz="0 0 0" rpy="0 0 0 " />
         <geometry>
-          <mesh filename="package://robotnik_description/meshes/bases/rbvogui/rbvogui_xl_chassis.stl"/>
+          <mesh filename="package://robotnik_description/meshes/bases/rbvogui_xl/rbvogui_xl_chassis.stl"/>
         </geometry>
       </collision>
@@ -68,10 +68,10 @@
         <xacro:if value="${hq}">
           <geometry>
-             <mesh filename="package://robotnik_description/meshes/bases/rbvogui/rbvogui_xl_battery.stl"/>
+             <mesh filename="package://robotnik_description/meshes/bases/rbvogui_xl/rbvogui_xl_battery.stl"/>
           </geometry>
         </xacro:if>
         <xacro:unless value="${hq}">
           <geometry>
-             <mesh filename="package://robotnik_description/meshes/bases/rbvogui/rbvogui_xl_battery.stl"/>
+             <mesh filename="package://robotnik_description/meshes/bases/rbvogui_xl/rbvogui_xl_battery.stl"/>
           </geometry>
         </xacro:unless>
@@ -83,5 +83,5 @@
         <origin xyz="0 0 0" rpy="0 0 0 " />
         <geometry>
-           <mesh filename="package://robotnik_description/meshes/bases/rbvogui/rbvogui_xl_battery.stl"/>
+           <mesh filename="package://robotnik_description/meshes/bases/rbvogui_xl/rbvogui_xl_battery.stl"/>
         </geometry>
       </collision>
@@ -99,10 +99,10 @@
         <xacro:if value="${hq}">
           <geometry>
-            <mesh filename="package://robotnik_description/meshes/bases/rbvogui/rbvogui_contactors.stl" />
+            <mesh filename="package://robotnik_description/meshes/bases/rbvogui_xl/rbvogui_contactors.stl" />
           </geometry>
         </xacro:if>
         <xacro:unless value="${hq}">
           <geometry>
-            <mesh filename="package://robotnik_description/meshes/bases/rbvogui/rbvogui_contactors.stl" />
+            <mesh filename="package://robotnik_description/meshes/bases/rbvogui_xl/rbvogui_contactors.stl" />
           </geometry>
         </xacro:unless>
@@ -124,10 +124,10 @@
         <xacro:if value="${hq}">
           <geometry>
-            <mesh filename="package://robotnik_description/meshes/bases/rbvogui/rbvogui_logos.stl" scale="1.24 1.24 1"/>
+            <mesh filename="package://robotnik_description/meshes/bases/rbvogui_xl/rbvogui_logos.stl" scale="1.24 1.24 1"/>
           </geometry>
         </xacro:if>
         <xacro:unless value="${hq}">
           <geometry>
-            <mesh filename="package://robotnik_description/meshes/bases/rbvogui/rbvogui_logos.dae" scale="1.3 1.3 1"/>
+            <mesh filename="package://robotnik_description/meshes/bases/rbvogui_xl/rbvogui_logos.dae" scale="1.3 1.3 1"/>
           </geometry>
         </xacro:unless>
@@ -147,5 +147,5 @@
         <origin xyz="0 0 0" rpy="0 0 0.0" />
           <geometry>
-              <mesh filename="package://robotnik_description/meshes/bases/rbvogui/rbvogui_xl_leds.stl" />
+              <mesh filename="package://robotnik_description/meshes/bases/rbvogui_xl/rbvogui_xl_leds.stl" />
           </geometry>
         <material name="lightgreen">

Commit message: fix: rbvogui_xl_logos and rbvogui_xl_contactors stl

File: robots/rbvogui_xl/rbvogui_xl.urdf.xacro (robot description, xacro)
@@ -68,4 +68,12 @@
         <origin xyz="-0.64555 -0.39595 0.1145" rpy="${PI} 0 -2.35219"/>
     </xacro:sensor_sick_tim571>
+    <xacro:sensor_robosense_helios_16p
+        frame_prefix="$(arg prefix)top_3d_laser_"
+        parent="$(arg prefix)chassis_link"
+        node_namespace="$(arg namespace)"
+        node_name="top_3d_laser"
+        gazebo_ignition="$(arg gazebo_ignition)">
+        <origin xyz="0.60955 0.0 -0.0145" rpy="${PI} 0 0"/>
+    </xacro:sensor_robosense_helios_16p>
 	<!-- Controllers -->
     <xacro:if value="$(arg gazebo_ignition)">

File: urdf/bodies/rbvogui_xl/rbvogui_xl_body.urdf.xacro (robot description, xacro)
@@ -99,10 +99,10 @@
         <xacro:if value="${hq}">
           <geometry>
-            <mesh filename="package://robotnik_description/meshes/bases/rbvogui_xl/rbvogui_contactors.stl" />
+            <mesh filename="package://robotnik_description/meshes/bases/rbvogui_xl/rbvogui_xl_contactors.stl" />
           </geometry>
         </xacro:if>
         <xacro:unless value="${hq}">
           <geometry>
-            <mesh filename="package://robotnik_description/meshes/bases/rbvogui_xl/rbvogui_contactors.stl" />
+            <mesh filename="package://robotnik_description/meshes/bases/rbvogui_xl/rbvogui_xl_contactors.stl" />
           </geometry>
         </xacro:unless>
@@ -124,10 +124,10 @@
         <xacro:if value="${hq}">
           <geometry>
-            <mesh filename="package://robotnik_description/meshes/bases/rbvogui_xl/rbvogui_logos.stl" scale="1.24 1.24 1"/>
+            <mesh filename="package://robotnik_description/meshes/bases/rbvogui_xl/rbvogui_xl_logos.stl" scale="1.24 1.24 1"/>
           </geometry>
         </xacro:if>
         <xacro:unless value="${hq}">
           <geometry>
-            <mesh filename="package://robotnik_description/meshes/bases/rbvogui_xl/rbvogui_logos.dae" scale="1.3 1.3 1"/>
+            <mesh filename="package://robotnik_description/meshes/bases/rbvogui_xl/rbvogui_xl_logos.dae" scale="1.3 1.3 1"/>
           </geometry>
         </xacro:unless>
