Commit message: missing files from standard vogui

File: simulators/gazebo_ignition/rbvogui_xl/rbvogui_xl_control.urdf.xacro (robot description, xacro)
@@ -1,5 +1,5 @@
 <?xml version="1.0"?>
 <robot xmlns:xacro="http://wiki.ros.org/xacro">
-    <xacro:macro name="rbvogui_gz_ignition_control"  params="namespace prefix">
+    <xacro:macro name="rbvogui_xl_gz_ignition_control"  params="namespace prefix">
         <gazebo>
             <plugin name="gz_ros2_control::GazeboSimROS2ControlPlugin" filename="gz_ros2_control-system">
