Commit message: robot: added rbvogui_xl robot (#73)
* added rbvogui_xl robot

* change sensors

* add base_docking_contact link to vogui

* add missing simmulation and remove gazebo stuff

* moved vogui xl to its own folder

* added missing files

* fix: rbvogui_xl_logos and rbvogui_xl_contactors stl

* missing files from standard vogui

* gazebo can use meshes from local built packages

---------

Co-authored-by: Marc Bosch <mbosch@robotnik.es>

File: urdf/bodies/rbvogui_xl/rbvogui_xl_body.urdf.xacro (robot description, xacro)
@@ -1,6 +1,6 @@
 <?xml version="1.0"?>
 <robot xmlns:xacro="http://www.ros.org/wiki/xacro">
-  <xacro:include filename="$(find robotnik_description)/urdf/bodies/rbvogui/rbvogui_base.gazebo.xacro" />
-  <xacro:macro name="rbvogui_body" params="prefix:=robot_ hq:=true">
+  <xacro:include filename="$(find robotnik_description)/urdf/bodies/rbvogui_xl/rbvogui_xl_base.gazebo.xacro" />
+  <xacro:macro name="rbvogui_xl_body" params="prefix:=robot_ hq:=true">
     <!-- Robot mechanical and motor parameters -->
     <xacro:property name="PI" value="3.1415926535897931"/>
@@ -17,5 +17,5 @@
     <!-- Chassis -->
     <joint name="${prefix}chassis_joint" type="fixed">
-      <origin xyz="-0.012 0 0.1775" rpy="0 0 0" />
+      <origin xyz="0 0 0.23376" rpy="0 0 0" />
       <parent link="${prefix}base_link"/>
       <child link="${prefix}chassis_link" />
@@ -32,17 +32,20 @@
         <xacro:if value="${hq}">
           <geometry>
-            <mesh filename="package://robotnik_description/meshes/bases/rbvogui/rbvogui_chassis_color.dae"/>
+            <mesh filename="package://robotnik_description/meshes/bases/rbvogui_xl/rbvogui_xl_chassis.stl"/>
           </geometry>
         </xacro:if>
         <xacro:unless value="${hq}">
           <geometry>
-            <mesh filename="package://robotnik_description/meshes/bases/rbvogui/rbvogui_chassis.stl"/>
+            <mesh filename="package://robotnik_description/meshes/bases/rbvogui_xl/rbvogui_xl_chassis.stl"/>
           </geometry>
         </xacro:unless>
+        <material name="darkgrey">
+          <color rgba="0.1 0.1 0.1 1"/>
+        </material>
       </visual>
       <collision>
         <origin xyz="0 0 0" rpy="0 0 0 " />
         <geometry>
-          <mesh filename="package://robotnik_description/meshes/bases/rbvogui/rbvogui_chassis_color.dae"/>
+          <mesh filename="package://robotnik_description/meshes/bases/rbvogui_xl/rbvogui_xl_chassis.stl"/>
         </geometry>
       </collision>
@@ -50,5 +53,5 @@
     <!-- Battery -->
     <joint name="${prefix}battery_joint" type="fixed">
-      <origin xyz="0.02952 0 0" rpy="0 0 0 " />
+      <origin xyz="0 0 0" rpy="0 0 0 " />
       <parent link="${prefix}chassis_link"/>
       <child link="${prefix}battery_link" />
@@ -65,10 +68,10 @@
         <xacro:if value="${hq}">
           <geometry>
-             <mesh filename="package://robotnik_description/meshes/bases/rbvogui/rbvogui_battery.stl"/>
+             <mesh filename="package://robotnik_description/meshes/bases/rbvogui_xl/rbvogui_xl_battery.stl"/>
           </geometry>
         </xacro:if>
         <xacro:unless value="${hq}">
           <geometry>
-             <mesh filename="package://robotnik_description/meshes/bases/rbvogui/rbvogui_battery.stl"/>
+             <mesh filename="package://robotnik_description/meshes/bases/rbvogui_xl/rbvogui_xl_battery.stl"/>
           </geometry>
         </xacro:unless>
@@ -80,5 +83,5 @@
         <origin xyz="0 0 0" rpy="0 0 0 " />
         <geometry>
-           <mesh filename="package://robotnik_description/meshes/bases/rbvogui/rbvogui_battery.stl"/>
+           <mesh filename="package://robotnik_description/meshes/bases/rbvogui_xl/rbvogui_xl_battery.stl"/>
         </geometry>
       </collision>
@@ -86,5 +89,5 @@
     <!-- Contactors -->
     <joint name="${prefix}contactors_joint" type="fixed">
-      <origin xyz="0.5235 0 0.09265" rpy="0 0 0 " />
+      <origin xyz="0.6405 0 0.10264" rpy="0 0 0 " />
       <parent link="${prefix}chassis_link"/>
       <child link="${prefix}contactors_link" />
@@ -96,10 +99,10 @@
         <xacro:if value="${hq}">
           <geometry>
-            <mesh filename="package://robotnik_description/meshes/bases/rbvogui/rbvogui_contactors.stl" />
+            <mesh filename="package://robotnik_description/meshes/bases/rbvogui_xl/rbvogui_xl_contactors.stl" />
           </geometry>
         </xacro:if>
         <xacro:unless value="${hq}">
           <geometry>
-            <mesh filename="package://robotnik_description/meshes/bases/rbvogui/rbvogui_contactors.stl" />
+            <mesh filename="package://robotnik_description/meshes/bases/rbvogui_xl/rbvogui_xl_contactors.stl" />
           </geometry>
         </xacro:unless>
@@ -111,5 +114,5 @@
     <!-- Logos -->
     <joint name="${prefix}base_logos_joint" type="fixed">
-      <origin xyz="0 0 -0.1775" rpy="0 0 0" />
+      <origin xyz="0 0 -0.08376" rpy="0 0 0 " />
       <parent link="${prefix}chassis_link"/>
       <child link="${prefix}base_logos_link" />
@@ -118,13 +121,13 @@
     <link name="${prefix}base_logos_link">
       <visual>
-        <origin xyz="-0.015 0 0" rpy="0 0 0 " />
+        <origin xyz="0 0 -0.06" rpy="0 0 0" />
         <xacro:if value="${hq}">
           <geometry>
-            <mesh filename="package://robotnik_description/meshes/bases/rbvogui/rbvogui_logos.stl" scale="1.001 1.076 1.001"/>
+            <mesh filename="package://robotnik_description/meshes/bases/rbvogui_xl/rbvogui_xl_logos.stl" scale="1.24 1.24 1"/>
           </geometry>
         </xacro:if>
         <xacro:unless value="${hq}">
           <geometry>
-            <mesh filename="package://robotnik_description/meshes/bases/rbvogui/rbvogui_logos.dae" scale="1.001 1.076 1.001"/>
+            <mesh filename="package://robotnik_description/meshes/bases/rbvogui_xl/rbvogui_xl_logos.dae" scale="1.3 1.3 1"/>
           </geometry>
         </xacro:unless>
@@ -136,5 +139,5 @@
     <!-- Leds -->
     <joint name="${prefix}leds_joint" type="fixed">
-      <origin xyz="0 0 0.1025" rpy="0 0 0 " />
+      <origin xyz="0 0 0.12624" rpy="0 0 0 " />
       <parent link="${prefix}chassis_link"/>
       <child link="${prefix}leds_link" />
@@ -144,5 +147,5 @@
         <origin xyz="0 0 0" rpy="0 0 0.0" />
           <geometry>
-              <mesh filename="package://robotnik_description/meshes/bases/rbvogui/rbvogui_leds.stl" />
+              <mesh filename="package://robotnik_description/meshes/bases/rbvogui_xl/rbvogui_xl_leds.stl" />
           </geometry>
         <material name="lightgreen">
