Commit message: fix: rename robot rbficus as rbfiqus

File: robots/rbfiqus/rbfiqus.urdf.xacro (robot description, xacro)
@@ -1,8 +1,8 @@
 <?xml version="1.0" ?>
 <robot
-  name="rbficus"
+  name="rbfiqus"
   xmlns:xacro="http://wiki.ros.org/xacro">
   <xacro:include
-    filename="$(find robotnik_description)/urdf/bases/rbficus/rbficus_base.urdf.xacro" />
+    filename="$(find robotnik_description)/urdf/bases/rbfiqus/rbfiqus_base.urdf.xacro" />
   <xacro:include
     filename="$(find robotnik_sensors)/urdf/all_sensors.urdf.xacro" />
@@ -18,5 +18,5 @@
     default="false" />
   <!-- RB-VOGUI -->
-  <xacro:rbficus
+  <xacro:rbfiqus
     prefix="$(arg prefix)"
     gazebo_ignition="$(arg gazebo_ignition)"

File: robots/rbrobout/rbrobout.urdf.xacro (robot description, xacro)
@@ -53,3 +53,14 @@
       rpy="0 0 ${-3/4*pi}" />
   </xacro:sensor_sick_microscan3>
+  <!-- CAMERAS -->
+  <xacro:sensor_intel_realsense_d435
+    frame_prefix="$(arg prefix)front_rgbd_camera_"
+    parent="$(arg prefix)base_link"
+    node_namespace="$(arg namespace)"
+    node_name="front_camera"
+    gazebo_ignition="$(arg gazebo_ignition)">
+    <origin
+      xyz="0.835 0 0.1555"
+      rpy="0 0 0" />
+  </xacro:sensor_intel_realsense_d435>
 </robot>

File: robots/rbrobout/rbrobout_plus.urdf.xacro (robot description, xacro)
@@ -86,3 +86,14 @@
       rpy="0 0 ${-3/4*pi}" />
   </xacro:sensor_sick_microscan3>
+  <!-- CAMERAS -->
+  <xacro:sensor_intel_realsense_d435
+    frame_prefix="$(arg prefix)front_rgbd_camera_"
+    parent="$(arg prefix)base_link"
+    node_namespace="$(arg namespace)"
+    node_name="front_camera"
+    gazebo_ignition="$(arg gazebo_ignition)">
+    <origin
+      xyz="0.835 0 0.1555"
+      rpy="0 0 0" />
+  </xacro:sensor_intel_realsense_d435>
 </robot>

File: simulators/gazebo_ignition/rbfiqus/rbfiqus_control.urdf.xacro (robot description, xacro)
@@ -2,5 +2,5 @@
 <robot xmlns:xacro="http://wiki.ros.org/xacro">
   <xacro:macro
-    name="rbficus_gz_ignition_control"
+    name="rbfiqus_gz_ignition_control"
     params="namespace prefix">
     <gazebo>
@@ -10,5 +10,5 @@
         <robot_param>robot_description</robot_param>
         <robot_param_node>robot_state_publisher</robot_param_node>
-        <parameters>$(find robotnik_description)/simulators/gazebo_ignition/rbficus/rbficus_controller_params.yaml</parameters>
+        <parameters>$(find robotnik_description)/simulators/gazebo_ignition/rbfiqus/rbfiqus_controller_params.yaml</parameters>
         <ros>
           <namespace>/${namespace}</namespace>

File: urdf/bases/rbfiqus/rbfiqus_base.urdf.xacro (robot description, xacro)
@@ -1,12 +1,12 @@
 <?xml version="1.0" ?>
 <robot
-  name="rbficus_base"
+  name="rbfiqus_base"
   xmlns:xacro="http://www.ros.org/wiki/xacro">
   <xacro:include
-    filename="$(find robotnik_description)/urdf/bodies/rbficus/rbficus_body.urdf.xacro" />
+    filename="$(find robotnik_description)/urdf/bodies/rbfiqus/rbfiqus_body.urdf.xacro" />
   <xacro:include
-    filename="$(find robotnik_description)/urdf/wheels/steering_wheel/steering_wheel_rbficus.urdf.xacro" />
+    filename="$(find robotnik_description)/urdf/wheels/steering_wheel/steering_wheel_rbfiqus.urdf.xacro" />
   <xacro:include
-    filename="$(find robotnik_description)/simulators/gazebo_ignition/rbficus/rbficus_control.urdf.xacro" />
+    filename="$(find robotnik_description)/simulators/gazebo_ignition/rbfiqus/rbfiqus_control.urdf.xacro" />
   <!-- WHEELS PROPERTIES -->
   <xacro:property
@@ -20,5 +20,5 @@
     value="0.27319" />
   <xacro:macro
-    name="rbficus"
+    name="rbfiqus"
     params="
       prefix:=robot_
@@ -29,5 +29,5 @@
       name="hq"
       value="true" />
-    <xacro:rbficus_body
+    <xacro:rbfiqus_body
       prefix="${prefix}"
       hq="${hq}" />
@@ -69,5 +69,5 @@
     </xacro:steering_wheel_rbfiqus>
     <xacro:if value="$(arg gazebo_ignition)">
-      <xacro:rbficus_gz_ignition_control
+      <xacro:rbfiqus_gz_ignition_control
         namespace="${namespace}"
         prefix="${prefix}" />

File: urdf/bodies/rbfiqus/rbfiqus_body.urdf.xacro (robot description, xacro)
@@ -2,7 +2,7 @@
 <robot xmlns:xacro="http://www.ros.org/wiki/xacro">
   <xacro:include
-    filename="$(find robotnik_description)/urdf/bodies/rbficus/rbficus_body.gazebo.xacro" />
+    filename="$(find robotnik_description)/urdf/bodies/rbfiqus/rbfiqus_body.gazebo.xacro" />
   <xacro:macro
-    name="rbficus_body"
+    name="rbfiqus_body"
     params="prefix:=robot_ hq:=true">
     <!-- Robot mechanical and motor parameters -->
@@ -36,5 +36,5 @@
                 <origin xyz="0 0 0" rpy="0 0 0" />
                 <geometry>
-                    <mesh filename="package://robotnik_description/meshes/bases/rbficus/chasis.stl" />
+                    <mesh filename="package://robotnik_description/meshes/bases/rbfiqus/chasis.stl" />
                 </geometry>
                 <material name="grey">
@@ -65,5 +65,5 @@
                 <origin xyz="0.0 0.0 0.0" rpy="0 0 0" />
                 <geometry>
-                    <mesh filename="package://robotnik_description/meshes/bases/rbficus/rocker.stl" />
+                    <mesh filename="package://robotnik_description/meshes/bases/rbfiqus/rocker.stl" />
                 </geometry>
                 <material name="grey">
@@ -94,5 +94,5 @@
                 <origin xyz="0 0 0" rpy="0 0 0" />
                 <geometry>
-                    <mesh filename="package://robotnik_description/meshes/bases/rbficus/left_box.stl" />
+                    <mesh filename="package://robotnik_description/meshes/bases/rbfiqus/left_box.stl" />
                 </geometry>
                 <material name="grey">
@@ -123,5 +123,5 @@
                 <origin xyz="0 0 0" rpy="0 0 0" />
                 <geometry>
-                    <mesh filename="package://robotnik_description/meshes/bases/rbficus/right_box.stl" />
+                    <mesh filename="package://robotnik_description/meshes/bases/rbfiqus/right_box.stl" />
                 </geometry>
                 <material name="grey">

File: urdf/wheels/steering_wheel/steering_wheel_rbfiqus.urdf.xacro (robot description, xacro)
@@ -77,5 +77,5 @@
           <geometry>
             <mesh
-              filename="package://robotnik_description/meshes/wheels/steering_wheel/mw_frame_rbficus.stl" />
+              filename="package://robotnik_description/meshes/wheels/steering_wheel/mw_frame_rbfiqus.stl" />
           </geometry>
         </xacro:if>
@@ -93,5 +93,5 @@
           <geometry>
             <mesh
-              filename="package://robotnik_description/meshes/wheels/steering_wheel/mw_frame_rbficus.stl" />
+              filename="package://robotnik_description/meshes/wheels/steering_wheel/mw_frame_rbfiqus.stl" />
           </geometry>
         </xacro:unless>
@@ -113,5 +113,5 @@
         <geometry>
           <mesh
-            filename="package://robotnik_description/meshes/wheels/steering_wheel/mw_frame_rbficus.stl" />
+            filename="package://robotnik_description/meshes/wheels/steering_wheel/mw_frame_rbfiqus.stl" />
         </geometry>
       </collision>
