Commit message: added rb-watcher

File: robots/rbwatcher/rbwatcher.urdf.xacro (robot description, xacro)
@@ -2,7 +2,7 @@
 <robot
   name="rbwatcher"
-  xmlns:xacro="http://www.ros.org/wiki/xacro">
+  xmlns:xacro="http://wiki.ros.org/xacro">
   <xacro:include
-    filename="$(find robotnik_description)/urdf/bases/rb1/rb1_base.xacro" />
+    filename="$(find robotnik_description)/urdf/bases/rbwatcher/rbwatcher_base.xacro" />
   <xacro:include
     filename="$(find robotnik_sensors)/urdf/all_sensors.urdf.xacro" />
@@ -17,6 +17,6 @@
     name="gazebo_ignition"
     default="false" />
-  <!-- RB-1 -->
-  <xacro:rb1
+  <!-- RB-WATCHER -->
+  <xacro:rbwatcher
     prefix="$(arg prefix)"
     gazebo_ignition="$(arg gazebo_ignition)"
@@ -29,18 +29,18 @@
     gazebo_ignition="$(arg gazebo_ignition)">
     <origin
-      xyz="-0.1975 0.0 0.1098"
+      xyz="-0.03534 0.132 0.16109"
       rpy="0 0 0" />
   </xacro:sensor_vectornav>
   <!-- LASERS -->
-  <xacro:sensor_hokuyo_ust20lx
-    frame_prefix="$(arg prefix)front_laser_"
+  <xacro:sensor_robosense_helios_16p
+    frame_prefix="$(arg prefix)top_3d_laser_"
     parent="$(arg prefix)base_link"
     node_namespace="$(arg namespace)"
-    node_name="front_laser"
+    node_name="top_lidar"
     gazebo_ignition="$(arg gazebo_ignition)">
     <origin
-      xyz="0.210 0.0 0.1588"
-      rpy="0 ${pi} ${pi}" />
-  </xacro:sensor_hokuyo_ust20lx>
+      xyz="-0.11924 0 0.38609"
+      rpy="0 0 0" />
+  </xacro:sensor_robosense_helios_16p>
   <!-- CAMERAS -->
   <xacro:sensor_intel_realsense_d435
@@ -51,6 +51,17 @@
     gazebo_ignition="$(arg gazebo_ignition)">
     <origin
-      xyz="0.234 0.0 0.0408"
+      xyz="0.29881 0.0 0.15243"
       rpy="0 0 0" />
   </xacro:sensor_intel_realsense_d435>
+  <!-- GPS -->
+  <xacro:sensor_ublox_with_mast
+    frame_prefix="$(arg prefix)gps_"
+    parent="$(arg prefix)base_link"
+    node_namespace="$(arg namespace)"
+    node_name="gps"
+    gazebo_ignition="$(arg gazebo_ignition)">
+    <origin
+      xyz="-0.24824 0.095 0.76359"
+      rpy="0 0 0" />
+  </xacro:sensor_ublox_with_mast>
 </robot>

Commit message: feat: add top ptz camera  to rbwatcher & update control params

File: robots/rbwatcher/rbwatcher.urdf.xacro (robot description, xacro)
@@ -54,4 +54,14 @@
       rpy="0 0 0" />
   </xacro:sensor_intel_realsense_d435>
+  <xacro:sensor_link_750_nh
+    frame_prefix="$(arg prefix)top_ptz_camera_"
+    parent="$(arg prefix)base_link"
+    node_namespace="$(arg namespace)"
+    node_name="top_ptz_camera"
+    gazebo_ignition="$(arg gazebo_ignition)">
+    <origin
+      xyz="-0.11808 0 0.55429"
+      rpy="0 0 0" />
+  </xacro:sensor_link_750_nh>
   <!-- GPS -->
   <xacro:sensor_ublox_with_mast
