Commit message: moved kairos_plus base to kairos, created rbsummit_steel

File: urdf/bases/rbsummit_steel/rbsummit_steel_base.xacro (robot description, xacro)
@@ -1,24 +1,24 @@
 <?xml version="1.0" ?>
 <robot
-  name="rbkairos_base"
-  xmlns:xacro="http://wiki.ros.org/xacro">
+  name="summit_steel_base"
+  xmlns:xacro="http://www.ros.org/wiki/xacro">
   <xacro:include
-    filename="$(find robotnik_description)/urdf/bodies/rbkairos/rbkairos_body.urdf.xacro" />
+    filename="$(find robotnik_description)/urdf/bodies/rbsummit_steel/rbsummit_steel_body.urdf.xacro" />
   <xacro:include
     filename="$(find robotnik_description)/urdf/wheels/mecanum_wheel/rbkairos_mecanum_wheel.urdf.xacro" />
   <xacro:include
-    filename="$(find robotnik_description)/simulators/gazebo_ignition/rbkairos/rbkairos_control.urdf.xacro" />
+    filename="$(find robotnik_description)/simulators/gazebo_ignition/rbsummit_steel/rbsummit_steel_control.urdf.xacro" />
   <!-- WHEELS PROPERTIES -->
   <xacro:property
     name="wheel_offset_x"
-    value="0.21528" />
+    value="0.2225" />
   <xacro:property
     name="wheel_offset_y"
-    value="0.2590" />
+    value="0.2045" />
   <xacro:property
     name="wheel_offset_z"
     value="0.0" />
   <xacro:macro
-    name="rbkairos"
+    name="rbsummit_steel"
     params="
       prefix:=robot_
@@ -29,5 +29,6 @@
       name="hq"
       value="true" />
-    <xacro:rbkairos_body prefix="${prefix}" />
+    <xacro:rbsummit_steel_body
+      prefix="${prefix}" />
     <!-- WHEELS -->
     <xacro:rbkairos_mecanum_wheel
@@ -60,5 +61,5 @@
       xyz="-${wheel_offset_x} -${wheel_offset_y} ${wheel_offset_z}" />
     <xacro:if value="$(arg gazebo_ignition)">
-      <xacro:rbkairos_gz_ignition_control
+      <xacro:rbsummit_steel_gz_ignition_control
         namespace="${namespace}"
         prefix="${prefix}" />

File: urdf/bodies/rbkairos/rbkairos_body.urdf.xacro (robot description, xacro)
@@ -73,5 +73,5 @@
       <visual>
         <origin
-          xyz="0 0 0"
+          xyz="0 0 0.0065"
           rpy="0 0 0" />
         <geometry>
@@ -88,5 +88,5 @@
       type="fixed">
       <origin
-        xyz="0.0 0 0.38062"
+        xyz="0.0 0 0.56162"
         rpy="0 0 0" />
       <parent link="${prefix}base_link" />
@@ -112,5 +112,5 @@
       type="fixed">
       <origin
-        xyz="0.0 0.28931 0.29062"
+        xyz="0.0 0.2894 0.35562"
         rpy="0 0 0" />
       <parent link="${prefix}base_link" />
@@ -136,5 +136,5 @@
       type="fixed">
       <origin
-        xyz="0.0 -0.28931 0.29062"
+        xyz="0.0 -0.28931 0.35562"
         rpy="0 0 ${pi}" />
       <parent link="${prefix}base_link" />

File: urdf/bodies/rbsummit_steel/rbsummit_steel_body.urdf.xacro (robot description, xacro)
@@ -1,8 +1,8 @@
 <?xml version="1.0" ?>
 <robot
-  name="rbkairos"
+  name="rbsummit_steel"
   xmlns:xacro="http://wiki.ros.org/xacro">
   <xacro:macro
-    name="rbkairos_plus_body"
+    name="rbsummit_steel_body"
     params="prefix:=robot_">
     <!-- Robot mechanical and motor parameters -->
@@ -50,5 +50,5 @@
         <geometry>
           <mesh
-            filename="package://robotnik_description/meshes/bases/rbkairos/rbkairos_plus_chassis.stl" />
+            filename="package://robotnik_description/meshes/bases/rbsummit_steel/rbsummit_steel_chassis.stl" />
         </geometry>
         <material name="black">
@@ -62,5 +62,5 @@
         <geometry>
           <mesh
-            filename="package://robotnik_description/meshes/bases/rbkairos/rbkairos_plus_chassis.stl" />
+            filename="package://robotnik_description/meshes/bases/rbsummit_steel/rbsummit_steel_chassis.stl" />
         </geometry>
       </collision>
@@ -73,9 +73,9 @@
       <visual>
         <origin
-          xyz="0 0 0.0065"
-          rpy="0 0 0" />
-        <geometry>
-          <mesh
-            filename="package://robotnik_description/meshes/bases/rbkairos/rbkairos_top_cover.stl" />
+          xyz="0 0 0"
+          rpy="0 0 0" />
+        <geometry>
+          <mesh
+            filename="package://robotnik_description/meshes/bases/rbsummit_steel/rbsummit_steel_top_cover.stl" />
         </geometry>
         <material name="darkgrey">
@@ -88,5 +88,5 @@
       type="fixed">
       <origin
-        xyz="0.0 0 0.56162"
+        xyz="0.0 0 0.38062"
         rpy="0 0 0" />
       <parent link="${prefix}base_link" />
@@ -112,5 +112,5 @@
       type="fixed">
       <origin
-        xyz="0.0 0.2894 0.35562"
+        xyz="0.0 0.28931 0.29062"
         rpy="0 0 0" />
       <parent link="${prefix}base_link" />
@@ -136,5 +136,5 @@
       type="fixed">
       <origin
-        xyz="0.0 -0.28931 0.35562"
+        xyz="0.0 -0.28931 0.29062"
         rpy="0 0 ${pi}" />
       <parent link="${prefix}base_link" />

Commit message: Apply prettier format  in rbsummit_steel, rbwatcher & rbfiqus

File: urdf/bases/rbsummit_steel/rbsummit_steel_base.xacro (robot description, xacro)
@@ -29,6 +29,5 @@
       name="hq"
       value="true" />
-    <xacro:rbsummit_steel_body
-      prefix="${prefix}" />
+    <xacro:rbsummit_steel_body prefix="${prefix}" />
     <!-- WHEELS -->
     <xacro:rbkairos_mecanum_wheel

File: urdf/bodies/rbfiqus/rbfiqus_body.urdf.xacro (robot description, xacro)
@@ -34,27 +34,42 @@
         <link name="${prefix}chassis_link">
             <visual>
-                <origin xyz="0 0 0" rpy="0 0 0" />
-                <geometry>
-                    <mesh filename="package://robotnik_description/meshes/bases/rbfiqus/chasis.stl" />
-                </geometry>
-                <material name="grey">
-                    <color rgba="0.2 0.2 0.2 1" />
-                </material>
-            </visual>
-            <collision>
-                <origin xyz="0 0 0" rpy="0 0 0 " />
-                <geometry>
-                    <box size="1.1 0.9 0.1"/>
-                </geometry>
-            </collision>
-            <inertial>
-                <origin xyz="0.0 0.0 0.0" rpy="0.0 0.0 0.0" />
+                <origin
+          xyz="0 0 0"
+          rpy="0 0 0" />
+                <geometry>
+                    <mesh
+            filename="package://robotnik_description/meshes/bases/rbfiqus/chasis.stl" />
+                </geometry>
+                <material name="grey">
+                    <color rgba="0.2 0.2 0.2 1" />
+                </material>
+            </visual>
+            <collision>
+                <origin
+          xyz="0 0 0"
+          rpy="0 0 0 " />
+                <geometry>
+                    <box size="1.1 0.9 0.1" />
+                </geometry>
+            </collision>
+            <inertial>
+                <origin
+          xyz="0.0 0.0 0.0"
+          rpy="0.0 0.0 0.0" />
                 <mass value="50.0" />
-                <xacro:solid_cuboid_inertia w="1.1" h="0.9" d="0.1" m="50" />
+                <xacro:solid_cuboid_inertia
+          w="1.1"
+          h="0.9"
+          d="0.1"
+          m="50" />
             </inertial>
         </link>
         <!-- Rocker Chassis Joint -->
-            <joint name="${prefix}rocker_chassis" type="fixed">
-                <origin xyz="-0.835 0 0.047" rpy="0 0 0" />
+            <joint
+      name="${prefix}rocker_chassis"
+      type="fixed">
+                <origin
+        xyz="-0.835 0 0.047"
+        rpy="0 0 0" />
                 <parent link="${prefix}chassis_link" />
                 <child link="${prefix}rocker_link" />
@@ -63,80 +78,123 @@
         <link name="${prefix}rocker_link">
             <visual>
-                <origin xyz="0.0 0.0 0.0" rpy="0 0 0" />
-                <geometry>
-                    <mesh filename="package://robotnik_description/meshes/bases/rbfiqus/rocker.stl" />
-                </geometry>
-                <material name="grey">
-                    <color rgba="0.2 0.2 0.2 1" />
-                </material>
-            </visual>
-            <collision>
-                <origin xyz="0 0 0" rpy="0 0 0 " />
-                <geometry>
-                    <box size="0.2 1.55 0.3"/>
-                </geometry>
-            </collision>
-            <inertial>
-                <origin xyz="0.0 0.0 0.0" rpy="0.0 0.0 0.0" />
+                <origin
+          xyz="0.0 0.0 0.0"
+          rpy="0 0 0" />
+                <geometry>
+                    <mesh
+            filename="package://robotnik_description/meshes/bases/rbfiqus/rocker.stl" />
+                </geometry>
+                <material name="grey">
+                    <color rgba="0.2 0.2 0.2 1" />
+                </material>
+            </visual>
+            <collision>
+                <origin
+          xyz="0 0 0"
+          rpy="0 0 0 " />
+                <geometry>
+                    <box size="0.2 1.55 0.3" />
+                </geometry>
+            </collision>
+            <inertial>
+                <origin
+          xyz="0.0 0.0 0.0"
+          rpy="0.0 0.0 0.0" />
                 <mass value="5.0" />
-                <xacro:solid_cuboid_inertia w="0.2" h="1.55" d="0.3" m="5" />
+                <xacro:solid_cuboid_inertia
+          w="0.2"
+          h="1.55"
+          d="0.3"
+          m="5" />
             </inertial>
         </link>
         <!-- Left Rear Protection Rocker Joint -->
-        <joint name="${prefix}left_rear_protection" type="fixed">
-            <origin xyz="-0.008 0.505 0.23619" rpy="0 0 0" />
+        <joint
+      name="${prefix}left_rear_protection"
+      type="fixed">
+            <origin
+        xyz="-0.008 0.505 0.23619"
+        rpy="0 0 0" />
             <parent link="${prefix}rocker_link" />
-            <child link="${prefix}left_rear_protection_link" />
+            <child
+        link="${prefix}left_rear_protection_link" />
         </joint>
         <!-- Left Rear Protection -->
         <link name="${prefix}left_rear_protection_link">
             <visual>
-                <origin xyz="0 0 0" rpy="0 0 0" />
-                <geometry>
-                    <mesh filename="package://robotnik_description/meshes/bases/rbfiqus/left_box.stl" />
-                </geometry>
-                <material name="grey">
-                    <color rgba="0.2 0.2 0.2 1" />
-                </material>
-            </visual>
-            <collision>
-                <origin xyz="0.15 0.17 0.12" rpy="0 0 0 " />
-                <geometry>
-                    <box size="0.3 0.27 0.2"/>
-                </geometry>
-            </collision>
-            <inertial>
-                <origin xyz="0.0 0.0 0.0" rpy="0.0 0.0 0.0" />
+                <origin
+          xyz="0 0 0"
+          rpy="0 0 0" />
+                <geometry>
+                    <mesh
+            filename="package://robotnik_description/meshes/bases/rbfiqus/left_box.stl" />
+                </geometry>
+                <material name="grey">
+                    <color rgba="0.2 0.2 0.2 1" />
+                </material>
+            </visual>
+            <collision>
+                <origin
+          xyz="0.15 0.17 0.12"
+          rpy="0 0 0 " />
+                <geometry>
+                    <box size="0.3 0.27 0.2" />
+                </geometry>
+            </collision>
+            <inertial>
+                <origin
+          xyz="0.0 0.0 0.0"
+          rpy="0.0 0.0 0.0" />
                 <mass value="3.0" />
-                <xacro:solid_cuboid_inertia w="0.3" h="0.27" d="0.2" m="3" />
+                <xacro:solid_cuboid_inertia
+          w="0.3"
+          h="0.27"
+          d="0.2"
+          m="3" />
             </inertial>
         </link>
         <!-- Right Rear Protection Rocker Joint-->
-        <joint name="${prefix}right_rear_protection" type="fixed">
-            <origin xyz="-0.008 -0.505 0.23619" rpy="0 0 0" />
+        <joint
+      name="${prefix}right_rear_protection"
+      type="fixed">
+            <origin
+        xyz="-0.008 -0.505 0.23619"
+        rpy="0 0 0" />
             <parent link="${prefix}rocker_link" />
-            <child link="${prefix}right_rear_protection_link" />
+            <child
+        link="${prefix}right_rear_protection_link" />
         </joint>
         <!-- Right Rear Protection -->
         <link name="${prefix}right_rear_protection_link">
             <visual>
-                <origin xyz="0 0 0" rpy="0 0 0" />
-                <geometry>
-                    <mesh filename="package://robotnik_description/meshes/bases/rbfiqus/right_box.stl" />
-                </geometry>
-                <material name="grey">
-                    <color rgba="0.2 0.2 0.2 1" />
-                </material>
-            </visual>
-            <collision>
-                <origin xyz="0.15 -0.17 0.12" rpy="0 0 0 " />
-                <geometry>
-                    <box size="0.3 0.27 0.2"/>
-                </geometry>
-            </collision>
-            <inertial>
-                <origin xyz="0.0 0.0 0.0" rpy="0.0 0.0 0.0" />
+                <origin
+          xyz="0 0 0"
+          rpy="0 0 0" />
+                <geometry>
+                    <mesh
+            filename="package://robotnik_description/meshes/bases/rbfiqus/right_box.stl" />
+                </geometry>
+                <material name="grey">
+                    <color rgba="0.2 0.2 0.2 1" />
+                </material>
+            </visual>
+            <collision>
+                <origin
+          xyz="0.15 -0.17 0.12"
+          rpy="0 0 0 " />
+                <geometry>
+                    <box size="0.3 0.27 0.2" />
+                </geometry>
+            </collision>
+            <inertial>
+                <origin
+          xyz="0.0 0.0 0.0"
+          rpy="0.0 0.0 0.0" />
                 <mass value="3.0" />
-                <xacro:solid_cuboid_inertia w="0.3" h="0.27" d="0.2" m="3" />
+                <xacro:solid_cuboid_inertia
+          w="0.3"
+          h="0.27"
+          d="0.2"
+          m="3" />
             </inertial>
         </link>

File: urdf/bodies/rbwatcher/rbwatcher_body.urdf.xacro (robot description, xacro)
@@ -1,3 +1,3 @@
-<?xml version="1.0"?>
+<?xml version="1.0" ?>
 <robot
   name="rbwatcher_body"
@@ -75,9 +75,11 @@
     </link>
     <!-- TOP STRUCTURE -->
-    <joint name="${prefix}top_structure_joint" type="fixed">
+    <joint
+      name="${prefix}top_structure_joint"
+      type="fixed">
       <axis xyz="0 0 1" />
  			<origin
         xyz="-0.17024 0 0.27609"
-        rpy="0 0 0"/>
+        rpy="0 0 0" />
       <parent link="${prefix}base_link" />
       <child link="${prefix}top_structure_link" />
@@ -85,16 +87,22 @@
     <link name="${prefix}top_structure_link">
       <visual>
-        <origin rpy="0 0 0" xyz="0 0 0" />
+        <origin
+          rpy="0 0 0"
+          xyz="0 0 0" />
         <material name="${prefix}top_structure_color">
           <color rgba="0.5 0.5 0.5 1" />
         </material>
         <geometry>
-          <mesh filename="package://robotnik_description/meshes/bases/rbwatcher/rbwatcher_top_structure.dae" />
+          <mesh
+            filename="package://robotnik_description/meshes/bases/rbwatcher/rbwatcher_top_structure.dae" />
         </geometry>
       </visual>
       <collision>
-        <origin rpy="0 0 0" xyz="0 0 0" />
+        <origin
+          rpy="0 0 0"
+          xyz="0 0 0" />
         <geometry>
-          <mesh filename="package://robotnik_description/meshes/bases/rbwatcher/rbwatcher_top_structure.stl" />
+          <mesh
+            filename="package://robotnik_description/meshes/bases/rbwatcher/rbwatcher_top_structure.stl" />
         </geometry>
       </collision>
