Commit message: Fix wheels collisions and base inertia rbrobout

File: urdf/bodies/rbrobout/rbrobout_body.urdf.xacro (robot description, xacro)
@@ -22,7 +22,7 @@
       <link name="${prefix}base_link">
           <inertial>
-            <mass value="200.0" />
-            <origin xyz="0 0 0" />
-            <inertia  ixx="1.391" ixy="0.004"  ixz="0.0"  iyy="6.853"  iyz="0.0"  izz="6.125" />
+        <mass value="200.0" />
+        <origin xyz="0 0 0.10" />
+        <xacro:solid_cuboid_inertia w="2.0" h="1.5" d="0.2" m="200.0"/>
           </inertial>
           <visual>

File: urdf/wheels/omni_wheel/rbrobout_omni_wheel.urdf.xacro (robot description, xacro)
@@ -39,5 +39,5 @@
       </visual>
       <collision>
-				<origin xyz="0 0 0" rpy="0 0 0" />
+				<origin xyz="0 0 0" rpy="${PI/2} 0 0" />
         <geometry>
 					<cylinder length="${omni_wheel_height}" radius="${omni_wheel_radius}" />
@@ -51,10 +51,9 @@
     </link>
     <gazebo reference="${prefix}_wheel_link">
-		<mu1 value="0.0"/>
-		<mu2 value="0.0"/>
-		<kp value="10000000.0" />
-		<kd value="1.0" />
-		<fdir1 value="1 0 0"/>
-        <turnGravityOff>false</turnGravityOff>
+      <mu1>0.90</mu1>
+      <mu2>0.85</mu2>
+      <kp>2.75e6</kp>
+      <kd>8.25e1</kd>
+      <fdir1>0 0 0</fdir1>
     </gazebo>
   </xacro:macro>

Commit message: robout contact fixed

File: urdf/bodies/rbrobout/rbrobout_body.urdf.xacro (robot description, xacro)
@@ -43,11 +43,11 @@
       </link>
         <!-- DOCKING CONTACTS -->
-        <!-- <joint name="${prefix}base_docking_joint" type="fixed">
-            <origin xyz="0.284 0.012 0.068" rpy="0 0 0 " />
-            <parent link="${prefix}base_link"/>
+        <joint name="${prefix}base_docking_joint" type="fixed">
+            <origin xyz="0.858 0.02 0.008" rpy="0 0 0 " />
+            <parent link="${prefix}base_footprint"/>
             <child link="${prefix}base_docking_contact_link" />
-        </joint> -->
+        </joint>
         <!-- DOCKING LINK -->
-        <!-- <link name="${prefix}base_docking_contact_link" /> -->
+        <link name="${prefix}base_docking_contact_link" />
   </xacro:macro>
 </robot>

Commit message: fix

File: urdf/bodies/rbrobout/rbrobout_body.urdf.xacro (robot description, xacro)
@@ -44,5 +44,5 @@
         <!-- DOCKING CONTACTS -->
         <joint name="${prefix}base_docking_joint" type="fixed">
-            <origin xyz="0.858 0.02 0.008" rpy="0 0 0 " />
+            <origin xyz="0.858 0.01 0.008" rpy="0 0 0 " />
             <parent link="${prefix}base_footprint"/>
             <child link="${prefix}base_docking_contact_link" />

Commit message: fix

File: urdf/bodies/rbrobout/rbrobout_body.urdf.xacro (robot description, xacro)
@@ -44,5 +44,5 @@
         <!-- DOCKING CONTACTS -->
         <joint name="${prefix}base_docking_joint" type="fixed">
-            <origin xyz="0.858 0.01 0.008" rpy="0 0 0 " />
+            <origin xyz="0.86 -0.005 0.008" rpy="0 0 0 " />
             <parent link="${prefix}base_footprint"/>
             <child link="${prefix}base_docking_contact_link" />
