Commit message: Standardize docking_contact link naming across all body URDFs
Co-authored-by: jamendezib <126663352+jamendezib@users.noreply.github.com>

File: urdf/bodies/rbsummit/rbsummit_body.urdf.xacro (robot description, xacro)
@@ -82,8 +82,8 @@
         rpy="0 0 0 " />
       <parent link="${prefix}base_link" />
-      <child link="${prefix}base_docking_contact_link" />
+      <child link="${prefix}base_docking_contact" />
     </joint>
     <!-- DOCKING LINK -->
-    <link name="${prefix}base_docking_contact_link" />
+    <link name="${prefix}base_docking_contact" />
   </xacro:macro>
 </robot>

File: urdf/bodies/rbwatcher/rbwatcher_body.urdf.xacro (robot description, xacro)
@@ -116,8 +116,8 @@
         rpy="0 0 0 " />
       <parent link="${prefix}base_link" />
-      <child link="${prefix}base_docking_contact_link" />
+      <child link="${prefix}base_docking_contact" />
     </joint>
     <!-- DOCKING LINK -->
-    <link name="${prefix}base_docking_contact_link" />
+    <link name="${prefix}base_docking_contact" />
   </xacro:macro>
 </robot>
