Commit message: rbfiqus_agrimate/first_commit

File: simulators/gazebo_ignition/rbfiqus/rbfiqus_control.urdf.xacro (robot description, xacro)
@@ -53,10 +53,10 @@
         jmin="-2"
         jmax="2"
-        name="${prefix}back_left_steering_joint" />
+        name="${prefix}back_right_steering_joint" />
       <xacro:ros2_joint
         interface="position"
         jmin="-2"
         jmax="2"
-        name="${prefix}back_right_steering_joint" />
+        name="${prefix}back_left_steering_joint" />
       <xacro:ros2_joint
         interface="velocity"

File: urdf/arms/ur_macro.urdf.xacro (robot description, xacro)
@@ -34,6 +34,5 @@
       kinematics_parameters_file="${kinematics_params}"
       physical_parameters_file="${physical_params}"
-      visual_parameters_file="${visual_params}"
-      generate_ros2_control_tag="false">
+      visual_parameters_file="${visual_params}">
       <xacro:insert_block name="origin" />
     </xacro:ur_robot>

File: urdf/wheels/steering_wheel/steering_wheel_rbfiqus_agrimate.urdf.xacro (robot description, xacro)
@@ -4,8 +4,8 @@
     filename="$(find robotnik_description)/urdf/wheels/wheel.gazebo.xacro" />
   <xacro:include
-    filename="$(find robotnik_description)/urdf/wheels/rubber_wheel/rubber_wheel_220.urdf.xacro" />
+    filename="$(find robotnik_description)/urdf/wheels/rubber_wheel/fiqus_agrimate_wheel_front.urdf.xacro" />
   <xacro:property
     name="wheel_radius"
-    value="0.193" />
+    value="0.195" />
   <xacro:property
     name="wheel_width"
@@ -15,5 +15,5 @@
     value="7.5" />
   <xacro:macro
-    name="steering_wheel_rbfiqus"
+    name="steering_wheel_rbfiqus_agrimate"
     params="prefix parent *origin reflect hq">
     <xacro:macro
@@ -36,14 +36,14 @@
     <xacro:property
       name="steer_joint_damping"
-      value="1.0" />
+      value="0.1" />
     <xacro:property
       name="steer_joint_friction"
-      value="1.0" />
+      value="0.5" />
     <xacro:property
       name="steer_joint_effort_limit"
-      value="200.0" />
+      value="5000.0" />
     <xacro:property
       name="steer_joint_velocity_limit"
-      value="100.0" />
+      value="2.0" />
     <joint
       name="${prefix}steering_joint"
@@ -67,15 +67,15 @@
           <xacro:if value="${reflect}">
             <origin
-              xyz="0 0 0.0"
+              xyz="0 0 0"
               rpy="0 0 0" />
           </xacro:if>
           <xacro:unless value="${reflect}">
             <origin
-              xyz="0 0 0.0"
+              xyz="0 0 0"
               rpy="0 0 ${pi}" />
           </xacro:unless>
           <geometry>
             <mesh
-              filename="package://robotnik_description/meshes/wheels/steering_wheel/mw_frame_rbfiqus.stl" />
+              filename="package://robotnik_description/meshes/bases/rbfiqus/agrimate/L_Delantera.STL" />
           </geometry>
         </xacro:if>
@@ -93,5 +93,5 @@
           <geometry>
             <mesh
-              filename="package://robotnik_description/meshes/wheels/steering_wheel/mw_frame_rbfiqus.stl" />
+              filename="package://robotnik_description/meshes/bases/rbfiqus/agrimate/L_Delantera.STL" />
           </geometry>
         </xacro:unless>
@@ -113,5 +113,5 @@
         <geometry>
           <mesh
-            filename="package://robotnik_description/meshes/wheels/steering_wheel/mw_frame_rbfiqus.stl" />
+            filename="package://robotnik_description/meshes/bases/rbfiqus/agrimate/L_Delantera.STL" />
         </geometry>
       </collision>
@@ -136,5 +136,5 @@
     <xacro:gazebo_steering_frame_physics
       name="${prefix}base_wheel" />
-    <xacro:rubber_wheel
+    <xacro:fiqus_agrimate_wheel_front
       prefix="${prefix}"
       parent="${prefix}base_wheel"
@@ -144,8 +144,15 @@
       rubber_wheel_width="${wheel_width}"
       rubber_wheel_mass="${wheel_mass}">
-      <origin
-        xyz="0 0 -0.27319"
-        rpy="0 0 0" />
-    </xacro:rubber_wheel>
+      <xacro:if value="${reflect}">
+          <origin
+            xyz="0 -0.041 -0.0765"
+            rpy="0 0 0" />
+      </xacro:if>
+      <xacro:unless value="${reflect}">
+          <origin
+            xyz="0 0.041 -0.0765"
+            rpy="0 0 0" />
+      </xacro:unless>
+    </xacro:fiqus_agrimate_wheel_front>
   </xacro:macro>
 </robot>

File: urdf/wheels/steering_wheel/wheel_rbfiqus_agrimate_back.urdf.xacro (robot description, xacro)
@@ -4,8 +4,8 @@
     filename="$(find robotnik_description)/urdf/wheels/wheel.gazebo.xacro" />
   <xacro:include
-    filename="$(find robotnik_description)/urdf/wheels/rubber_wheel/rubber_wheel_220.urdf.xacro" />
+    filename="$(find robotnik_description)/urdf/wheels/rubber_wheel/fiqus_agrimate_wheel_back.urdf.xacro" />
   <xacro:property
-    name="wheel_radius"
-    value="0.193" />
+    name="wheel_big_radius"
+    value="0.29" />
   <xacro:property
     name="wheel_width"
@@ -13,8 +13,8 @@
   <xacro:property
     name="wheel_mass"
-    value="7.5" />
+    value="12.8" />
   <xacro:macro
-    name="steering_wheel_rbfiqus"
-    params="prefix parent *origin reflect hq">
+    name="wheel_rbfiqus_agrimate_back"
+    params="prefix parent *origin reflect hq left">
     <xacro:macro
       name="cylinder_inertia"
@@ -30,5 +30,5 @@
     <xacro:property
       name="steering_support_mass"
-      value="10" />
+      value="37.5" />
     <xacro:property
       name="steering_support_width"
@@ -46,19 +46,11 @@
       name="steer_joint_velocity_limit"
       value="100.0" />
-    <joint
-      name="${prefix}steering_joint"
-      type="revolute">
+    <joint name="${prefix}steering_joint" type="prismatic">
       <parent link="${parent}" />
       <child link="${prefix}base_wheel" />
       <xacro:insert_block name="origin" />
       <axis xyz="0 0 1" />
-      <limit
-        effort="${steer_joint_effort_limit}"
-        velocity="${steer_joint_velocity_limit}"
-        lower="-3.00"
-        upper="3.00" />
-      <dynamics
-        damping="${steer_joint_damping}"
-        friction="${steer_joint_friction}" />
+      <limit effort="100.0" lower="-0.05" upper="0.0" velocity="1.0"/>
+      <dynamics damping="100.0" friction="0.0" spring_reference="0.0" spring_stiffness="5000.0"/>
     </joint>
     <link name="${prefix}base_wheel">
@@ -76,6 +68,12 @@
           </xacro:unless>
           <geometry>
-            <mesh
-              filename="package://robotnik_description/meshes/wheels/steering_wheel/mw_frame_rbfiqus.stl" />
+            <xacro:if value="${left}">
+              <mesh
+                filename="package://robotnik_description/meshes/bases/rbfiqus/agrimate/Brazo_Agrimate_1.STL" />
+            </xacro:if>
+            <xacro:unless value="${left}">
+              <mesh
+                filename="package://robotnik_description/meshes/bases/rbfiqus/agrimate/Brazo_Agrimate_2.STL" />
+            </xacro:unless>
           </geometry>
         </xacro:if>
@@ -92,6 +90,12 @@
           </xacro:unless>
           <geometry>
-            <mesh
-              filename="package://robotnik_description/meshes/wheels/steering_wheel/mw_frame_rbfiqus.stl" />
+            <xacro:if value="${left}">
+              <mesh
+                filename="package://robotnik_description/meshes/bases/rbfiqus/agrimate/Brazo_Agrimate_1.STL" />
+            </xacro:if>
+            <xacro:unless value="${left}">
+              <mesh
+                filename="package://robotnik_description/meshes/bases/rbfiqus/agrimate/Brazo_Agrimate_2.STL" />
+            </xacro:unless>
           </geometry>
         </xacro:unless>
@@ -112,6 +116,12 @@
         </xacro:unless>
         <geometry>
-          <mesh
-            filename="package://robotnik_description/meshes/wheels/steering_wheel/mw_frame_rbfiqus.stl" />
+          <xacro:if value="${left}">
+              <mesh
+                filename="package://robotnik_description/meshes/bases/rbfiqus/agrimate/Brazo_Agrimate_1.STL" />
+            </xacro:if>
+            <xacro:unless value="${left}">
+              <mesh
+                filename="package://robotnik_description/meshes/bases/rbfiqus/agrimate/Brazo_Agrimate_2.STL" />
+            </xacro:unless>
         </geometry>
       </collision>
@@ -120,15 +130,15 @@
         <xacro:if value="${reflect}">
           <origin
-            xyz="0 0 ${wheel_radius/1.5}"
+            xyz="0 0 ${wheel_big_radius/1.5}"
             rpy="${pi/2.0} ${pi/2.0} 0" />
         </xacro:if>
         <xacro:unless value="${reflect}">
           <origin
-            xyz="0 0 ${wheel_radius/1.5}"
+            xyz="0 0 ${wheel_big_radius/1.5}"
             rpy="${pi/2.0} ${pi/2.0} ${pi/2.0}" />
         </xacro:unless>
         <xacro:cylinder_inertia
           m="${steering_support_mass}"
-          r="${wheel_radius}"
+          r="${wheel_big_radius}"
           h="${steering_support_width}" />
       </inertial>
@@ -136,16 +146,23 @@
     <xacro:gazebo_steering_frame_physics
       name="${prefix}base_wheel" />
-    <xacro:rubber_wheel
+    <xacro:fiqus_agrimate_wheel_back
       prefix="${prefix}"
       parent="${prefix}base_wheel"
       reflect="${reflect}"
       hq="${hq}"
-      rubber_wheel_radius="${wheel_radius}"
+      rubber_big_wheel_radius="${wheel_big_radius}"
       rubber_wheel_width="${wheel_width}"
       rubber_wheel_mass="${wheel_mass}">
-      <origin
-        xyz="0 0 -0.27319"
-        rpy="0 0 0" />
-    </xacro:rubber_wheel>
+      <xacro:if value="${left}">
+            <origin
+              xyz="0 0.18044 0"
+              rpy="0 0 0" />
+      </xacro:if>
+      <xacro:unless value="${left}">
+            <origin
+              xyz="0 -0.18044 0"
+              rpy="0 0 0" />
+      </xacro:unless>
+    </xacro:fiqus_agrimate_wheel_back>
   </xacro:macro>
 </robot>
