Commit message: Adding and registering proper joints for ackermann control

File: simulators/gazebo_ignition/rbcar/rbcar_control.urdf.xacro (robot description, xacro)
@@ -48,12 +48,23 @@
       <xacro:ros2_joint interface="position" jmin="-0.785398163" jmax="0.785398163" name="${prefix}left_steering_joint" />
       <xacro:ros2_joint interface="position" jmin="-0.785398163" jmax="0.785398163" name="${prefix}right_steering_joint" />
-      <!-- Front wheel axles (velocity control) -->
-      <xacro:ros2_joint interface="velocity" jmin="-39.02" jmax="39.02" name="${prefix}left_front_axle" />
-      <xacro:ros2_joint interface="velocity" jmin="-39.02" jmax="39.02" name="${prefix}right_front_axle" />
-      <!-- Rear wheel axles (velocity control) -->
+      <!-- Front wheel axles - NOT registered (passive rotation) -->
+      <!-- <xacro:ros2_joint interface="velocity" jmin="-39.02" jmax="39.02" name="${prefix}left_front_axle" /> -->
+      <!-- <xacro:ros2_joint interface="velocity" jmin="-39.02" jmax="39.02" name="${prefix}right_front_axle" /> -->
+      <joint name="${prefix}left_front_axle">
+        <state_interface name="position" />
+        <state_interface name="velocity" />
+        <state_interface name="effort" />
+      </joint>
+      <joint name="${prefix}right_front_axle">
+        <state_interface name="position" />
+        <state_interface name="velocity" />
+        <state_interface name="effort" />
+      </joint>
+      <!-- Rear wheel axles (velocity control for traction) -->
       <xacro:ros2_joint interface="velocity" jmin="-39.02" jmax="39.02" name="${prefix}left_rear_axle" />
       <xacro:ros2_joint interface="velocity" jmin="-39.02" jmax="39.02" name="${prefix}right_rear_axle" />
       <!-- Rear axle joint (effort control) -->
-      <xacro:ros2_joint interface="effort" jmin="-600" jmax="600" name="${prefix}rear_axle_joint" />
+      <!-- <xacro:ros2_joint interface="effort" jmin="-600" jmax="600" name="${prefix}rear_axle_joint" /> -->
+      <!-- <xacro:ros2_joint interface="velocity" jmin="-1000" jmax="1000" name="${prefix}rear_axle_joint" /> -->
     </ros2_control>
   </xacro:macro>

File: urdf/bases/rbcar/rbcar_base.urdf.xacro (robot description, xacro)
@@ -38,41 +38,4 @@
       hq="${hq}" />
     <!-- WHEELS -->
-    <!-- <xacro:rubber_wheel
-      prefix="${prefix}front_right_"
-      parent="${prefix}base_link"
-      reflect="false"
-      hq="${hq}">
-      <origin
-        xyz="${wheel_offset_x} -${wheel_offset_y} ${wheel_offset_z}"
-        rpy="0 0 0" />
-    </xacro:rubber_wheel>
-    <xacro:rubber_wheel
-      prefix="${prefix}front_left_"
-      parent="${prefix}base_link"
-      reflect="true"
-      hq="${hq}">
-      <origin
-        xyz="${wheel_offset_x} ${wheel_offset_y} ${wheel_offset_z}"
-        rpy="0 0 0" />
-    </xacro:rubber_wheel>
-    <xacro:rubber_wheel
-      prefix="${prefix}back_left_"
-      parent="${prefix}base_link"
-      reflect="true"
-      hq="${hq}">
-      <origin
-        xyz="0 ${wheel_offset_y} ${wheel_offset_z}"
-        rpy="0 0 0" />
-    </xacro:rubber_wheel>
-    <xacro:rubber_wheel
-      prefix="${prefix}back_right_"
-      parent="${prefix}base_link"
-      reflect="false"
-      hq="${hq}">
-      <origin
-        xyz="0 -${wheel_offset_y} ${wheel_offset_z}"
-        rpy="0 0 0" />
-    </xacro:rubber_wheel> -->
-    <!-- Wheels -->
     <xacro:front_wheel
       lr_prefix="$(arg prefix)left"
@@ -99,5 +62,5 @@
       fr_reflect="-1"
       parent="$(arg prefix)base_link" />
-    <xacro:rear_axle
+    <!-- <xacro:rear_axle
       prefix="$(arg prefix)rear_axle"
       parent="$(arg prefix)base_link">
@@ -105,5 +68,5 @@
         xyz="0 0.0 0"
         rpy="1.57079633 0 3.14159265"/>
-    </xacro:rear_axle>
+    </xacro:rear_axle> -->
     <!-- CONTROL -->
     <xacro:if value="$(arg gazebo_ignition)">
