Commit message: Comment unused material

File: urdf/wheels/rbcar/suspension_wheel_v2.urdf.xacro (robot description, xacro)
@@ -149,5 +149,5 @@
           <mesh filename="package://robotnik_description/meshes/wheels/rbcar/rbcar_wheel.stl"/>
         </geometry>
-        <material name="tire_mat"/>
+        <!-- <material name="tire_mat"/> -->
       </visual>
       <collision>
