Commit message: Update suspnesion xacro an delete deprecate rear_axle

File: urdf/wheels/rbcar/suspension_wheel_v4.urdf.xacro (robot description, xacro)
@@ -1,51 +1,29 @@
 <?xml version="1.0"?>
 <robot name="wheel" xmlns:xacro="http://wiki.ros.org/xacro">
-  <!-- hub_dia and tire_dia are the diameters of the hub and tire,
-       respectively. hex_hub_depth is the distance that the hex hub is
-       inset from the outer edge of the tire. It is set so that each wheel
-       is a "zero offset" wheel. hex_hub_depth = tire_width / 2 -
-       axle_length. -->
+  <!-- Geometry from v3, mechanical behaviour from v2 -->
   <xacro:property name="hub_dia" value="0.235"/>
-  <xacro:property name="tire_dia" value="0.634"/>
-  <xacro:property name="tire_width" value="0.322"/>
-  <xacro:property name="hex_hub_depth" value="0.120"/> <!-- or +0.072 -->
-  <xacro:property name="wheel_mass" value="8.0"/>   <!-- check -->
-  <!-- hex_hub_dist is the distance between left and right hex hubs when
-       the shock absorbers are fully extended. axle_length is the distance
-       from a U joint to the corresponding hex hub. wheel_travel is the
-       vertical wheel travel. -->
-  <xacro:property name="wheelbase" value="1.83"/>
-  <!--xacro:property name="hex_hub_dist" value="1.2385"/-->  <!-- 1.127 0.742 0.900 check -->
-  <xacro:property name="axle_length" value="0.120"/>
+  <xacro:property name="tire_dia" value="0.639"/>
+  <xacro:property name="wheel_radius" value="${tire_dia / 2.0}"/>
+  <xacro:property name="tire_width" value="0.245"/>
+  <xacro:property name="hex_hub_depth" value="0.0"/>
+  <xacro:property name="wheel_mass" value="8.0"/>
+  <xacro:property name="wheelbase" value="1.83323"/>
+  <xacro:property name="axle_length" value="0.12"/>
   <xacro:property name="wheel_travel" value="0.1"/>
   <xacro:property name="shock_z_offset" value="0.05"/>
-  <!-- Degree-to-radian conversions -->
-  <xacro:property name="degrees_34" value="0.60822457"/> <!-- this is used as the limit of the steering of the wheels -->
+  <xacro:property name="degrees_34" value="0.60822457"/>
   <xacro:property name="degrees_45" value="0.785398163"/>
   <xacro:property name="degrees_90" value="1.57079633"/>
   <xacro:property name="degrees_180" value="3.14159265"/>
-  <!-- shock_eff_limit is 2 * ((shock_stroke / 2) * shock_spring_constant) N. -->
   <xacro:property name="shock_eff_limit" value="100"/>
   <xacro:property name="shock_vel_limit" value="1000"/>
   <xacro:property name="wheel_joint_damping" value="0.2" />
   <xacro:property name="wheel_joint_friction" value="0.7" />
-  <xacro:property name="suspension_joint_damping" value="0.2" />
-  <xacro:property name="suspension_joint_friction" value="0.7" />
-  <!-- axle eff limit = 2 * stall_torque
-       as a function of the max gradient (15%) with overall max payload (600Kg) * wheel_radius
-       (calculating this way, it should be divided by 2 if 2 motors are used)
-       axle_eff_limit = 204.95 / 2 N m = ~102.5 -->
-  <!-- xacro:property name="axle_eff_limit" value="102.5"/ -->
+  <xacro:property name="suspension_joint_damping" value="0.1" />
+  <xacro:property name="suspension_joint_friction" value="0.1" />
   <xacro:property name="axle_eff_limit" value="204.95"/>
-  <!-- max_speed = 33 Km/h = 9.17 m/s
-       axle_vel_limit = (2 * pi) * (max_speed / (pi * tire_dia)) =  39.02 rad/s -->
   <xacro:property name="axle_vel_limit" value="39.02"/>
-  <!-- Servo_stall_torque of the direction axis in Nm. servo_no_load_speed is
-       measured in rad/s. -->
-  <xacro:property name="servo_stall_torque" value="50"/>  <!-- check -->
-  <xacro:property name="servo_no_load_speed" value="25"/> <!-- check -->
-  <!-- Inertia of a thick-walled cylindrical tube with open ends. Height is
-       measured along the z axis, which is the tube's axis. inner_rad and
-       outer_rad are the tube's inner and outer radii, respectively. -->
+  <xacro:property name="servo_stall_torque" value="50"/>
+  <xacro:property name="servo_no_load_speed" value="25"/>
   <xacro:macro name="thick_walled_tube_inertial"
                params="inner_rad outer_rad height mass">
@@ -62,6 +40,4 @@
     </inertial>
   </xacro:macro>
-  <!-- Null inertial element. This is needed to make the model work with
-       Gazebo. -->
   <xacro:macro name="null_inertial">
     <inertial>
@@ -70,5 +46,5 @@
     </inertial>
   </xacro:macro>
-  <!-- Shock absorber -->
+  <!-- Keep v2 prismatic suspension, but place the wheelset using v3 geometry -->
   <xacro:macro name="shock"
                params="lr_prefix fr_prefix lr_reflect fr_reflect child parent">
@@ -76,11 +52,6 @@
       <parent link="${parent}"/>
       <child link="${child}"/>
-      <xacro:if value="${fr_prefix=='front'}">
-        <xacro:property name="hex_hub_dist" value="1.03802"/>
-      </xacro:if>
-      <xacro:if value="${fr_prefix=='rear'}">
-        <xacro:property name="hex_hub_dist" value="1.2385"/>
-      </xacro:if>
-      <origin xyz="${fr_reflect * wheelbase / 2 + 0.917}
+      <xacro:property name="hex_hub_dist" value="1.45802"/>
+      <origin xyz="${fr_reflect * wheelbase / 2 + 1}
                    ${lr_reflect * ((hex_hub_dist / 2) - axle_length)}
                    ${(wheel_travel / 2) - shock_z_offset}"/>
@@ -100,27 +71,12 @@
     </transmission>
   </xacro:macro>
-  <!-- The "wheel" macro defines an axle carrier, axle, and wheel. -->
   <xacro:macro name="wheel" params="lr_prefix fr_prefix lr_reflect">
     <link name="${lr_prefix}_${fr_prefix}_axle_carrier">
-	  <!-- visual>
-        <origin xyz="0 0 0"/>
-        <geometry>
-          <cylinder radius="0.1" length="0.1"/>
-        </geometry>
-	  </visual>
-	  <collision>
-        <origin xyz="0 0 0"/>
-        <geometry>
-          <cylinder radius="0.1" length="0.1"/>
-        </geometry>
-	  </collision -->
       <xacro:null_inertial/>
     </link>
-    <!-- The left and right axles have the same axis so that identical
-         rotation values cause the wheels to rotate in the same direction. -->
     <joint name="${lr_prefix}_${fr_prefix}_axle" type="continuous">
       <parent link="${lr_prefix}_${fr_prefix}_axle_carrier"/>
       <child link="${lr_prefix}_${fr_prefix}_wheel"/>
-      <origin rpy="-${degrees_90} 0 0"/>
+      <origin rpy="${degrees_90} 0 ${degrees_180}"/>
       <axis xyz="0 0 1"/>
       <limit effort="${axle_eff_limit}" velocity="${axle_vel_limit}"/>
@@ -130,5 +86,4 @@
       <type>transmission_interface/SimpleTransmission</type>
       <joint name="${lr_prefix}_${fr_prefix}_axle">
-        <!-- hardwareInterface>hardware_interface/EffortJointInterface</hardwareInterface -->
         <hardwareInterface>hardware_interface/VelocityJointInterface</hardwareInterface>
       </joint>
@@ -142,12 +97,30 @@
     <link name="${lr_prefix}_${fr_prefix}_wheel">
       <visual>
+        <xacro:if value="${lr_reflect == 1}">
           <origin xyz="0
                        0
-                       ${lr_reflect * (axle_length - (tire_width / 2 - hex_hub_depth))}" rpy = "${lr_reflect * degrees_90} 0 ${degrees_180}"/>
+                       ${lr_reflect * (axle_length - (tire_width / 2 - hex_hub_depth)) - 0.08}"
+                  rpy="-${degrees_90} 0 ${degrees_180}"/>
+        </xacro:if>
+        <xacro:unless value="${lr_reflect == 1}">
+          <origin xyz="0
+                       0
+                       ${lr_reflect * (axle_length - (tire_width / 2 - hex_hub_depth)) + 0.08}"
+                  rpy="${degrees_90} 0 ${degrees_180}"/>
+        </xacro:unless>
         <geometry>
-          <!--cylinder radius="${tire_dia / 2}" length="${tire_width}"/-->
-          <mesh filename="package://robotnik_description/meshes/wheels/rbcar/rbcar_wheel.stl"/>
+          <xacro:if value="${lr_reflect == 1 and fr_prefix == 'front'}">
+            <mesh filename="package://robotnik_description/meshes/wheels/rbcar/polaris/left_front_wheel.STL"/>
+          </xacro:if>
+          <xacro:if value="${lr_reflect == -1 and fr_prefix == 'front'}">
+            <mesh filename="package://robotnik_description/meshes/wheels/rbcar/polaris/right_front_wheel.STL"/>
+          </xacro:if>
+          <xacro:if value="${lr_reflect == 1 and fr_prefix == 'rear'}">
+            <mesh filename="package://robotnik_description/meshes/wheels/rbcar/polaris/left_rear_wheel.STL"/>
+          </xacro:if>
+          <xacro:if value="${lr_reflect == -1 and fr_prefix == 'rear'}">
+            <mesh filename="package://robotnik_description/meshes/wheels/rbcar/polaris/right_rear_wheel.STL"/>
+          </xacro:if>
         </geometry>
-        <!-- <material name="tire_mat"/> -->
       </visual>
       <collision>
@@ -156,9 +129,9 @@
                      ${lr_reflect * (axle_length - (tire_width / 2 - hex_hub_depth))}"/>
         <geometry>
-          <cylinder radius="${tire_dia / 2}" length="${tire_width}"/>
+          <cylinder radius="${wheel_radius}" length="${tire_width}"/>
         </geometry>
       </collision>
       <xacro:thick_walled_tube_inertial
-          inner_rad="${hub_dia / 2}" outer_rad="${tire_dia / 2}"
+          inner_rad="${hub_dia / 2}" outer_rad="${wheel_radius}"
           height="${tire_width}" mass="${wheel_mass}"/>
     </link>
@@ -167,6 +140,4 @@
     </gazebo>
   </xacro:macro>
-  <!-- xacro:macro name="rubber_wheel" params="name parent *origin reflect hq" -->
-  <!-- Front wheel -->
   <xacro:macro name="front_wheel"
                params="lr_prefix fr_prefix lr_reflect fr_reflect parent">
@@ -175,16 +146,4 @@
                  child="${lr_prefix}_steering_link" parent="${parent}"/>
     <link name="${lr_prefix}_steering_link">
-	  <!-- visual>
-		<origin xyz="0 0 0"/>
-        <geometry>
-          <cylinder radius="0.1" length="0.1"/>
-        </geometry>
-	  </visual>
-	  <collision>
-		<origin xyz="0 0 0"/>
-        <geometry>
-          <cylinder radius="0.1" length="0.1"/>
-        </geometry>
-	  </collision -->
       <xacro:null_inertial/>
     </link>
@@ -193,11 +152,11 @@
       <child link="${lr_prefix}_${fr_prefix}_axle_carrier"/>
       <axis xyz="0 0 1"/>
-      <xacro:if value="${lr_reflect == 1}"> <!-- this applies if we are setting the left wheel -->
+      <xacro:if value="${lr_reflect == 1}">
         <limit lower="${-degrees_34}" upper="${degrees_45}"
-             effort="${servo_stall_torque}" velocity="${servo_no_load_speed}"/>
-        </xacro:if>
-      <xacro:unless value="${lr_reflect == 1}"> <!-- this applies if we are setting the right wheel -->
+               effort="${servo_stall_torque}" velocity="${servo_no_load_speed}"/>
+      </xacro:if>
+      <xacro:unless value="${lr_reflect == 1}">
         <limit lower="${-degrees_45}" upper="${degrees_34}"
-             effort="${servo_stall_torque}" velocity="${servo_no_load_speed}"/>
+               effort="${servo_stall_torque}" velocity="${servo_no_load_speed}"/>
       </xacro:unless>
     </joint>
@@ -205,5 +164,4 @@
       <type>transmission_interface/SimpleTransmission</type>
       <joint name="${lr_prefix}_steering_joint">
-        <!--<hardwareInterface>hardware_interface/EffortJointInterface</hardwareInterface>-->
         <hardwareInterface>hardware_interface/PositionJointInterface</hardwareInterface>
       </joint>
@@ -218,5 +176,4 @@
                  lr_reflect="${lr_reflect}"/>
   </xacro:macro>
-  <!-- Rear wheel -->
   <xacro:macro name="rear_wheel"
                params="lr_prefix fr_prefix lr_reflect fr_reflect parent">
@@ -227,3 +184,3 @@
                  lr_reflect="${lr_reflect}"/>
   </xacro:macro>
- </robot>
+</robot>
