Commit message: Update suspension wheels xacro for use the mechanical data from v2 and use the new model of wheel

File: urdf/wheels/rbcar/suspension_wheel_v4.urdf.xacro (robot description, xacro)
@@ -1,29 +1,53 @@
 <?xml version="1.0"?>
 <robot name="wheel" xmlns:xacro="http://wiki.ros.org/xacro">
-  <!-- Geometry from v3, mechanical behaviour from v2 -->
+  <!-- hub_dia and tire_dia are the diameters of the hub and tire,
+       respectively. hex_hub_depth is the distance that the hex hub is
+       inset from the outer edge of the tire. It is set so that each wheel
+       is a "zero offset" wheel. hex_hub_depth = tire_width / 2 -
+       axle_length. -->
   <xacro:property name="hub_dia" value="0.235"/>
   <xacro:property name="tire_dia" value="0.639"/>
   <xacro:property name="wheel_radius" value="${tire_dia / 2.0}"/>
   <xacro:property name="tire_width" value="0.245"/>
-  <xacro:property name="hex_hub_depth" value="0.0"/>
-  <xacro:property name="wheel_mass" value="8.0"/>
+  <xacro:property name="hex_hub_depth" value="0.0"/> <!-- or +0.072 -->
+  <xacro:property name="wheel_mass" value="8.0"/>   <!-- check -->
+  <!-- hex_hub_dist is the distance between left and right hex hubs when
+       the shock absorbers are fully extended. axle_length is the distance
+       from a U joint to the corresponding hex hub. wheel_travel is the
+       vertical wheel travel. -->
   <xacro:property name="wheelbase" value="1.83323"/>
+  <!--xacro:property name="hex_hub_dist" value="1.2385"/-->  <!-- 1.127 0.742 0.900 check -->
+  <!--xacro:property name="axle_length" value="0.120"/-->
   <xacro:property name="axle_length" value="0.12"/>
   <xacro:property name="wheel_travel" value="0.1"/>
   <xacro:property name="shock_z_offset" value="0.05"/>
-  <xacro:property name="degrees_34" value="0.60822457"/>
+  <!-- Degree-to-radian conversions -->
+  <xacro:property name="degrees_34" value="0.60822457"/> <!-- this is used as the limit of the steering of the wheels -->
   <xacro:property name="degrees_45" value="0.785398163"/>
   <xacro:property name="degrees_90" value="1.57079633"/>
   <xacro:property name="degrees_180" value="3.14159265"/>
+  <!-- shock_eff_limit is 2 * ((shock_stroke / 2) * shock_spring_constant) N. -->
   <xacro:property name="shock_eff_limit" value="100"/>
   <xacro:property name="shock_vel_limit" value="1000"/>
   <xacro:property name="wheel_joint_damping" value="0.2" />
   <xacro:property name="wheel_joint_friction" value="0.7" />
-  <xacro:property name="suspension_joint_damping" value="0.1" />
-  <xacro:property name="suspension_joint_friction" value="0.1" />
+  <xacro:property name="suspension_joint_damping" value="0.2" />
+  <xacro:property name="suspension_joint_friction" value="0.7" />
+  <!-- axle eff limit = 2 * stall_torque
+       as a function of the max gradient (15%) with overall max payload (600Kg) * wheel_radius
+       (calculating this way, it should be divided by 2 if 2 motors are used)
+       axle_eff_limit = 204.95 / 2 N m = ~102.5 -->
+  <!-- xacro:property name="axle_eff_limit" value="102.5"/ -->
   <xacro:property name="axle_eff_limit" value="204.95"/>
+  <!-- max_speed = 33 Km/h = 9.17 m/s
+       axle_vel_limit = (2 * pi) * (max_speed / (pi * tire_dia)) =  39.02 rad/s -->
   <xacro:property name="axle_vel_limit" value="39.02"/>
-  <xacro:property name="servo_stall_torque" value="50"/>
-  <xacro:property name="servo_no_load_speed" value="25"/>
+  <!-- Servo_stall_torque of the direction axis in Nm. servo_no_load_speed is
+       measured in rad/s. -->
+  <xacro:property name="servo_stall_torque" value="50"/>  <!-- check -->
+  <xacro:property name="servo_no_load_speed" value="25"/> <!-- check -->
+  <!-- Inertia of a thick-walled cylindrical tube with open ends. Height is
+       measured along the z axis, which is the tube's axis. inner_rad and
+       outer_rad are the tube's inner and outer radii, respectively. -->
   <xacro:macro name="thick_walled_tube_inertial"
                params="inner_rad outer_rad height mass">
@@ -40,4 +64,6 @@
     </inertial>
   </xacro:macro>
+  <!-- Null inertial element. This is needed to make the model work with
+       Gazebo. -->
   <xacro:macro name="null_inertial">
     <inertial>
@@ -46,13 +72,18 @@
     </inertial>
   </xacro:macro>
-  <!-- Keep v2 prismatic suspension, but place the wheelset using v3 geometry -->
+  <!-- Shock absorber -->
   <xacro:macro name="shock"
-               params="lr_prefix fr_prefix lr_reflect fr_reflect child parent">
-    <joint name="${lr_prefix}_${fr_prefix}_shock" type="prismatic">
+               params="prefix lr_prefix fr_prefix lr_reflect fr_reflect child parent">
+    <joint name="${prefix}${lr_prefix}_${fr_prefix}_shock" type="prismatic">
       <parent link="${parent}"/>
       <child link="${child}"/>
-      <xacro:property name="hex_hub_dist" value="1.45802"/>
+      <xacro:if value="${fr_prefix=='front'}">
+        <xacro:property name="hex_hub_dist" value="1.45802"/>
+      </xacro:if>
+      <xacro:if value="${fr_prefix=='rear'}">
+        <xacro:property name="hex_hub_dist" value="1.45802"/>
+      </xacro:if>
       <origin xyz="${fr_reflect * wheelbase / 2 + 1}
-                   ${lr_reflect * ((hex_hub_dist / 2) - axle_length)}
+                   ${lr_reflect * ((hex_hub_dist / 2) - axle_length )}
                    ${(wheel_travel / 2) - shock_z_offset}"/>
       <axis xyz="0 0 -1"/>
@@ -61,21 +92,33 @@
       <joint_properties damping="${suspension_joint_damping}" friction="${suspension_joint_friction}"/>
     </joint>
-    <transmission name="${lr_prefix}_${fr_prefix}_shock_trans">
+    <transmission name="${prefix}${lr_prefix}_${fr_prefix}_shock_trans">
       <type>transmission_interface/SimpleTransmission</type>
-      <joint name="${lr_prefix}_${fr_prefix}_shock">
+      <joint name="${prefix}${lr_prefix}_${fr_prefix}_shock">
         <hardwareInterface>hardware_interface/EffortJointInterface</hardwareInterface>
       </joint>
-      <actuator name="${lr_prefix}_${fr_prefix}_shock_act">
+      <actuator name="${prefix}${lr_prefix}_${fr_prefix}_shock_act">
         <mechanicalReduction>1</mechanicalReduction>
       </actuator>
     </transmission>
   </xacro:macro>
-  <xacro:macro name="wheel" params="lr_prefix fr_prefix lr_reflect">
-    <link name="${lr_prefix}_${fr_prefix}_axle_carrier">
+  <!-- The "wheel" macro defines an axle carrier, axle, and wheel. -->
+  <xacro:macro name="wheel" params="prefix lr_prefix fr_prefix lr_reflect">
+    <xacro:property
+      name="wheel_mesh"
+      value="package://robotnik_description/meshes/wheels/rbcar/rbcar_wheel.STL"/>
+    <xacro:property
+      name="wheel_visual_z"
+      value="${lr_reflect * (axle_length - (tire_width / 2 - hex_hub_depth))}"/>
+    <xacro:property
+      name="wheel_visual_roll"
+      value="${lr_reflect * degrees_90}"/>
+    <link name="${prefix}${lr_prefix}_${fr_prefix}_axle_carrier">
       <xacro:null_inertial/>
     </link>
-    <joint name="${lr_prefix}_${fr_prefix}_axle" type="continuous">
-      <parent link="${lr_prefix}_${fr_prefix}_axle_carrier"/>
-      <child link="${lr_prefix}_${fr_prefix}_wheel"/>
+    <!-- The left and right axles have the same axis so that identical
+         rotation values cause the wheels to rotate in the same direction. -->
+    <joint name="${prefix}${lr_prefix}_${fr_prefix}_axle" type="continuous">
+      <parent link="${prefix}${lr_prefix}_${fr_prefix}_axle_carrier"/>
+      <child link="${prefix}${lr_prefix}_${fr_prefix}_wheel"/>
       <origin rpy="${degrees_90} 0 ${degrees_180}"/>
       <axis xyz="0 0 1"/>
@@ -83,43 +126,24 @@
       <joint_properties damping="${wheel_joint_damping}" friction="${wheel_joint_friction}"/>
     </joint>
-    <transmission name="${lr_prefix}_${fr_prefix}_axle_trans">
+    <transmission name="${prefix}${lr_prefix}_${fr_prefix}_axle_trans">
       <type>transmission_interface/SimpleTransmission</type>
-      <joint name="${lr_prefix}_${fr_prefix}_axle">
+      <joint name="${prefix}${lr_prefix}_${fr_prefix}_axle">
+        <!-- hardwareInterface>hardware_interface/EffortJointInterface</hardwareInterface -->
         <hardwareInterface>hardware_interface/VelocityJointInterface</hardwareInterface>
       </joint>
-      <actuator name="${lr_prefix}_${fr_prefix}_axle_act">
+      <actuator name="${prefix}${lr_prefix}_${fr_prefix}_axle_act">
         <mechanicalReduction>1</mechanicalReduction>
       </actuator>
     </transmission>
-    <gazebo reference="${lr_prefix}_${fr_prefix}_axle_carrier">
+    <gazebo reference="${prefix}${lr_prefix}_${fr_prefix}_axle_carrier">
       <material>Gazebo/Black</material>
     </gazebo>
-    <link name="${lr_prefix}_${fr_prefix}_wheel">
+    <link name="${prefix}${lr_prefix}_${fr_prefix}_wheel">
       <visual>
-        <xacro:if value="${lr_reflect == 1}">
-          <origin xyz="0
-                       0
-                       ${lr_reflect * (axle_length - (tire_width / 2 - hex_hub_depth)) - 0.08}"
-                  rpy="-${degrees_90} 0 ${degrees_180}"/>
-        </xacro:if>
-        <xacro:unless value="${lr_reflect == 1}">
-          <origin xyz="0
-                       0
-                       ${lr_reflect * (axle_length - (tire_width / 2 - hex_hub_depth)) + 0.08}"
-                  rpy="${degrees_90} 0 ${degrees_180}"/>
-        </xacro:unless>
-        <geometry>
-          <xacro:if value="${lr_reflect == 1 and fr_prefix == 'front'}">
-            <mesh filename="package://robotnik_description/meshes/wheels/rbcar/polaris/left_front_wheel.STL"/>
-          </xacro:if>
-          <xacro:if value="${lr_reflect == -1 and fr_prefix == 'front'}">
-            <mesh filename="package://robotnik_description/meshes/wheels/rbcar/polaris/right_front_wheel.STL"/>
-          </xacro:if>
-          <xacro:if value="${lr_reflect == 1 and fr_prefix == 'rear'}">
-            <mesh filename="package://robotnik_description/meshes/wheels/rbcar/polaris/left_rear_wheel.STL"/>
-          </xacro:if>
-          <xacro:if value="${lr_reflect == -1 and fr_prefix == 'rear'}">
-            <mesh filename="package://robotnik_description/meshes/wheels/rbcar/polaris/right_rear_wheel.STL"/>
-          </xacro:if>
+        <origin
+          xyz="0 0 ${wheel_visual_z}"
+          rpy="${wheel_visual_roll} 0 ${degrees_180}"/>
+        <geometry>
+          <mesh filename="${wheel_mesh}"/>
         </geometry>
       </visual>
@@ -129,5 +153,5 @@
                      ${lr_reflect * (axle_length - (tire_width / 2 - hex_hub_depth))}"/>
         <geometry>
-          <cylinder radius="${wheel_radius}" length="${tire_width}"/>
+          <cylinder radius="${tire_dia / 2}" length="${tire_width}"/>
         </geometry>
       </collision>
@@ -136,51 +160,67 @@
           height="${tire_width}" mass="${wheel_mass}"/>
     </link>
-    <gazebo reference="${lr_prefix}_${fr_prefix}_wheel">
+    <gazebo reference="${prefix}${lr_prefix}_${fr_prefix}_wheel">
       <material>Gazebo/Black</material>
     </gazebo>
   </xacro:macro>
+  <!-- xacro:macro name="rubber_wheel" params="name parent *origin reflect hq" -->
+  <!-- Front wheel -->
   <xacro:macro name="front_wheel"
-               params="lr_prefix fr_prefix lr_reflect fr_reflect parent">
-    <xacro:shock lr_prefix="${lr_prefix}" fr_prefix="${fr_prefix}"
+               params="prefix lr_prefix fr_prefix lr_reflect fr_reflect parent">
+    <xacro:shock prefix="${prefix}" lr_prefix="${lr_prefix}" fr_prefix="${fr_prefix}"
                  lr_reflect="${lr_reflect}" fr_reflect="${fr_reflect}"
-                 child="${lr_prefix}_steering_link" parent="${parent}"/>
-    <link name="${lr_prefix}_steering_link">
+                 child="${prefix}${lr_prefix}_steering_link" parent="${parent}"/>
+    <link name="${prefix}${lr_prefix}_steering_link">
+	  <!-- visual>
+		<origin xyz="0 0 0"/>
+        <geometry>
+          <cylinder radius="0.1" length="0.1"/>
+        </geometry>
+	  </visual>
+	  <collision>
+		<origin xyz="0 0 0"/>
+        <geometry>
+          <cylinder radius="0.1" length="0.1"/>
+        </geometry>
+	  </collision -->
       <xacro:null_inertial/>
     </link>
-    <joint name="${lr_prefix}_steering_joint" type="revolute">
-      <parent link="${lr_prefix}_steering_link"/>
-      <child link="${lr_prefix}_${fr_prefix}_axle_carrier"/>
+    <joint name="${prefix}${lr_prefix}_steering_joint" type="revolute">
+      <parent link="${prefix}${lr_prefix}_steering_link"/>
+      <child link="${prefix}${lr_prefix}_${fr_prefix}_axle_carrier"/>
       <axis xyz="0 0 1"/>
-      <xacro:if value="${lr_reflect == 1}">
+      <xacro:if value="${lr_reflect == 1}"> <!-- this applies if we are setting the left wheel -->
         <limit lower="${-degrees_34}" upper="${degrees_45}"
-               effort="${servo_stall_torque}" velocity="${servo_no_load_speed}"/>
-      </xacro:if>
-      <xacro:unless value="${lr_reflect == 1}">
+             effort="${servo_stall_torque}" velocity="${servo_no_load_speed}"/>
+        </xacro:if>
+      <xacro:unless value="${lr_reflect == 1}"> <!-- this applies if we are setting the right wheel -->
         <limit lower="${-degrees_45}" upper="${degrees_34}"
-               effort="${servo_stall_torque}" velocity="${servo_no_load_speed}"/>
+             effort="${servo_stall_torque}" velocity="${servo_no_load_speed}"/>
       </xacro:unless>
     </joint>
-    <transmission name="${lr_prefix}_steering_trans">
+    <transmission name="${prefix}${lr_prefix}_steering_trans">
       <type>transmission_interface/SimpleTransmission</type>
-      <joint name="${lr_prefix}_steering_joint">
+      <joint name="${prefix}${lr_prefix}_steering_joint">
+        <!--<hardwareInterface>hardware_interface/EffortJointInterface</hardwareInterface>-->
         <hardwareInterface>hardware_interface/PositionJointInterface</hardwareInterface>
       </joint>
-      <actuator name="${lr_prefix}_steering_act">
+      <actuator name="${prefix}${lr_prefix}_steering_act">
         <mechanicalReduction>1</mechanicalReduction>
       </actuator>
     </transmission>
-    <gazebo reference="${lr_prefix}_steering_link">
+    <gazebo reference="${prefix}${lr_prefix}_steering_link">
       <material>Gazebo/Black</material>
     </gazebo>
-    <xacro:wheel lr_prefix="${lr_prefix}" fr_prefix="${fr_prefix}"
+    <xacro:wheel prefix="${prefix}" lr_prefix="${lr_prefix}" fr_prefix="${fr_prefix}"
                  lr_reflect="${lr_reflect}"/>
   </xacro:macro>
+  <!-- Rear wheel -->
   <xacro:macro name="rear_wheel"
-               params="lr_prefix fr_prefix lr_reflect fr_reflect parent">
-    <xacro:shock lr_prefix="${lr_prefix}" fr_prefix="${fr_prefix}"
+               params="prefix lr_prefix fr_prefix lr_reflect fr_reflect parent">
+    <xacro:shock prefix="${prefix}" lr_prefix="${lr_prefix}" fr_prefix="${fr_prefix}"
                  lr_reflect="${lr_reflect}" fr_reflect="${fr_reflect}"
-                 child="${lr_prefix}_${fr_prefix}_axle_carrier" parent="${parent}"/>
-    <xacro:wheel lr_prefix="${lr_prefix}" fr_prefix="${fr_prefix}"
+                 child="${prefix}${lr_prefix}_${fr_prefix}_axle_carrier" parent="${parent}"/>
+    <xacro:wheel prefix="${prefix}" lr_prefix="${lr_prefix}" fr_prefix="${fr_prefix}"
                  lr_reflect="${lr_reflect}"/>
   </xacro:macro>
-</robot>
+ </robot>
