Commit message: Vacuum gripper meshes added

File: urdf/grippers/suction_gripper/suction_gripper.urdf.xacro (robot description, xacro)
@@ -21,5 +21,5 @@
         <origin xyz="0 0 0" rpy="0 0 0" />
         <geometry>
-          <mesh filename="package://robotnik_description/meshes/structures/suction_gripper/gripper.dae" />
+          <mesh filename="package://robotnik_description/meshes/grippers/suction_gripper/gripper.dae" />
         </geometry>
       </visual>
@@ -30,5 +30,5 @@
         <origin xyz="0 0 0" rpy="0 0 0" />
         <geometry>
-          <mesh filename="package://robotnik_description/meshes/structures/suction_gripper/my_gripper.stl" />
+          <mesh filename="package://robotnik_description/meshes/grippers/suction_gripper/my_gripper.stl" />
         </geometry>
       </collision>
