Commit message: add ewellix offset

File: urdf/structures/ewellix/ewellix_lift_900mm.urdf.xacro (robot description, xacro)
@@ -5,5 +5,5 @@
   <xacro:macro name="ewellix_lift_900mm" params="prefix parent cut_model:=false *origin">
     <!-- Lift base link -->
-    <link name="${prefix}ewellix_lift_base_link">
+    <link name="${prefix}base_link">
       <visual>
         <origin xyz="0 0 0" rpy="0 0 0"/>
@@ -28,11 +28,11 @@
     </link>
     <!-- Lift base link joint -->
-    <joint name="${prefix}ewellix_lift_base_joint" type="fixed">
+    <joint name="${prefix}base_joint" type="fixed">
       <xacro:insert_block name="origin" />
       <parent link="${parent}"/>
-      <child link="${prefix}ewellix_lift_base_link" />
+      <child link="${prefix}base_link" />
     </joint>
     <!-- Lift top link -->
-    <link name="${prefix}ewellix_lift_top_link">
+    <link name="${prefix}link">
       <visual>
         <origin xyz="0 0 0" rpy="0 0 0"/>
@@ -67,8 +67,9 @@
     </link>
     <!-- Lift top link joint -->
-    <joint name="${prefix}ewellix_lift_top_joint" type="prismatic">
-      <parent link="${prefix}ewellix_lift_base_link"/>
-      <child link="${prefix}ewellix_lift_top_link" />
-      <origin xyz="0 0 0.730" rpy="0 0 0" />
+    <joint name="${prefix}joint" type="prismatic">
+      <parent link="${prefix}base_link"/>
+      <child link="${prefix}link" />
+      <!-- <origin xyz="0 0 0.730" rpy="0 0 0" /> -->
+      <origin xyz="0 0 0" rpy="0 0 0" />
       <limit effort="1000" lower="0.0" upper="0.9" velocity="0.088"/>
       <axis xyz="0 0 1" />
@@ -79,8 +80,8 @@
         EffortJointInterface
     -->
-    <gazebo reference="${prefix}ewellix_lift_base_link">
+    <gazebo reference="${prefix}base_link">
       <material>Gazebo/Grey</material>
     </gazebo>
-    <gazebo reference="${prefix}ewellix_lift_top_link">
+    <gazebo reference="${prefix}link">
       <material>Gazebo/Grey</material>
     </gazebo>

Commit message: fix: add ewellix offset (#80)

File: urdf/structures/ewellix/ewellix_lift_900mm.urdf.xacro (robot description, xacro)
@@ -8,5 +8,5 @@
     params="prefix parent cut_model:=false *origin">
     <!-- Lift base link -->
-    <link name="${prefix}ewellix_lift_base_link">
+    <link name="${prefix}base_link">
       <visual>
         <origin
@@ -48,12 +48,12 @@
     <!-- Lift base link joint -->
     <joint
-      name="${prefix}ewellix_lift_base_joint"
+      name="${prefix}base_joint"
       type="fixed">
       <xacro:insert_block name="origin" />
       <parent link="${parent}" />
-      <child link="${prefix}ewellix_lift_base_link" />
+      <child link="${prefix}base_link" />
     </joint>
     <!-- Lift top link -->
-    <link name="${prefix}ewellix_lift_top_link">
+    <link name="${prefix}link">
       <visual>
         <origin
@@ -105,13 +105,13 @@
     <!-- Lift top link joint -->
     <joint
-      name="${prefix}ewellix_lift_top_joint"
+      name="${prefix}joint"
       type="prismatic">
-      <parent link="${prefix}ewellix_lift_base_link" />
-      <child link="${prefix}ewellix_lift_top_link" />
+      <parent link="${prefix}base_link" />
+      <child link="${prefix}link" />
       <origin
-        xyz="0 0 0.730"
+        xyz="0 0 0"
         rpy="0 0 0" />
       <limit
-        effort="1000000"
+        effort="1000"
         lower="0.0"
         upper="0.9"
@@ -119,8 +119,8 @@
       <axis xyz="0 0 1" />
     </joint>
-    <gazebo reference="${prefix}ewellix_lift_base_link">
+    <gazebo reference="${prefix}base_link">
       <material>Gazebo/Grey</material>
     </gazebo>
-    <gazebo reference="${prefix}ewellix_lift_top_link">
+    <gazebo reference="${prefix}link">
       <material>Gazebo/Grey</material>
     </gazebo>

Commit message: Cambiado el urdf del lift

File: urdf/structures/ewellix/ewellix_lift_900mm.urdf.xacro (robot description, xacro)
@@ -7,5 +7,13 @@
     name="ewellix_lift_900mm"
     params="prefix parent cut_model:=false *origin">
-    <!-- Lift base link -->
+    <!--
+      Offset vertical para alinear:
+      - malla del lift_link (visual/collision)
+      - centro de masas del lift_link (inertial)
+      - frame superior de montaje del brazo (ewellix_lift_top_link)
+      Ajusta este valor (por ejemplo 0.9, 1.0, 1.05...) hasta que brazo + eje lineal queden bien.
+    -->
+    <xacro:property name="lift_z_offset" value="0.7"/>
+    <!-- Lift base link (fixed part of the linear axis) -->
     <link name="${prefix}base_link">
       <visual>
@@ -46,5 +54,5 @@
       </inertial>
     </link>
-    <!-- Lift base link joint -->
+    <!-- Mount lift to parent robot link -->
     <joint
       name="${prefix}base_joint"
@@ -54,9 +62,9 @@
       <child link="${prefix}base_link" />
     </joint>
-    <!-- Lift top link -->
+    <!-- Lift moving link (carriage / upper moving part) -->
     <link name="${prefix}link">
       <visual>
         <origin
-          xyz="0 0 0"
+          xyz="0 0 ${lift_z_offset}"
           rpy="0 0 0" />
         <geometry>
@@ -67,5 +75,5 @@
           <xacro:unless value="${cut_model}">
             <mesh
-              filename="package://robotnik_description/meshes/structures/ewellix/ewellix_lift_top_900mm.stl" />
+              filename="package://robotnik_description/meshes/structures/ewellix/ewellix_lift_top_900mm_cut.stl" />
           </xacro:unless>
         </geometry>
@@ -76,5 +84,5 @@
       <collision>
         <origin
-          xyz="-0.005 0 0.00235"
+          xyz="-0.005 0 ${0.00235 + lift_z_offset}"
           rpy="0 0 0" />
         <geometry>
@@ -85,12 +93,13 @@
           <xacro:unless value="${cut_model}">
             <mesh
-              filename="package://robotnik_description/meshes/structures/ewellix/ewellix_lift_top_900mm.stl" />
+              filename="package://robotnik_description/meshes/structures/ewellix/ewellix_lift_top_900mm_cut.stl" />
           </xacro:unless>
         </geometry>
       </collision>
+      <!-- Coherencia física con el desplazamiento visual/collision -->
       <inertial>
         <mass value="2" />
         <origin
-          xyz="0 0 0"
+          xyz="0 0 ${lift_z_offset}"
           rpy="0 0 0" />
         <inertia
@@ -103,5 +112,5 @@
       </inertial>
     </link>
-    <!-- Lift top link joint -->
+    <!-- Actuated prismatic joint (REAL linear axis joint) -->
     <joint
       name="${prefix}joint"
@@ -119,4 +128,20 @@
       <axis xyz="0 0 1" />
     </joint>
+    <!-- Extra top mounting frame (3rd frame) for arm/payload attachment -->
+    <link name="${prefix}ewellix_lift_top_link" />
+    <!--
+      Este frame es el que usa el brazo como parent.
+      Si quieres que el brazo quede alineado con la geometría desplazada del lift_link,
+      este origin debe llevar el mismo offset (lift_z_offset).
+    -->
+    <joint
+      name="${prefix}ewellix_lift_top_joint"
+      type="fixed">
+      <parent link="${prefix}link" />
+      <child link="${prefix}ewellix_lift_top_link" />
+      <origin
+        xyz="0 0 ${lift_z_offset}"
+        rpy="0 0 0" />
+    </joint>
     <gazebo reference="${prefix}base_link">
       <material>Gazebo/Grey</material>
@@ -125,4 +150,5 @@
       <material>Gazebo/Grey</material>
     </gazebo>
+    <!-- ros2_control MUST control the actuated prismatic joint -->
     <ros2_control
       name="${prefix}ewellix_lift_control"
@@ -131,9 +157,10 @@
         <plugin>gz_ros2_control/GazeboSimSystem</plugin>
       </hardware>
-      <joint name="${prefix}ewellix_lift_top_joint">
+      <joint name="${prefix}joint">
         <command_interface name="position" />
         <command_interface name="velocity" />
         <state_interface name="position">
-          <param name="initial_value">0.2</param>
+          <!-- Replegado al iniciar -->
+          <param name="initial_value">0.0</param>
         </state_interface>
         <state_interface name="velocity" />
