Commit message: add ewellix 700mm

File: urdf/structures/ewellix/ewellix_lift_700mm.urdf.xacro (robot description, xacro)
@@ -8,5 +8,5 @@
     params="prefix parent cut_model:=false *origin">
     <!-- Lift base link -->
-    <link name="${prefix}ewellix_lift_base_link">
+    <link name="${prefix}base_link">
       <visual>
         <origin
@@ -15,5 +15,6 @@
         <geometry>
           <mesh
-            filename="package://robotnik_description/meshes/structures/ewellix/ewellix_lift_base_700mm.stl" />
+            filename="package://robotnik_description/meshes/structures/ewellix/ewellix_lift_base_700mm.stl"
+            scale="0.95 0.95 1" />
         </geometry>
         <material name="grey">
@@ -27,5 +28,6 @@
         <geometry>
           <mesh
-            filename="package://robotnik_description/meshes/structures/ewellix/ewellix_lift_base_700mm.stl" />
+            filename="package://robotnik_description/meshes/structures/ewellix/ewellix_lift_base_700mm.stl"
+            scale="0.95 0.95 1" />
         </geometry>
       </collision>
@@ -46,12 +48,12 @@
     <!-- Lift base link joint -->
     <joint
-      name="${prefix}ewellix_lift_base_joint"
+      name="${prefix}base_joint"
       type="fixed">
       <xacro:insert_block name="origin" />
       <parent link="${parent}" />
-      <child link="${prefix}ewellix_lift_base_link" />
+      <child link="${prefix}base_link" />
     </joint>
     <!-- Lift top link -->
-    <link name="${prefix}ewellix_lift_top_link">
+    <link name="${prefix}link">
       <visual>
         <origin
@@ -103,10 +105,10 @@
     <!-- Lift top link joint -->
     <joint
-      name="${prefix}ewellix_lift_top_joint"
+      name="${prefix}joint"
       type="prismatic">
-      <parent link="${prefix}ewellix_lift_base_link" />
-      <child link="${prefix}ewellix_lift_top_link" />
+      <parent link="${prefix}base_link" />
+      <child link="${prefix}link" />
       <origin
-        xyz="0 0 0.730"
+        xyz="0 0 0"
         rpy="0 0 0" />
       <limit
@@ -117,8 +119,8 @@
       <axis xyz="0 0 1" />
     </joint>
-    <gazebo reference="${prefix}ewellix_lift_base_link">
+    <gazebo reference="${prefix}base_link">
       <material>Gazebo/Grey</material>
     </gazebo>
-    <gazebo reference="${prefix}ewellix_lift_top_link">
+    <gazebo reference="${prefix}link">
       <material>Gazebo/Grey</material>
     </gazebo>
@@ -129,5 +131,5 @@
         <plugin>gz_ros2_control/GazeboSimSystem</plugin>
       </hardware>
-      <joint name="${prefix}ewellix_lift_top_joint">
+      <joint name="${prefix}joint">
         <command_interface name="position" />
         <command_interface name="velocity" />

Commit message: Updated lift urdfs, now they load correctly for robot description. However, lift does not seem to hold position. To be fixed

File: urdf/structures/ewellix/ewellix_lift_700mm.urdf.xacro (robot description, xacro)
@@ -3,5 +3,5 @@
   name="ewellix_lift_700mm"
   xmlns:xacro="http://www.ros.org/wiki/xacro">
-  <!-- EWELLIX LIFT  -->
+  <!-- EWELLIX LIFT -->
   <xacro:macro
     name="ewellix_lift_700mm"
@@ -55,5 +55,5 @@
     </joint>
     <!-- Lift top link -->
-    <link name="${prefix}link">
+    <link name="${prefix}top_link">
       <visual>
         <origin
@@ -105,31 +105,34 @@
     <!-- Lift top link joint -->
     <joint
-      name="${prefix}joint"
+      name="${prefix}top_joint"
       type="prismatic">
       <parent link="${prefix}base_link" />
-      <child link="${prefix}link" />
+      <child link="${prefix}top_link" />
       <origin
-        xyz="0 0 0"
+        xyz="0 0 0.72"
         rpy="0 0 0" />
       <limit
-        effort="1000"
+        effort="700.0"
         lower="0.0"
-        upper="0.7"
+        upper="0.9"
         velocity="0.088" />
       <axis xyz="0 0 1" />
+      <dynamics damping="0.0" friction="0.0" />
     </joint>
     <gazebo reference="${prefix}base_link">
       <material>Gazebo/Grey</material>
+      <gravity>true</gravity>
     </gazebo>
-    <gazebo reference="${prefix}link">
+    <gazebo reference="${prefix}top_link">
       <material>Gazebo/Grey</material>
+      <gravity>true</gravity>
     </gazebo>
     <ros2_control
-      name="${prefix}ewellix_lift_control"
+      name="${prefix}lift_control"
       type="system">
       <hardware>
         <plugin>gz_ros2_control/GazeboSimSystem</plugin>
       </hardware>
-      <joint name="${prefix}joint">
+      <joint name="${prefix}top_joint">
         <command_interface name="position" />
         <command_interface name="velocity" />

File: urdf/structures/ewellix/ewellix_lift_900mm.urdf.xacro (robot description, xacro)
@@ -55,5 +55,5 @@
     </joint>
     <!-- Lift top link -->
-    <link name="${prefix}link">
+    <link name="${prefix}top_link">
       <visual>
         <origin
@@ -105,31 +105,34 @@
     <!-- Lift top link joint -->
     <joint
-      name="${prefix}joint"
+      name="${prefix}top_joint"
       type="prismatic">
       <parent link="${prefix}base_link" />
-      <child link="${prefix}link" />
+      <child link="${prefix}top_link" />
       <origin
-        xyz="0 0 0"
+        xyz="0 0 0.72"
         rpy="0 0 0" />
       <limit
-        effort="1000"
+        effort="700.0"
         lower="0.0"
         upper="0.9"
         velocity="0.088" />
       <axis xyz="0 0 1" />
+      <dynamics damping="0.0" friction="0.0" />
     </joint>
     <gazebo reference="${prefix}base_link">
       <material>Gazebo/Grey</material>
+      <gravity>true</gravity>
     </gazebo>
-    <gazebo reference="${prefix}link">
+    <gazebo reference="${prefix}top_link">
       <material>Gazebo/Grey</material>
+      <gravity>true</gravity>
     </gazebo>
     <ros2_control
-      name="${prefix}ewellix_lift_control"
+      name="${prefix}lift_control"
       type="system">
       <hardware>
         <plugin>gz_ros2_control/GazeboSimSystem</plugin>
       </hardware>
-      <joint name="${prefix}ewellix_lift_top_joint">
+      <joint name="${prefix}top_joint">
         <command_interface name="position" />
         <command_interface name="velocity" />

Commit message: Updated mass values for ewelix lifts, so it does not fall to below 0.0 position after spawning

File: urdf/structures/ewellix/ewellix_lift_700mm.urdf.xacro (robot description, xacro)
@@ -33,5 +33,5 @@
       </collision>
       <inertial>
-        <mass value="20" />
+        <mass value="0" />
         <origin
           xyz="0 0 0"

File: urdf/structures/ewellix/ewellix_lift_900mm.urdf.xacro (robot description, xacro)
@@ -33,5 +33,5 @@
       </collision>
       <inertial>
-        <mass value="20" />
+        <mass value="0" />
         <origin
           xyz="0 0 0"

Commit message: Feat/jazzy/moveit manipulation support (#88)
* Updated ur macro to be compatible with official ur gazebo package

* Updated lift urdfs, now they load correctly for robot description. However, lift does not seem to hold position. To be fixed

* Updated rbkarios urdf to work correctly with MoveIt in Gazebo simulation

* Updated rbrobout urdf to work correctly with MoveIt in Gazebo simulation

* Add arm_type argument to robot_description launch file for arm model

* Updated mass values for ewelix lifts, so it does not fall to below 0.0 position after spawning

File: urdf/structures/ewellix/ewellix_lift_700mm.urdf.xacro (robot description, xacro)
@@ -3,5 +3,5 @@
   name="ewellix_lift_700mm"
   xmlns:xacro="http://www.ros.org/wiki/xacro">
-  <!-- EWELLIX LIFT  -->
+  <!-- EWELLIX LIFT -->
   <xacro:macro
     name="ewellix_lift_700mm"
@@ -33,5 +33,5 @@
       </collision>
       <inertial>
-        <mass value="20" />
+        <mass value="0" />
         <origin
           xyz="0 0 0"
@@ -55,5 +55,5 @@
     </joint>
     <!-- Lift top link -->
-    <link name="${prefix}link">
+    <link name="${prefix}top_link">
       <visual>
         <origin
@@ -105,31 +105,34 @@
     <!-- Lift top link joint -->
     <joint
-      name="${prefix}joint"
+      name="${prefix}top_joint"
       type="prismatic">
       <parent link="${prefix}base_link" />
-      <child link="${prefix}link" />
+      <child link="${prefix}top_link" />
       <origin
-        xyz="0 0 0"
+        xyz="0 0 0.72"
         rpy="0 0 0" />
       <limit
-        effort="1000"
+        effort="700.0"
         lower="0.0"
-        upper="0.7"
+        upper="0.9"
         velocity="0.088" />
       <axis xyz="0 0 1" />
+      <dynamics damping="0.0" friction="0.0" />
     </joint>
     <gazebo reference="${prefix}base_link">
       <material>Gazebo/Grey</material>
+      <gravity>true</gravity>
     </gazebo>
-    <gazebo reference="${prefix}link">
+    <gazebo reference="${prefix}top_link">
       <material>Gazebo/Grey</material>
+      <gravity>true</gravity>
     </gazebo>
     <ros2_control
-      name="${prefix}ewellix_lift_control"
+      name="${prefix}lift_control"
       type="system">
       <hardware>
         <plugin>gz_ros2_control/GazeboSimSystem</plugin>
       </hardware>
-      <joint name="${prefix}joint">
+      <joint name="${prefix}top_joint">
         <command_interface name="position" />
         <command_interface name="velocity" />

File: urdf/structures/ewellix/ewellix_lift_900mm.urdf.xacro (robot description, xacro)
@@ -33,5 +33,5 @@
       </collision>
       <inertial>
-        <mass value="20" />
+        <mass value="0" />
         <origin
           xyz="0 0 0"
@@ -55,5 +55,5 @@
     </joint>
     <!-- Lift top link -->
-    <link name="${prefix}link">
+    <link name="${prefix}top_link">
       <visual>
         <origin
@@ -105,31 +105,34 @@
     <!-- Lift top link joint -->
     <joint
-      name="${prefix}joint"
+      name="${prefix}top_joint"
       type="prismatic">
       <parent link="${prefix}base_link" />
-      <child link="${prefix}link" />
+      <child link="${prefix}top_link" />
       <origin
-        xyz="0 0 0"
+        xyz="0 0 0.72"
         rpy="0 0 0" />
       <limit
-        effort="1000"
+        effort="700.0"
         lower="0.0"
         upper="0.9"
         velocity="0.088" />
       <axis xyz="0 0 1" />
+      <dynamics damping="0.0" friction="0.0" />
     </joint>
     <gazebo reference="${prefix}base_link">
       <material>Gazebo/Grey</material>
+      <gravity>true</gravity>
     </gazebo>
-    <gazebo reference="${prefix}link">
+    <gazebo reference="${prefix}top_link">
       <material>Gazebo/Grey</material>
+      <gravity>true</gravity>
     </gazebo>
     <ros2_control
-      name="${prefix}ewellix_lift_control"
+      name="${prefix}lift_control"
       type="system">
       <hardware>
         <plugin>gz_ros2_control/GazeboSimSystem</plugin>
       </hardware>
-      <joint name="${prefix}ewellix_lift_top_joint">
+      <joint name="${prefix}top_joint">
         <command_interface name="position" />
         <command_interface name="velocity" />
