Commit message: another spanish word

File: urdf/bodies/rbvogui/rbvogui_body.urdf.xacro (robot description, xacro)
@@ -17,5 +17,5 @@
     <!-- Chassis -->
     <joint name="${prefix}chassis_joint" type="fixed">
-      <origin xyz="-0.012 0 0.1775" rpy="0 0 0" /> <!-- Modificar para cada vogui -->
+      <origin xyz="-0.012 0 0.1775" rpy="0 0 0" />
       <parent link="${prefix}base_link"/>
       <child link="${prefix}chassis_link" />

Commit message: Restore xacro:if/unless hq blocks in base_docking_contact for rbvogui and rbvogui_xl
Agent-Logs-Url: https://github.com/RobotnikAutomation/robotnik_description/sessions/8f892b32-8b2e-422f-9012-d775b8413ad1

Co-authored-by: jamendezib <126663352+jamendezib@users.noreply.github.com>

File: urdf/bodies/rbvogui/rbvogui_body.urdf.xacro (robot description, xacro)
@@ -191,8 +191,16 @@
           xyz="0 0 0"
           rpy="0 0 0" />
-        <geometry>
-          <mesh
-            filename="package://robotnik_description/meshes/bases/rbvogui/rbvogui_contactors.stl" />
-        </geometry>
+        <xacro:if value="${hq}">
+          <geometry>
+            <mesh
+              filename="package://robotnik_description/meshes/bases/rbvogui/rbvogui_contactors.stl" />
+          </geometry>
+        </xacro:if>
+        <xacro:unless value="${hq}">
+          <geometry>
+            <mesh
+              filename="package://robotnik_description/meshes/bases/rbvogui/rbvogui_contactors.stl" />
+          </geometry>
+        </xacro:unless>
         <material name="lighbrown">
           <color rgba="0.7 0.3 0.0 1" />

File: urdf/bodies/rbvogui_xl/rbvogui_xl_body.urdf.xacro (robot description, xacro)
@@ -194,8 +194,16 @@
           xyz="0 0 0"
           rpy="0 0 0" />
-        <geometry>
-          <mesh
-            filename="package://robotnik_description/meshes/bases/rbvogui_xl/rbvogui_xl_contactors.stl" />
-        </geometry>
+        <xacro:if value="${hq}">
+          <geometry>
+            <mesh
+              filename="package://robotnik_description/meshes/bases/rbvogui_xl/rbvogui_xl_contactors.stl" />
+          </geometry>
+        </xacro:if>
+        <xacro:unless value="${hq}">
+          <geometry>
+            <mesh
+              filename="package://robotnik_description/meshes/bases/rbvogui_xl/rbvogui_xl_contactors.stl" />
+          </geometry>
+        </xacro:unless>
         <material name="lighbrown">
           <color rgba="0.7 0.3 0.0 1" />
