Commit message: Standardize body URDFs: merge contactors_link into base_docking_contact (#87)
* Standardize body URDFs: merge contactors_link into base_docking_contact for rbvogui and rbvogui_xl

Agent-Logs-Url: https://github.com/RobotnikAutomation/robotnik_description/sessions/2c2639ff-218e-48b2-91dd-85696a1957c6

Co-authored-by: jamendezib <126663352+jamendezib@users.noreply.github.com>

* Restore xacro:if/unless hq blocks in base_docking_contact for rbvogui and rbvogui_xl

Agent-Logs-Url: https://github.com/RobotnikAutomation/robotnik_description/sessions/8f892b32-8b2e-422f-9012-d775b8413ad1

Co-authored-by: jamendezib <126663352+jamendezib@users.noreply.github.com>

* Fix rvbogui_xl xacro

* Mesh naming more coherent

---------

Co-authored-by: copilot-swe-agent[bot] <198982749+Copilot@users.noreply.github.com>
Co-authored-by: jamendezib <126663352+jamendezib@users.noreply.github.com>
Co-authored-by: Jose Antonio Mendez <jamendez@robotnik.es>

File: urdf/bodies/rbvogui/rbvogui_base.gazebo.xacro (robot description, xacro)
@@ -31,5 +31,5 @@
   </xacro:macro>
   <xacro:macro
-    name="gazebo_color_logo_link"
+    name="gazebo_color_base_logos_link"
     params="prefix">
     <gazebo reference="${prefix}base_logos_link">
@@ -59,7 +59,7 @@
   </xacro:macro>
   <xacro:macro
-    name="gazebo_color_contactors_link"
+    name="gazebo_color_base_docking_contact"
     params="prefix">
-    <gazebo reference="${prefix}contactors_link">
+    <gazebo reference="${prefix}base_docking_contact">
       <visual>
         <material>

File: urdf/bodies/rbvogui/rbvogui_body.urdf.xacro (robot description, xacro)
@@ -49,5 +49,5 @@
           <geometry>
             <mesh
-              filename="package://robotnik_description/meshes/bases/rbvogui/rbvogui_chassis_color.dae" />
+              filename="package://robotnik_description/meshes/bases/rbvogui/rbvogui_chassis.dae" />
           </geometry>
         </xacro:if>
@@ -65,5 +65,5 @@
         <geometry>
           <mesh
-            filename="package://robotnik_description/meshes/bases/rbvogui/rbvogui_chassis_color.dae" />
+            filename="package://robotnik_description/meshes/bases/rbvogui/rbvogui_chassis.dae" />
         </geometry>
       </collision>
@@ -120,37 +120,4 @@
       </collision>
     </link>
-    <!-- Contactors -->
-    <joint
-      name="${prefix}contactors_joint"
-      type="fixed">
-      <origin
-        xyz="0.5235 0 0.09265"
-        rpy="0 0 0 " />
-      <parent link="${prefix}chassis_link" />
-      <child link="${prefix}contactors_link" />
-    </joint>
-    <!-- Contactors -->
-    <link name="${prefix}contactors_link">
-      <visual>
-        <origin
-          xyz="0 0 0"
-          rpy="0 0 0" />
-        <xacro:if value="${hq}">
-          <geometry>
-            <mesh
-              filename="package://robotnik_description/meshes/bases/rbvogui/rbvogui_contactors.stl" />
-          </geometry>
-        </xacro:if>
-        <xacro:unless value="${hq}">
-          <geometry>
-            <mesh
-              filename="package://robotnik_description/meshes/bases/rbvogui/rbvogui_contactors.stl" />
-          </geometry>
-        </xacro:unless>
-        <material name="lighbrown">
-          <color rgba="0.7 0.3 0.0 1" />
-        </material>
-      </visual>
-    </link>
     <!-- Logos -->
     <joint
@@ -172,5 +139,5 @@
           <geometry>
             <mesh
-              filename="package://robotnik_description/meshes/bases/rbvogui/rbvogui_logos.stl"
+              filename="package://robotnik_description/meshes/bases/rbvogui/rbvogui_base_logos.stl"
               scale="1.001 1.076 1.001" />
           </geometry>
@@ -179,5 +146,5 @@
           <geometry>
             <mesh
-              filename="package://robotnik_description/meshes/bases/rbvogui/rbvogui_logos.dae"
+              filename="package://robotnik_description/meshes/bases/rbvogui/rbvogui_base_logos.dae"
               scale="1.001 1.076 1.001" />
           </geometry>
@@ -214,15 +181,36 @@
     <xacro:gazebo_color_base_link prefix="${prefix}" />
     <xacro:gazebo_color_battery_link prefix="${prefix}" />
-    <xacro:gazebo_color_contactors_link
+    <xacro:gazebo_color_base_docking_contact
       prefix="${prefix}" />
-    <xacro:gazebo_color_logo_link prefix="${prefix}" />
+    <xacro:gazebo_color_base_logos_link prefix="${prefix}" />
     <xacro:gazebo_color_leds_link prefix="${prefix}" />
     <!-- DOCKING CONTACT -->
-    <link name="${prefix}base_docking_contact" />
+    <link name="${prefix}base_docking_contact">
+      <visual>
+        <origin
+          xyz="0 0 0"
+          rpy="0 0 0" />
+        <xacro:if value="${hq}">
+          <geometry>
+            <mesh
+              filename="package://robotnik_description/meshes/bases/rbvogui/rbvogui_base_docking_contact.stl" />
+          </geometry>
+        </xacro:if>
+        <xacro:unless value="${hq}">
+          <geometry>
+            <mesh
+              filename="package://robotnik_description/meshes/bases/rbvogui/rbvogui_base_docking_contact.stl" />
+          </geometry>
+        </xacro:unless>
+        <material name="lighbrown">
+          <color rgba="0.7 0.3 0.0 1" />
+        </material>
+      </visual>
+    </link>
     <joint
       name="${prefix}base_docking_joint"
       type="fixed">
       <origin
-        xyz="0.6405 0 0.10264"
+        xyz="0.5235 0 0.09265"
         rpy="0 0 0" />
       <parent link="${prefix}chassis_link" />

File: urdf/bodies/rbvogui_xl/rbvogui_xl_body.urdf.xacro (robot description, xacro)
@@ -123,37 +123,4 @@
       </collision>
     </link>
-    <!-- Contactors -->
-    <joint
-      name="${prefix}contactors_joint"
-      type="fixed">
-      <origin
-        xyz="0.6405 0 0.10264"
-        rpy="0 0 0 " />
-      <parent link="${prefix}chassis_link" />
-      <child link="${prefix}contactors_link" />
-    </joint>
-    <!-- Contactors -->
-    <link name="${prefix}contactors_link">
-      <visual>
-        <origin
-          xyz="0 0 0"
-          rpy="0 0 0" />
-        <xacro:if value="${hq}">
-          <geometry>
-            <mesh
-              filename="package://robotnik_description/meshes/bases/rbvogui_xl/rbvogui_xl_contactors.stl" />
-          </geometry>
-        </xacro:if>
-        <xacro:unless value="${hq}">
-          <geometry>
-            <mesh
-              filename="package://robotnik_description/meshes/bases/rbvogui_xl/rbvogui_xl_contactors.stl" />
-          </geometry>
-        </xacro:unless>
-        <material name="lighbrown">
-          <color rgba="0.7 0.3 0.0 1" />
-        </material>
-      </visual>
-    </link>
     <!-- Logos -->
     <joint
@@ -175,5 +142,5 @@
           <geometry>
             <mesh
-              filename="package://robotnik_description/meshes/bases/rbvogui_xl/rbvogui_xl_logos.stl"
+              filename="package://robotnik_description/meshes/bases/rbvogui_xl/rbvogui_xl_base_logos.stl"
               scale="1.24 1.24 1" />
           </geometry>
@@ -182,5 +149,5 @@
           <geometry>
             <mesh
-              filename="package://robotnik_description/meshes/bases/rbvogui_xl/rbvogui_xl_logos.dae"
+              filename="package://robotnik_description/meshes/bases/rbvogui_xl/rbvogui_xl_base_logos.dae"
               scale="1.3 1.3 1" />
           </geometry>
@@ -217,10 +184,31 @@
     <xacro:gazebo_color_base_link prefix="${prefix}" />
     <xacro:gazebo_color_battery_link prefix="${prefix}" />
-    <xacro:gazebo_color_contactors_link
+    <xacro:gazebo_color_base_docking_contact
       prefix="${prefix}" />
-    <xacro:gazebo_color_logo_link prefix="${prefix}" />
+    <xacro:gazebo_color_base_logos_link prefix="${prefix}" />
     <xacro:gazebo_color_leds_link prefix="${prefix}" />
     <!-- DOCKING CONTACT -->
-    <link name="${prefix}base_docking_contact" />
+    <link name="${prefix}base_docking_contact">
+      <visual>
+        <origin
+          xyz="0 0 0"
+          rpy="0 0 0" />
+        <xacro:if value="${hq}">
+          <geometry>
+            <mesh
+              filename="package://robotnik_description/meshes/bases/rbvogui_xl/rbvogui_xl_base_docking_contact.stl" />
+          </geometry>
+        </xacro:if>
+        <xacro:unless value="${hq}">
+          <geometry>
+            <mesh
+              filename="package://robotnik_description/meshes/bases/rbvogui_xl/rbvogui_xl_base_docking_contact.stl" />
+          </geometry>
+        </xacro:unless>
+        <material name="lighbrown">
+          <color rgba="0.7 0.3 0.0 1" />
+        </material>
+      </visual>
+    </link>
     <joint
       name="${prefix}base_docking_joint"
