Commit message: fix: replace Ogre1 Gazebo/* material names with inline RGBA
Gazebo Harmonic uses Ogre2/HLMS. Legacy Ogre1 script names such as
Gazebo/Black, Gazebo/Yellow, Gazebo/Grey and Gazebo/Gray are not
loaded by the Ogre2 renderer and cause models to render white or
throw warnings. Replaced with equivalent inline ambient/diffuse/
specular RGBA values inside each <gazebo reference> block.

Affected files (13 occurrences across 8 files):
  urdf/bodies/rb1/rb1_body.urdf.xacro
  urdf/bodies/rbkairos/rbkairos_body.urdf.xacro
  urdf/bodies/rbsummit_steel/rbsummit_steel_body.urdf.xacro
  urdf/bodies/rbtheron/rbtheron_body.urdf.xacro
  urdf/structures/ewellix/ewellix_lift_700mm.urdf.xacro (x2)
  urdf/structures/ewellix/ewellix_lift_900mm.urdf.xacro (x2)
  urdf/wheels/caster_wheel/rbtheron_caster.urdf.xacro
  urdf/wheels/rubber_wheel/gazebo/rubber_wheel.gazebo.xacro (x2)

File: urdf/bodies/rb1/rb1_body.urdf.xacro (robot description, xacro)
@@ -77,5 +77,10 @@
     </link>
     <gazebo reference="${prefix}base_link">
-      <material>Gazebo/Black</material>
+      <!-- Ogre2/HLMS (Gazebo Harmonic): inline RGBA replaces Gazebo/Black script -->
+      <material>
+        <ambient>0.0 0.0 0.0 1.0</ambient>
+        <diffuse>0.1 0.1 0.1 1.0</diffuse>
+        <specular>0.4 0.4 0.4 1.0</specular>
+      </material>
     </gazebo>
     <joint

File: urdf/bodies/rbkairos/rbkairos_body.urdf.xacro (robot description, xacro)
@@ -67,5 +67,10 @@
     </link>
     <gazebo reference="${prefix}base_link">
-      <material>Gazebo/Black</material>
+      <!-- Ogre2/HLMS (Gazebo Harmonic): inline RGBA replaces Gazebo/Black script -->
+      <material>
+        <ambient>0.0 0.0 0.0 1.0</ambient>
+        <diffuse>0.1 0.1 0.1 1.0</diffuse>
+        <specular>0.4 0.4 0.4 1.0</specular>
+      </material>
     </gazebo>
     <!-- TOP COVER -->

File: urdf/bodies/rbsummit_steel/rbsummit_steel_body.urdf.xacro (robot description, xacro)
@@ -67,5 +67,10 @@
     </link>
     <gazebo reference="${prefix}base_link">
-      <material>Gazebo/Black</material>
+      <!-- Ogre2/HLMS (Gazebo Harmonic): inline RGBA replaces Gazebo/Black script -->
+      <material>
+        <ambient>0.0 0.0 0.0 1.0</ambient>
+        <diffuse>0.1 0.1 0.1 1.0</diffuse>
+        <specular>0.4 0.4 0.4 1.0</specular>
+      </material>
     </gazebo>
     <!-- TOP COVER -->

File: urdf/bodies/rbtheron/rbtheron_body.urdf.xacro (robot description, xacro)
@@ -75,5 +75,10 @@
     </link>
     <gazebo reference="${prefix}base_link">
-      <material>Gazebo/Black</material>
+      <!-- Ogre2/HLMS (Gazebo Harmonic): inline RGBA replaces Gazebo/Black script -->
+      <material>
+        <ambient>0.0 0.0 0.0 1.0</ambient>
+        <diffuse>0.1 0.1 0.1 1.0</diffuse>
+        <specular>0.4 0.4 0.4 1.0</specular>
+      </material>
     </gazebo>
     <!-- LOGO ROBOTNIK IZQUIERDO -->

File: urdf/structures/ewellix/ewellix_lift_700mm.urdf.xacro (robot description, xacro)
@@ -120,8 +120,18 @@
     </joint>
     <gazebo reference="${prefix}base_link">
-      <material>Gazebo/Grey</material>
+      <!-- Ogre2/HLMS (Gazebo Harmonic): inline RGBA replaces Gazebo/Grey script -->
+      <material>
+        <ambient>0.5 0.5 0.5 1.0</ambient>
+        <diffuse>0.5 0.5 0.5 1.0</diffuse>
+        <specular>0.3 0.3 0.3 1.0</specular>
+      </material>
     </gazebo>
     <gazebo reference="${prefix}link">
-      <material>Gazebo/Grey</material>
+      <!-- Ogre2/HLMS (Gazebo Harmonic): inline RGBA replaces Gazebo/Grey script -->
+      <material>
+        <ambient>0.5 0.5 0.5 1.0</ambient>
+        <diffuse>0.5 0.5 0.5 1.0</diffuse>
+        <specular>0.3 0.3 0.3 1.0</specular>
+      </material>
     </gazebo>
     <ros2_control

File: urdf/structures/ewellix/ewellix_lift_900mm.urdf.xacro (robot description, xacro)
@@ -120,8 +120,18 @@
     </joint>
     <gazebo reference="${prefix}base_link">
-      <material>Gazebo/Grey</material>
+      <!-- Ogre2/HLMS (Gazebo Harmonic): inline RGBA replaces Gazebo/Grey script -->
+      <material>
+        <ambient>0.5 0.5 0.5 1.0</ambient>
+        <diffuse>0.5 0.5 0.5 1.0</diffuse>
+        <specular>0.3 0.3 0.3 1.0</specular>
+      </material>
     </gazebo>
     <gazebo reference="${prefix}link">
-      <material>Gazebo/Grey</material>
+      <!-- Ogre2/HLMS (Gazebo Harmonic): inline RGBA replaces Gazebo/Grey script -->
+      <material>
+        <ambient>0.5 0.5 0.5 1.0</ambient>
+        <diffuse>0.5 0.5 0.5 1.0</diffuse>
+        <specular>0.3 0.3 0.3 1.0</specular>
+      </material>
     </gazebo>
     <ros2_control

File: urdf/wheels/caster_wheel/rbtheron_caster.urdf.xacro (robot description, xacro)
@@ -202,5 +202,10 @@
       <kp>1.0</kp>
       <kd>1.0</kd>
-      <material>Gazebo/Black</material>
+      <!-- Ogre2/HLMS (Gazebo Harmonic): inline RGBA replaces Gazebo/Black script -->
+      <material>
+        <ambient>0.0 0.0 0.0 1.0</ambient>
+        <diffuse>0.1 0.1 0.1 1.0</diffuse>
+        <specular>0.4 0.4 0.4 1.0</specular>
+      </material>
     </gazebo>
   </xacro:macro>

File: urdf/wheels/rubber_wheel/gazebo/rubber_wheel.gazebo.xacro (robot description, xacro)
@@ -10,5 +10,10 @@
       <kp>0.0001</kp>
       <kd>1.0</kd> -->
-      <material>Gazebo/Yellow</material>
+      <!-- Ogre2/HLMS (Gazebo Harmonic): inline RGBA replaces Gazebo/Yellow script -->
+      <material>
+        <ambient>1.0 0.85 0.0 1.0</ambient>
+        <diffuse>1.0 0.85 0.0 1.0</diffuse>
+        <specular>0.3 0.3 0.3 1.0</specular>
+      </material>
       <minDepth>0.1</minDepth>
     </gazebo>
@@ -23,5 +28,10 @@
       <slip1>0.05</slip1>
       <slip2>0.05</slip2>
-      <material>Gazebo/Gray</material>
+      <!-- Ogre2/HLMS (Gazebo Harmonic): inline RGBA replaces Gazebo/Gray script -->
+      <material>
+        <ambient>0.5 0.5 0.5 1.0</ambient>
+        <diffuse>0.5 0.5 0.5 1.0</diffuse>
+        <specular>0.3 0.3 0.3 1.0</specular>
+      </material>
     </gazebo>
   </xacro:macro>
