Commit message: Feat/jazzy/add rbcar (#95)
* Standardize docking_contact link naming to base_docking_contact (#81)

* Standardize body URDFs: merge contactors_link into base_docking_contact (#87)

* Standardize body URDFs: merge contactors_link into base_docking_contact for rbvogui and rbvogui_xl

Agent-Logs-Url: https://github.com/RobotnikAutomation/robotnik_description/sessions/2c2639ff-218e-48b2-91dd-85696a1957c6

Co-authored-by: jamendezib <126663352+jamendezib@users.noreply.github.com>

* Restore xacro:if/unless hq blocks in base_docking_contact for rbvogui and rbvogui_xl

Agent-Logs-Url: https://github.com/RobotnikAutomation/robotnik_description/sessions/8f892b32-8b2e-422f-9012-d775b8413ad1

Co-authored-by: jamendezib <126663352+jamendezib@users.noreply.github.com>

* Fix rvbogui_xl xacro

* Mesh naming more coherent

---------

Co-authored-by: copilot-swe-agent[bot] <198982749+Copilot@users.noreply.github.com>
Co-authored-by: jamendezib <126663352+jamendezib@users.noreply.github.com>
Co-authored-by: Jose Antonio Mendez <jamendez@robotnik.es>

* fix: remove rear RGB-D camera from RB-THERON configuration (#89)

* rbtheron: Set picoscan120 as default laser (#90)

* Feat/jazzy/moveit manipulation support (#88)

* Updated ur macro to be compatible with official ur gazebo package

* Updated lift urdfs, now they load correctly for robot description. However, lift does not seem to hold position. To be fixed

* Updated rbkarios urdf to work correctly with MoveIt in Gazebo simulation

* Updated rbrobout urdf to work correctly with MoveIt in Gazebo simulation

* Add arm_type argument to robot_description launch file for arm model

* Updated mass values for ewelix lifts, so it does not fall to below 0.0 position after spawning

* Add ur_simulation_gz dependency

* Remove deprecate wheel model and suspension xacro

* Update suspnesion xacro an delete deprecate rear_axle

* Update rbcar base urdf for new suspension

* Update body to add better parametes definition an new hq model reference with textures

* Add elevator structure for rbcar if needed

* Add new version with textures for rbcar model

* Add textures for new rbcar model

* delete older wheels

* Add new wheel stl

* Update base xacro to use new wheel version

* Update body to use textured version

* Update suspension wheels xacro for use the mechanical data from v2 and use the new model of wheel

* Add ros2_control params to use ackermann controller from ros2

---------

Co-authored-by: Copilot <198982749+Copilot@users.noreply.github.com>
Co-authored-by: jamendezib <126663352+jamendezib@users.noreply.github.com>
Co-authored-by: Jose Antonio Mendez <jamendez@robotnik.es>
Co-authored-by: Román Navarro García <rnavarro@robotnik.es>
Co-authored-by: Robert Vasquez Zavaleta <59690050+robert-ros@users.noreply.github.com>
Co-authored-by: Łukasz Granat <122286182+LokneyRobotnik@users.noreply.github.com>
Co-authored-by: Ángel Soriano <asoriano@robotnik.es>

File: urdf/bases/rbcar/rbcar_base.urdf.xacro (robot description, xacro)
@@ -5,10 +5,6 @@
   <xacro:include
     filename="$(find robotnik_description)/urdf/bodies/rbcar/rbcar_body.urdf.xacro" />
-  <!-- <xacro:include
-    filename="$(find robotnik_description)/urdf/wheels/rubber_wheel/rubber_wheel.urdf.xacro" /> -->
   <xacro:include
-    filename="$(find robotnik_description)/urdf/wheels/rbcar/suspension_wheel_v2.urdf.xacro" />
-  <xacro:include
-    filename="$(find robotnik_description)/urdf/wheels/rbcar/rear_axle.urdf.xacro" />
+    filename="$(find robotnik_description)/urdf/wheels/rbcar/suspension_wheel_v4.urdf.xacro" />
   <xacro:include
     filename="$(find robotnik_description)/simulators/gazebo_ignition/rbcar/rbcar_control.urdf.xacro" />
@@ -16,5 +12,5 @@
   <xacro:property
     name="wheel_offset_x"
-    value="1.85" />
+    value="0.91131" />
   <xacro:property
     name="wheel_offset_y"
@@ -22,5 +18,5 @@
   <xacro:property
     name="wheel_offset_z"
-    value="0.0" />
+    value="-0.05" />
   <xacro:macro
     name="rbcar"
@@ -30,5 +26,4 @@
       namespace:=''
       ">
-    <!-- BODY -->
     <xacro:property
       name="hq"
@@ -36,37 +31,35 @@
     <xacro:rbcar_body
       prefix="${prefix}"
-      hq="${hq}" />
+      hq="${hq}"
+      clearance="${wheel_radius}" />
     <!-- WHEELS -->
     <xacro:front_wheel
-      lr_prefix="$(arg prefix)left"
+      prefix="${prefix}"
+      lr_prefix="left"
       fr_prefix="front"
       lr_reflect="1"
       fr_reflect="1"
-      parent="$(arg prefix)base_link" />
+      parent="${prefix}base_link" />
     <xacro:front_wheel
-      lr_prefix="$(arg prefix)right"
+      prefix="${prefix}"
+      lr_prefix="right"
       fr_prefix="front"
       lr_reflect="-1"
       fr_reflect="1"
-      parent="$(arg prefix)base_link" />
+      parent="${prefix}base_link" />
     <xacro:rear_wheel
-      lr_prefix="$(arg prefix)left"
+      prefix="${prefix}"
+      lr_prefix="left"
       fr_prefix="rear"
       lr_reflect="1"
       fr_reflect="-1"
-      parent="$(arg prefix)base_link" />
+      parent="${prefix}base_link" />
     <xacro:rear_wheel
-      lr_prefix="$(arg prefix)right"
+      prefix="${prefix}"
+      lr_prefix="right"
       fr_prefix="rear"
       lr_reflect="-1"
       fr_reflect="-1"
-      parent="$(arg prefix)base_link" />
-    <!-- <xacro:rear_axle
-      prefix="$(arg prefix)rear_axle"
-      parent="$(arg prefix)base_link">
-      <origin
-        xyz="0 0.0 0"
-        rpy="1.57079633 0 3.14159265"/>
-    </xacro:rear_axle> -->
+      parent="${prefix}base_link" />
     <!-- CONTROL -->
     <xacro:if value="$(arg gazebo_ignition)">

File: urdf/bodies/rbcar/rbcar_body.urdf.xacro (robot description, xacro)
@@ -1,23 +1,19 @@
 <?xml version="1.0"?>
 <robot name="rbcar" xmlns:xacro="http://wiki.ros.org/xacro">
-  <xacro:macro name="rbcar_body" params="prefix:='' hq">
-  <!-- Robot mechanical and motor parameters -->
-  <xacro:property
-    name="wheel_width"
-    value="0.317" />
-  <xacro:property
-    name="clearance"
-    value="${tire_dia/2.0}" />
+  <xacro:macro
+    name="rbcar_body"
+    params="prefix:='' hq:=true clearance:=${wheel_radius}">
   <!-- BASE FOOTPRINT -->
   <link name="${prefix}base_footprint">
     <visual>
-        <origin xyz="0 0 0" rpy="0 0 0" />
-        <geometry>
-            <box size="0.001 0.001 0.001" />
-        </geometry>
+      <origin xyz="0 0 0" rpy="0 0 0" />
+      <geometry>
+        <box size="0.001 0.001 0.001" />
+      </geometry>
     </visual>
   </link>
   <joint name="${prefix}base_footprint_joint" type="fixed">
-    <origin xyz="0 0 ${clearance}" rpy="0 0 0" />  <!-- height is the clearance -->
+    <origin xyz="0 0 ${clearance}" rpy="0 0 0" />
+    <!-- height is the clearance -->
     <parent link="${prefix}base_footprint"/>
     <child link="${prefix}base_link" />
@@ -33,16 +29,16 @@
        <origin xyz="0.917 0 0" rpy="0 0 0" />
        <xacro:if value="${hq}">
-       <geometry>
-	     <mesh filename="package://robotnik_description/meshes/bases/rbcar/rbcar_chassis_hq.stl"/>
-       </geometry>
+         <geometry>
+           <mesh filename="package://robotnik_description/meshes/bases/rbcar/rbcar_hq.dae"/>
+         </geometry>
        </xacro:if>
        <xacro:unless value="${hq}">
-       <geometry>
-	     <mesh filename="package://robotnik_description/meshes/bases/rbcar/rbcar_chassis.stl"/>
-       </geometry>
+         <geometry>
+           <mesh filename="package://robotnik_description/meshes/bases/rbcar/rbcar_chassis.stl"/>
+         </geometry>
        </xacro:unless>
-       <material name="gray">
+       <!-- <material name="gray">
          <color rgba="0.8 0.8 0.8 1"/>
-       </material>
+       </material> -->
     </visual>
     <collision>
@@ -53,4 +49,13 @@
     </collision>
   </link>
+  <!-- DOCKING CONTACT -->
+  <!--
+  <link name="${prefix}base_docking_contact" />
+  <joint name="${prefix}base_docking_joint" type="fixed">
+    <origin xyz="0.0 0.0 0.0" rpy="0 0 0" />
+    <parent link="${prefix}base_link" />
+    <child link="${prefix}base_docking_contact" />
+  </joint>
+  -->
   </xacro:macro>
 </robot>
