Commit message: No control. Can spawn be spawned if commenting controller spawner.

File: robots/rbcar/rbcar.urdf.xacro (robot description, xacro)
@@ -13,4 +13,6 @@
 <!-- Flag to select the high or low quality model -->
 <xacro:property name="hq" value="true" />
+<xacro:arg name="gazebo_ignition" default="false"/>
+<xacro:arg name="namespace" default="robot"/>
 <xacro:arg name="prefix" default="robot_"/>
 <xacro:arg name="gpu" default="true"/>

File: urdf/bases/rbcar/rbcar_base.urdf.xacro (robot description, xacro)
@@ -5,15 +5,19 @@
   <xacro:include
     filename="$(find robotnik_description)/urdf/bodies/rbcar/rbcar_body.urdf.xacro" />
+  <!-- <xacro:include
+    filename="$(find robotnik_description)/urdf/wheels/rubber_wheel/rubber_wheel.urdf.xacro" /> -->
   <xacro:include
     filename="$(find robotnik_description)/urdf/wheels/rbcar/suspension_wheel_v2.urdf.xacro" />
   <xacro:include
     filename="$(find robotnik_description)/urdf/wheels/rbcar/rear_axle.urdf.xacro" />
+  <!-- <xacro:include
+    filename="$(find robotnik_description)/simulators/gazebo_ignition/rbcar/rbcar_control.urdf.xacro" /> -->
   <!-- WHEELS PROPERTIES -->
   <xacro:property
     name="wheel_offset_x"
-    value="1.0" />
+    value="1.85" />
   <xacro:property
     name="wheel_offset_y"
-    value="0.75" />
+    value="0.62124" />
   <xacro:property
     name="wheel_offset_z"
@@ -26,4 +30,5 @@
       namespace:=''
       ">
+    <!-- BODY -->
     <xacro:property
       name="hq"
@@ -32,16 +37,4 @@
       prefix="${prefix}"
       hq="${hq}" />
-    <!-- Wheels -->
-<!-- <xacro:front_wheel lr_prefix="$(arg prefix)left" fr_prefix="front"
-          lr_reflect="1" fr_reflect="1" parent="$(arg prefix)base_link" />
-<xacro:front_wheel lr_prefix="$(arg prefix)right" fr_prefix="front"
-          lr_reflect="-1" fr_reflect="1" parent="$(arg prefix)base_link" />
-<xacro:rear_wheel lr_prefix="$(arg prefix)left" fr_prefix="rear"
-        lr_reflect="1" fr_reflect="-1" parent="$(arg prefix)base_link" />
-<xacro:rear_wheel lr_prefix="$(arg prefix)right" fr_prefix="rear"
-        lr_reflect="-1" fr_reflect="-1" parent="$(arg prefix)base_link" />
-  <xacro:rear_axle prefix="$(arg prefix)rear_axle" parent="$(arg prefix)base_link">
-  <origin xyz="0 0.0 0" rpy="1.57079633 0 3.14159265"/>
-  </xacro:rear_axle> -->
     <!-- WHEELS -->
     <!-- <xacro:rubber_wheel
@@ -69,5 +62,5 @@
       hq="${hq}">
       <origin
-        xyz="-${wheel_offset_x} ${wheel_offset_y} ${wheel_offset_z}"
+        xyz="0 ${wheel_offset_y} ${wheel_offset_z}"
         rpy="0 0 0" />
     </xacro:rubber_wheel>
@@ -78,9 +71,42 @@
       hq="${hq}">
       <origin
-        xyz="-${wheel_offset_x} -${wheel_offset_y} ${wheel_offset_z}"
+        xyz="0 -${wheel_offset_y} ${wheel_offset_z}"
         rpy="0 0 0" />
-    </xacro:rubber_wheel>
-    <xacro:if value="$(arg gazebo_ignition)">
-      <xacro:rbwatcher_gz_ignition_control
+    </xacro:rubber_wheel> -->
+    <!-- Wheels -->
+    <xacro:front_wheel
+      lr_prefix="$(arg prefix)left"
+      fr_prefix="front"
+      lr_reflect="1"
+      fr_reflect="1"
+      parent="$(arg prefix)base_link" />
+    <xacro:front_wheel
+      lr_prefix="$(arg prefix)right"
+      fr_prefix="front"
+      lr_reflect="-1"
+      fr_reflect="1"
+      parent="$(arg prefix)base_link" />
+    <xacro:rear_wheel
+      lr_prefix="$(arg prefix)left"
+      fr_prefix="rear"
+      lr_reflect="1"
+      fr_reflect="-1"
+      parent="$(arg prefix)base_link" />
+    <xacro:rear_wheel
+      lr_prefix="$(arg prefix)right"
+      fr_prefix="rear"
+      lr_reflect="-1"
+      fr_reflect="-1"
+      parent="$(arg prefix)base_link" />
+    <xacro:rear_axle
+      prefix="$(arg prefix)rear_axle"
+      parent="$(arg prefix)base_link">
+      <origin
+        xyz="0 0.0 0"
+        rpy="1.57079633 0 3.14159265"/>
+    </xacro:rear_axle>
+    <!-- CONTROL -->
+    <!-- <xacro:if value="$(arg gazebo_ignition)">
+      <xacro:rbcar_gz_ignition_control
         namespace="${namespace}"
         prefix="${prefix}" />

File: urdf/wheels/rbcar/suspension_wheel_v2.urdf.xacro (robot description, xacro)
@@ -147,5 +147,5 @@
         <geometry>
           <!--cylinder radius="${tire_dia / 2}" length="${tire_width}"/-->
-          <mesh filename="package://rbcar_description/meshes/wheels/rbcar_wheel.stl"/>
+          <mesh filename="package://robotnik_description/meshes/wheels/rbcar/rbcar_wheel.stl"/>
         </geometry>
         <material name="tire_mat"/>

Commit message: Add sensors to rbcar

File: robots/rbcar/rbcar.urdf.xacro (robot description, xacro)
@@ -23,25 +23,56 @@
     namespace="$(arg namespace)" />
 <!-- Sensors-->
-<!--
-  <xacro:macro name="sensor_rslidar_m1" params="prefix parent prefix_topic:='laser_front' *origin gpu:=false">
-    <sensor_rslidar prefix="${prefix}" parent="${parent}" prefix_topic="${prefix_topic}" range_min="0.4" range_max="250.0" hfov="360.0" hres="0.1" vfov="40.0" vres="0.1" fps="20.0" gpu="${gpu}" >
-      <xacro:insert_block name="origin" />
-    </sensor_rslidar>
-  </xacro:macro>
-<xacro:sensor_ublox prefix="$(arg prefix)gps" parent="$(arg prefix)base_link">
-  <origin xyz="-0.58 0 1.503" rpy="0 0 0"/>
+<!-- IMU -->
+<xacro:sensor_vectornav
+  frame_prefix="$(arg prefix)imu_"
+  parent="$(arg prefix)base_link"
+  node_namespace="$(arg namespace)"
+  gazebo_ignition="$(arg gazebo_ignition)">
+  <origin xyz="0.319 0.018 0.676" rpy="0 0 0"/>
+</xacro:sensor_vectornav>
+<!-- GPS -->
+<xacro:sensor_ublox
+  frame_prefix="$(arg prefix)gps_"
+  parent="$(arg prefix)base_link"
+  node_namespace="$(arg namespace)"
+  node_name="gps"
+  gazebo_ignition="$(arg gazebo_ignition)">
+  <origin xyz="0.58 0 1.503" rpy="0 0 0"/>
 </xacro:sensor_ublox>
-<xacro:sensor_imu_hector prefix="$(arg prefix)imu" parent="$(arg prefix)base_link">
-  <origin xyz="0.319 0.018 0.676" rpy="0 0 0"/>
-</xacro:sensor_imu_hector> -->
-      <!--xacro:sensor_rslidar_16 prefix="$(arg prefix)top_3d_laser" parent="$(arg prefix)base_link"  gpu="$(arg gpu)">
-        <origin xyz="1.32252 0.0 1.20341" rpy="0 0.288 0"/>
-      </xacro:sensor_rslidar_16-->
-<!-- <xacro:sensor_rslidar_m1 prefix="$(arg prefix)laser_front" parent="$(arg prefix)base_link"  gpu="$(arg gpu)">
-  <origin xyz="2.14 0.0 0.24" rpy="0 3.015 3.14159"/>
+<!-- 3D LiDAR -->
+<xacro:sensor_rslidar_16
+  frame_prefix="$(arg prefix)top_3d_laser_"
+  parent="$(arg prefix)base_link"
+  node_namespace="$(arg namespace)"
+  node_name="top_lidar"
+  gazebo_ignition="$(arg gazebo_ignition)"
+  max_angle="3.14159"
+  min_angle="-3.14159"
+  gpu="$(arg gpu)">
+  <origin xyz="1.40252 0.0 1.40341" rpy="0 0.288 0"/>
+</xacro:sensor_rslidar_16>
+<!-- Front 3D LiDAR -->
+<xacro:sensor_rslidar_m1
+  frame_prefix="$(arg prefix)front_laser_"
+  parent="$(arg prefix)base_link"
+  node_namespace="$(arg namespace)"
+  node_name="front_lidar"
+  gazebo_ignition="$(arg gazebo_ignition)"
+  max_angle="3.14159"
+  min_angle="-3.14159"
+  gpu="$(arg gpu)">
+  <origin xyz="2.28 0.0 0.30" rpy="0 3.015 3.14159"/>
 </xacro:sensor_rslidar_m1>
-<xacro:sensor_hokuyo_utm30lx prefix="$(arg prefix)rear_laser" parent="$(arg prefix)base_link" prefix_topic="rear_laser" min_angle="-2.35" max_angle="2.35">
-  <origin xyz="-0.8 0.0 0.20" rpy="0 0 3.14159"/>
-</xacro:sensor_hokuyo_utm30lx> -->
+<!-- Rear 2D LiDAR -->
+<xacro:sensor_hokuyo_utm30lx
+  frame_prefix="$(arg prefix)rear_laser_"
+  parent="$(arg prefix)base_link"
+  node_namespace="$(arg namespace)"
+  node_name="rear_laser"
+  gazebo_ignition="$(arg gazebo_ignition)"
+  min_angle="-2.35"
+  max_angle="2.35">
+  <origin xyz="-0.4 0.0 0.20" rpy="0 0 3.14159"/>
+</xacro:sensor_hokuyo_utm30lx>
 <!--Gazebo plugins-->
 <!-- <gazebo>
