Commit message: Updated centauro rb vogui tool frames

File: urdf/structures/tools/pilz_d435f_arduino.urdf.xacro (robot description, xacro)
@@ -15,5 +15,5 @@
             *origin
             gazebo_ignition:=false
-            node_name:=photoneo_motioncam
+            node_name:=realsense_d435i
             node_namespace:=${None}
             topic_prefix:=~/">
@@ -24,14 +24,14 @@
     </xacro:if>
     <xacro:property
-      name="photoneo_motioncam_depth_horizontal_fov"
+      name="realsense_d435i_depth_horizontal_fov"
       value="52.71264861" />
     <xacro:property
-      name="photoneo_motioncam_depth_vertical_fov"
+      name="realsense_d435i_depth_vertical_fov"
       value="42.24943829" />
     <xacro:property
-      name="photoneo_motioncam_color_horizontal_fov"
+      name="realsense_d435i_color_horizontal_fov"
       value="52.71264861" />
     <xacro:property
-      name="photoneo_motioncam_color_vertical_fov"
+      name="realsense_d435i_color_vertical_fov"
       value="42.24943829" />
     <!-- Lift base link -->
@@ -43,5 +43,5 @@
         <geometry>
           <mesh
-            filename="package://robotnik_description/meshes/structures/CENTAURO/pilz_d435f_arduino_simplified.STL"
+            filename="package://robotnik_description/meshes/structures/CENTAURO/Pilz_d435f_arduino_simplified.STL"
             scale="1 1 1" />
         </geometry>
@@ -56,5 +56,5 @@
         <geometry>
           <mesh
-            filename="package://robotnik_description/meshes/structures/CENTAURO/pilz_d435f_arduino_simplified.STL"
+            filename="package://robotnik_description/meshes/structures/CENTAURO/Pilz_d435f_arduino_simplified.STL"
             scale="1 1 1" />
         </geometry>
@@ -82,68 +82,68 @@
       <child link="${prefix}tool_link" />
     </joint>
-    <!-- sander link joint -->
-    <joint
-      name="${prefix}sander_joint"
-      type="fixed">
-      <origin
-        xyz="0 0 0.123"
+    <!-- arduino link joint -->
+    <joint
+      name="${prefix}arduino_joint"
+      type="fixed">
+      <origin
+        xyz="0 0 0.0523"
         rpy="0 0 0" />
       <parent link="${prefix}tool_link" />
-      <child link="${prefix}sander_link" />
-    </joint>
-    <link name="${prefix}sander_link" />
-    <!-- photoneo_motioncam link joint -->
-    <joint
-      name="${prefix}photoneo_motioncam_joint"
-      type="fixed">
-      <origin
-        xyz="0 -0.1155 0.075 "
-        rpy="${radians(15)} 0 0" />
+      <child link="${prefix}arduino_link" />
+    </joint>
+    <link name="${prefix}arduino_link" />
+    <!-- realsense_d435i link joint -->
+    <joint
+      name="${prefix}realsense_d435i_joint"
+      type="fixed">
+      <origin
+        xyz="-0.042 0 0.1064 "
+        rpy="0 0 0" />
       <parent link="${prefix}tool_link" />
-      <child link="${prefix}photoneo_motioncam_link" />
-    </joint>
-    <link name="${prefix}photoneo_motioncam_link" />
-    <!-- photoneo_motioncam depth joints and links -->
-    <joint
-      name="${prefix}photoneo_motioncam_depth_joint"
-      type="fixed">
-      <origin
-        xyz="0 0 0"
-        rpy="0 0 0" />
-      <parent link="${prefix}photoneo_motioncam_link" />
-      <child link="${prefix}photoneo_motioncam_depth_frame" />
-    </joint>
-    <link name="${prefix}photoneo_motioncam_depth_frame" />
-    <joint
-      name="${prefix}photoneo_motioncam_depth_optical_joint"
-      type="fixed">
-      <origin
-        xyz="0 0 0"
-        rpy="0 0 0" />
-      <parent link="${prefix}photoneo_motioncam_depth_frame" />
-      <child link="${prefix}photoneo_motioncam_depth_optical_frame" />
-    </joint>
-    <link name="${prefix}photoneo_motioncam_depth_optical_frame" />
-    <!-- photoneo_motioncam color joints and links -->
-    <joint
-      name="${prefix}photoneo_motioncam_color_joint"
-      type="fixed">
-      <origin
-        xyz="0 0 0"
-        rpy="0 0 0" />
-      <parent link="${prefix}photoneo_motioncam_link" />
-      <child link="${prefix}photoneo_motioncam_color_frame" />
-    </joint>
-    <link name="${prefix}photoneo_motioncam_color_frame" />
-    <joint
-      name="${prefix}photoneo_motioncam_color_optical_joint"
+      <child link="${prefix}realsense_d435i_link" />
+    </joint>
+    <link name="${prefix}realsense_d435i_link" />
+    <!-- realsense_d435i depth joints and links -->
+    <joint
+      name="${prefix}realsense_d435i_depth_joint"
+      type="fixed">
+      <origin
+        xyz="0 0 0"
+        rpy="0 0 0" />
+      <parent link="${prefix}realsense_d435i_link" />
+      <child link="${prefix}realsense_d435i_depth_frame" />
+    </joint>
+    <link name="${prefix}realsense_d435i_depth_frame" />
+    <joint
+      name="${prefix}realsense_d435i_depth_optical_joint"
+      type="fixed">
+      <origin
+        xyz="0 0 0"
+        rpy="0 0 0" />
+      <parent link="${prefix}realsense_d435i_depth_frame" />
+      <child link="${prefix}realsense_d435i_depth_optical_frame" />
+    </joint>
+    <link name="${prefix}realsense_d435i_depth_optical_frame" />
+    <!-- realsense_d435i color joints and links -->
+    <joint
+      name="${prefix}realsense_d435i_color_joint"
+      type="fixed">
+      <origin
+        xyz="0 0 0"
+        rpy="0 0 0" />
+      <parent link="${prefix}realsense_d435i_link" />
+      <child link="${prefix}realsense_d435i_color_frame" />
+    </joint>
+    <link name="${prefix}realsense_d435i_color_frame" />
+    <joint
+      name="${prefix}realsense_d435i_color_optical_joint"
       type="fixed">
       <origin
         xyz="0 0 0"
         rpy="${radians(0)} ${radians(-90)} ${radians(90)}" />
-      <parent link="${prefix}photoneo_motioncam_color_frame" />
-      <child link="${prefix}photoneo_motioncam_color_optical_frame" />
-    </joint>
-    <link name="${prefix}photoneo_motioncam_color_optical_frame" />
+      <parent link="${prefix}realsense_d435i_color_frame" />
+      <child link="${prefix}realsense_d435i_color_optical_frame" />
+    </joint>
+    <link name="${prefix}realsense_d435i_color_optical_frame" />
     <xacro:depth_camera_plugin
       node_namespace="${node_namespace}"
@@ -151,8 +151,8 @@
       topic_prefix="${topic_prefix}_depth"
       gazebo_ignition="${gazebo_ignition}"
-      optical_frame="${prefix}photoneo_motioncam_depth_optical_frame"
-      reference_frame="${prefix}photoneo_motioncam_depth_optical_frame"
-      horizontal_fov="${photoneo_motioncam_depth_horizontal_fov}"
-      vertical_fov="${photoneo_motioncam_depth_vertical_fov}"
+      optical_frame="${prefix}realsense_d435i_depth_optical_frame"
+      reference_frame="${prefix}realsense_d435i_depth_optical_frame"
+      horizontal_fov="${realsense_d435i_depth_horizontal_fov}"
+      vertical_fov="${realsense_d435i_depth_vertical_fov}"
       video_width="1280"
       video_height="720"
@@ -165,8 +165,8 @@
       topic_prefix="${topic_prefix}_color"
       gazebo_ignition="${gazebo_ignition}"
-      optical_frame="${prefix}photoneo_motioncam_color_optical_frame"
-      reference_frame="${prefix}photoneo_motioncam_color_optical_frame"
-      horizontal_fov="${photoneo_motioncam_color_horizontal_fov}"
-      vertical_fov="${photoneo_motioncam_color_vertical_fov}"
+      optical_frame="${prefix}realsense_d435i_color_optical_frame"
+      reference_frame="${prefix}realsense_d435i_color_optical_frame"
+      horizontal_fov="${realsense_d435i_color_horizontal_fov}"
+      vertical_fov="${realsense_d435i_color_vertical_fov}"
       video_width="2448"
       video_height="2048"
@@ -175,5 +175,5 @@
       rate="30" />
     <xacro:unless value="${gazebo_ignition}">
-      <gazebo reference="${prefix}photoneo_motioncam_color_optical_frame">
+      <gazebo reference="${prefix}realsense_d435i_color_optical_frame">
         <sensor name="${prefix}" type="depth">
             <always_on>true</always_on>
@@ -203,5 +203,5 @@
                 </ros>
                 <camera_name>${prefix}</camera_name>
-                <frame_name>${prefix}photoneo_motioncam_color_optical_frame</frame_name>
+                <frame_name>${prefix}realsense_d435i_color_optical_frame</frame_name>
                 <hack_baseline>0.07</hack_baseline>
                 <min_depth>0.05</min_depth>
