Commit message: Increase 1cm ptz height for rbwatcher v2

File: robots/versions/rbwatcher/rbwatcher_v2.urdf.xacro (robot description, xacro)
@@ -70,5 +70,5 @@
 		<!-- PTZ camera -->
 		<xacro:sensor_link_750_nh prefix="${prefix}top_ptz_camera" prefix_topic="top_ptz_camera" parent="${prefix}base_link" fps="15.0">
-			<origin xyz="-0.11808 0 0.60038" rpy="0 0 0"/>
+			<origin xyz="-0.11808 0 0.61038" rpy="0 0 0"/>
 		</xacro:sensor_link_750_nh>
 		<!-- Gazebo ros control pluggins -->
